File: PMod_Neopixel/PMod_Neopixel.sch (KiCad schematic (older format))
At the start: 14 parts, among them J1 Conn_02x06_Counter_Clockwise, J2 Conn_01x02

Commit message: Minor Scematic changes
Parts:
- gave numbers to parts that had none: 2
Changed lines of the file:
@@
 NoConn ~ 2100 1650
 $Comp
-L Device:R R?
+L Device:R R1
 U 1 1 608892A1
 P 2350 3850
-F 0 "R?" V 2143 3850 50  0000 C CNN
+F 0 "R1" V 2143 3850 50  0000 C CNN
 F 1 "0" V 2234 3850 50  0000 C CNN
 F 2 "Resistor_SMD:R_0603_1608Metric" V 2280 3850 50  0001 C CNN
@@
 $EndComp
 $Comp
-L Device:R R?
+L Device:R R2
 U 1 1 6088B93D
 P 2350 4500
-F 0 "R?" V 2143 4500 50  0000 C CNN
+F 0 "R2" V 2143 4500 50  0000 C CNN
 F 1 "0" V 2234 4500 50  0000 C CNN
 F 2 "Resistor_SMD:R_0603_1608Metric" V 2280 4500 50  0001 C CNN
@@
 $EndComp
 $Comp
-L power:+3V3 #PWR?
+L power:+3V3 #PWR0127
 U 1 1 608967EB
 P 2050 3850
-F 0 "#PWR?" H 2050 3700 50  0001 C CNN
+F 0 "#PWR0127" H 2050 3700 50  0001 C CNN
 F 1 "+3V3" V 1950 3950 50  0000 L CNN
 F 2 "" H 2050 3850 50  0001 C CNN
@@
 $EndComp
 $Comp
-L power:VCC #PWR?
+L power:VCC #PWR0128
 U 1 1 608967F1
 P 2650 3850
-F 0 "#PWR?" H 2650 3700 50  0001 C CNN
+F 0 "#PWR0128" H 2650 3700 50  0001 C CNN
 F 1 "VCC" V 2750 4050 50  0000 C CNN
 F 2 "" H 2650 3850 50  0001 C CNN
