File: PMod_Neopixel/PMod_Neopixel.kicad_pcb (KiCad board)
At the start: 2 copper layers, 80 x 17 mm, 14 parts, among them J1 Conn_02x06_Counter_Clockwise, J2 Conn_01x02

Commit message: Updates to silk screen before sent to be produced
Parts:
- added G***: LOGO, jjh:Untitled, B.Cu at (164.2, 102.8)
Other:
- board text added: "@JamesjHorton JJHorton.co.uk"
- board text added: "NeoPixel PMod Strip"
