File: PMod_Neopixel/PMod_Neopixel_compact.kicad_pcb (KiCad board)
At the start: 2 copper layers, 49.4 x 17 mm, 14 parts, among them J1 Conn_02x06_Counter_Clockwise, J2 Conn_01x02

Commit message: Update the silkscreen
Parts:
- moved R1 3.15 mm to (118.3, 101.9), turned to 90 degrees
- moved R2 2.83 mm to (118.3, 97.1)
- moved J2 1.64 mm to (118.4, 104.9)
Routing:
- net VCC: track 116.1 -> 108.7 mm
- net Din_Vcc: track 6.40 -> 3.43 mm
- net Din_3v3: track 3.62 -> 6.59 mm
- net +3V3: track 15.8 -> 17.3 mm
- net GND: vias 20 -> 21
Other:
- board text added: "3V3"
- board text added: "DIN"
- board text added: "GND"
- board text removed: "WS2812B PMod Board @Jamesjhorton jjhorton.co.uk"

Commit message: Updates to silk screen before sent to be produced
Parts:
- added G***: LOGO, jjh:Untitled, B.Cu at (138.5, 103.2)
Other:
- board text added: "@JamesjHorton jjhorton.co.uk"
- board text added: "NeoPixel PMod Board"
- board text removed: "WS2812B PMod Board @JamesjHorton jjhorton.co.uk"
