File: PMod_LED/PMod_LED.sch (KiCad schematic (older format))
At the start: 17 parts

Commit message: update names in schematic
Parts:
- gave numbers to parts that had none: 9
Changed lines of the file:
@@
 $EndDescr
 $Comp
-L Connector_Generic:Conn_02x06_Odd_Even J?
+L Connector_Generic:Conn_02x06_Odd_Even J1
 U 1 1 60870F83
 P 2700 1750
-F 0 "J?" H 2750 2167 50  0000 C CNN
+F 0 "J1" H 2750 2167 50  0000 C CNN
 F 1 "Conn_02x06_Odd_Even" H 2750 2076 50  0000 C CNN
 F 2 "Connector_PinSocket_2.54mm:PinSocket_2x06_P2.54mm_Vertical" H 2700 1750 50  0001 C CNN
@@
 $EndComp
 $Comp
-L Device:R R?
+L Device:R R1
 U 1 1 60873A1F
 P 5900 1450
-F 0 "R?" H 5970 1496 50  0000 L CNN
+F 0 "R1" H 5970 1496 50  0000 L CNN
 F 1 "330" H 5970 1405 50  0000 L CNN
 F 2 "Resistor_SMD:R_0603_1608Metric" V 5830 1450 50  0001 C CNN
@@
 LED0
 $Comp
-L power:GND #PWR?
+L power:GND #PWR0101
 U 1 1 60874556
 P 5900 2250
-F 0 "#PWR?" H 5900 2000 50  0001 C CNN
+F 0 "#PWR0101" H 5900 2000 50  0001 C CNN
 F 1 "GND" H 5905 2077 50  0000 C CNN
 F 2 "" H 5900 2250 50  0001 C CNN
@@
 $EndComp
 $Comp
-L Device:R R?
+L Device:R R2
 U 1 1 608761F7
 P 6350 1450
-F 0 "R?" H 6420 1496 50  0000 L CNN
+F 0 "R2" H 6420 1496 50  0000 L CNN
 F 1 "330" H 6420 1405 50  0000 L CNN
 F 2 "Resistor_SMD:R_0603_1608Metric" V 6280 1450 50  0001 C CNN
@@
 LED1
 $Comp
-L power:GND #PWR?
+L power:GND #PWR0102
 U 1 1 608761FE
 P 6350 2250
-F 0 "#PWR?" H 6350 2000 50  0001 C CNN
+F 0 "#PWR0102" H 6350 2000 50  0001 C CNN
 F 1 "GND" H 6355 2077 50  0000 C CNN
 F 2 "" H 6350 2250 50  0001 C CNN
@@
 $EndComp
 $Comp
-L Device:R R?
+L Device:R R3
 U 1 1 608794FE
 P 6750 1450
-F 0 "R?" H 6820 1496 50  0000 L CNN
+F 0 "R3" H 6820 1496 50  0000 L CNN
 F 1 "330" H 6820 1405 50  0000 L CNN
 F 2 "Resistor_SMD:R_0603_1608Metric" V 6680 1450 50  0001 C CNN
@@
 LED2
 $Comp
-L power:GND #PWR?
+L power:GND #PWR0103
 U 1 1 60879505
 P 6750 2250
-F 0 "#PWR?" H 6750 2000 50  0001 C CNN
+F 0 "#PWR0103" H 6750 2000 50  0001 C CNN
 F 1 "GND" H 6755 2077 50  0000 C CNN
 F 2 "" H 6750 2250 50  0001 C CNN
@@
 $EndComp
 $Comp
-L Device:R R?
+L Device:R R4
 U 1 1 60879514
 P 7200 1450
-F 0 "R?" H 7270 1496 50  0000 L CNN
+F 0 "R4" H 7270 1496 50  0000 L CNN
 F 1 "330" H 7270 1405 50  0000 L CNN
 F 2 "Resistor_SMD:R_0603_1608Metric" V 7130 1450 50  0001 C CNN
@@
 LED3
 $Comp
-L power:GND #PWR?
+L power:GND #PWR0104
 U 1 1 6087951B
 P 7200 2250
-F 0 "#PWR?" H 7200 2000 50  0001 C CNN
+F 0 "#PWR0104" H 7200 2000 50  0001 C CNN
 F 1 "GND" H 7205 2077 50  0000 C CNN
 F 2 "" H 7200 2250 50  0001 C CNN
@@
 $EndComp
 $Comp
-L Device:R R?
+L Device:R R5
 U 1 1 6087FA40
 P 7600 1450
-F 0 "R?" H 7670 1496 50  0000 L CNN
+F 0 "R5" H 7670 1496 50  0000 L CNN
 F 1 "330" H 7670 1405 50  0000 L CNN
 F 2 "Resistor_SMD:R_0603_1608Metric" V 7530 1450 50  0001 C CNN
@@
 LED4
 $Comp
-L power:GND #PWR?
+L power:GND #PWR0105
 U 1 1 6087FA47
 P 7600 2250
-F 0 "#PWR?" H 7600 2000 50  0001 C CNN
+F 0 "#PWR0105" H 7600 2000 50  0001 C CNN
 F 1 "GND" H 7605 2077 50  0000 C CNN
 F 2 "" H 7600 2250 50  0001 C CNN
@@
 $EndComp
 $Comp
-L Device:R R?
+L Device:R R6
 U 1 1 6087FA56
 P 8050 1450
-F 0 "R?" H 8120 1496 50  0000 L CNN
+F 0 "R6" H 8120 1496 50  0000 L CNN
 F 1 "330" H 8120 1405 50  0000 L CNN
 F 2 "Resistor_SMD:R_0603_1608Metric" V 7980 1450 50  0001 C CNN
@@
 LED5
 $Comp
-L power:GND #PWR?
+L power:GND #PWR0106
 U 1 1 6087FA5D
 P 8050 2250
-F 0 "#PWR?" H 8050 2000 50  0001 C CNN
+F 0 "#PWR0106" H 8050 2000 50  0001 C CNN
 F 1 "GND" H 8055 2077 50  0000 C CNN
 F 2 "" H 8050 2250 50  0001 C CNN
@@
 $EndComp
 $Comp
-L Device:R R?
+L Device:R R7
 U 1 1 6087FA6C
 P 8450 1450
-F 0 "R?" H 8520 1496 50  0000 L CNN
+F 0 "R7" H 8520 1496 50  0000 L CNN
 F 1 "330" H 8520 1405 50  0000 L CNN
 F 2 "Resistor_SMD:R_0603_1608Metric" V 8380 1450 50  0001 C CNN
@@
 LED6
 $Comp
-L power:GND #PWR?
+L power:GND #PWR0107
 U 1 1 6087FA73
 P 8450 2250
-F 0 "#PWR?" H 8450 2000 50  0001 C CNN
+F 0 "#PWR0107" H 8450 2000 50  0001 C CNN
 F 1 "GND" H 8455 2077 50  0000 C CNN
 F 2 "" H 8450 2250 50  0001 C CNN
@@
 $EndComp
 $Comp
-L Device:R R?
+L Device:R R8
 U 1 1 6087FA82
 P 8900 1450
-F 0 "R?" H 8970 1496 50  0000 L CNN
+F 0 "R8" H 8970 1496 50  0000 L CNN
 F 1 "330" H 8970 1405 50  0000 L CNN
 F 2 "Resistor_SMD:R_0603_1608Metric" V 8830 1450 50  0001 C CNN
@@
 LED7
 $Comp
-L power:GND #PWR?
+L power:GND #PWR0108
 U 1 1 6087FA89
 P 8900 2250
-F 0 "#PWR?" H 8900 2000 50  0001 C CNN
+F 0 "#PWR0108" H 8900 2000 50  0001 C CNN
 F 1 "GND" H 8905 2077 50  0000 C CNN
 F 2 "" H 8900 2250 50  0001 C CNN
@@
 	2500 1550 2350 1550
 $Comp
-L power:GND #PWR?
+L power:GND #PWR0109
 U 1 1 608849A4
 P 2350 1950
-F 0 "#PWR?" H 2350 1700 50  0001 C CNN
+F 0 "#PWR0109" H 2350 1700 50  0001 C CNN
 F 1 "GND" V 2355 1822 50  0000 R CNN
 F 2 "" H 2350 1950 50  0001 C CNN
@@
 $EndComp
 $Comp
-L power:GND #PWR?
+L power:GND #PWR0110
 U 1 1 608851EE
 P 3150 1950
-F 0 "#PWR?" H 3150 1700 50  0001 C CNN
+F 0 "#PWR0110" H 3150 1700 50  0001 C CNN
 F 1 "GND" V 3155 1822 50  0000 R CNN
 F 2 "" H 3150 1950 50  0001 C CNN
