File: PMod_Infrared_Array/PMod_Infrared_Array.sch (KiCad schematic (older format))
At the start: 12 parts

Commit message: Add LEDs and lable components
Parts:
- added D? (x2): LED, LED_SMD:LED_0603_1608Metric, symbol Device:LED
- added R1, R2: R, Resistor_SMD:R_0603_1608Metric, symbol Device:R
- C? (x4): footprint (none) -> Capacitor_SMD:C_0603_1608Metric
- R3, R4, R5, R6, R7: renamed from R?; footprint (none) -> Resistor_SMD:R_0603_1608Metric
- R?: footprint (none) -> Resistor_SMD:R_0603_1608Metric
Connections:
- net GND: now also D?.1 (K), D?.1 (K)
- net INT: now also J?.10 (Pin_10)
- net SCL: now also J?.9 (Pin_9)
- net SDA: now also J?.4 (Pin_4)
- net LED0: now reaches J?.1 (Pin_1)
- net LED0: now also R1.1
- net LED1: now reaches J?.12 (Pin_12)
- net LED1: now also R2.1
- new net: D?.2 (A), R1.2
- new net: D?.2 (A), R2.2
- no-connect marks 5 -> 8
Changed lines of the file:
@@
 Text GLabel 8150 2850 2    50   Input ~ 0
 INT
-Text GLabel 3000 2550 2    50   Input ~ 0
+Text GLabel 1650 2900 0    50   Input ~ 0
 SDA
-Text GLabel 3000 2650 2    50   Input ~ 0
+Text GLabel 2650 2900 2    50   Input ~ 0
 SCL
-Text GLabel 3000 2750 2    50   Input ~ 0
+Text GLabel 2650 2800 2    50   Input ~ 0
 INT
 $Comp
@@
 F 0 "C?" H 4415 2396 50  0000 L CNN
 F 1 "0.1u" H 4415 2305 50  0000 L CNN
-F 2 "" H 4338 2200 50  0001 C CNN
+F 2 "Capacitor_SMD:C_0603_1608Metric" H 4338 2200 50  0001 C CNN
 F 3 "~" H 4300 2350 50  0001 C CNN
 	1    4300 2350
@@
 F 0 "C?" H 4415 3396 50  0000 L CNN
 F 1 "10u" H 4415 3305 50  0000 L CNN
-F 2 "" H 4338 3200 50  0001 C CNN
+F 2 "Capacitor_SMD:C_0603_1608Metric" H 4338 3200 50  0001 C CNN
 F 3 "~" H 4300 3350 50  0001 C CNN
 	1    4300 3350
@@
 F 0 "C?" H 7765 3846 50  0000 L CNN
 F 1 "1.5u" H 7765 3755 50  0000 L CNN
-F 2 "" H 7688 3650 50  0001 C CNN
+F 2 "Capacitor_SMD:C_0603_1608Metric" H 7688 3650 50  0001 C CNN
 F 3 "~" H 7650 3800 50  0001 C CNN
 	1    7650 3800
@@
 F 0 "C?" H 8215 3846 50  0000 L CNN
 F 1 "1u" H 8215 3755 50  0000 L CNN
-F 2 "" H 8138 3650 50  0001 C CNN
+F 2 "Capacitor_SMD:C_0603_1608Metric" H 8138 3650 50  0001 C CNN
 F 3 "~" H 8100 3800 50  0001 C CNN
 	1    8100 3800
@@
 $EndComp
 $Comp
-L Device:R R?
+L Device:R R7
 U 1 1 60947081
 P 8100 4150
-F 0 "R?" H 8170 4196 50  0000 L CNN
+F 0 "R7" H 8170 4196 50  0000 L CNN
 F 1 "20" H 8170 4105 50  0000 L CNN
-F 2 "" V 8030 4150 50  0001 C CNN
+F 2 "Resistor_SMD:R_0603_1608Metric" V 8030 4150 50  0001 C CNN
 F 3 "~" H 8100 4150 50  0001 C CNN
 	1    8100 4150
@@
 	7300 3650 7650 3650
 $Comp
-L Device:R R?
+L Device:R R3
 U 1 1 609496B6
 P 7400 2250
-F 0 "R?" H 7470 2296 50  0000 L CNN
+F 0 "R3" H 7470 2296 50  0000 L CNN
 F 1 "10K" H 7470 2205 50  0000 L CNN
-F 2 "" V 7330 2250 50  0001 C CNN
+F 2 "Resistor_SMD:R_0603_1608Metric" V 7330 2250 50  0001 C CNN
 F 3 "~" H 7400 2250 50  0001 C CNN
 	1    7400 2250
@@
 $EndComp
 $Comp
-L Device:R R?
+L Device:R R4
 U 1 1 60949E91
 P 7700 2250
-F 0 "R?" H 7770 2296 50  0000 L CNN
+F 0 "R4" H 7770 2296 50  0000 L CNN
 F 1 "10K" H 7770 2205 50  0000 L CNN
-F 2 "" V 7630 2250 50  0001 C CNN
+F 2 "Resistor_SMD:R_0603_1608Metric" V 7630 2250 50  0001 C CNN
 F 3 "~" H 7700 2250 50  0001 C CNN
 	1    7700 2250
@@
 $EndComp
 $Comp
-L Device:R R?
+L Device:R R5
 U 1 1 6094A276
 P 8000 2250
-F 0 "R?" H 8070 2296 50  0000 L CNN
+F 0 "R5" H 8070 2296 50  0000 L CNN
 F 1 "10K" H 8070 2205 50  0000 L CNN
-F 2 "" V 7930 2250 50  0001 C CNN
+F 2 "Resistor_SMD:R_0603_1608Metric" V 7930 2250 50  0001 C CNN
 F 3 "~" H 8000 2250 50  0001 C CNN
 	1    8000 2250
@@
 F 0 "R?" H 9070 3246 50  0000 L CNN
 F 1 "0" H 9070 3155 50  0000 L CNN
-F 2 "" V 8930 3200 50  0001 C CNN
+F 2 "Resistor_SMD:R_0603_1608Metric" V 8930 3200 50  0001 C CNN
 F 3 "~" H 9000 3200 50  0001 C CNN
 	1    9000 3200
@@
 	8100 4300 8100 4400
 $Comp
-L Device:R R?
+L Device:R R6
 U 1 1 60953239
 P 9000 2650
-F 0 "R?" H 9070 2696 50  0000 L CNN
+F 0 "R6" H 9070 2696 50  0000 L CNN
 F 1 "10k" H 9070 2605 50  0000 L CNN
-F 2 "" V 8930 2650 50  0001 C CNN
+F 2 "Resistor_SMD:R_0603_1608Metric" V 8930 2650 50  0001 C CNN
 F 3 "~" H 9000 2650 50  0001 C CNN
 	1    9000 2650
@@
 Text Notes 4450 2150 0    50   ~ 0
 VPP Decoupling
+Wire Wire Line
+	2650 2800 2400 2800
+Wire Wire Line
+	2400 2900 2650 2900
+Wire Wire Line
+	1900 2900 1650 2900
+NoConn ~ 2400 2700
+NoConn ~ 1900 2700
+NoConn ~ 1900 2800
+Text GLabel 1650 2600 0    50   Input ~ 0
+LED0
+Text GLabel 2650 2600 2    50   Input ~ 0
+LED1
+Wire Wire Line
+	2650 2600 2400 2600
+Wire Wire Line
+	1900 2600 1650 2600
+Text GLabel 1600 4150 0    50   Input ~ 0
+LED0
+Text GLabel 2700 4150 0    50   Input ~ 0
+LED1
+$Comp
+L Device:R R1
+U 1 1 6094A679
+P 1900 4350
+F 0 "R1" H 1970 4396 50  0000 L CNN
+F 1 "R" H 1970 4305 50  0000 L CNN
+F 2 "Resistor_SMD:R_0603_1608Metric" V 1830 4350 50  0001 C CNN
+F 3 "~" H 1900 4350 50  0001 C CNN
+	1    1900 4350
+	1    0    0    -1
+$EndComp
+$Comp
+L Device:R R2
+U 1 1 6094AADD
+P 2950 4350
+F 0 "R2" H 3020 4396 50  0000 L CNN
+F 1 "R" H 3020 4305 50  0000 L CNN
+F 2 "Resistor_SMD:R_0603_1608Metric" V 2880 4350 50  0001 C CNN
+F 3 "~" H 2950 4350 50  0001 C CNN
+	1    2950 4350
+	1    0    0    -1
+$EndComp
+$Comp
+L Device:LED D?
+U 1 1 6094B201
+P 1900 4850
+F 0 "D?" V 1939 4732 50  0000 R CNN
+F 1 "LED" V 1848 4732 50  0000 R CNN
+F 2 "LED_SMD:LED_0603_1608Metric" H 1900 4850 50  0001 C CNN
+F 3 "~" H 1900 4850 50  0001 C CNN
+	1    1900 4850
+	0    -1   -1   0
+$EndComp
+$Comp
+L Device:LED D?
+U 1 1 6094BA91
+P 2950 4850
+F 0 "D?" V 2989 4732 50  0000 R CNN
+F 1 "LED" V 2898 4732 50  0000 R CNN
+F 2 "LED_SMD:LED_0603_1608Metric" H 2950 4850 50  0001 C CNN
+F 3 "~" H 2950 4850 50  0001 C CNN
+	1    2950 4850
+	0    -1   -1   0
+$EndComp
+$Comp
+L power:GND #PWR?
+U 1 1 6094C265
+P 1900 5150
+F 0 "#PWR?" H 1900 4900 50  0001 C CNN
+F 1 "GND" H 1905 4977 50  0000 C CNN
+F 2 "" H 1900 5150 50  0001 C CNN
+F 3 "" H 1900 5150 50  0001 C CNN
+	1    1900 5150
+	1    0    0    -1
+$EndComp
+$Comp
+L power:GND #PWR?
+U 1 1 6094C94C
+P 2950 5150
+F 0 "#PWR?" H 2950 4900 50  0001 C CNN
+F 1 "GND" H 2955 4977 50  0000 C CNN
+F 2 "" H 2950 5150 50  0001 C CNN
+F 3 "" H 2950 5150 50  0001 C CNN
+	1    2950 5150
+	1    0    0    -1
+$EndComp
+Wire Wire Line
+	2950 4200 2950 4150
+Wire Wire Line
+	2950 4150 2700 4150
+Wire Wire Line
+	1900 4200 1900 4150
+Wire Wire Line
+	1900 4150 1600 4150
+Wire Wire Line
+	1900 4500 1900 4700
+Wire Wire Line
+	1900 5000 1900 5150
+Wire Wire Line
+	2950 5150 2950 5000
+Wire Wire Line
+	2950 4700 2950 4500
 $EndSCHEMATC

Commit message: Initial PCB layout of the board
Parts:
- J1: renamed from J?; footprint (none) -> Connector_PinHeader_2.54mm:PinHeader_2x06_P2.54mm_Vertical; symbol Connector_Generic:Conn_02x06_Counter_Clockwise -> Connector_Generic:Conn_02x06_Odd_Even
- gave numbers to parts that had none: 8
Connections:
- net +3V3: now also J1.11 (Pin_11), J1.12 (Pin_12); no longer J1.6 (Pin_6), J1.7 (Pin_7)
- net GND: now also J1.10 (Pin_10), J1.9 (Pin_9); no longer J1.5 (Pin_5), J1.8 (Pin_8)
- net INT: now also J1.6 (Pin_6); no longer J1.10 (Pin_10)
- net LED1: now also J1.2 (Pin_2); no longer J1.12 (Pin_12)
- net SCL: now also J1.8 (Pin_8); no longer J1.9 (Pin_9)
- net SDA: now also J1.7 (Pin_7); no longer J1.4 (Pin_4)
Changed lines of the file:
@@
 $EndDescr
 $Comp
-L JJH_Library:AMG8834 IC?
+L JJH_Library:AMG8834 IC1
 U 1 1 60937256
 P 5800 2650
-F 0 "IC?" H 6550 2915 50  0000 C CNN
+F 0 "IC1" H 6550 2915 50  0000 C CNN
 F 1 "AMG8834" H 6550 2824 50  0000 C CNN
 F 2 "AMG8834" H 7150 2750 50  0001 L CNN
@@
 NoConn ~ 5800 3650
 $Comp
-L power:+3V3 #PWR?
+L power:+3V3 #PWR0101
 U 1 1 60938147
 P 5700 2350
-F 0 "#PWR?" H 5700 2200 50  0001 C CNN
+F 0 "#PWR0101" H 5700 2200 50  0001 C CNN
 F 1 "+3V3" H 5715 2523 50  0000 C CNN
 F 2 "" H 5700 2350 50  0001 C CNN
@@
 $EndComp
 $Comp
-L power:+3V3 #PWR?
+L power:+3V3 #PWR0102
 U 1 1 609384E2
 P 4300 3200
-F 0 "#PWR?" H 4300 3050 50  0001 C CNN
+F 0 "#PWR0102" H 4300 3050 50  0001 C CNN
 F 1 "+3V3" H 4315 3373 50  0000 C CNN
 F 2 "" H 4300 3200 50  0001 C CNN
@@
 $EndComp
 $Comp
-L power:+3V3 #PWR?
+L power:+3V3 #PWR0103
 U 1 1 609388E3
 P 4300 2200
-F 0 "#PWR?" H 4300 2050 50  0001 C CNN
+F 0 "#PWR0103" H 4300 2050 50  0001 C CNN
 F 1 "+3V3" H 4315 2373 50  0000 C CNN
 F 2 "" H 4300 2200 50  0001 C CNN
@@
 $EndComp
 $Comp
-L power:GND #PWR?
+L power:GND #PWR0104
 U 1 1 60938E6A
 P 5700 2900
-F 0 "#PWR?" H 5700 2650 50  0001 C CNN
+F 0 "#PWR0104" H 5700 2650 50  0001 C CNN
 F 1 "GND" H 5705 2727 50  0000 C CNN
 F 2 "" H 5700 2900 50  0001 C CNN
@@
 	5700 2650 5700 2350
 $Comp
-L Connector_Generic:Conn_02x06_Counter_Clockwise J?
+L Connector_Generic:Conn_02x06_Odd_Even J1
 U 1 1 6093A1DB
 P 2100 2800
-F 0 "J?" H 2150 3217 50  0000 C CNN
+F 0 "J1" H 2150 3217 50  0000 C CNN
 F 1 "Conn_02x06_Counter_Clockwise" H 2150 3126 50  0000 C CNN
-F 2 "" H 2100 2800 50  0001 C CNN
+F 2 "Connector_PinHeader_2.54mm:PinHeader_2x06_P2.54mm_Vertical" H 2100 2800 50  0001 C CNN
 F 3 "~" H 2100 2800 50  0001 C CNN
 	1    2100 2800
@@
 $EndComp
 $Comp
-L power:+3V3 #PWR?
+L power:+3V3 #PWR0105
 U 1 1 6093D9B8
 P 2650 3100
-F 0 "#PWR?" H 2650 2950 50  0001 C CNN
+F 0 "#PWR0105" H 2650 2950 50  0001 C CNN
 F 1 "+3V3" V 2650 3350 50  0000 C CNN
 F 2 "" H 2650 3100 50  0001 C CNN
@@
 $EndComp
 $Comp
-L power:+3V3 #PWR?
+L power:+3V3 #PWR0106
 U 1 1 6093E45C
 P 1650 3100
-F 0 "#PWR?" H 1650 2950 50  0001 C CNN
+F 0 "#PWR0106" H 1650 2950 50  0001 C CNN
 F 1 "+3V3" V 1650 3350 50  0000 C CNN
 F 2 "" H 1650 3100 50  0001 C CNN
@@
 $EndComp
 $Comp
-L power:GND #PWR?
+L power:GND #PWR0107
 U 1 1 6093E951
 P 2650 3000
-F 0 "#PWR?" H 2650 2750 50  0001 C CNN
+F 0 "#PWR0107" H 2650 2750 50  0001 C CNN
 F 1 "GND" V 2650 2800 50  0000 R CNN
 F 2 "" H 2650 3000 50  0001 C CNN
@@
 $EndComp
 $Comp
-L power:GND #PWR?
+L power:GND #PWR0108
 U 1 1 6093F149
 P 1650 3000
-F 0 "#PWR?" H 1650 2750 50  0001 C CNN
+F 0 "#PWR0108" H 1650 2750 50  0001 C CNN
 F 1 "GND" V 1650 2850 50  0000 R CNN
 F 2 "" H 1650 3000 50  0001 C CNN
@@
 INT
 $Comp
-L power:GND #PWR?
+L power:GND #PWR0109
 U 1 1 609422BD
 P 4300 2500
-F 0 "#PWR?" H 4300 2250 50  0001 C CNN
+F 0 "#PWR0109" H 4300 2250 50  0001 C CNN
 F 1 "GND" H 4305 2327 50  0000 C CNN
 F 2 "" H 4300 2500 50  0001 C CNN
@@
 $EndComp
 $Comp
-L power:GND #PWR?
+L power:GND #PWR0110
 U 1 1 609425A2
 P 4300 3500
-F 0 "#PWR?" H 4300 3250 50  0001 C CNN
+F 0 "#PWR0110" H 4300 3250 50  0001 C CNN
 F 1 "GND" H 4305 3327 50  0000 C CNN
 F 2 "" H 4300 3500 50  0001 C CNN
@@
 $EndComp
 $Comp
-L Device:C C?
+L Device:C C1
 U 1 1 60942A0D
 P 4300 2350
-F 0 "C?" H 4415 2396 50  0000 L CNN
+F 0 "C1" H 4415 2396 50  0000 L CNN
 F 1 "0.1u" H 4415 2305 50  0000 L CNN
 F 2 "Capacitor_SMD:C_0603_1608Metric" H 4338 2200 50  0001 C CNN
@@
 $EndComp
 $Comp
-L Device:C C?
+L Device:C C2
 U 1 1 609434D9
 P 4300 3350
-F 0 "C?" H 4415 3396 50  0000 L CNN
+F 0 "C2" H 4415 3396 50  0000 L CNN
 F 1 "10u" H 4415 3305 50  0000 L CNN
 F 2 "Capacitor_SMD:C_0603_1608Metric" H 4338 3200 50  0001 C CNN
@@
 $EndComp
 $Comp
-L power:GND #PWR?
+L power:GND #PWR0111
 U 1 1 609466CF
 P 7650 3950
-F 0 "#PWR?" H 7650 3700 50  0001 C CNN
+F 0 "#PWR0111" H 7650 3700 50  0001 C CNN
 F 1 "GND" H 7655 3777 50  0000 C CNN
 F 2 "" H 7650 3950 50  0001 C CNN
@@
 $EndComp
 $Comp
-L power:GND #PWR?
+L power:GND #PWR0112
 U 1 1 609466D5
 P 8100 4400
-F 0 "#PWR?" H 8100 4150 50  0001 C CNN
+F 0 "#PWR0112" H 8100 4150 50  0001 C CNN
 F 1 "GND" H 8105 4227 50  0000 C CNN
 F 2 "" H 8100 4400 50  0001 C CNN
@@
 $EndComp
 $Comp
-L Device:C C?
+L Device:C C3
 U 1 1 609466DB
 P 7650 3800
-F 0 "C?" H 7765 3846 50  0000 L CNN
+F 0 "C3" H 7765 3846 50  0000 L CNN
 F 1 "1.5u" H 7765 3755 50  0000 L CNN
 F 2 "Capacitor_SMD:C_0603_1608Metric" H 7688 3650 50  0001 C CNN
@@
 $EndComp
 $Comp
-L Device:C C?
+L Device:C C4
 U 1 1 609466E1
 P 8100 3800
-F 0 "C?" H 8215 3846 50  0000 L CNN
+F 0 "C4" H 8215 3846 50  0000 L CNN
 F 1 "1u" H 8215 3755 50  0000 L CNN
 F 2 "Capacitor_SMD:C_0603_1608Metric" H 8138 3650 50  0001 C CNN
@@
 Connection ~ 7400 2650
 $Comp
-L power:+3V3 #PWR?
+L power:+3V3 #PWR0113
 U 1 1 6094CCD1
 P 7400 1950
-F 0 "#PWR?" H 7400 1800 50  0001 C CNN
+F 0 "#PWR0113" H 7400 1800 50  0001 C CNN
 F 1 "+3V3" H 7415 2123 50  0000 C CNN
 F 2 "" H 7400 1950 50  0001 C CNN
@@
 $EndComp
 $Comp
-L power:+3V3 #PWR?
+L power:+3V3 #PWR0114
 U 1 1 6094CFF8
 P 7700 1950
-F 0 "#PWR?" H 7700 1800 50  0001 C CNN
+F 0 "#PWR0114" H 7700 1800 50  0001 C CNN
 F 1 "+3V3" H 7715 2123 50  0000 C CNN
 F 2 "" H 7700 1950 50  0001 C CNN
@@
 $EndComp
 $Comp
-L power:+3V3 #PWR?
+L power:+3V3 #PWR0115
 U 1 1 6094D331
 P 8000 1950
-F 0 "#PWR?" H 8000 1800 50  0001 C CNN
+F 0 "#PWR0115" H 8000 1800 50  0001 C CNN
 F 1 "+3V3" H 8015 2123 50  0000 C CNN
 F 2 "" H 8000 1950 50  0001 C CNN
@@
 	7400 2100 7400 1950
 $Comp
-L Device:R R?
+L Device:R R8
 U 1 1 6094ED1F
 P 9000 3200
-F 0 "R?" H 9070 3246 50  0000 L CNN
+F 0 "R8" H 9070 3246 50  0000 L CNN
 F 1 "0" H 9070 3155 50  0000 L CNN
 F 2 "Resistor_SMD:R_0603_1608Metric" V 8930 3200 50  0001 C CNN
@@
 $EndComp
 $Comp
-L power:GND #PWR?
+L power:GND #PWR0116
 U 1 1 6094F9F4
 P 9000 3450
-F 0 "#PWR?" H 9000 3200 50  0001 C CNN
+F 0 "#PWR0116" H 9000 3200 50  0001 C CNN
 F 1 "GND" H 9005 3277 50  0000 C CNN
 F 2 "" H 9000 3450 50  0001 C CNN
@@
 $EndComp
 $Comp
-L power:+3V3 #PWR?
+L power:+3V3 #PWR0117
 U 1 1 6095383F
 P 9000 2400
-F 0 "#PWR?" H 9000 2250 50  0001 C CNN
+F 0 "#PWR0117" H 9000 2250 50  0001 C CNN
 F 1 "+3V3" H 9015 2573 50  0000 C CNN
 F 2 "" H 9000 2400 50  0001 C CNN
@@
 $EndComp
 $Comp
-L Device:LED D?
+L Device:LED D1
 U 1 1 6094B201
 P 1900 4850
-F 0 "D?" V 1939 4732 50  0000 R CNN
+F 0 "D1" V 1939 4732 50  0000 R CNN
 F 1 "LED" V 1848 4732 50  0000 R CNN
 F 2 "LED_SMD:LED_0603_1608Metric" H 1900 4850 50  0001 C CNN
@@
 $EndComp
 $Comp
-L Device:LED D?
+L Device:LED D2
 U 1 1 6094BA91
 P 2950 4850
-F 0 "D?" V 2989 4732 50  0000 R CNN
+F 0 "D2" V 2989 4732 50  0000 R CNN
 F 1 "LED" V 2898 4732 50  0000 R CNN
 F 2 "LED_SMD:LED_0603_1608Metric" H 2950 4850 50  0001 C CNN
@@
 $EndComp
 $Comp
-L power:GND #PWR?
+L power:GND #PWR0118
 U 1 1 6094C265
 P 1900 5150
-F 0 "#PWR?" H 1900 4900 50  0001 C CNN
+F 0 "#PWR0118" H 1900 4900 50  0001 C CNN
 F 1 "GND" H 1905 4977 50  0000 C CNN
 F 2 "" H 1900 5150 50  0001 C CNN
@@
 $EndComp
 $Comp
-L power:GND #PWR?
+L power:GND #PWR0119
 U 1 1 6094C94C
 P 2950 5150
-F 0 "#PWR?" H 2950 4900 50  0001 C CNN
+F 0 "#PWR0119" H 2950 4900 50  0001 C CNN
 F 1 "GND" H 2955 4977 50  0000 C CNN
 F 2 "" H 2950 5150 50  0001 C CNN
