File: PMod_Infrared_Array/PMod_Infrared_Array.kicad_pcb (KiCad board)
At the start: 2 copper layers, 50 x 18 mm, 17 parts, among them IC1 AMG8834, J1 Conn_02x06_Counter_Clockwise

Commit message: Add PMod connector labels on PCB
Other:
- board text added: "3V3"
- board text added: "GND"
- board text added: "INT"
- board text added: "LED 0"
- board text added: "LED 1"
- board text added: "PMod"
- board text added: "SCL"
- board text added: "SDA"
Changed lines of the file:
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@@
   (general
     (thickness 1.6)
-    (drawings 13)
+    (drawings 37)
     (tracks 152)
     (zones 0)
@@
     (34 B.Paste user)
     (35 F.Paste user)
-    (36 B.SilkS user)
+    (36 B.SilkS user hide)
     (37 F.SilkS user)
     (38 B.Mask user)
@@
     (tags resistor)
     (attr smd)
-    (fp_text reference R6 (at -2.7 0) (layer F.SilkS)
+    (fp_text reference R6 (at -2.825 0) (layer F.SilkS)
       (effects (font (size 1 1) (thickness 0.15)))
     )
@@
     (tags resistor)
     (attr smd)
-    (fp_text reference R5 (at -2.7 0) (layer F.SilkS)
+    (fp_text reference R5 (at -2.825 0) (layer F.SilkS)
       (effects (font (size 1 1) (thickness 0.15)))
     )
@@
     (tags resistor)
     (attr smd)
-    (fp_text reference R4 (at -2.5 0) (layer F.SilkS)
+    (fp_text reference R4 (at -2.825 0) (layer F.SilkS)
       (effects (font (size 1 1) (thickness 0.15)))
     )
@@
     (tags resistor)
     (attr smd)
-    (fp_text reference R3 (at -2.6 0.1) (layer F.SilkS)
+    (fp_text reference R3 (at -2.825 0) (layer F.SilkS)
       (effects (font (size 1 1) (thickness 0.15)))
     )
@@
     (tags resistor)
     (attr smd)
-    (fp_text reference R2 (at -2.575 0) (layer F.SilkS)
+    (fp_text reference R2 (at -2.825 0) (layer F.SilkS)
       (effects (font (size 1 1) (thickness 0.15)))
     )
@@
     (tags resistor)
     (attr smd)
-    (fp_text reference R1 (at -2.5 0) (layer F.SilkS)
+    (fp_text reference R1 (at -2.675 0) (layer F.SilkS)
       (effects (font (size 1 1) (thickness 0.15)))
     )
@@
     (tags LED)
     (attr smd)
-    (fp_text reference D2 (at 2.6 0) (layer F.SilkS)
+    (fp_text reference D2 (at 2.7875 0) (layer F.SilkS)
       (effects (font (size 1 1) (thickness 0.15)))
     )
@@
     (tags LED)
     (attr smd)
-    (fp_text reference D1 (at 2.4875 0) (layer F.SilkS)
+    (fp_text reference D1 (at 2.7875 0) (layer F.SilkS)
       (effects (font (size 1 1) (thickness 0.15)))
     )
@@
     (tags capacitor)
     (attr smd)
-    (fp_text reference C4 (at 3 0) (layer F.SilkS)
+    (fp_text reference C4 (at 2.775 0) (layer F.SilkS)
       (effects (font (size 1 1) (thickness 0.15)))
     )
@@
     (tags capacitor)
     (attr smd)
-    (fp_text reference C3 (at 3 0) (layer F.SilkS)
+    (fp_text reference C3 (at 2.775 0) (layer F.SilkS)
       (effects (font (size 1 1) (thickness 0.15)))
     )
@@
     (tags capacitor)
     (attr smd)
-    (fp_text reference C2 (at 3 0) (layer F.SilkS)
+    (fp_text reference C2 (at 2.775 0) (layer F.SilkS)
       (effects (font (size 1 1) (thickness 0.15)))
     )
@@
     (tags capacitor)
     (attr smd)
-    (fp_text reference C1 (at 3.025 0) (layer F.SilkS)
+    (fp_text reference C1 (at 2.775 0) (layer F.SilkS)
       (effects (font (size 1 1) (thickness 0.15)))
     )
@@
     )
   )
+  (gr_text 3V3 (at 119 92) (layer F.SilkS)
+    (effects (font (size 1 1) (thickness 0.15)))
+  )
+  (gr_text GND (at 119 89.25) (layer F.SilkS)
+    (effects (font (size 1 1) (thickness 0.15)))
+  )
+  (gr_line (start 117.5 77.25) (end 117.25 77.25) (layer F.SilkS) (width 0.12))
+  (gr_line (start 114 77.25) (end 117.25 77.25) (layer F.SilkS) (width 0.12))
+  (gr_line (start 113 78.25) (end 114 77.25) (layer F.SilkS) (width 0.12))
+  (gr_line (start 116.25 79.75) (end 115.75 79.25) (layer F.SilkS) (width 0.12))
+  (gr_line (start 117.5 79.75) (end 116.25 79.75) (layer F.SilkS) (width 0.12))
+  (gr_line (start 117.5 83.5) (end 115.75 83.5) (layer F.SilkS) (width 0.12))
+  (gr_line (start 114 85.25) (end 112.75 86.5) (layer F.SilkS) (width 0.12))
+  (gr_line (start 117.5 85.25) (end 114 85.25) (layer F.SilkS) (width 0.12))
+  (gr_line (start 116 86.75) (end 117.5 86.75) (layer F.SilkS) (width 0.12))
+  (gr_text SCL (at 119 86.75) (layer F.SilkS)
+    (effects (font (size 1 1) (thickness 0.15)))
+  )
+  (gr_text SDA (at 119 85.25) (layer F.SilkS)
+    (effects (font (size 1 1) (thickness 0.15)))
+  )
+  (gr_text INT (at 118.75 83.5) (layer F.SilkS)
+    (effects (font (size 1 1) (thickness 0.15)))
+  )
+  (gr_text "LED 1" (at 119.75 79.75) (layer F.SilkS)
+    (effects (font (size 1 1) (thickness 0.15)))
+  )
+  (gr_text "LED 0" (at 119.75 78) (layer F.SilkS)
+    (effects (font (size 1 1) (thickness 0.15)))
+  )
+  (gr_text PMod (at 122.75 82.75 90) (layer F.SilkS)
+    (effects (font (size 1 1) (thickness 0.15)))
+  )
+  (gr_line (start 116.5 88) (end 123.75 88) (layer F.SilkS) (width 0.12))
+  (gr_line (start 116.5 90.5) (end 123.75 90.5) (layer F.SilkS) (width 0.12))
+  (gr_line (start 110.5 93.5) (end 117 93.5) (layer F.SilkS) (width 0.12))
+  (gr_line (start 110.5 77) (end 110.5 93.5) (layer F.SilkS) (width 0.12))
+  (gr_line (start 123.75 77) (end 110.5 77) (layer F.SilkS) (width 0.12))
+  (gr_line (start 123.75 93.5) (end 123.75 77) (layer F.SilkS) (width 0.12))
+  (gr_line (start 117 93.5) (end 123.75 93.5) (layer F.SilkS) (width 0.12))
   (gr_text "8x8 Infrared Array\nTemperature Sensor\nPMod Board" (at 152 85 -90) (layer B.SilkS)
     (effects (font (size 1 1) (thickness 0.15)) (justify mirror))
