File: PMod_Neopixel/Hardware/Compact/PMod_Neopixel.sch (KiCad schematic (older format))
At the start: 14 parts, among them J1 Conn_02x06_Counter_Clockwise, J2 Conn_01x02

Commit message: Address design rules issues on the PCB
Changed lines of the file:
@@
 $EndComp
-Wire Wire Line
-	5100 1550 5100 1650
 Wire Wire Line
 	6250 1550 6250 1650
@@
 Wire Wire Line
 	8500 2250 8500 2350
-Wire Wire Line
-	7350 2350 7350 2250
 Wire Wire Line
 	6250 2250 6250 2350
@@
 Wire Wire Line
 	6250 3100 6250 3200
-Wire Wire Line
-	7350 3200 7350 3100
 Wire Wire Line
 	8500 3100 8500 3200
@@
 Wire Wire Line
 	2100 2150 1700 2150
-Wire Wire Line
-	1700 2050 2100 2050
 $Comp
 L Connector_Generic:Conn_01x02 J2
@@
 	2050 4500 2200 4500
 Wire Wire Line
+	2500 3850 2650 3850
+Wire Wire Line
+	7350 2250 7350 2350
+Wire Wire Line
+	5100 1650 5100 1550
+Wire Wire Line
+	1700 2050 2100 2050
+Wire Wire Line
+	7350 3200 7350 3100
+Wire Wire Line
 	2050 3850 2200 3850
-Wire Wire Line
-	2500 3850 2650 3850
 $EndSCHEMATC
