File: PMod_Neopixel/Hardware/Compact/PMod_Neopixel_compact.kicad_pcb (KiCad board)
At the start: 2 copper layers, 49.4 x 17 mm, 15 parts, among them J1 Conn_02x06_Counter_Clockwise, J2 Conn_01x02

Commit message: Address design rules issues on the PCB
Parts:
- moved R1 0.58 mm to (118.3, 101.3)
Routing:
- net +3V3: track 17.3 -> 17.9 mm
