File: PMod_Infrared_Array/Hardware/PMod_Infrared_Array.sch (KiCad schematic (older format))
At the start: 16 parts, among them IC1 AMG8834, J1 Conn_02x06_Counter_Clockwise

Commit message: Tidy up the schematic layout
Other:
- note added: "Decoupling"
- note added: "PMod Connector"
- note added: "SDA and SCL are placed to match the outputs \non the Pico PMod host board, so it can easily \nbe used with that board."
- note added: "Status LED 0"
- note added: "Status LED 1"
- note added: "Value for VDD Decoupling Capasitor \ntaken from Datashet"
- note added: "Value for Vpp Decoupling taken from Datashet"
- moved on the sheet: C1, C2, C3, C4, D1, D2, IC1, J1, R1, R2, R3, R4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

Commit message: Add values for the LED resistors
Parts:
- R1, R2: value R -> 330
Changed lines of the file:
@@
 P 1600 5450
 F 0 "R1" H 1670 5496 50  0000 L CNN
-F 1 "R" H 1670 5405 50  0000 L CNN
+F 1 "330" H 1670 5405 50  0000 L CNN
 F 2 "Resistor_SMD:R_0603_1608Metric" V 1530 5450 50  0001 C CNN
 F 3 "~" H 1600 5450 50  0001 C CNN
@@
 P 3400 5450
 F 0 "R2" H 3470 5496 50  0000 L CNN
-F 1 "R" H 3470 5405 50  0000 L CNN
+F 1 "330" H 3470 5405 50  0000 L CNN
 F 2 "Resistor_SMD:R_0603_1608Metric" V 3330 5450 50  0001 C CNN
 F 3 "~" H 3400 5450 50  0001 C CNN
