File: PMod_Infrared_Array/Hardware/PMod_Infrared_Array.kicad_pcb (KiCad board)
At the start: 2 copper layers, 50 x 18 mm, 17 parts, among them IC1 AMG8834, J1 Conn_02x06_Counter_Clockwise

Commit message: change the logo reference
Parts:
- renumbered G*** to L1
Changed lines of the file:
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@@
     (at 135 85.5 180)
     (attr through_hole)
-    (fp_text reference "G***" (at 0 0) (layer "B.SilkS") hide
+    (fp_text reference "L1" (at 0 0) (layer "B.SilkS") hide
         (effects (font (size 1.524 1.524) (thickness 0.3)) (justify mirror))
     )
