File: PMod_Infrared_Array/Hardware/PMod_Infrared_Array.kicad_pcb (KiCad board)
At the start: 2 copper layers, 50 x 18 mm, 17 parts, among them IC1 AMG8834, J1 Conn_02x06_Counter_Clockwise

Commit message: update the design rukes for thermal releif
Routing:
- net GND: track 7.55 -> 5.18 mm
Changed lines of the file:
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@@
     (tags "Through hole pin header THT 2x06 2.54mm double row")
     (attr exclude_from_pos_files exclude_from_bom)
-    (fp_text reference "J1" (at 1.27 -2.33) (layer "F.SilkS")
-        (effects (font (size 1 1) (thickness 0.15)))
+    (fp_text reference "J1" (at 1.24 -2.48) (layer "F.SilkS")
+        (effects (font (size 0.8 0.8) (thickness 0.15)))
     )
     (fp_text value "Conn_02x06_Counter_Clockwise" (at 1.27 15.03) (layer "F.Fab")
@@
     (style (thickness 0.15) (arrow_length 1.27) (text_position_mode 0) (extension_height 0.58642) (extension_offset 0) keep_text_aligned)
   )
-  (segment (start 115.86 89.14) (end 115.1 89.14) (width 0.25) (layer "F.Cu") (net 1))
   (segment (start 137 88.5) (end 137 89) (width 0.25) (layer "F.Cu") (net 1))
-  (segment (start 117 90) (end 116 89) (width 0.25) (layer "F.Cu") (net 1))
   (segment (start 131.15 85.35) (end 131.15 85.5) (width 0.25) (layer "F.Cu") (net 1))
-  (segment (start 116 89) (end 115.86 89.14) (width 0.25) (layer "F.Cu") (net 1))
   (segment (start 138.5 87.5) (end 138 87.5) (width 0.25) (layer "F.Cu") (net 1))
   (segment (start 133 83.5) (end 131.15 85.35) (width 0.25) (layer "F.Cu") (net 1))
@@
   (segment (start 129.5 81) (end 126.755009 78.255009) (width 0.25) (layer "F.Cu") (net 18))
   (zone (net 1) (net_name "GND") (layer "F.Cu") (hatch edge 0.508)
-    (connect_pads (clearance 0.508))
-    (min_thickness 0.254) (filled_areas_thickness no)
-    (fill yes (thermal_gap 0.508) (thermal_bridge_width 0.508))
+    (connect_pads (clearance 0.5))
+    (min_thickness 0.2) (filled_areas_thickness no)
+    (fill yes (thermal_gap 0.5) (thermal_bridge_width 0.5))
     (polygon
       (pts

Commit message: edit the design rules for libary error
Parts:
- R1, R2: value R -> 330
Connections:
- IC1 pad 1: Net-(IC1-Pad1) -> unconnected-(IC1-NC_1-Pad1)
- IC1 pad 11: Net-(IC1-Pad11) -> unconnected-(IC1-NC_4-Pad11)
- IC1 pad 14: Net-(IC1-Pad14) -> unconnected-(IC1-NC_5-Pad14)
- IC1 pad 7: Net-(IC1-Pad7) -> unconnected-(IC1-NC_2-Pad7)
- IC1 pad 8: Net-(IC1-Pad8) -> unconnected-(IC1-NC_3-Pad8)
- J1 pad 3: Net-(J1-Pad3) -> unconnected-(J1-Pin_3-Pad3)
- J1 pad 4: Net-(J1-Pad4) -> unconnected-(J1-Pin_4-Pad4)
- J1 pad 5: Net-(J1-Pad5) -> unconnected-(J1-Pin_5-Pad5)
