File: PMod_CC1101/Hardware/cc1101.kicad_pcb (KiCad board)
At the start: 4 copper layers, 40.5 x 17 mm, 18 parts, among them J1 Conn_Coaxial, J2 Conn_02x06_Odd_Even, U1 CC1101RGPR

Commit message: Update pin layout to match RP2040 PMod Board
Connections:
- J2 pad 3: SPI_TX -> GDO2
- J2 pad 4: SPI_CLK -> GDO0
- J2 pad 5: SPI_CSN -> SPI_CLK
- J2 pad 6: SPI_RX -> SPI_TX
- J2 pad 7: GDO2 -> SPI_RX
- J2 pad 8: GDO0 -> SPI_CSN
- U1 pad PAD: (no net) -> GND
Routing:
- net SPI_CSN: track 20.8 -> 13.8 mm
- net GND: track 26.6 -> 31.0 mm
- net GDO0: track 12.5 -> 16.7 mm, vias 0 -> 1
- net SPI_TX: track 15.3 -> 11.3 mm
- net SPI_RX: track 10.4 -> 13.4 mm
- net SPI_CLK: track 11.3 -> 13.6 mm
- net GDO2: track 13.2 -> 15.5 mm, vias 0 -> 1
