File: PMod_CC1101/Hardware/cc1101.kicad_pcb (KiCad board)
At the start: 2 copper layers, 16 parts, among them J1 Conn_Coaxial, J2 Conn_02x06_Odd_Even

Commit message: initial footprint for the CC1101 part
Parts:
- added C131: 3.9pF, Capacitor_SMD:C_0603_1608Metric, F.Cu at (162.5, 70.8)
- added U1: CC1101RGPR, Package_DFN_QFN:UQFN-20-1EP_4x4mm_P0.5mm_EP2.8x2.8mm, F.Cu at (145.8, 61.8)
- moved J1 30.7 mm to (173.5, 62.2), turned to 90 degrees
- moved C51 16.4 mm to (156.3, 76.0)
- moved L123 16.3 mm to (165.8, 65.0)
- moved C101 14.9 mm to (151.0, 69.2), turned to 90 degrees
- moved C123 14.1 mm to (156.2, 53.2)
- moved XTAL1 13.3 mm to (145.8, 69.0), turned to 180 degrees
- moved R171 12.7 mm to (145.8, 56.0)
- moved C81 12.4 mm to (140.5, 69.0), turned to 90 degrees
- moved C125 12.0 mm to (165.8, 62.0)
- moved C122 11.5 mm to (156.0, 70.5)
- moved C121 10.8 mm to (160.5, 65.0)
- moved L131 9.56 mm to (155.8, 65.2)
- moved L122 6.82 mm to (160.5, 62.0)
- moved L121 2.49 mm to (161.2, 58.0)

Commit message: Component positioned within board edges
Parts:
- moved C51 18.1 mm to (139.8, 68.5), turned to 90 degrees
- moved C131 14.7 mm to (154.7, 58.2)
- moved C123 12.9 mm to (163.0, 64.2)
- moved C122 12.7 mm to (159.2, 58.2)
- moved L121 11.2 mm to (154.5, 67.0), turned to 180 degrees
- moved C124 9.27 mm to (159.3, 67.0)
- moved L123 7.54 mm to (159.2, 61.2)
- moved C121 5.82 mm to (154.7, 64.2), turned to 180 degrees
- moved L131 4.13 mm to (154.7, 61.2)
- moved J1 4.07 mm to (169.5, 63.0)
- moved C125 2.85 mm to (163.0, 61.2), turned to 180 degrees
- moved L122 2.57 mm to (159.2, 64.2)
- moved C81 1.35 mm to (141.8, 68.5)
- moved C101 1.03 mm to (150.2, 68.5)
- moved XTAL1 0.56 mm to (146.0, 68.5)
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Other:
- board outline added: 40.5 x 17 mm

Commit message: line up the RF componnents on the board
Parts:
- moved C124 6.03 mm to (153.3, 67.8), turned to 180 degrees
- moved L122 2.84 mm to (156.7, 63.0)
- moved C125 2.46 mm to (164.7, 63.0)
- moved U1 2.44 mm to (148.0, 62.7)
- moved C122 2.39 mm to (158.8, 60.6), turned to 90 degrees
- moved L123 2.30 mm to (160.7, 63.0)
- moved C131 2.17 mm to (152.7, 59.0), turned to 270 degrees
- moved L121 1.51 mm to (153.3, 66.1)
- moved C121 1.41 mm to (153.3, 64.4)
- moved L131 1.34 mm to (153.4, 61.5)
- moved C123 1.16 mm to (162.7, 65.4), turned to 270 degrees
- moved C81 0.70 mm to (141.8, 69.2)
- moved XTAL1 0.70 mm to (146.0, 69.2)
- moved C101 0.70 mm to (150.2, 69.2)
- moved C51 0.69 mm to (140.1, 69.1)

Commit message: initial PCB routing
Parts:
- U1: footprint Package_DFN_QFN:UQFN-20-1EP_4x4mm_P0.5mm_EP2.8x2.8mm -> jjh:QFN50P400X400X100-21N-D
- moved C51 5.72 mm to (142.7, 64.0), turned to 0 degrees
- moved R171 2.48 mm to (147.7, 57.2)
- moved U1 0.28 mm to (148.2, 62.9)
Connections:
- U1 pad PAD: GND -> (no net)
Routing:
- net GND: track 0.00 -> 26.6 mm, vias 0 -> 14
- net SPI_CSN: track 0.00 -> 20.8 mm
- net SPI_TX: track 0.00 -> 15.3 mm
- net +3V3: track 0.00 -> 14.6 mm, vias 0 -> 6
- net GDO2: track 0.00 -> 13.2 mm
- net GDO0: track 0.00 -> 12.5 mm
- net SPI_CLK: track 0.00 -> 11.3 mm
- net Net-(C81-Pad1): track 0.00 -> 10.7 mm
- net SPI_RX: track 0.00 -> 10.4 mm
- net Net-(C101-Pad2): track 0.00 -> 6.30 mm
- net Net-(C121-Pad2): track 0.00 -> 5.83 mm
- net Net-(C131-Pad2): track 0.00 -> 4.87 mm
- net Net-(C121-Pad1): track 0.00 -> 4.74 mm
- net Net-(C125-Pad1): track 0.00 -> 4.20 mm
- net Net-(C122-Pad1): track 0.00 -> 4.10 mm
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- added copper zone on In2.Cu, net +3V3
- added copper zone on In1.Cu, net GND
Other:
- copper layers 2 -> 4

Commit message: Add GND filled zones
Routing:
- net GND: vias 14 -> 45
- added copper zone on B.Cu, net GND
- added copper zone on F.Cu, net GND
Changed lines of the file:
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@@
     (thickness 1.6)
     (drawings 10)
-    (tracks 139)
+    (tracks 170)
     (zones 0)
     (modules 18)
@@
     (1 In1.Cu signal hide)
     (2 In2.Cu signal hide)
-    (31 B.Cu signal)
+    (31 B.Cu signal hide)
     (32 B.Adhes user)
     (33 F.Adhes user)
@@
   (segment (start 142.95 68.05) (end 142.1 67.2) (width 0.2) (layer F.Cu) (net 2))
   (segment (start 144.1 68.05) (end 142.95 68.05) (width 0.2) (layer F.Cu) (net 2))
+  (via (at 158.7 64.2) (size 0.8) (drill 0.4) (layers F.Cu B.Cu) (net 2))
+  (via (at 157.2 61.5) (size 0.8) (drill 0.4) (layers F.Cu B.Cu) (net 2))
+  (via (at 160.3 61.5) (size 0.8) (drill 0.4) (layers F.Cu B.Cu) (net 2))
+  (via (at 162.7 61.8) (size 0.8) (drill 0.4) (layers F.Cu B.Cu) (net 2))
+  (via (at 161.2 64.5) (size 0.8) (drill 0.4) (layers F.Cu B.Cu) (net 2))
+  (via (at 164.2 64.5) (size 0.8) (drill 0.4) (layers F.Cu B.Cu) (net 2))
+  (via (at 166.6 64.1) (size 0.8) (drill 0.4) (layers F.Cu B.Cu) (net 2))
+  (via (at 166.6 61.8) (size 0.8) (drill 0.4) (layers F.Cu B.Cu) (net 2))
+  (via (at 164.7 61.7) (size 0.8) (drill 0.4) (layers F.Cu B.Cu) (net 2))
+  (via (at 156.7 64.3) (size 0.8) (drill 0.4) (layers F.Cu B.Cu) (net 2))
+  (via (at 154.2 60) (size 0.8) (drill 0.4) (layers F.Cu B.Cu) (net 2))
+  (via (at 155.3 65.3) (size 0.8) (drill 0.4) (layers F.Cu B.Cu) (net 2))
+  (via (at 155.3 66.9) (size 0.8) (drill 0.4) (layers F.Cu B.Cu) (net 2))
+  (via (at 155.2 68.9) (size 0.8) (drill 0.4) (layers F.Cu B.Cu) (net 2))
+  (via (at 153.3 69.1) (size 0.8) (drill 0.4) (layers F.Cu B.Cu) (net 2))
+  (via (at 155.5 61) (size 0.8) (drill 0.4) (layers F.Cu B.Cu) (net 2))
+  (via (at 170 70) (size 0.8) (drill 0.4) (layers F.Cu B.Cu) (net 2))
+  (via (at 167.5 70) (size 0.8) (drill 0.4) (layers F.Cu B.Cu) (net 2))
+  (via (at 165 70) (size 0.8) (drill 0.4) (layers F.Cu B.Cu) (net 2))
+  (via (at 162.5 70) (size 0.8) (drill 0.4) (layers F.Cu B.Cu) (net 2))
+  (via (at 160 70) (size 0.8) (drill 0.4) (layers F.Cu B.Cu) (net 2))
+  (via (at 157.5 70) (size 0.8) (drill 0.4) (layers F.Cu B.Cu) (net 2))
+  (via (at 170 67.5) (size 0.8) (drill 0.4) (layers F.Cu B.Cu) (net 2))
+  (via (at 170 56) (size 0.8) (drill 0.4) (layers F.Cu B.Cu) (net 2))
+  (via (at 167.5 56) (size 0.8) (drill 0.4) (layers F.Cu B.Cu) (net 2))
+  (via (at 165 56) (size 0.8) (drill 0.4) (layers F.Cu B.Cu) (net 2))
+  (via (at 162.5 56) (size 0.8) (drill 0.4) (layers F.Cu B.Cu) (net 2))
+  (via (at 160 56) (size 0.8) (drill 0.4) (layers F.Cu B.Cu) (net 2))
+  (via (at 155 56) (size 0.8) (drill 0.4) (layers F.Cu B.Cu) (net 2))
+  (via (at 157.5 56) (size 0.8) (drill 0.4) (layers F.Cu B.Cu) (net 2))
+  (via (at 152 56) (size 0.8) (drill 0.4) (layers F.Cu B.Cu) (net 2))
   (segment (start 148.2 64.8) (end 148.2 65.475) (width 0.2) (layer F.Cu) (net 3))
   (segment (start 146.2 68.25) (end 144.1 70.35) (width 0.2) (layer F.Cu) (net 3))
@@
     (connect_pads (clearance 0.508))
     (min_thickness 0.254)
+    (fill yes (arc_segments 32) (thermal_gap 0.508) (thermal_bridge_width 0.508))
+    (polygon
+      (pts
+        (xy 171.5 71.5) (xy 131 71.5) (xy 131 54.5) (xy 171.5 54.5)
+      )
+    )
+  )
+  (zone (net 2) (net_name GND) (layer F.Cu) (hatch edge 0.508)
+    (connect_pads (clearance 0.508))
+    (min_thickness 0.254)
+    (fill yes (arc_segments 32) (thermal_gap 0.508) (thermal_bridge_width 0.508))
+    (polygon
+      (pts
+        (xy 171.5 71.4) (xy 131 71.5) (xy 131 54.5) (xy 171.5 54.5)
+      )
+    )
+  )
+  (zone (net 2) (net_name GND) (layer B.Cu) (hatch edge 0.508)
+    (connect_pads (clearance 0.508))
+    (min_thickness 0.254)

Commit message: change the clearance for drc rules of cc1101 part
Other:
- net class Default: clearance 0.2 -> 0.1
- rule trace_clearance: 0.2 -> 0.1
Changed lines of the file:
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@@
     (thickness 1.6)
     (drawings 10)
-    (tracks 170)
+    (tracks 171)
     (zones 0)
     (modules 18)
@@
     (1 In1.Cu signal hide)
     (2 In2.Cu signal hide)
-    (31 B.Cu signal hide)
+    (31 B.Cu signal)
     (32 B.Adhes user)
     (33 F.Adhes user)
@@
     (user_trace_width 0.25)
     (user_trace_width 0.34036)
-    (trace_clearance 0.2)
+    (trace_clearance 0.1)
     (zone_clearance 0.508)
     (zone_45_only no)
@@
   (net 21 "Net-(R171-Pad2)")
   (net_class Default "This is the default net class."
-    (clearance 0.2)
+    (clearance 0.1)
     (trace_width 0.25)
     (via_dia 0.8)
@@
   (via (at 142.1 67.2) (size 0.8) (drill 0.4) (layers F.Cu B.Cu) (net 2))
   (via (at 144.9 63.5) (size 0.8) (drill 0.4) (layers F.Cu B.Cu) (net 11))
-  (via (at 148.3 66.6) (size 0.8) (drill 0.4) (layers F.Cu B.Cu) (net 11))
+  (via (at 148.5 66.5) (size 0.8) (drill 0.4) (layers F.Cu B.Cu) (net 11))
   (via (at 151.5 70.1) (size 0.8) (drill 0.4) (layers F.Cu B.Cu) (net 2))
   (via (at 146.4 70.4) (size 0.8) (drill 0.4) (layers F.Cu B.Cu) (net 2))
@@
   (via (at 150.1 59.8) (size 0.8) (drill 0.4) (layers F.Cu B.Cu) (net 11))
   (segment (start 148.7 66.2) (end 148.7 64.8) (width 0.2) (layer F.Cu) (net 11))
-  (segment (start 148.3 66.6) (end 148.7 66.2) (width 0.2) (layer F.Cu) (net 11))
   (segment (start 150.1 63.9) (end 150.9 63.9) (width 0.2) (layer F.Cu) (net 11))
   (segment (start 150.9 63.9) (end 151.2 64.2) (width 0.2) (layer F.Cu) (net 11))
@@
   (segment (start 145 63.4) (end 144.9 63.5) (width 0.2) (layer F.Cu) (net 11))
   (segment (start 146.3 63.4) (end 145 63.4) (width 0.2) (layer F.Cu) (net 11))
+  (segment (start 148.5 66.5) (end 148.7 66.3) (width 0.2) (layer F.Cu) (net 11))
+  (segment (start 148.7 66.3) (end 148.7 66.2) (width 0.2) (layer F.Cu) (net 11))
   (segment (start 140.9 65.8) (end 139.33 64.23) (width 0.2) (layer F.Cu) (net 12))
   (segment (start 146.875 65.8) (end 140.9 65.8) (width 0.2) (layer F.Cu) (net 12))

Commit message: Add logos and move reference about
Parts:
- added G***: LOGO, jjh:Untitled, B.Cu at (153.3, 63.5)
Other:
- board text added: "@JamesjHorton jjhorton.co.uk"
- board text added: "CC1101 PMod"

Commit message: Update the connector layout
Connections:
- J2 pad 3: SPI_TX -> GDO2
- J2 pad 4: SPI_CLK -> GDO0
- J2 pad 5: SPI_CSN -> SPI_CLK
- J2 pad 6: SPI_RX -> SPI_TX
- J2 pad 7: GDO2 -> SPI_RX
- J2 pad 8: GDO0 -> SPI_CSN
- U1 pad PAD: (no net) -> GND
Routing:
- net SPI_CSN: track 20.8 -> 14.4 mm
- net GDO2: track 13.2 -> 18.2 mm, vias 0 -> 1
- net GND: track 26.6 -> 31.0 mm
- net GDO0: track 12.5 -> 16.4 mm, vias 0 -> 1
- net SPI_TX: track 15.3 -> 11.4 mm
- net SPI_RX: track 10.4 -> 13.4 mm
- net SPI_CLK: track 11.3 -> 13.5 mm
