File: PMod_CC1101/Hardware/cc1101.sch (KiCad schematic (older format))
At the start: 17 parts

Commit message: update the layout of the schematic
Parts:
- J?: footprint (none) -> Connector_PinHeader_2.54mm:PinHeader_2x06_P2.54mm_Vertical
Connections:
- no-connect marks 0 -> 2
Other:
- note added: "PMod Connector"
- moved on the sheet: C?, J?, L?, R?, U?, Y?

Commit message: update the reference values and add a suitable crystal
Parts:
- removed Y?: 26MHz, symbol Device:Crystal
- added C51: 100nF, Capacitor_SMD:C_0603_1608Metric, symbol Device:C
- added Y?: 26MHz, Crystal:Crystal_SMD_Abracon_ABM3C-4Pin_5.0x3.2mm, symbol Device:Crystal_GND24_Small
- R171: renamed from R?; value R -> 56K; footprint (none) -> Resistor_SMD:R_0603_1608Metric
- gave numbers to parts that had none: 11
Connections:
- net +3V3: now also U1.18 (DGUARD)
- net GND: now also C51.1, Y?.2, Y?.4
- net at C?.2, U1.10 (XOSC_Q2): now also Y?.1
- net at U1.5 (DCOUPL): now also C51.2
- net at C?.1, U1.8 (XOSC_Q1): now also Y?.3
Other:
- note added: "Designed optermised for 433MHz based on:\nhttps://www.ti.com/lit/ds/symlink/cc1101.pdf\n\nPage 25/26 for circuit and values selected \n"
Changed lines of the file:
@@
 $EndComp
 $Comp
-L Device:C C?
+L Device:C C125
 U 1 1 60A35692
 P 8350 1850
-F 0 "C?" V 8098 1850 50  0000 C CNN
+F 0 "C125" V 8098 1850 50  0000 C CNN
 F 1 "220pF" V 8189 1850 50  0000 C CNN
 F 2 "Capacitor_SMD:C_0603_1608Metric" H 8388 1700 50  0001 C CNN
@@
 $EndComp
 $Comp
-L Device:C C?
+L Device:C C123
 U 1 1 60A35E36
 P 7950 2100
-F 0 "C?" H 8065 2146 50  0000 L CNN
+F 0 "C123" H 8065 2146 50  0000 L CNN
 F 1 "5.6pF" H 8065 2055 50  0000 L CNN
 F 2 "Capacitor_SMD:C_0603_1608Metric" H 7988 1950 50  0001 C CNN
@@
 $EndComp
 $Comp
-L Device:C C?
+L Device:C C122
 U 1 1 60A36923
 P 7450 2100
-F 0 "C?" H 7565 2146 50  0000 L CNN
+F 0 "C122" H 7565 2146 50  0000 L CNN
 F 1 "8.2pF" H 7565 2055 50  0000 L CNN
 F 2 "Capacitor_SMD:C_0603_1608Metric" H 7488 1950 50  0001 C CNN
@@
 $EndComp
 $Comp
-L Device:C C?
+L Device:C C121
 U 1 1 60A36D2F
 P 6800 1750
-F 0 "C?" V 6750 1600 50  0000 C CNN
+F 0 "C121" V 6750 1600 50  0000 C CNN
 F 1 "3.9pF" V 6750 1900 50  0000 C CNN
 F 2 "Capacitor_SMD:C_0603_1608Metric" H 6838 1600 50  0001 C CNN
@@
 $EndComp
 $Comp
-L Device:C C?
+L Device:C C131
 U 1 1 60A3755B
 P 6400 2100
-F 0 "C?" H 6515 2146 50  0000 L CNN
+F 0 "C131" H 6515 2146 50  0000 L CNN
 F 1 "3.9pF" H 6515 2055 50  0000 L CNN
 F 2 "" H 6438 1950 50  0001 C CNN
@@
 $EndComp
 $Comp
-L Device:C C?
+L Device:C C124
 U 1 1 60A37995
 P 6400 1200
-F 0 "C?" H 6285 1154 50  0000 R CNN
+F 0 "C124" H 6285 1154 50  0000 R CNN
 F 1 "220pF" H 6285 1245 50  0000 R CNN
 F 2 "Capacitor_SMD:C_0603_1608Metric" H 6438 1050 50  0001 C CNN
@@
 $EndComp
 $Comp
-L Device:L L?
+L Device:L L121
 U 1 1 60A38065
 P 6400 1600
-F 0 "L?" H 6356 1554 50  0000 R CNN
+F 0 "L121" H 6356 1554 50  0000 R CNN
 F 1 "27nH" H 6356 1645 50  0000 R CNN
 F 2 "Inductor_SMD:L_0603_1608Metric" H 6400 1600 50  0001 C CNN
@@
 $EndComp
 $Comp
-L Device:L L?
+L Device:L L131
 U 1 1 60A38A26
 P 6800 1950
-F 0 "L?" V 6750 2100 50  0000 C CNN
+F 0 "L131" V 6750 2100 50  0000 C CNN
 F 1 "27nH" V 6750 1800 50  0000 C CNN
 F 2 "Inductor_SMD:L_0603_1608Metric" H 6800 1950 50  0001 C CNN
@@
 $EndComp
 $Comp
-L Device:L L?
+L Device:L L122
 U 1 1 60A39321
 P 7200 1850
-F 0 "L?" V 7390 1850 50  0000 C CNN
+F 0 "L122" V 7390 1850 50  0000 C CNN
 F 1 "22nH" V 7299 1850 50  0000 C CNN
 F 2 "Inductor_SMD:L_0603_1608Metric" H 7200 1850 50  0001 C CNN
@@
 $EndComp
 $Comp
-L Device:L L?
+L Device:L L123
 U 1 1 60A3A077
 P 7700 1850
-F 0 "L?" V 7890 1850 50  0000 C CNN
+F 0 "L123" V 7890 1850 50  0000 C CNN
 F 1 "27nH" V 7799 1850 50  0000 C CNN
 F 2 "Inductor_SMD:L_0603_1608Metric" H 7700 1850 50  0001 C CNN
@@
 	6400 2250 6400 2350
 $Comp
-L JJH_Library:CC1101RGPR U?
+L JJH_Library:CC1101RGPR U1
 U 1 1 60A502FE
 P 4600 1900
-F 0 "U?" H 4575 2315 50  0000 C CNN
+F 0 "U1" H 4575 2315 50  0000 C CNN
 F 1 "CC1101RGPR" H 4575 2224 50  0000 C CNN
 F 2 "" H 4250 1900 50  0001 C CNN
@@
 	0    1    1    0
 $EndComp
-$Comp
-L Device:Crystal Y?
-U 1 1 60A6E09E
-P 3150 2800
-F 0 "Y?" V 3100 2950 50  0000 L CNN
-F 1 "26MHz" V 3250 2950 50  0000 L CNN
-F 2 "" H 3150 2800 50  0001 C CNN
-F 3 "~" H 3150 2800 50  0001 C CNN
-	1    3150 2800
-	0    1    1    0
-$EndComp
 Wire Wire Line
 	3900 2700 3900 2600
-Wire Wire Line
-	3150 2650 3150 2600
 Connection ~ 3150 2600
 Wire Wire Line
@@
 Wire Wire Line
 	3050 3000 3150 3000
-Wire Wire Line
-	3150 3000 3150 2950
 Wire Wire Line
 	3900 2900 3900 3000
@@
 	3750 1800 3900 1800
 $Comp
-L Device:R R?
+L Device:R R171
 U 1 1 60A8D230
 P 5550 3300
-F 0 "R?" V 5450 3300 50  0000 C CNN
-F 1 "R" V 5650 3300 50  0000 C CNN
-F 2 "" V 5480 3300 50  0001 C CNN
+F 0 "R171" V 5450 3300 50  0000 C CNN
+F 1 "56K" V 5650 3300 50  0000 C CNN
+F 2 "Resistor_SMD:R_0603_1608Metric" V 5480 3300 50  0001 C CNN
 F 3 "~" H 5550 3300 50  0001 C CNN
 	1    5550 3300
@@
 NoConn ~ 3600 5950
 NoConn ~ 3100 5950
+$Comp
+L Device:C C51
+U 1 1 60E263E0
+P 3150 3450
+F 0 "C51" H 3035 3404 50  0000 R CNN
+F 1 "100nF" H 3035 3495 50  0000 R CNN
+F 2 "Capacitor_SMD:C_0603_1608Metric" H 3188 3300 50  0001 C CNN
+F 3 "~" H 3150 3450 50  0001 C CNN
+	1    3150 3450
+	-1   0    0    1
+$EndComp
+Wire Wire Line
+	3150 3300 3150 3200
+Wire Wire Line
+	3150 3200 3900 3200
+$Comp
+L power:GND #PWR?
+U 1 1 60E2AE47
+P 3150 3700
+F 0 "#PWR?" H 3150 3450 50  0001 C CNN
+F 1 "GND" H 3155 3527 50  0000 C CNN
+F 2 "" H 3150 3700 50  0001 C CNN
+F 3 "" H 3150 3700 50  0001 C CNN
+	1    3150 3700
+	1    0    0    -1
+$EndComp
+$Comp
+L power:+3V3 #PWR?
+U 1 1 60E2B410
+P 3750 3700
+F 0 "#PWR?" H 3750 3550 50  0001 C CNN
+F 1 "+3V3" H 3765 3873 50  0000 C CNN
+F 2 "" H 3750 3700 50  0001 C CNN
+F 3 "" H 3750 3700 50  0001 C CNN
+	1    3750 3700
+	-1   0    0    1
+$EndComp
+Wire Wire Line
+	3750 3700 3750 3300
+Wire Wire Line
+	3750 3300 3900 3300
+Wire Wire Line
+	3150 3700 3150 3600
+Text Notes 6350 3350 0    55   ~ 0
+Designed optermised for 433MHz based on:\nhttps://www.ti.com/lit/ds/symlink/cc1101.pdf\n\nPage 25/26 for circuit and values selected \n
+$Comp
+L Device:Crystal_GND24_Small Y?
+U 1 1 60E33551
+P 3150 2800
+F 0 "Y?" V 3250 2550 50  0000 L CNN
+F 1 "26MHz" V 3050 2450 50  0000 L CNN
+F 2 "Crystal:Crystal_SMD_Abracon_ABM3C-4Pin_5.0x3.2mm" H 3150 2800 50  0001 C CNN
+F 3 "https://www.mouser.co.uk/datasheet/2/3/abrcs02719_1-2258580.pdf" H 3150 2800 50  0001 C CNN
+F 4 "815-ABM3C-26-D4YT" H 3150 2800 50  0001 C CNN "Mouser No."
+	1    3150 2800
+	0    -1   -1   0
+$EndComp
+Wire Wire Line
+	3150 2600 3150 2700
+Wire Wire Line
+	3150 2900 3150 3000
+$Comp
+L power:GND #PWR?
+U 1 1 60E3F2C7
+P 3000 2800
+F 0 "#PWR?" H 3000 2550 50  0001 C CNN
+F 1 "GND" V 3005 2672 50  0000 R CNN
+F 2 "" H 3000 2800 50  0001 C CNN
+F 3 "" H 3000 2800 50  0001 C CNN
+	1    3000 2800
+	0    1    1    0
+$EndComp
+$Comp
+L power:GND #PWR?
+U 1 1 60E3FC31
+P 3300 2800
+F 0 "#PWR?" H 3300 2550 50  0001 C CNN
+F 1 "GND" V 3305 2672 50  0000 R CNN
+F 2 "" H 3300 2800 50  0001 C CNN
+F 3 "" H 3300 2800 50  0001 C CNN
+	1    3300 2800
+	0    -1   -1   0
+$EndComp
+Wire Wire Line
+	3300 2800 3250 2800
+Wire Wire Line
+	3050 2800 3000 2800
 $EndSCHEMATC

Commit message: Add references to values
Parts:
- J1: renamed from J?; footprint (none) -> Connector_Coaxial:SMA_Samtec_SMA-J-P-X-ST-EM1_EdgeMount
- gave numbers to parts that had none: 4
Changed lines of the file:
@@
 $EndDescr
 $Comp
-L Connector_Generic:Conn_02x06_Odd_Even J?
+L Connector_Generic:Conn_02x06_Odd_Even J2
 U 1 1 60A2E9D0
 P 3300 6150
-F 0 "J?" H 3350 6567 50  0000 C CNN
+F 0 "J2" H 3350 6567 50  0000 C CNN
 F 1 "Conn_02x06_Odd_Even" H 3350 6476 50  0000 C CNN
 F 2 "Connector_PinHeader_2.54mm:PinHeader_2x06_P2.54mm_Vertical" H 3300 6150 50  0001 C CNN
@@
 $EndComp
 $Comp
-L power:GND #PWR?
+L power:GND #PWR0101
 U 1 1 60A2F9D4
 P 3850 6350
-F 0 "#PWR?" H 3850 6100 50  0001 C CNN
+F 0 "#PWR0101" H 3850 6100 50  0001 C CNN
 F 1 "GND" V 3855 6222 50  0000 R CNN
 F 2 "" H 3850 6350 50  0001 C CNN
@@
 $EndComp
 $Comp
-L power:GND #PWR?
+L power:GND #PWR0102
 U 1 1 60A2FFBC
 P 2800 6350
-F 0 "#PWR?" H 2800 6100 50  0001 C CNN
+F 0 "#PWR0102" H 2800 6100 50  0001 C CNN
 F 1 "GND" V 2805 6222 50  0000 R CNN
 F 2 "" H 2800 6350 50  0001 C CNN
@@
 $EndComp
 $Comp
-L power:+3V3 #PWR?
+L power:+3V3 #PWR0103
 U 1 1 60A3030B
 P 2800 6450
-F 0 "#PWR?" H 2800 6300 50  0001 C CNN
+F 0 "#PWR0103" H 2800 6300 50  0001 C CNN
 F 1 "+3V3" V 2815 6578 50  0000 L CNN
 F 2 "" H 2800 6450 50  0001 C CNN
@@
 $EndComp
 $Comp
-L power:+3V3 #PWR?
+L power:+3V3 #PWR0104
 U 1 1 60A3054F
 P 3850 6450
-F 0 "#PWR?" H 3850 6300 50  0001 C CNN
+F 0 "#PWR0104" H 3850 6300 50  0001 C CNN
 F 1 "+3V3" V 3865 6578 50  0000 L CNN
 F 2 "" H 3850 6450 50  0001 C CNN
@@
 	3100 6050 2800 6050
 $Comp
-L Connector:Conn_Coaxial J?
+L Connector:Conn_Coaxial J1
 U 1 1 60A31A03
 P 8800 1850
-F 0 "J?" H 8900 1825 50  0000 L CNN
+F 0 "J1" H 8900 1825 50  0000 L CNN
 F 1 "Conn_Coaxial" H 8900 1734 50  0000 L CNN
-F 2 "" H 8800 1850 50  0001 C CNN
+F 2 "Connector_Coaxial:SMA_Samtec_SMA-J-P-X-ST-EM1_EdgeMount" H 8800 1850 50  0001 C CNN
 F 3 " ~" H 8800 1850 50  0001 C CNN
 	1    8800 1850
@@
 $EndComp
 $Comp
-L power:GND #PWR?
+L power:GND #PWR0105
 U 1 1 60A326FB
 P 8800 2050
-F 0 "#PWR?" H 8800 1800 50  0001 C CNN
+F 0 "#PWR0105" H 8800 1800 50  0001 C CNN
 F 1 "GND" H 8805 1877 50  0000 C CNN
 F 2 "" H 8800 2050 50  0001 C CNN
@@
 $EndComp
 $Comp
-L power:GND #PWR?
+L power:GND #PWR0106
 U 1 1 60A3B067
 P 7950 2350
-F 0 "#PWR?" H 7950 2100 50  0001 C CNN
+F 0 "#PWR0106" H 7950 2100 50  0001 C CNN
 F 1 "GND" H 7955 2177 50  0000 C CNN
 F 2 "" H 7950 2350 50  0001 C CNN
@@
 $EndComp
 $Comp
-L power:GND #PWR?
+L power:GND #PWR0107
 U 1 1 60A3B334
 P 7450 2350
-F 0 "#PWR?" H 7450 2100 50  0001 C CNN
+F 0 "#PWR0107" H 7450 2100 50  0001 C CNN
 F 1 "GND" H 7455 2177 50  0000 C CNN
 F 2 "" H 7450 2350 50  0001 C CNN
@@
 $EndComp
 $Comp
-L power:GND #PWR?
+L power:GND #PWR0108
 U 1 1 60A3B60D
 P 6400 950
-F 0 "#PWR?" H 6400 700 50  0001 C CNN
+F 0 "#PWR0108" H 6400 700 50  0001 C CNN
 F 1 "GND" H 6405 777 50  0000 C CNN
 F 2 "" H 6400 950 50  0001 C CNN
@@
 $EndComp
 $Comp
-L power:GND #PWR?
+L power:GND #PWR0109
 U 1 1 60A3B8F2
 P 6400 2350
-F 0 "#PWR?" H 6400 2100 50  0001 C CNN
+F 0 "#PWR0109" H 6400 2100 50  0001 C CNN
 F 1 "GND" H 6405 2177 50  0000 C CNN
 F 2 "" H 6400 2350 50  0001 C CNN
@@
 $EndComp
 $Comp
-L power:+3V3 #PWR?
+L power:+3V3 #PWR0110
 U 1 1 60A55E7E
 P 5550 2350
-F 0 "#PWR?" H 5550 2200 50  0001 C CNN
+F 0 "#PWR0110" H 5550 2200 50  0001 C CNN
 F 1 "+3V3" V 5565 2478 50  0000 L CNN
 F 2 "" H 5550 2350 50  0001 C CNN
@@
 	5400 2250 5400 2150
 $Comp
-L power:GND #PWR?
+L power:GND #PWR0111
 U 1 1 60A59036
 P 5550 2900
-F 0 "#PWR?" H 5550 2650 50  0001 C CNN
+F 0 "#PWR0111" H 5550 2650 50  0001 C CNN
 F 1 "GND" V 5555 2772 50  0000 R CNN
 F 2 "" H 5550 2900 50  0001 C CNN
@@
 	5950 1900 5250 1900
 $Comp
-L Device:C C?
+L Device:C C81
 U 1 1 60A6949A
 P 2900 2600
-F 0 "C?" V 3000 2450 50  0000 C CNN
+F 0 "C81" V 3000 2450 50  0000 C CNN
 F 1 "27pF" V 2750 2600 50  0000 C CNN
 F 2 "Capacitor_SMD:C_0603_1608Metric" H 2938 2450 50  0001 C CNN
@@
 $EndComp
 $Comp
-L Device:C C?
+L Device:C C101
 U 1 1 60A69C8B
 P 2900 3000
-F 0 "C?" V 2950 3150 50  0000 C CNN
+F 0 "C101" V 2950 3150 50  0000 C CNN
 F 1 "27pF" V 2750 3000 50  0000 C CNN
 F 2 "Capacitor_SMD:C_0603_1608Metric" H 2938 2850 50  0001 C CNN
@@
 $EndComp
 $Comp
-L power:GND #PWR?
+L power:GND #PWR0112
 U 1 1 60A6D454
 P 2600 2600
-F 0 "#PWR?" H 2600 2350 50  0001 C CNN
+F 0 "#PWR0112" H 2600 2350 50  0001 C CNN
 F 1 "GND" V 2605 2472 50  0000 R CNN
 F 2 "" H 2600 2600 50  0001 C CNN
@@
 $EndComp
 $Comp
-L power:GND #PWR?
+L power:GND #PWR0113
 U 1 1 60A6D7EE
 P 2600 3000
-F 0 "#PWR?" H 2600 2750 50  0001 C CNN
+F 0 "#PWR0113" H 2600 2750 50  0001 C CNN
 F 1 "GND" V 2605 2872 50  0000 R CNN
 F 2 "" H 2600 3000 50  0001 C CNN
@@
 $EndComp
 $Comp
-L power:GND #PWR?
+L power:GND #PWR0114
 U 1 1 60A8E43F
 P 5850 3300
-F 0 "#PWR?" H 5850 3050 50  0001 C CNN
+F 0 "#PWR0114" H 5850 3050 50  0001 C CNN
 F 1 "GND" V 5855 3172 50  0000 R CNN
 F 2 "" H 5850 3300 50  0001 C CNN
@@
 	3150 3200 3900 3200
 $Comp
-L power:GND #PWR?
+L power:GND #PWR0115
 U 1 1 60E2AE47
 P 3150 3700
-F 0 "#PWR?" H 3150 3450 50  0001 C CNN
+F 0 "#PWR0115" H 3150 3450 50  0001 C CNN
 F 1 "GND" H 3155 3527 50  0000 C CNN
 F 2 "" H 3150 3700 50  0001 C CNN
@@
 $EndComp
 $Comp
-L power:+3V3 #PWR?
+L power:+3V3 #PWR0116
 U 1 1 60E2B410
 P 3750 3700
-F 0 "#PWR?" H 3750 3550 50  0001 C CNN
+F 0 "#PWR0116" H 3750 3550 50  0001 C CNN
 F 1 "+3V3" H 3765 3873 50  0000 C CNN
 F 2 "" H 3750 3700 50  0001 C CNN
@@
 Designed optermised for 433MHz based on:\nhttps://www.ti.com/lit/ds/symlink/cc1101.pdf\n\nPage 25/26 for circuit and values selected \n
 $Comp
-L Device:Crystal_GND24_Small Y?
+L Device:Crystal_GND24_Small XTAL1
 U 1 1 60E33551
 P 3150 2800
-F 0 "Y?" V 3250 2550 50  0000 L CNN
+F 0 "XTAL1" V 3250 2550 50  0000 L CNN
 F 1 "26MHz" V 3050 2450 50  0000 L CNN
 F 2 "Crystal:Crystal_SMD_Abracon_ABM3C-4Pin_5.0x3.2mm" H 3150 2800 50  0001 C CNN
@@
 	3150 2900 3150 3000
 $Comp
-L power:GND #PWR?
+L power:GND #PWR0117
 U 1 1 60E3F2C7
 P 3000 2800
-F 0 "#PWR?" H 3000 2550 50  0001 C CNN
+F 0 "#PWR0117" H 3000 2550 50  0001 C CNN
 F 1 "GND" V 3005 2672 50  0000 R CNN
 F 2 "" H 3000 2800 50  0001 C CNN
@@
 $EndComp
 $Comp
-L power:GND #PWR?
+L power:GND #PWR0118
 U 1 1 60E3FC31
 P 3300 2800
-F 0 "#PWR?" H 3300 2550 50  0001 C CNN
+F 0 "#PWR0118" H 3300 2550 50  0001 C CNN
 F 1 "GND" V 3305 2672 50  0000 R CNN
 F 2 "" H 3300 2800 50  0001 C CNN

Commit message: initial footprint for the CC1101 part
Parts:
- U1: footprint (none) -> Package_DFN_QFN:UQFN-20-1EP_4x4mm_P0.5mm_EP2.8x2.8mm
Changed lines of the file:
@@
 F 0 "U1" H 4575 2315 50  0000 C CNN
 F 1 "CC1101RGPR" H 4575 2224 50  0000 C CNN
-F 2 "" H 4250 1900 50  0001 C CNN
+F 2 "Package_DFN_QFN:UQFN-20-1EP_4x4mm_P0.5mm_EP2.8x2.8mm" H 4250 1900 50  0001 C CNN
 F 3 "" H 4250 1900 50  0001 C CNN
 	1    4600 1900

Commit message: add footprint missing on cap
Parts:
- C131: footprint (none) -> Capacitor_SMD:C_0603_1608Metric
Changed lines of the file:
@@
 F 0 "C131" H 6515 2146 50  0000 L CNN
 F 1 "3.9pF" H 6515 2055 50  0000 L CNN
-F 2 "" H 6438 1950 50  0001 C CNN
+F 2 "Capacitor_SMD:C_0603_1608Metric" H 6438 1950 50  0001 C CNN
 F 3 "~" H 6400 2100 50  0001 C CNN
 	1    6400 2100

Commit message: update schematic part for cc1101
Parts:
- U1: footprint Package_DFN_QFN:UQFN-20-1EP_4x4mm_P0.5mm_EP2.8x2.8mm -> jjh:QFN50P400X400X100-21N-D
Changed lines of the file:
@@
 F 0 "U1" H 4575 2315 50  0000 C CNN
 F 1 "CC1101RGPR" H 4575 2224 50  0000 C CNN
-F 2 "Package_DFN_QFN:UQFN-20-1EP_4x4mm_P0.5mm_EP2.8x2.8mm" H 4250 1900 50  0001 C CNN
+F 2 "jjh:QFN50P400X400X100-21N-D" H 4250 1900 50  0001 C CNN
 F 3 "" H 4250 1900 50  0001 C CNN
 	1    4600 1900

Commit message: Update the connector layout
Connections:
- net GDO0: now also J2.4 (Pin_4); no longer J2.8 (Pin_8)
- net GDO2: now also J2.3 (Pin_3); no longer J2.7 (Pin_7)
- net SPI_CLK: now also J2.5 (Pin_5); no longer J2.4 (Pin_4)
- net SPI_CSN: now also J2.8 (Pin_8); no longer J2.5 (Pin_5)
- net SPI_RX: now also J2.7 (Pin_7); no longer J2.6 (Pin_6)
- net SPI_TX: now also J2.6 (Pin_6); no longer J2.3 (Pin_3)
Changed lines of the file:
@@
 	0    1    1    0
 $EndComp
-Text GLabel 3850 6050 2    50   Input ~ 0
+Text GLabel 2800 6150 0    50   Input ~ 0
 SPI_CLK
+Text GLabel 2800 6250 0    50   Input ~ 0
+SPI_RX
+Text GLabel 3850 6250 2    50   Input ~ 0
+SPI_CSN
 Text GLabel 3850 6150 2    50   Input ~ 0
-SPI_RX
-Text GLabel 2800 6150 0    50   Input ~ 0
-SPI_CSN
-Text GLabel 2800 6050 0    50   Input ~ 0
 SPI_TX
 Wire Wire Line
@@
 Wire Wire Line
 	5400 3300 5250 3300
-Text GLabel 2800 6250 0    50   Input ~ 0
+Text GLabel 2800 6050 0    50   Input ~ 0
 GDO2
-Text GLabel 3850 6250 2    50   Input ~ 0
+Text GLabel 3850 6050 2    50   Input ~ 0
 GDO0
 Wire Wire Line
