File: PMod_Neopixel_Array/Neopixel_Array.sch (KiCad schematic (older format))
At the start: 130 parts

Commit message: update the schematic
Parts:
- gave numbers to parts that had none: 130

Commit message: Add footprints for connectors and place on PCB
Parts:
- J1, J2: footprint (none) -> Connector_PinHeader_2.54mm:PinHeader_1x06_P2.54mm_Vertical
Changed lines of the file:
@@
 F 0 "J1" H 7450 6100 50  0000 L CNN
 F 1 "Conn_01x06" H 7250 5350 50  0000 L CNN
-F 2 "" H 7500 5750 50  0001 C CNN
+F 2 "Connector_PinHeader_2.54mm:PinHeader_1x06_P2.54mm_Vertical" H 7500 5750 50  0001 C CNN
 F 3 "~" H 7500 5750 50  0001 C CNN
 	1    7500 5750
@@
 F 0 "J2" H 9700 6150 50  0000 L CNN
 F 1 "Conn_01x06" H 9550 5400 50  0000 L CNN
-F 2 "" H 9750 5800 50  0001 C CNN
+F 2 "Connector_PinHeader_2.54mm:PinHeader_1x06_P2.54mm_Vertical" H 9750 5800 50  0001 C CNN
 F 3 "~" H 9750 5800 50  0001 C CNN
 	1    9750 5800
