File: PMod_Neopixel_Array/Neopixel_Array.kicad_pcb (KiCad board)
At the start: 2 copper layers, 69 x 80 mm, 128 parts

Commit message: Add footprints for connectors and place on PCB
Parts:
- added J1: Conn_01x06, Connector_PinHeader_2.54mm:PinHeader_1x06_P2.54mm_Vertical, F.Cu at (128.5, 68.0)
- added J2: Conn_01x06, Connector_PinHeader_2.54mm:PinHeader_1x06_P2.54mm_Vertical, F.Cu at (178.0, 68.0)
Routing:
- net VCC: track 711.6 -> 793.6 mm
- net DIN: track 0.00 -> 72.4 mm

Commit message: Add logo's to complete PCB
Parts:
- added G***: LOGO, jjh:Untitled, B.Cu at (160.0, 127.0)
- added G***: LOGO, jjh:j2h_small, F.Cu at (159.0, 69.0)
Other:
- board text added: "NeoPixel 8x8 @jamesjhorton jjhorton.co.uk"
