File: PMod_7Segment/hardware/PMod_7Segement.kicad_pcb (KiCad board)
At the start: 2 copper layers, 100 x 19.5 mm, 3 parts, among them U1 GN1640

Commit message: Add pmod connector and start the layout of data bus
Parts:
- added J1: Conn_02x06_Odd_Even, Connector_PinHeader_2.54mm:PinHeader_2x06_P2.54mm_Vertical, F.Cu at (173.0, 96.0)
Changed lines of the file:
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@@
     (tracks 0)
     (zones 0)
-    (modules 3)
-    (nets 53)
+    (modules 4)
+    (nets 65)
   )
   (page A4)
@@
   (net 51 "Net-(U1-Pad2)")
   (net 52 "Net-(U1-Pad1)")
+  (net 53 "Net-(J1-Pad12)")
+  (net 54 "Net-(J1-Pad11)")
+  (net 55 "Net-(J1-Pad10)")
+  (net 56 "Net-(J1-Pad9)")
+  (net 57 "Net-(J1-Pad8)")
+  (net 58 "Net-(J1-Pad7)")
+  (net 59 "Net-(J1-Pad6)")
+  (net 60 "Net-(J1-Pad5)")
+  (net 61 "Net-(J1-Pad4)")
+  (net 62 "Net-(J1-Pad3)")
+  (net 63 "Net-(J1-Pad2)")
+  (net 64 "Net-(J1-Pad1)")
   (net_class Default "This is the default net class."
     (clearance 0.2)
@@
     (add_net "Net-(DS2-Pad8)")
     (add_net "Net-(DS2-Pad9)")
+    (add_net "Net-(J1-Pad1)")
+    (add_net "Net-(J1-Pad10)")
+    (add_net "Net-(J1-Pad11)")
+    (add_net "Net-(J1-Pad12)")
+    (add_net "Net-(J1-Pad2)")
+    (add_net "Net-(J1-Pad3)")
+    (add_net "Net-(J1-Pad4)")
+    (add_net "Net-(J1-Pad5)")
+    (add_net "Net-(J1-Pad6)")
+    (add_net "Net-(J1-Pad7)")
+    (add_net "Net-(J1-Pad8)")
+    (add_net "Net-(J1-Pad9)")
     (add_net "Net-(U1-Pad1)")
     (add_net "Net-(U1-Pad10)")
@@
     (add_net "Net-(U1-Pad9)")
   )
+  (module Connector_PinHeader_2.54mm:PinHeader_2x06_P2.54mm_Vertical (layer F.Cu)
+    (at 173 96)
+    (descr "Through hole straight pin header, 2x06, 2.54mm pitch, double rows")
+    (tags "Through hole pin header THT 2x06 2.54mm double row")
+    (fp_text reference J1 (at 1.27 -2.33) (layer F.SilkS)
+      (effects (font (size 1 1) (thickness 0.15)))
+    )
+    (fp_text value Conn_02x06_Odd_Even (at 1.27 15.03) (layer F.Fab)
+      (effects (font (size 1 1) (thickness 0.15)))
+    )
+    (fp_text user %R (at 1.27 6.35 90) (layer F.Fab)
+      (effects (font (size 1 1) (thickness 0.15)))
+    )
+    (fp_line (start 0 -1.27) (end 3.81 -1.27) (layer F.Fab) (width 0.1))
+    (fp_line (start 3.81 -1.27) (end 3.81 13.97) (layer F.Fab) (width 0.1))
+    (fp_line (start 3.81 13.97) (end -1.27 13.97) (layer F.Fab) (width 0.1))
+    (fp_line (start -1.27 13.97) (end -1.27 0) (layer F.Fab) (width 0.1))
+    (fp_line (start -1.27 0) (end 0 -1.27) (layer F.Fab) (width 0.1))
+    (fp_line (start -1.33 14.03) (end 3.87 14.03) (layer F.SilkS) (width 0.12))
+    (fp_line (start -1.33 1.27) (end -1.33 14.03) (layer F.SilkS) (width 0.12))
+    (fp_line (start 3.87 -1.33) (end 3.87 14.03) (layer F.SilkS) (width 0.12))
+    (fp_line (start -1.33 1.27) (end 1.27 1.27) (layer F.SilkS) (width 0.12))
+    (fp_line (start 1.27 1.27) (end 1.27 -1.33) (layer F.SilkS) (width 0.12))
+    (fp_line (start 1.27 -1.33) (end 3.87 -1.33) (layer F.SilkS) (width 0.12))
+    (fp_line (start -1.33 0) (end -1.33 -1.33) (layer F.SilkS) (width 0.12))
+    (fp_line (start -1.33 -1.33) (end 0 -1.33) (layer F.SilkS) (width 0.12))
+    (fp_line (start -1.8 -1.8) (end -1.8 14.5) (layer F.CrtYd) (width 0.05))
+    (fp_line (start -1.8 14.5) (end 4.35 14.5) (layer F.CrtYd) (width 0.05))
+    (fp_line (start 4.35 14.5) (end 4.35 -1.8) (layer F.CrtYd) (width 0.05))
+    (fp_line (start 4.35 -1.8) (end -1.8 -1.8) (layer F.CrtYd) (width 0.05))
+    (pad 12 thru_hole oval (at 2.54 12.7) (size 1.7 1.7) (drill 1) (layers *.Cu *.Mask)
+      (net 53 "Net-(J1-Pad12)"))
+    (pad 11 thru_hole oval (at 0 12.7) (size 1.7 1.7) (drill 1) (layers *.Cu *.Mask)
+      (net 54 "Net-(J1-Pad11)"))
+    (pad 10 thru_hole oval (at 2.54 10.16) (size 1.7 1.7) (drill 1) (layers *.Cu *.Mask)
+      (net 55 "Net-(J1-Pad10)"))
+    (pad 9 thru_hole oval (at 0 10.16) (size 1.7 1.7) (drill 1) (layers *.Cu *.Mask)
+      (net 56 "Net-(J1-Pad9)"))
+    (pad 8 thru_hole oval (at 2.54 7.62) (size 1.7 1.7) (drill 1) (layers *.Cu *.Mask)
+      (net 57 "Net-(J1-Pad8)"))
+    (pad 7 thru_hole oval (at 0 7.62) (size 1.7 1.7) (drill 1) (layers *.Cu *.Mask)
+      (net 58 "Net-(J1-Pad7)"))
+    (pad 6 thru_hole oval (at 2.54 5.08) (size 1.7 1.7) (drill 1) (layers *.Cu *.Mask)
+      (net 59 "Net-(J1-Pad6)"))
+    (pad 5 thru_hole oval (at 0 5.08) (size 1.7 1.7) (drill 1) (layers *.Cu *.Mask)
+      (net 60 "Net-(J1-Pad5)"))
+    (pad 4 thru_hole oval (at 2.54 2.54) (size 1.7 1.7) (drill 1) (layers *.Cu *.Mask)
+      (net 61 "Net-(J1-Pad4)"))
+    (pad 3 thru_hole oval (at 0 2.54) (size 1.7 1.7) (drill 1) (layers *.Cu *.Mask)
+      (net 62 "Net-(J1-Pad3)"))
+    (pad 2 thru_hole oval (at 2.54 0) (size 1.7 1.7) (drill 1) (layers *.Cu *.Mask)
+      (net 63 "Net-(J1-Pad2)"))
+    (pad 1 thru_hole rect (at 0 0) (size 1.7 1.7) (drill 1) (layers *.Cu *.Mask)
+      (net 64 "Net-(J1-Pad1)"))
+    (model ${KISYS3DMOD}/Connector_PinHeader_2.54mm.3dshapes/PinHeader_2x06_P2.54mm_Vertical.wrl
+      (at (xyz 0 0 0))
+      (scale (xyz 1 1 1))
+      (rotate (xyz 0 0 0))
+    )
+  )
   (module Package_SO:SSOP-28_5.3x10.2mm_P0.65mm (layer B.Cu)

Commit message: Add pull up resitors and work on layout
Connections:
- net Net-(DS1-Pad12) renamed /GRDI1
- net Net-(U1-Pad18) renamed /GRID1
- DS1 pad 1: Net-(DS1-Pad1) -> /SEG5
- DS1 pad 10: Net-(DS1-Pad10) -> /SEG6
- DS1 pad 11: Net-(DS1-Pad11) -> /SEG1
- DS1 pad 2: Net-(DS1-Pad2) -> /SEG4
- DS1 pad 3: Net-(DS1-Pad3) -> /SEG8
- DS1 pad 4: Net-(DS1-Pad4) -> /SEG3
- DS1 pad 5: Net-(DS1-Pad5) -> /SEG7
- DS1 pad 6: Net-(DS1-Pad6) -> /GRID4
- DS1 pad 7: Net-(DS1-Pad7) -> /SEG2
- DS1 pad 8: Net-(DS1-Pad8) -> /GRID3
- DS1 pad 9: Net-(DS1-Pad9) -> /GRID2
- DS2 pad 1: Net-(DS2-Pad1) -> /SEG5
- DS2 pad 10: Net-(DS2-Pad10) -> /SEG6
- DS2 pad 11: Net-(DS2-Pad11) -> /SEG1
- DS2 pad 12: Net-(DS2-Pad12) -> /GRID5
- DS2 pad 2: Net-(DS2-Pad2) -> /SEG4
- DS2 pad 3: Net-(DS2-Pad3) -> /SEG8
- DS2 pad 4: Net-(DS2-Pad4) -> /SEG3
- DS2 pad 5: Net-(DS2-Pad5) -> /SEG7
- DS2 pad 6: Net-(DS2-Pad6) -> /GRID8
- DS2 pad 7: Net-(DS2-Pad7) -> /SEG2
- DS2 pad 8: Net-(DS2-Pad8) -> /GRID7
- DS2 pad 9: Net-(DS2-Pad9) -> /GRID6
- J1 pad 10: Net-(J1-Pad10) -> GND
- J1 pad 11: Net-(J1-Pad11) -> +3V3
- J1 pad 12: Net-(J1-Pad12) -> +3V3
- J1 pad 5: Net-(J1-Pad5) -> CLK
- J1 pad 7: Net-(J1-Pad7) -> DATA
- J1 pad 9: Net-(J1-Pad9) -> GND
- U1 pad 10: Net-(U1-Pad10) -> /SEG2
- U1 pad 11: Net-(U1-Pad11) -> /SEG3
- U1 pad 12: Net-(U1-Pad12) -> /SEG4
- U1 pad 13: Net-(U1-Pad13) -> /SEG5
- U1 pad 14: Net-(U1-Pad14) -> /SEG6
- U1 pad 15: Net-(U1-Pad15) -> /SEG7
- U1 pad 16: Net-(U1-Pad16) -> /SEG8
- U1 pad 17: Net-(U1-Pad17) -> +3V3
- U1 pad 19: Net-(U1-Pad19) -> /GRID2
- U1 pad 20: Net-(U1-Pad20) -> /GRID3
- U1 pad 21: Net-(U1-Pad21) -> /GRID4
- U1 pad 22: Net-(U1-Pad22) -> /GRID5
- U1 pad 23: Net-(U1-Pad23) -> /GRID6
- U1 pad 24: Net-(U1-Pad24) -> /GRID7
- U1 pad 25: Net-(U1-Pad25) -> /GRID8
- U1 pad 6: Net-(U1-Pad6) -> GND
- U1 pad 7: Net-(U1-Pad7) -> DATA
- U1 pad 8: Net-(U1-Pad8) -> CLK
- U1 pad 9: Net-(U1-Pad9) -> /SEG1
Routing:
- net /SEG6: track 0.00 -> 99.0 mm
- net /SEG8: track 0.00 -> 76.6 mm, vias 0 -> 2
- net /SEG2: track 0.00 -> 75.7 mm, vias 0 -> 2
- net /SEG7: track 0.00 -> 72.7 mm, vias 0 -> 2
- net /SEG1: track 0.00 -> 71.3 mm, vias 0 -> 1
- net /SEG5: track 0.00 -> 55.7 mm
- net /SEG4: track 0.00 -> 51.7 mm
- net /GRID8: track 0.00 -> 42.7 mm
- net /SEG3: track 0.00 -> 40.9 mm
- net /GRID7: track 0.00 -> 38.2 mm
- net /GRID6: track 0.00 -> 37.9 mm
- net /GRID5: track 0.00 -> 29.3 mm
- net /GRID2: track 0.00 -> 17.6 mm
- net /GRID4: track 0.00 -> 17.2 mm, vias 0 -> 1
- net /GRID3: track 0.00 -> 15.7 mm

Commit message: Add in and route the pull up resistors
Parts:
- added C1: 10uF, Resistor_SMD:R_0603_1608Metric, B.Cu at (197.8, 106.0)
- added R1: 10k, Resistor_SMD:R_0603_1608Metric, B.Cu at (197.8, 100.0)
- added R2: 10k, Resistor_SMD:R_0603_1608Metric, B.Cu at (197.8, 103.0)
Routing:
- net CLK: track 0.00 -> 67.4 mm, vias 0 -> 2
- net DATA: track 0.00 -> 64.6 mm, vias 0 -> 2
- net +3V3: track 0.00 -> 32.8 mm
- net /SEG4: track 51.7 -> 80.4 mm, vias 0 -> 1
- net /SEG3: track 40.9 -> 67.0 mm, vias 0 -> 2
- net /SEG5: track 55.7 -> 80.2 mm, vias 0 -> 1
- net /SEG6: track 99.0 -> 99.9 mm

Commit message: Correct label spelling error and re-route signals
Connections:
- DS1 pad 12: /GRDI1 -> /GRID1
Routing:
- net +3V3: track 32.8 -> 69.9 mm, vias 0 -> 2
- net /GRID1: track 0.00 -> 26.1 mm
- net /SEG6: track 99.9 -> 102.2 mm

Commit message: Add ground fill zones
Routing:
- net GND: track 0.00 -> 8.44 mm, vias 0 -> 13
- added copper zone on B.Cu, net GND
- added copper zone on F.Cu, net GND
Changed lines of the file:
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@@
     (thickness 1.6)
     (drawings 6)
-    (tracks 265)
+    (tracks 282)
     (zones 0)
     (modules 7)
@@
   (gr_line (start 270 112) (end 170 112) (layer Edge.Cuts) (width 0.05))
   (gr_line (start 270 92.5) (end 270 112) (layer Edge.Cuts) (width 0.05))
+  (via (at 250.75 99.5) (size 0.8) (drill 0.4) (layers F.Cu B.Cu) (net 31))
   (segment (start 221.100001 105.399999) (end 221.025 105.475) (width 0.25) (layer B.Cu) (net 15))
   (segment (start 241.170001 105.399999) (end 221.100001 105.399999) (width 0.25) (layer B.Cu) (net 15))
@@
   (segment (start 195.5 108.7) (end 195.5 108.7) (width 0.25) (layer F.Cu) (net 30))
   (via (at 195.5 108.7) (size 0.8) (drill 0.4) (layers F.Cu B.Cu) (net 30))
+  (via (at 230 107.75) (size 0.8) (drill 0.4) (layers F.Cu B.Cu) (net 31))
+  (via (at 240 107.75) (size 0.8) (drill 0.4) (layers F.Cu B.Cu) (net 31))
+  (via (at 230.25 99.75) (size 0.8) (drill 0.4) (layers F.Cu B.Cu) (net 31))
+  (via (at 240.25 99.5) (size 0.8) (drill 0.4) (layers F.Cu B.Cu) (net 31))
+  (via (at 266.5 95.25) (size 0.8) (drill 0.4) (layers F.Cu B.Cu) (net 31))
+  (via (at 266.25 108.5) (size 0.8) (drill 0.4) (layers F.Cu B.Cu) (net 31))
+  (segment (start 223.489997 108.149999) (end 229.600001 108.149999) (width 0.25) (layer B.Cu) (net 31))
+  (segment (start 229.600001 108.149999) (end 230 107.75) (width 0.25) (layer B.Cu) (net 31))
+  (segment (start 222.975 107.635002) (end 223.489997 108.149999) (width 0.25) (layer B.Cu) (net 31))
+  (segment (start 222.975 106.6) (end 222.975 107.635002) (width 0.25) (layer B.Cu) (net 31))
+  (via (at 214.25 94.75) (size 0.8) (drill 0.4) (layers F.Cu B.Cu) (net 31))
+  (via (at 222 94.75) (size 0.8) (drill 0.4) (layers F.Cu B.Cu) (net 31))
+  (via (at 230 95.75) (size 0.8) (drill 0.4) (layers F.Cu B.Cu) (net 31))
+  (via (at 245.75 96) (size 0.8) (drill 0.4) (layers F.Cu B.Cu) (net 31))
+  (via (at 205.75 106) (size 0.8) (drill 0.4) (layers F.Cu B.Cu) (net 31))
+  (via (at 202.25 102.75) (size 0.8) (drill 0.4) (layers F.Cu B.Cu) (net 31))
   (segment (start 196.444999 102.444999) (end 197 103) (width 0.25) (layer B.Cu) (net 32))
   (segment (start 174.175001 102.444999) (end 196.444999 102.444999) (width 0.25) (layer B.Cu) (net 32))
@@
   (segment (start 198.650001 93.879999) (end 203.210001 93.879999) (width 0.25) (layer B.Cu) (net 34))
   (segment (start 197.65 94.88) (end 198.650001 93.879999) (width 0.25) (layer B.Cu) (net 34))
+  (zone (net 31) (net_name GND) (layer B.Cu) (hatch edge 0.508)
+    (connect_pads (clearance 0.508))
+    (min_thickness 0.254)
+    (fill yes (arc_segments 32) (thermal_gap 0.508) (thermal_bridge_width 0.508))
+    (polygon
+      (pts
+        (xy 270 112) (xy 170 112) (xy 170 92.5) (xy 270 92.5)
+      )
+    )
+  )
+  (zone (net 31) (net_name GND) (layer F.Cu) (hatch edge 0.508)
+    (connect_pads (clearance 0.508))
+    (min_thickness 0.254)
+    (fill yes (arc_segments 32) (thermal_gap 0.508) (thermal_bridge_width 0.508))
+    (polygon
+      (pts
+        (xy 270 112) (xy 170 112) (xy 170 92.5) (xy 270 92.5)
+      )
+    )
+  )
 )

Commit message: Update to use correct footrpint for GN1640
Parts:
- added G***: LOGO, jjh:Untitled, B.Cu at (255.0, 103.5)
- added G***: LOGO, jjh:j2h_small, F.Cu at (186.0, 102.0)
- U1: footprint Package_SO:SSOP-28_5.3x10.2mm_P0.65mm -> jjh:TM1640
- moved U1 4.04 mm to (226.0, 102.4), turned to 180 degrees
Routing:
- net GND: track 8.44 -> 0.00 mm, vias 13 -> 9
- net /GRID4: track 17.2 -> 23.1 mm
- net /GRID8: track 42.7 -> 37.2 mm
- net /GRID5: track 29.3 -> 24.3 mm
- net /GRID7: track 38.2 -> 33.5 mm
- net /GRID6: track 37.9 -> 33.9 mm
- net CLK: track 67.4 -> 64.0 mm
- net /GRID3: track 16.0 -> 18.9 mm
- net /SEG7: track 72.7 -> 75.4 mm
- net /GRID2: track 17.6 -> 20.2 mm
- net +3V3: track 69.9 -> 72.5 mm
- net /SEG4: track 80.4 -> 82.7 mm
- net /SEG6: track 102.2 -> 100.0 mm
- net DATA: track 64.6 -> 66.8 mm
- net /SEG8: track 76.6 -> 78.7 mm
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Other:
- board text added: "PMOD 7 segment Display @jamesjhorton jjhorton.co.uk"
