File: PMod_7Segment/hardware/PMod_7Segement.kicad_pcb (KiCad board)
At the start: 2 copper layers, 100 x 19.5 mm, 9 parts, among them J1 Conn_02x06_Odd_Even, U1 GN1640

Commit message: fix the DRC errors in PCB on v6
Routing:
- net /SEG4: track 82.7 -> 81.7 mm
- net /SEG2: track 77.5 -> 76.6 mm
- net /SEG7: track 75.4 -> 74.6 mm
- net +3V3: track 72.5 -> 71.9 mm
Other:
- net class Default removed
