File: PMod_7Segment/hardware/PMod_7Segement.sch (KiCad schematic (older format))
At the start: 3 parts, among them U1 GN1640

Commit message: Add pmod connector and start the layout of data bus
Parts:
- added J1: Conn_02x06_Odd_Even, Connector_PinHeader_2.54mm:PinHeader_2x06_P2.54mm_Vertical, symbol Connector_Generic:Conn_02x06_Odd_Even
Connections:
- net SEG2: now reaches U1.10 (SEG2)
- net SEG3: now reaches U1.11 (SEG3)
- net SEG4: now reaches U1.12 (SEG4)
- net SEG5: now reaches U1.13 (SEG5)
- net SEG6: now reaches U1.14 (SEG6)
- net SEG7: now reaches U1.15 (SEG7)
- net SEG8: now reaches U1.16 (SEG8)
- net +3V3: now reaches U1.17 (VDD)
- net +3V3: now also J1.11 (Pin_11), J1.12 (Pin_12)
- net GND: now reaches U1.6 (GND)
- net GND: now also J1.10 (Pin_10), J1.9 (Pin_9)
- net DATA: now reaches U1.7 (DATA)
- net DATA: now also J1.7 (Pin_7)
- net CLK: now reaches U1.8 (CLK)
- net CLK: now also J1.5 (Pin_5)
- net SEG1: now reaches U1.9 (SEG1)
- no-connect marks 0 -> 6
Other:
- moved on the sheet: DS1, DS2

Commit message: Add pull up resitors and work on layout
Parts:
- added C?: 10uF, Resistor_SMD:R_0603_1608Metric, symbol Device:C
- added R? (x2): 10k, Resistor_SMD:R_0603_1608Metric, symbol Device:R
Connections:
- net +3V3: now also C?.1, R?.1, R?.1
- net CLK: now also R?.2
- net DATA: now also R?.2
- net GND: now also C?.2
- net SEG1: now also DS1.11 (A_A), DS2.11 (A_A)
- net SEG2: now also DS1.7 (A_B), DS2.7 (A_B)
- net SEG3: now also DS1.4 (A_C), DS2.4 (A_C)
- net SEG4: now also DS1.2 (A_D), DS2.2 (A_D)
- net SEG5: now also DS1.1 (A_E), DS2.1 (A_E)
- net SEG6: now also DS1.10 (A_F), DS2.10 (A_F)
- net SEG7: now also DS1.5 (A_G), DS2.5 (A_G)
- net SEG8: now also DS1.3 (A_D.P.), DS2.3 (A_D.P.)
- net GRID1: now reaches U1.18 (GRID1)
- net GRID2: now reaches U1.19 (GRID2)
- net GRID2: now also DS1.9 (COMMON_K_(DIGIT_2))
- net GRID3: now reaches U1.20 (GRID3)
- net GRID3: now also DS1.8 (COMMON_K_(DIGIT_3))
- net GRID4: now reaches U1.21 (GRID4)
- net GRID4: now also DS1.6 (COMMON_K_(DIGIT_4))
- net GRID5: now reaches U1.22 (GRID5)
- net GRID5: now also DS2.12 (COMMON_K_(DIGIT_1))
- net GRID6: now reaches U1.23 (GRID6)
- net GRID6: now also DS2.9 (COMMON_K_(DIGIT_2))
- net GRID7: now reaches U1.24 (GRID7)
- net GRID7: now also DS2.8 (COMMON_K_(DIGIT_3))
- net GRID8: now reaches U1.25 (GRID8)
- net GRID8: now also DS2.6 (COMMON_K_(DIGIT_4))
- net GRDI1: now reaches DS1.12 (COMMON_K_(DIGIT_1))
- no-connect marks 6 -> 14
Changed lines of the file:
@@
 DATA
 $Comp
-L power:GND #PWR?
+L power:GND #PWR0101
 U 1 1 61091D57
 P 2250 5250
-F 0 "#PWR?" H 2250 5000 50  0001 C CNN
+F 0 "#PWR0101" H 2250 5000 50  0001 C CNN
 F 1 "GND" V 2255 5122 50  0000 R CNN
 F 2 "" H 2250 5250 50  0001 C CNN
@@
 $EndComp
 $Comp
-L power:GND #PWR?
+L power:GND #PWR0102
 U 1 1 61091FA9
 P 3300 5250
-F 0 "#PWR?" H 3300 5000 50  0001 C CNN
+F 0 "#PWR0102" H 3300 5000 50  0001 C CNN
 F 1 "GND" V 3305 5122 50  0000 R CNN
 F 2 "" H 3300 5250 50  0001 C CNN
@@
 $EndComp
 $Comp
-L power:+3V3 #PWR?
+L power:+3V3 #PWR0103
 U 1 1 610924B4
 P 3300 5350
-F 0 "#PWR?" H 3300 5200 50  0001 C CNN
+F 0 "#PWR0103" H 3300 5200 50  0001 C CNN
 F 1 "+3V3" V 3315 5478 50  0000 L CNN
 F 2 "" H 3300 5350 50  0001 C CNN
@@
 $EndComp
 $Comp
-L power:+3V3 #PWR?
+L power:+3V3 #PWR0104
 U 1 1 61092748
 P 2250 5350
-F 0 "#PWR?" H 2250 5200 50  0001 C CNN
+F 0 "#PWR0104" H 2250 5200 50  0001 C CNN
 F 1 "+3V3" V 2265 5478 50  0000 L CNN
 F 2 "" H 2250 5350 50  0001 C CNN
@@
 	3300 5250 3050 5250
 $Comp
-L power:+3V3 #PWR?
+L power:+3V3 #PWR0105
 U 1 1 61093001
 P 1600 1400
-F 0 "#PWR?" H 1600 1250 50  0001 C CNN
+F 0 "#PWR0105" H 1600 1250 50  0001 C CNN
 F 1 "+3V3" V 1615 1528 50  0000 L CNN
 F 2 "" H 1600 1400 50  0001 C CNN
@@
 $EndComp
 $Comp
-L power:GND #PWR?
+L power:GND #PWR0106
 U 1 1 61093663
 P 1600 1500
-F 0 "#PWR?" H 1600 1250 50  0001 C CNN
+F 0 "#PWR0106" H 1600 1250 50  0001 C CNN
 F 1 "GND" V 1605 1372 50  0000 R CNN
 F 2 "" H 1600 1500 50  0001 C CNN
@@
 Wire Wire Line
 	9750 2050 10200 2050
-Wire Bus Line
-	3700 950  3700 1900
+Entry Wire Line
+	3700 2900 3600 3000
+Entry Wire Line
+	3700 3000 3600 3100
+Entry Wire Line
+	3700 3100 3600 3200
+Entry Wire Line
+	3700 3200 3600 3300
+Entry Wire Line
+	3700 3300 3600 3400
+Entry Wire Line
+	3700 3400 3600 3500
+Entry Wire Line
+	3700 3500 3600 3600
+Entry Wire Line
+	3700 3600 3600 3700
+Wire Wire Line
+	3200 3000 3600 3000
+Wire Wire Line
+	3600 3700 3200 3700
+Wire Wire Line
+	3200 3100 3600 3100
+Wire Wire Line
+	3600 3200 3200 3200
+Wire Wire Line
+	3200 3300 3600 3300
+Wire Wire Line
+	3600 3400 3200 3400
+Wire Wire Line
+	3200 3500 3600 3500
+Wire Wire Line
+	3600 3600 3200 3600
+Text Label 3250 3700 0    50   ~ 0
+GRID1
+Text Label 3250 3600 0    50   ~ 0
+GRID2
+Text Label 3250 3500 0    50   ~ 0
+GRID3
+Text Label 3250 3400 0    50   ~ 0
+GRID4
+Text Label 3250 3300 0    50   ~ 0
+GRID5
+Text Label 3250 3200 0    50   ~ 0
+GRID6
+Text Label 3250 3100 0    50   ~ 0
+GRID7
+Text Label 3250 3000 0    50   ~ 0
+GRID8
+Text Label 9800 1550 0    50   ~ 0
+GRDI1
+Text Label 9800 1850 0    50   ~ 0
+GRID2
+Text Label 9800 1950 0    50   ~ 0
+GRID3
+Text Label 6850 2050 0    50   ~ 0
+GRID4
+Text Label 9800 2550 0    50   ~ 0
+GRID5
+Text Label 9800 2850 0    50   ~ 0
+GRID6
+Text Label 9800 2950 0    50   ~ 0
+GRID7
+Text Label 6850 3050 0    50   ~ 0
+GRID8
+Text Label 9800 1650 0    50   ~ 0
+SEG1
+Text Label 9800 2650 0    50   ~ 0
+SEG1
+Text Label 9800 2050 0    50   ~ 0
+SEG2
+Text Label 9800 3050 0    50   ~ 0
+SEG2
+Text Label 6850 2850 0    50   ~ 0
+SEG3
+Text Label 6850 1850 0    50   ~ 0
+SEG3
+Text Label 6850 1650 0    50   ~ 0
+SEG4
+Text Label 6850 2650 0    50   ~ 0
+SEG4
+Text Label 6850 2550 0    50   ~ 0
+SEG5
+Text Label 6850 1550 0    50   ~ 0
+SEG5
+Text Label 9800 1750 0    50   ~ 0
+SEG6
+Text Label 9800 2750 0    50   ~ 0
+SEG6
+Text Label 6850 2950 0    50   ~ 0
+SEG7
+Text Label 6850 1950 0    50   ~ 0
+SEG7
+Text Label 6850 1750 0    50   ~ 0
+SEG8
+Text Label 6850 2750 0    50   ~ 0
+SEG8
+NoConn ~ 3200 2900
+NoConn ~ 3200 2800
+NoConn ~ 3200 2700
+NoConn ~ 3200 2600
+NoConn ~ 3200 2500
+NoConn ~ 3200 2400
+NoConn ~ 3200 2300
+NoConn ~ 3200 2200
+$Comp
+L Device:R R?
+U 1 1 610CEB3C
+P 6300 4950
+F 0 "R?" H 6370 4996 50  0000 L CNN
+F 1 "10k" H 6370 4905 50  0000 L CNN
+F 2 "Resistor_SMD:R_0603_1608Metric" V 6230 4950 50  0001 C CNN
+F 3 "~" H 6300 4950 50  0001 C CNN
+	1    6300 4950
+	1    0    0    -1
+$EndComp
+$Comp
+L Device:R R?
+U 1 1 610CF026
+P 7000 4950
+F 0 "R?" H 7070 4996 50  0000 L CNN
+F 1 "10k" H 7070 4905 50  0000 L CNN
+F 2 "Resistor_SMD:R_0603_1608Metric" V 6930 4950 50  0001 C CNN
+F 3 "~" H 7000 4950 50  0001 C CNN
+	1    7000 4950
+	1    0    0    -1
+$EndComp
+$Comp
+L Device:C C?
+U 1 1 610CF6C9
+P 7800 4950
+F 0 "C?" H 7915 4996 50  0000 L CNN
+F 1 "10uF" H 7915 4905 50  0000 L CNN
+F 2 "Resistor_SMD:R_0603_1608Metric" H 7838 4800 50  0001 C CNN
+F 3 "~" H 7800 4950 50  0001 C CNN
+	1    7800 4950
+	1    0    0    -1
+$EndComp
+$Comp
+L power:+3V3 #PWR?
+U 1 1 610CFA76
+P 6300 4650
+F 0 "#PWR?" H 6300 4500 50  0001 C CNN
+F 1 "+3V3" H 6315 4823 50  0000 C CNN
+F 2 "" H 6300 4650 50  0001 C CNN
+F 3 "" H 6300 4650 50  0001 C CNN
+	1    6300 4650
+	1    0    0    -1
+$EndComp
+$Comp
+L power:+3V3 #PWR?
+U 1 1 610CFD5D
+P 7000 4650
+F 0 "#PWR?" H 7000 4500 50  0001 C CNN
+F 1 "+3V3" H 7015 4823 50  0000 C CNN
+F 2 "" H 7000 4650 50  0001 C CNN
+F 3 "" H 7000 4650 50  0001 C CNN
+	1    7000 4650
+	1    0    0    -1
+$EndComp
+$Comp
+L power:+3V3 #PWR?
+U 1 1 610D0056
+P 7800 4650
+F 0 "#PWR?" H 7800 4500 50  0001 C CNN
+F 1 "+3V3" H 7815 4823 50  0000 C CNN
+F 2 "" H 7800 4650 50  0001 C CNN
+F 3 "" H 7800 4650 50  0001 C CNN
+	1    7800 4650
+	1    0    0    -1
+$EndComp
+$Comp
+L power:GND #PWR?
+U 1 1 610D03B7
+P 7800 5300
+F 0 "#PWR?" H 7800 5050 50  0001 C CNN
+F 1 "GND" H 7805 5127 50  0000 C CNN
+F 2 "" H 7800 5300 50  0001 C CNN
+F 3 "" H 7800 5300 50  0001 C CNN
+	1    7800 5300
+	1    0    0    -1
+$EndComp
+Wire Wire Line
+	7800 4800 7800 4650
+Wire Wire Line
+	7800 5100 7800 5300
+Wire Wire Line
+	7000 4800 7000 4650
+Wire Wire Line
+	6300 4800 6300 4650
+Text GLabel 6100 5350 0    50   Input ~ 0
+CLK
+Text GLabel 6900 5350 0    50   Input ~ 0
+DATA
+Wire Wire Line
+	6900 5350 7000 5350
+Wire Wire Line
+	7000 5350 7000 5100
+Wire Wire Line
+	6300 5100 6300 5350
+Wire Wire Line
+	6300 5350 6100 5350
 Wire Bus Line
 	6500 950  6500 3000
 Wire Bus Line
 	10300 950  10300 3000
+Wire Bus Line
+	3700 950  3700 3600
 $EndSCHEMATC

Commit message: Correct label spelling error and re-route signals
Parts:
- gave numbers to parts that had none: 3
Connections:
- net GRDI1 is gone; now on net GRID1: DS1.12 (COMMON_K_(DIGIT_1))
Changed lines of the file:
@@
 GRID8
 Text Label 9800 1550 0    50   ~ 0
-GRDI1
+GRID1
 Text Label 9800 1850 0    50   ~ 0
 GRID2
@@
 NoConn ~ 3200 2200
 $Comp
-L Device:R R?
+L Device:R R1
 U 1 1 610CEB3C
 P 6300 4950
-F 0 "R?" H 6370 4996 50  0000 L CNN
+F 0 "R1" H 6370 4996 50  0000 L CNN
 F 1 "10k" H 6370 4905 50  0000 L CNN
 F 2 "Resistor_SMD:R_0603_1608Metric" V 6230 4950 50  0001 C CNN
@@
 $EndComp
 $Comp
-L Device:R R?
+L Device:R R2
 U 1 1 610CF026
 P 7000 4950
-F 0 "R?" H 7070 4996 50  0000 L CNN
+F 0 "R2" H 7070 4996 50  0000 L CNN
 F 1 "10k" H 7070 4905 50  0000 L CNN
 F 2 "Resistor_SMD:R_0603_1608Metric" V 6930 4950 50  0001 C CNN
@@
 $EndComp
 $Comp
-L Device:C C?
+L Device:C C1
 U 1 1 610CF6C9
 P 7800 4950
-F 0 "C?" H 7915 4996 50  0000 L CNN
+F 0 "C1" H 7915 4996 50  0000 L CNN
 F 1 "10uF" H 7915 4905 50  0000 L CNN
 F 2 "Resistor_SMD:R_0603_1608Metric" H 7838 4800 50  0001 C CNN
@@
 $EndComp
 $Comp
-L power:+3V3 #PWR?
+L power:+3V3 #PWR0107
 U 1 1 610CFA76
 P 6300 4650
-F 0 "#PWR?" H 6300 4500 50  0001 C CNN
+F 0 "#PWR0107" H 6300 4500 50  0001 C CNN
 F 1 "+3V3" H 6315 4823 50  0000 C CNN
 F 2 "" H 6300 4650 50  0001 C CNN
@@
 $EndComp
 $Comp
-L power:+3V3 #PWR?
+L power:+3V3 #PWR0108
 U 1 1 610CFD5D
 P 7000 4650
-F 0 "#PWR?" H 7000 4500 50  0001 C CNN
+F 0 "#PWR0108" H 7000 4500 50  0001 C CNN
 F 1 "+3V3" H 7015 4823 50  0000 C CNN
 F 2 "" H 7000 4650 50  0001 C CNN
@@
 $EndComp
 $Comp
-L power:+3V3 #PWR?
+L power:+3V3 #PWR0109
 U 1 1 610D0056
 P 7800 4650
-F 0 "#PWR?" H 7800 4500 50  0001 C CNN
+F 0 "#PWR0109" H 7800 4500 50  0001 C CNN
 F 1 "+3V3" H 7815 4823 50  0000 C CNN
 F 2 "" H 7800 4650 50  0001 C CNN
@@
 $EndComp
 $Comp
-L power:GND #PWR?
+L power:GND #PWR0110
 U 1 1 610D03B7
 P 7800 5300
-F 0 "#PWR?" H 7800 5050 50  0001 C CNN
+F 0 "#PWR0110" H 7800 5050 50  0001 C CNN
 F 1 "GND" H 7805 5127 50  0000 C CNN
 F 2 "" H 7800 5300 50  0001 C CNN

Commit message: Update to use correct footrpint for GN1640
Parts:
- U1: footprint Package_SO:SSOP-28_5.3x10.2mm_P0.65mm -> jjh:TM1640
Changed lines of the file:
@@
 F 0 "U1" H 2500 4465 50  0000 C CNN
 F 1 "GN1640" H 2500 4374 50  0000 C CNN
-F 2 "Package_SO:SSOP-28_5.3x10.2mm_P0.65mm" H 2550 1550 50  0001 C CNN
+F 2 "jjh:TM1640" H 2550 1550 50  0001 C CNN
 F 3 "https://datasheet.lcsc.com/lcsc/2009241905_GN-Semic-GN1640_C265478.pdf" H 2300 3600 50  0001 C CNN
 	1    2500 2750
