File: PMod_7Segment/hardware/PMod_7Segement.kicad_sch (KiCad schematic)
At the start: 7 parts

Commit message: update for schematic to pass erc
Parts:
- removed DS1, DS2: (no value), symbol JJH_Library:LTC-5723HR
- removed U1: (no value), symbol JJH_Library:GN1640
- added DS1, DS2: LTC-5723HR, DIP1524W75P254L5030H825Q12N, symbol jjh:LTC-5723HR
- added U1: GN1640, Package_SO:SSOP-28_5.3x10.2mm_P0.65mm, symbol jjh:GN1640
- C1: value (none) -> 10uF; footprint (none) -> Resistor_SMD:R_0603_1608Metric
- J1: value (none) -> Conn_02x06_Odd_Even; footprint (none) -> Connector_PinHeader_2.54mm:PinHeader_2x06_P2.54mm_Vertical
- R1, R2: value (none) -> 10k; footprint (none) -> Resistor_SMD:R_0603_1608Metric
Connections:
- net +3V3: now also U1.17 (VDD)
- net CLK: now also U1.8 (CLK)
- net DATA: now also U1.7 (DATA)
- net GND: now also U1.6 (GND)
- net GRID1: now also DS1.12 (COMMON_K_(DIGIT_1)), U1.18 (GRID1)
- net GRID2: now also DS1.9 (COMMON_K_(DIGIT_2)), U1.19 (GRID2)
- net GRID3: now also DS1.8 (COMMON_K_(DIGIT_3)), U1.20 (GRID3)
- net GRID4: now also DS1.6 (COMMON_K_(DIGIT_4)), U1.21 (GRID4)
- net GRID5: now also DS2.12 (COMMON_K_(DIGIT_1)), U1.22 (GRID5)
- net GRID6: now also DS2.9 (COMMON_K_(DIGIT_2)), U1.23 (GRID6)
- net GRID7: now also DS2.8 (COMMON_K_(DIGIT_3)), U1.24 (GRID7)
- net GRID8: now also DS2.6 (COMMON_K_(DIGIT_4)), U1.25 (GRID8)
- net SEG1: now also DS1.11 (A_A), DS2.11 (A_A), U1.9 (SEG1)
- net SEG2: now also DS1.7 (A_B), DS2.7 (A_B), U1.10 (SEG2)
- net SEG3: now also DS1.4 (A_C), DS2.4 (A_C), U1.11 (SEG3)
- net SEG4: now also DS1.2 (A_D), DS2.2 (A_D), U1.12 (SEG4)
- net SEG5: now also DS1.1 (A_E), DS2.1 (A_E), U1.13 (SEG5)
- net SEG6: now also DS1.10 (A_F), DS2.10 (A_F), U1.14 (SEG6)
- net SEG7: now also DS1.5 (A_G), DS2.5 (A_G), U1.15 (SEG7)
- net SEG8: now also DS1.3 (A_D.P.), DS2.3 (A_D.P.), U1.16 (SEG8)

Commit message: Schematic visual improvements and add license
Other:
- note added: "PMod Connector"
- note added: "Power Supply Capacitor"
- note added: "Pull up Resistors"
- company: (none) -> James Horton
- title: (none) -> PMod 7 Segment Display
- moved on the sheet: C1, J1, R1, R2
