File: PMOD_LEDArray/PMOD_LEDArray.sch (KiCad schematic (older format))
At the start: 130 parts

Commit message: Arrange the LED's in a 8*16 grid
Parts:
- gave numbers to parts that had none: 130
Connections:
- net GRID1: no longer D1.2 (A), D10.2 (A), D105.2 (A), D106.2 (A), D107.2 (A), D11.2 (A), D113.2 (A), D114.2 (A), D115.2 (A), D121.2 (A), D122.2 (A), D123.2 (A), D17.2 (A), D18.2 (A), D19.2 (A), D2.2 (A), D25.2 (A), D26.2 (A), D27.2 (A), D3.2 (A), D33.2 (A), D34.2 (A), D35.2 (A), D41.2 (A), D42.2 (A), D43.2 (A), D49.2 (A), D50.2 (A), D51.2 (A), D57.2 (A), D58.2 (A), D59.2 (A), D65.2 (A), D66.2 (A), D67.2 (A), D73.2 (A), D74.2 (A), D75.2 (A), D81.2 (A), D82.2 (A), D83.2 (A), D89.2 (A), D9.2 (A), D90.2 (A), D91.2 (A), D97.2 (A), D98.2 (A), D99.2 (A), U1.14 (SEG6), U1.15 (SEG7), U1.16 (SEG8)
- new net SEG6: D107.2 (A), D11.2 (A), D115.2 (A), D123.2 (A), D19.2 (A), D27.2 (A), D3.2 (A), D35.2 (A), D43.2 (A), D51.2 (A), D59.2 (A), D67.2 (A), D75.2 (A), D83.2 (A), D91.2 (A), D99.2 (A), U1.14 (SEG6)
- new net SEG7: D10.2 (A), D106.2 (A), D114.2 (A), D122.2 (A), D18.2 (A), D2.2 (A), D26.2 (A), D34.2 (A), D42.2 (A), D50.2 (A), D58.2 (A), D66.2 (A), D74.2 (A), D82.2 (A), D90.2 (A), D98.2 (A), U1.15 (SEG7)
- new net SEG8: D1.2 (A), D105.2 (A), D113.2 (A), D121.2 (A), D17.2 (A), D25.2 (A), D33.2 (A), D41.2 (A), D49.2 (A), D57.2 (A), D65.2 (A), D73.2 (A), D81.2 (A), D89.2 (A), D9.2 (A), D97.2 (A), U1.16 (SEG8)

Commit message: Add resitors and start removing LED number from silk screen
Parts:
- added C?: 100uF, Capacitor_SMD:C_0201_0603Metric, symbol Device:C
- added R? (x2): 10k, Resistor_SMD:R_0603_1608Metric, symbol Device:R
- J1: footprint (none) -> Connector_PinHeader_2.54mm:PinHeader_2x06_P2.54mm_Vertical
Connections:
- net +3V3: now also U1.17 (VDD), C?.1, R?.1, R?.1
- net CLK: now also U1.8 (CLK), R?.2
- net DATA: now also U1.7 (DATA), R?.2
- net GND: now also U1.6 (GND), C?.2
- no-connect marks 0 -> 6
Changed lines of the file:
@@
 F 0 "J1" H 1900 6367 50  0000 C CNN
 F 1 "Conn_02x06_Odd_Even" H 1900 6276 50  0000 C CNN
-F 2 "" H 1850 5950 50  0001 C CNN
+F 2 "Connector_PinHeader_2.54mm:PinHeader_2x06_P2.54mm_Vertical" H 1850 5950 50  0001 C CNN
 F 3 "~" H 1850 5950 50  0001 C CNN
 	1    1850 5950
@@
 Wire Wire Line
 	1500 850  1000 850
+Connection ~ 1500 850
+Connection ~ 1000 850
+Text GLabel 4150 5650 0    50   Input ~ 0
+DATA
+Text GLabel 4150 5750 0    50   Input ~ 0
+CLK
+Wire Wire Line
+	4150 5650 4450 5650
+Wire Wire Line
+	4450 5750 4150 5750
+$Comp
+L power:GND #PWR0105
+U 1 1 611A3A3C
+P 4150 5200
+F 0 "#PWR0105" H 4150 4950 50  0001 C CNN
+F 1 "GND" V 4155 5072 50  0000 R CNN
+F 2 "" H 4150 5200 50  0001 C CNN
+F 3 "" H 4150 5200 50  0001 C CNN
+	1    4150 5200
+	0    1    1    0
+$EndComp
+$Comp
+L power:+3V3 #PWR0106
+U 1 1 611A4CDD
+P 4150 5100
+F 0 "#PWR0106" H 4150 4950 50  0001 C CNN
+F 1 "+3V3" V 4165 5228 50  0000 L CNN
+F 2 "" H 4150 5100 50  0001 C CNN
+F 3 "" H 4150 5100 50  0001 C CNN
+	1    4150 5100
+	0    -1   -1   0
+$EndComp
+Wire Wire Line
+	4450 5200 4150 5200
+Wire Wire Line
+	4150 5100 4450 5100
+$Comp
+L Device:R R?
+U 1 1 6126C5AE
+P 7450 5700
+F 0 "R?" H 7520 5746 50  0000 L CNN
+F 1 "10k" H 7520 5655 50  0000 L CNN
+F 2 "Resistor_SMD:R_0603_1608Metric" V 7380 5700 50  0001 C CNN
+F 3 "~" H 7450 5700 50  0001 C CNN
+	1    7450 5700
+	1    0    0    -1
+$EndComp
+$Comp
+L Device:R R?
+U 1 1 6126E9D3
+P 8700 5750
+F 0 "R?" H 8770 5796 50  0000 L CNN
+F 1 "10k" H 8770 5705 50  0000 L CNN
+F 2 "Resistor_SMD:R_0603_1608Metric" V 8630 5750 50  0001 C CNN
+F 3 "~" H 8700 5750 50  0001 C CNN
+	1    8700 5750
+	1    0    0    -1
+$EndComp
+$Comp
+L Device:C C?
+U 1 1 61270DCB
+P 9800 5650
+F 0 "C?" H 9915 5696 50  0000 L CNN
+F 1 "100uF" H 9915 5605 50  0000 L CNN
+F 2 "Capacitor_SMD:C_0201_0603Metric" H 9838 5500 50  0001 C CNN
+F 3 "~" H 9800 5650 50  0001 C CNN
+	1    9800 5650
+	1    0    0    -1
+$EndComp
+$Comp
+L power:+3V3 #PWR?
+U 1 1 6127325E
+P 7450 5350
+F 0 "#PWR?" H 7450 5200 50  0001 C CNN
+F 1 "+3V3" H 7465 5523 50  0000 C CNN
+F 2 "" H 7450 5350 50  0001 C CNN
+F 3 "" H 7450 5350 50  0001 C CNN
+	1    7450 5350
+	1    0    0    -1
+$EndComp
+Text GLabel 7250 6050 0    50   Input ~ 0
+DATA
+Text GLabel 8500 6050 0    50   Input ~ 0
+CLK
+$Comp
+L power:+3V3 #PWR?
+U 1 1 6138EDB3
+P 9800 5350
+F 0 "#PWR?" H 9800 5200 50  0001 C CNN
+F 1 "+3V3" H 9815 5523 50  0000 C CNN
+F 2 "" H 9800 5350 50  0001 C CNN
+F 3 "" H 9800 5350 50  0001 C CNN
+	1    9800 5350
+	1    0    0    -1
+$EndComp
+$Comp
+L power:GND #PWR?
+U 1 1 6138F749
+P 9800 6000
+F 0 "#PWR?" H 9800 5750 50  0001 C CNN
+F 1 "GND" H 9805 5827 50  0000 C CNN
+F 2 "" H 9800 6000 50  0001 C CNN
+F 3 "" H 9800 6000 50  0001 C CNN
+	1    9800 6000
+	1    0    0    -1
+$EndComp
+Wire Wire Line
+	9800 5800 9800 6000
+Wire Wire Line
+	9800 5500 9800 5350
+Wire Wire Line
+	7450 5550 7450 5350
+Wire Wire Line
+	7450 5850 7450 6050
+Wire Wire Line
+	7450 6050 7250 6050
+$Comp
+L power:+3V3 #PWR?
+U 1 1 6148E456
+P 8700 5350
+F 0 "#PWR?" H 8700 5200 50  0001 C CNN
+F 1 "+3V3" H 8715 5523 50  0000 C CNN
+F 2 "" H 8700 5350 50  0001 C CNN
+F 3 "" H 8700 5350 50  0001 C CNN
+	1    8700 5350
+	1    0    0    -1
+$EndComp
+Wire Wire Line
+	8700 5350 8700 5600
+Wire Wire Line
+	8700 5900 8700 6050
+Wire Wire Line
+	8700 6050 8500 6050
+NoConn ~ 2150 6050
+NoConn ~ 2150 5950
+NoConn ~ 2150 5850
+NoConn ~ 2150 5750
+NoConn ~ 1650 5850
+NoConn ~ 1650 5750
 Wire Bus Line
 	750  650  750  4600
@@
 Wire Bus Line
 	6150 4600 6150 7550
-Connection ~ 1500 850
-Connection ~ 1000 850
 $EndSCHEMATC

Commit message: PCB initial layout complete
Parts:
- C1: renamed from C?; footprint Capacitor_SMD:C_0201_0603Metric -> Capacitor_SMD:C_0603_1608Metric
- gave numbers to parts that had none: 2
Connections:
- net GRDI16 is gone; now on net GRID16: U1.5 (GRID16)
Changed lines of the file:
@@
 	6050 7400 5850 7400
 Text Label 5850 5900 0    50   ~ 0
-GRDI16
+GRID16
 Text Label 5850 6000 0    50   ~ 0
 GRID15
@@
 	4150 5100 4450 5100
 $Comp
-L Device:R R?
+L Device:R R1
 U 1 1 6126C5AE
 P 7450 5700
-F 0 "R?" H 7520 5746 50  0000 L CNN
+F 0 "R1" H 7520 5746 50  0000 L CNN
 F 1 "10k" H 7520 5655 50  0000 L CNN
 F 2 "Resistor_SMD:R_0603_1608Metric" V 7380 5700 50  0001 C CNN
@@
 $EndComp
 $Comp
-L Device:R R?
+L Device:R R2
 U 1 1 6126E9D3
 P 8700 5750
-F 0 "R?" H 8770 5796 50  0000 L CNN
+F 0 "R2" H 8770 5796 50  0000 L CNN
 F 1 "10k" H 8770 5705 50  0000 L CNN
 F 2 "Resistor_SMD:R_0603_1608Metric" V 8630 5750 50  0001 C CNN
@@
 $EndComp
 $Comp
-L Device:C C?
+L Device:C C1
 U 1 1 61270DCB
 P 9800 5650
-F 0 "C?" H 9915 5696 50  0000 L CNN
+F 0 "C1" H 9915 5696 50  0000 L CNN
 F 1 "100uF" H 9915 5605 50  0000 L CNN
-F 2 "Capacitor_SMD:C_0201_0603Metric" H 9838 5500 50  0001 C CNN
+F 2 "Capacitor_SMD:C_0603_1608Metric" H 9838 5500 50  0001 C CNN
 F 3 "~" H 9800 5650 50  0001 C CNN
 	1    9800 5650
@@
 $EndComp
 $Comp
-L power:+3V3 #PWR?
+L power:+3V3 #PWR0107
 U 1 1 6127325E
 P 7450 5350
-F 0 "#PWR?" H 7450 5200 50  0001 C CNN
+F 0 "#PWR0107" H 7450 5200 50  0001 C CNN
 F 1 "+3V3" H 7465 5523 50  0000 C CNN
 F 2 "" H 7450 5350 50  0001 C CNN
@@
 CLK
 $Comp
-L power:+3V3 #PWR?
+L power:+3V3 #PWR0108
 U 1 1 6138EDB3
 P 9800 5350
-F 0 "#PWR?" H 9800 5200 50  0001 C CNN
+F 0 "#PWR0108" H 9800 5200 50  0001 C CNN
 F 1 "+3V3" H 9815 5523 50  0000 C CNN
 F 2 "" H 9800 5350 50  0001 C CNN
@@
 $EndComp
 $Comp
-L power:GND #PWR?
+L power:GND #PWR0109
 U 1 1 6138F749
 P 9800 6000
-F 0 "#PWR?" H 9800 5750 50  0001 C CNN
+F 0 "#PWR0109" H 9800 5750 50  0001 C CNN
 F 1 "GND" H 9805 5827 50  0000 C CNN
 F 2 "" H 9800 6000 50  0001 C CNN
@@
 	7450 6050 7250 6050
 $Comp
-L power:+3V3 #PWR?
+L power:+3V3 #PWR0110
 U 1 1 6148E456
 P 8700 5350
-F 0 "#PWR?" H 8700 5200 50  0001 C CNN
+F 0 "#PWR0110" H 8700 5200 50  0001 C CNN
 F 1 "+3V3" H 8715 5523 50  0000 C CNN
 F 2 "" H 8700 5350 50  0001 C CNN
