File: PMod_LEDArray/Hardware/PMOD_LEDArray.kicad_pcb (KiCad board)
At the start: 2 copper layers, 81.6 x 23 mm, 133 parts, among them J1 Conn_02x06_Odd_Even, U1 GN1640

Commit message: Add mounting holes
Parts:
- added REF**: MountingHole_2.2mm_M2, MountingHole:MountingHole_2.2mm_M2, F.Cu at (188.5, 109.0)
- added REF**: MountingHole_2.2mm_M2, MountingHole:MountingHole_2.2mm_M2, F.Cu at (188.5, 87.5)
- added REF**: MountingHole_2.2mm_M2, MountingHole:MountingHole_2.2mm_M2, F.Cu at (107.5, 109.0)
- added REF**: MountingHole_2.2mm_M2, MountingHole:MountingHole_2.2mm_M2, F.Cu at (107.5, 87.5)
- moved C1 7.73 mm to (115.8, 107.3), turned to 90 degrees
- moved R1 1.10 mm to (114.0, 107.3)
- moved R2 1.10 mm to (112.2, 107.3)
- moved J1 0.10 mm to (106.8, 92.0)
Routing:
- net +3V3: track 30.3 -> 26.4 mm
- net GND: track 34.8 -> 32.0 mm
- net DATA: track 24.4 -> 25.1 mm
- net CLK: track 26.2 -> 26.7 mm
- added copper zone on F.Cu, net GND
Other:
- board size 81.6 x 23 mm -> 86 x 26.5 mm

Commit message: add logos and ground planes to PCB
Parts:
- added G***: LOGO, jjh:Untitled, B.Cu at (176.8, 98.4)
- added G***: LOGO, jjh:j2h_small, F.Cu at (117.5, 89.1)
Routing:
- net /SEG7: track 97.3 -> 95.9 mm
- net /SEG8: track 95.7 -> 94.4 mm, vias 17 -> 16
- added copper zone on B.Cu, net GND
Other:
- board text added: "PMod LED Array @jamesjhorton jjhorton.co.uk"

Commit message: Add copper logo onto board
Parts:
- added G***: LOGO, jjh:j2h_small, F.Cu at (188.5, 98.5)
Routing:
- net /SEG8: track 94.4 -> 93.2 mm
Changed lines of the file:
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@@
     (tracks 741)
     (zones 0)
-    (modules 139)
+    (modules 140)
     (nets 35)
   )
@@
     (add_net "Net-(J1-Pad8)")
   )
+  (module jjh:j2h_small (layer F.Cu)
+    (at 188.5 98.5 90)
+    (fp_text reference G*** (at 0 0 90) (layer F.Cu) hide
+      (effects (font (size 1.524 1.524) (thickness 0.3)))
+    )
+    (fp_text value LOGO (at 0.75 0 90) (layer F.Cu) hide
+      (effects (font (size 1.524 1.524) (thickness 0.3)))
+    )
+    (fp_poly (pts (xy -0.916266 -2.009227) (xy -0.853482 -1.905249) (xy -0.846666 -1.779412) (xy -0.873808 -1.544377)
+      (xy -0.947163 -1.192884) (xy -1.054627 -0.767452) (xy -1.184096 -0.310597) (xy -1.323466 0.135162)
+      (xy -1.460632 0.527309) (xy -1.583491 0.823326) (xy -1.593507 0.843949) (xy -1.84552 1.254772)
+      (xy -2.138795 1.518476) (xy -2.508188 1.657156) (xy -2.933521 1.693333) (xy -3.263589 1.680518)
+      (xy -3.476315 1.633994) (xy -3.622307 1.541641) (xy -3.640666 1.524) (xy -3.743665 1.393135)
+      (xy -3.79329 1.236553) (xy -3.789599 1.019163) (xy -3.732647 0.70587) (xy -3.64259 0.338667)
+      (xy -3.490729 -0.121096) (xy -3.312754 -0.419638) (xy -3.103321 -0.563792) (xy -2.927834 -0.575511)
+      (xy -2.820682 -0.519823) (xy -2.766175 -0.376243) (xy -2.762291 -0.122477) (xy -2.807013 0.263767)
+      (xy -2.835438 0.4445) (xy -2.870183 0.685662) (xy -2.858652 0.803872) (xy -2.78396 0.842943)
+      (xy -2.68046 0.846667) (xy -2.529615 0.818556) (xy -2.398393 0.720882) (xy -2.276258 0.533626)
+      (xy -2.152674 0.236772) (xy -2.017104 -0.189696) (xy -1.88659 -0.661479) (xy -1.769102 -1.076097)
+      (xy -1.65248 -1.440471) (xy -1.549369 -1.717989) (xy -1.472416 -1.872037) (xy -1.465559 -1.880465)
+      (xy -1.280323 -1.994264) (xy -1.087544 -2.032) (xy -0.916266 -2.009227)) (layer F.Cu) (width 0.01))
+    (fp_poly (pts (xy 2.237663 -1.98957) (xy 2.315048 -1.909091) (xy 2.317395 -1.769299) (xy 2.277991 -1.521819)
+      (xy 2.206716 -1.225413) (xy 2.12553 -0.898368) (xy 2.114169 -0.702877) (xy 2.18633 -0.610734)
+      (xy 2.355712 -0.593731) (xy 2.506774 -0.60752) (xy 2.633231 -0.636476) (xy 2.720861 -0.712238)
+      (xy 2.792752 -0.872) (xy 2.871995 -1.152955) (xy 2.890385 -1.225482) (xy 2.984196 -1.534236)
+      (xy 3.089379 -1.783792) (xy 3.183707 -1.921744) (xy 3.186641 -1.923982) (xy 3.398254 -2.015938)
+      (xy 3.611894 -2.018021) (xy 3.761774 -1.933431) (xy 3.783231 -1.894971) (xy 3.781034 -1.761583)
+      (xy 3.735539 -1.498458) (xy 3.655356 -1.13665) (xy 3.549094 -0.707213) (xy 3.425361 -0.241201)
+      (xy 3.292766 0.230331) (xy 3.159919 0.67633) (xy 3.035428 1.06574) (xy 2.927903 1.36751)
+      (xy 2.845952 1.550583) (xy 2.817806 1.5875) (xy 2.614785 1.676754) (xy 2.404105 1.681246)
+      (xy 2.254233 1.603673) (xy 2.231205 1.564388) (xy 2.225391 1.419684) (xy 2.258883 1.168692)
+      (xy 2.318529 0.890821) (xy 2.38814 0.607242) (xy 2.437404 0.394221) (xy 2.455334 0.3001)
+      (xy 2.380384 0.27063) (xy 2.194237 0.25484) (xy 2.132988 0.254) (xy 1.810642 0.254)
+      (xy 1.656137 0.849699) (xy 1.514022 1.275408) (xy 1.343928 1.546476) (xy 1.135247 1.676698)
+      (xy 1.007528 1.693333) (xy 0.831352 1.632768) (xy 0.778031 1.585649) (xy 0.769726 1.471454)
+      (xy 0.803174 1.225705) (xy 0.870567 0.878769) (xy 0.964097 0.461011) (xy 1.075958 0.002795)
+      (xy 1.198342 -0.465513) (xy 1.323442 -0.913547) (xy 1.443449 -1.310942) (xy 1.550558 -1.627333)
+      (xy 1.636959 -1.832354) (xy 1.670065 -1.883733) (xy 1.842479 -1.991941) (xy 2.054555 -2.02812)
+      (xy 2.237663 -1.98957)) (layer F.Cu) (width 0.01))
+    (fp_poly (pts (xy 0.600871 -2.393282) (xy 0.644177 -2.334949) (xy 0.638427 -2.138705) (xy 0.512548 -1.933058)
+      (xy 0.302723 -1.773723) (xy 0.270019 -1.758832) (xy 0.118525 -1.689685) (xy 0.115652 -1.655199)
+      (xy 0.232834 -1.629997) (xy 0.39938 -1.562052) (xy 0.424049 -1.468015) (xy 0.32157 -1.386201)
+      (xy 0.127 -1.354667) (xy -0.081456 -1.376338) (xy -0.162652 -1.454071) (xy -0.168037 -1.502833)
+      (xy -0.110065 -1.730766) (xy 0.0774 -1.889396) (xy 0.192223 -1.939941) (xy 0.358612 -2.042927)
+      (xy 0.423334 -2.156905) (xy 0.379179 -2.273896) (xy 0.262158 -2.248576) (xy 0.187678 -2.185811)
+      (xy 0.071751 -2.12442) (xy 0.021186 -2.182195) (xy 0.071385 -2.311641) (xy 0.082969 -2.326287)
+      (xy 0.242541 -2.427061) (xy 0.440065 -2.449776) (xy 0.600871 -2.393282)) (layer F.Cu) (width 0.01))
+  )
   (module jjh:Untitled (layer B.Cu)
     (at 176.8 98.4 90)
@@
   (segment (start 145.5 88) (end 144.575 88) (width 0.125) (layer F.Cu) (net 22))
   (segment (start 153.5 88) (end 152.575 88) (width 0.125) (layer F.Cu) (net 22))
-  (segment (start 112.077498 94.825) (end 111.862499 94.610001) (width 0.125) (layer F.Cu) (net 22))
-  (segment (start 113 94.825) (end 112.077498 94.825) (width 0.125) (layer F.Cu) (net 22))
   (segment (start 141.5 88) (end 140.575 88) (width 0.25) (layer F.Cu) (net 22))
-  (segment (start 111.862499 90.656999) (end 113.344508 89.17499) (width 0.125) (layer F.Cu) (net 22))
-  (segment (start 111.862499 94.610001) (end 111.862499 90.656999) (width 0.125) (layer F.Cu) (net 22))
-  (segment (start 123.83749 87.26249) (end 124.575 88) (width 0.125) (layer F.Cu) (net 22))
-  (segment (start 122.581902 87.26249) (end 123.83749 87.26249) (width 0.125) (layer F.Cu) (net 22))
-  (segment (start 120.669402 89.17499) (end 122.581902 87.26249) (width 0.125) (layer F.Cu) (net 22))
-  (segment (start 113.344508 89.17499) (end 120.669402 89.17499) (width 0.125) (layer F.Cu) (net 22))
+  (segment (start 112.077498 94.825) (end 113 94.825) (width 0.125) (layer F.Cu) (net 22))
+  (segment (start 115.344508 89.17499) (end 111.862499 92.656999) (width 0.125) (layer F.Cu) (net 22))
+  (segment (start 111.862499 94.610001) (end 112.077498 94.825) (width 0.125) (layer F.Cu) (net 22))
+  (segment (start 120.669402 89.17499) (end 115.344508 89.17499) (width 0.125) (layer F.Cu) (net 22))
+  (segment (start 122.581902 87.26249) (end 120.669402 89.17499) (width 0.125) (layer F.Cu) (net 22))
+  (segment (start 123.83749 87.26249) (end 122.581902 87.26249) (width 0.125) (layer F.Cu) (net 22))
+  (segment (start 111.862499 92.656999) (end 111.862499 94.610001) (width 0.125) (layer F.Cu) (net 22))
+  (segment (start 124.575 88) (end 123.83749 87.26249) (width 0.125) (layer F.Cu) (net 22))
   (segment (start 184.575 91) (end 185.5 91) (width 0.125) (layer F.Cu) (net 23))
   (segment (start 180.575 91) (end 181.5 91) (width 0.125) (layer F.Cu) (net 23))

Commit message: refortmate the ground plane and ajust logos
Parts:
- moved G*** 1.89 mm to (115.9, 88.1)
Routing:
- net +3V3: track 26.4 -> 24.8 mm
- net /GRID5: track 51.1 -> 52.4 mm
- net /SEG8: track 93.2 -> 93.8 mm, vias 16 -> 17
- net GND: vias 0 -> 8

Commit message: Re-route the PCB to work with foorprint to work with #32
Parts:
- removed the G*** at (115.9, 88.1)
- U1: footprint Package_SO:SSOP-28_5.3x10.2mm_P0.65mm -> jjh:TM1640
- moved REF** 4.50 mm to (103.0, 109.0)
- moved REF** 4.50 mm to (103.0, 87.5)
- moved J1 4.34 mm to (102.5, 92.0)
- moved U1 3.54 mm to (114.0, 96.0), turned to 90 degrees
Routing:
- net GND: track 32.0 -> 71.2 mm, vias 8 -> 10
- net +3V3: track 24.8 -> 35.3 mm
- net DATA: track 25.1 -> 33.1 mm
- net /SEG1: track 92.4 -> 99.6 mm, vias 17 -> 19
- net CLK: track 26.7 -> 33.5 mm
- net /SEG5: track 85.7 -> 91.8 mm
- net /SEG4: track 83.8 -> 89.7 mm
- net /SEG2: track 89.3 -> 94.8 mm
- net /SEG6: track 80.8 -> 86.1 mm
- net /SEG3: track 86.3 -> 91.4 mm
- net /GRID5: track 52.4 -> 57.0 mm
- net /GRID6: track 52.8 -> 56.9 mm
- net /GRID7: track 56.5 -> 60.5 mm
- net /GRID8: track 60.2 -> 64.1 mm
- net /SEG7: track 95.9 -> 99.5 mm
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Other:
- board size 86 x 26.5 mm -> 90.5 x 26.5 mm

Commit message: Update hardware to kicad6
Connections:
- J1 pad 1: Net-(J1-Pad1) -> unconnected-(J1-Pad1)
- J1 pad 2: Net-(J1-Pad2) -> unconnected-(J1-Pad2)
- J1 pad 3: Net-(J1-Pad3) -> unconnected-(J1-Pad3)
- J1 pad 4: Net-(J1-Pad4) -> unconnected-(J1-Pad4)
- J1 pad 6: Net-(J1-Pad6) -> unconnected-(J1-Pad6)
- J1 pad 8: Net-(J1-Pad8) -> unconnected-(J1-Pad8)
Other:
- net class Default removed

Commit message: fix some ERC and DRC errors in the schematic
Routing:
- net /SEG2: track 94.8 -> 94.0 mm
- net /SEG1: track 99.6 -> 98.9 mm
