File: PMod_LEDArray/Hardware/PMOD_LEDArray.kicad_pcb (KiCad board)
At the start: 2 copper layers, 90.5 x 26.5 mm, 139 parts, among them J1 Conn_02x06_Odd_Even, U1 GN1640

Commit message: Change logo reference
Parts:
- renumbered G*** to LOGO1
Changed lines of the file:
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@@
     (at 176.8 98.4 90)
     (attr through_hole)
-    (fp_text reference "G***" (at 0 0 90) (layer "B.SilkS") hide
+    (fp_text reference "LOGO1" (at 0 0 90) (layer "B.SilkS") hide
       (effects (font (size 1.524 1.524) (thickness 0.3)) (justify mirror))
     )

Commit message: add designators to the mounting holes
Parts:
- renumbered REF** to H1, REF** to H2, REF** to H3, REF** to H4
Changed lines of the file:
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@@
     (tags "mounting hole 2.2mm no annular m2")
     (attr exclude_from_pos_files exclude_from_bom)
-    (fp_text reference "REF**" (at 0 -3.2) (layer "F.SilkS") hide
+    (fp_text reference "H4" (at 0 -3.2) (layer "F.SilkS") hide
       (effects (font (size 1 1) (thickness 0.15)))
     )
@@
     (tags "mounting hole 2.2mm no annular m2")
     (attr exclude_from_pos_files exclude_from_bom)
-    (fp_text reference "REF**" (at 0 -3.2) (layer "F.SilkS") hide
+    (fp_text reference "H2" (at 0 -3.2) (layer "F.SilkS") hide
       (effects (font (size 1 1) (thickness 0.15)))
     )
@@
     (tags "mounting hole 2.2mm no annular m2")
     (attr exclude_from_pos_files exclude_from_bom)
-    (fp_text reference "REF**" (at 0 -3.2) (layer "F.SilkS") hide
+    (fp_text reference "H1" (at 0 -3.2) (layer "F.SilkS") hide
       (effects (font (size 1 1) (thickness 0.15)))
     )
@@
     (tags "mounting hole 2.2mm no annular m2")
     (attr exclude_from_pos_files exclude_from_bom)
-    (fp_text reference "REF**" (at 0 -3.2) (layer "F.SilkS") hide
-      (effects (font (size 1 1) (thickness 0.15)))
-    )
+    (fp_text reference "H3" (at 0 -3.2) (layer "F.SilkS") hide
+      (effects (font (size 1 1) (thickness 0.15)))
+    )

Commit message: add designators to the copper logo
Parts:
- renumbered G*** to Logo2
Changed lines of the file:
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@@
     (at 188.5 98.5 90)
     (attr through_hole)
-    (fp_text reference "G***" (at 0 0 90) (layer "F.Cu") hide
+    (fp_text reference "Logo2" (at 0 0 90) (layer "F.Cu") hide
       (effects (font (size 1.524 1.524) (thickness 0.3)))
     )
