File: PMod_LEDArray/Hardware/PMOD_LEDArray.kicad_sch (KiCad schematic)
At the start: 133 parts, among them J1 Conn_02x06_Odd_Even, U1 GN1640

Commit message: fix some ERC and DRC errors in the schematic
Changed lines of the file:
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@@
   (junction (at 33.02 43.18) (diameter 0) (color 0 0 0 0)
   )
+  (junction (at 248.92 139.7) (diameter 0) (color 0 0 0 0)
+  )
   (junction (at 223.52 54.61) (diameter 0) (color 0 0 0 0)
   )
@@
   (junction (at 139.7 33.02) (diameter 0) (color 0 0 0 0)
   )
+  (junction (at 248.92 149.86) (diameter 0) (color 0 0 0 0)
+  )
   (junction (at 139.7 21.59) (diameter 0) (color 0 0 0 0)
   )
@@
     (stroke (width 0) (type default) (color 0 0 0 0))
   )
-  (bus_entry (at 157.48 16.51) (size 2.54 2.54)
-    (stroke (width 0) (type default) (color 0 0 0 0))
-  )
   (bus_entry (at 19.05 87.63) (size 2.54 2.54)
     (stroke (width 0) (type default) (color 0 0 0 0))
@@
     (stroke (width 0) (type default) (color 0 0 0 0))
   )
+  (bus_entry (at 157.48 16.51) (size 2.54 2.54)
+    (stroke (width 0) (type default) (color 0 0 0 0))
+  )
   (bus_entry (at 153.67 160.02) (size 2.54 2.54)
     (stroke (width 0) (type default) (color 0 0 0 0))
@@
     (stroke (width 0) (type default) (color 0 0 0 0))
   )
+  (wire (pts (xy 257.81 152.4) (xy 257.81 149.86))
+    (stroke (width 0) (type default) (color 0 0 0 0))
+  )
   (wire (pts (xy 25.4 31.75) (xy 33.02 31.75))
     (stroke (width 0) (type default) (color 0 0 0 0))
@@
     (stroke (width 0) (type default) (color 0 0 0 0))
   )
+  (wire (pts (xy 257.81 135.89) (xy 257.81 139.7))
+    (stroke (width 0) (type default) (color 0 0 0 0))
+  )
   (wire (pts (xy 190.5 86.36) (xy 190.5 88.9))
     (stroke (width 0) (type default) (color 0 0 0 0))
@@
     (stroke (width 0) (type default) (color 0 0 0 0))
   )
+  (wire (pts (xy 257.81 139.7) (xy 248.92 139.7))
+    (stroke (width 0) (type default) (color 0 0 0 0))
+  )
   (wire (pts (xy 177.8 78.74) (xy 190.5 78.74))
     (stroke (width 0) (type default) (color 0 0 0 0))
@@
     (stroke (width 0) (type default) (color 0 0 0 0))
   )
+  (wire (pts (xy 248.92 149.86) (xy 248.92 152.4))
+    (stroke (width 0) (type default) (color 0 0 0 0))
+  )
   (wire (pts (xy 223.52 19.05) (xy 223.52 31.75))
     (stroke (width 0) (type default) (color 0 0 0 0))
@@
     (stroke (width 0) (type default) (color 0 0 0 0))
   )
+  (wire (pts (xy 257.81 149.86) (xy 248.92 149.86))
+    (stroke (width 0) (type default) (color 0 0 0 0))
+  )
   (wire (pts (xy 177.8 100.33) (xy 185.42 100.33))
     (stroke (width 0) (type default) (color 0 0 0 0))
@@
   )
   (bus (pts (xy 132.08 16.51) (xy 144.78 16.51))
-    (stroke (width 0) (type default) (color 0 0 0 0))
+    (stroke (width 0) (type solid) (color 0 0 0 0))
   )
   (bus (pts (xy 156.21 162.56) (xy 156.21 165.1))
@@
     (stroke (width 0) (type default) (color 0 0 0 0))
   )
-  (wire (pts (xy 248.92 147.32) (xy 248.92 152.4))
+  (wire (pts (xy 248.92 147.32) (xy 248.92 149.86))
     (stroke (width 0) (type default) (color 0 0 0 0))
   )
@@
     (pin "9")
   )
+  (symbol (lib_id "power:PWR_FLAG") (at 257.81 135.89 0) (unit 1)
+    (in_bom yes) (on_board yes) (fields_autoplaced)
+    (property "Reference" "#FLG0101" (id 0) (at 257.81 133.985 0)
+      (effects (font (size 1.27 1.27)) hide)
+    )
+    (property "Value" "PWR_FLAG" (id 1) (at 257.81 132.2855 0))
+    (property "Footprint" "" (id 2) (at 257.81 135.89 0)
+      (effects (font (size 1.27 1.27)) hide)
+    )
+    (property "Datasheet" "~" (id 3) (at 257.81 135.89 0)
+      (effects (font (size 1.27 1.27)) hide)
+    )
+    (pin "1")
+  )
+  (symbol (lib_id "power:PWR_FLAG") (at 257.81 152.4 180) (unit 1)
+    (in_bom yes) (on_board yes) (fields_autoplaced)
+    (property "Reference" "#FLG0102" (id 0) (at 257.81 154.305 0)
+      (effects (font (size 1.27 1.27)) hide)
+    )
+    (property "Value" "PWR_FLAG" (id 1) (at 259.461 154.149 0)
+      (effects (font (size 1.27 1.27)) (justify right))
+    )
+    (property "Footprint" "" (id 2) (at 257.81 152.4 0)
+      (effects (font (size 1.27 1.27)) hide)
+    )
+    (property "Datasheet" "~" (id 3) (at 257.81 152.4 0)
+      (effects (font (size 1.27 1.27)) hide)
+    )
+    (pin "1")
+  )
   (sheet_instances
     (path "/" (page "1"))
   )
   (symbol_instances
+    (path "/5d51a283-21ad-4cc9-9423-ad024620aa95"
+      (reference "#FLG0101") (unit 1) (value "PWR_FLAG") (footprint "")
+    )
+    (path "/5f7fd090-8457-48c9-bf75-ed5257b4cbc5"
+      (reference "#FLG0102") (unit 1) (value "PWR_FLAG") (footprint "")
+    )
     (path "/00000000-0000-0000-0000-0000619ca441"
       (reference "#PWR0101") (unit 1) (value "GND") (footprint "")
