File: PMod_CC2500/Hardware/pmod_cc2500.sch (KiCad schematic (older format))
At the start: 1 part

Commit message: add CC2500 with poer supply and SPI connections
Parts:
- added U?: CC2500RGPR, symbol JJH_Library:CC2500RGPR
- J?: symbol Connector_Generic:Conn_02x06_Counter_Clockwise -> Connector_Generic:Conn_02x06_Odd_Even
Connections:
- net GND: now reaches J?.10 (Pin_10)
- net GND: now also J?.9 (Pin_9), U?.16 (GND), U?.19 (GND), U?.PAD (GND)
- net +3V3: now reaches J?.11 (Pin_11)
- net +3V3: now also J?.12 (Pin_12), U?.11 (AVDD), U?.14 (AVDD), U?.15 (AVDD), U?.4 (DVDD), U?.9 (AVDD)
- net GDO2: now reaches J?.3 (Pin_3)
- net GDO2: now also U?.3 (GDO2)
- net GDO0: now reaches J?.4 (Pin_4)
- net GDO0: now also U?.6 (GDO0)
- net SPI_CLK: now reaches J?.5 (Pin_5)
- net SPI_CLK: now also U?.1 (SCLK)
- net SPI_TX: now reaches J?.6 (Pin_6)
- net SPI_TX: now also U?.20 (SI)
- net SPI_RX: now reaches J?.7 (Pin_7)
- net SPI_RX: now also U?.2 (SO(GDO1))
- net SPI_CSN: now reaches J?.8 (Pin_8)
- net SPI_CSN: now also U?.7 (CSn)
- no-connect marks 0 -> 2
Other:
- moved on the sheet: J?
Changed lines of the file:
@@
 $EndDescr
 $Comp
-L Connector_Generic:Conn_02x06_Counter_Clockwise J?
+L Connector_Generic:Conn_02x06_Odd_Even J?
 U 1 1 619037E4
-P 2350 1700
-F 0 "J?" H 2400 2117 50  0000 C CNN
-F 1 "Conn_02x06_Counter_Clockwise" H 2400 2026 50  0000 C CNN
-F 2 "" H 2350 1700 50  0001 C CNN
-F 3 "~" H 2350 1700 50  0001 C CNN
-	1    2350 1700
+P 3250 6200
+F 0 "J?" H 3300 6617 50  0000 C CNN
+F 1 "Conn_02x06_Counter_Clockwise" H 3300 6526 50  0000 C CNN
+F 2 "" H 3250 6200 50  0001 C CNN
+F 3 "~" H 3250 6200 50  0001 C CNN
+	1    3250 6200
 	1    0    0    -1
 $EndComp
+NoConn ~ 3050 6000
+NoConn ~ 3550 6000
+Text GLabel 2800 6100 0    50   Input ~ 0
+GDO2
+Text GLabel 3750 6100 2    50   Input ~ 0
+GDO0
+Text GLabel 3750 6200 2    50   Input ~ 0
+SPI_TX
+Text GLabel 2800 6200 0    50   Input ~ 0
+SPI_CLK
+Text GLabel 2800 6300 0    50   Input ~ 0
+SPI_RX
+Text GLabel 3750 6300 2    50   Input ~ 0
+SPI_CSN
+$Comp
+L power:GND #PWR?
+U 1 1 622EEB9D
+P 3750 6400
+F 0 "#PWR?" H 3750 6150 50  0001 C CNN
+F 1 "GND" V 3755 6272 50  0000 R CNN
+F 2 "" H 3750 6400 50  0001 C CNN
+F 3 "" H 3750 6400 50  0001 C CNN
+	1    3750 6400
+	0    -1   -1   0
+$EndComp
+$Comp
+L power:GND #PWR?
+U 1 1 622EED68
+P 2800 6400
+F 0 "#PWR?" H 2800 6150 50  0001 C CNN
+F 1 "GND" V 2805 6272 50  0000 R CNN
+F 2 "" H 2800 6400 50  0001 C CNN
+F 3 "" H 2800 6400 50  0001 C CNN
+	1    2800 6400
+	0    1    1    0
+$EndComp
+$Comp
+L power:+3V3 #PWR?
+U 1 1 622EF08B
+P 2800 6500
+F 0 "#PWR?" H 2800 6350 50  0001 C CNN
+F 1 "+3V3" V 2815 6628 50  0000 L CNN
+F 2 "" H 2800 6500 50  0001 C CNN
+F 3 "" H 2800 6500 50  0001 C CNN
+	1    2800 6500
+	0    -1   -1   0
+$EndComp
+$Comp
+L power:+3V3 #PWR?
+U 1 1 622EF2B3
+P 3750 6500
+F 0 "#PWR?" H 3750 6350 50  0001 C CNN
+F 1 "+3V3" V 3765 6628 50  0000 L CNN
+F 2 "" H 3750 6500 50  0001 C CNN
+F 3 "" H 3750 6500 50  0001 C CNN
+	1    3750 6500
+	0    1    1    0
+$EndComp
+Wire Wire Line
+	2800 6100 3050 6100
+Wire Wire Line
+	3050 6200 2800 6200
+Wire Wire Line
+	2800 6300 3050 6300
+Wire Wire Line
+	3050 6400 2800 6400
+Wire Wire Line
+	2800 6500 3050 6500
+Wire Wire Line
+	3550 6500 3750 6500
+Wire Wire Line
+	3550 6400 3750 6400
+Wire Wire Line
+	3550 6300 3750 6300
+Wire Wire Line
+	3550 6200 3750 6200
+Wire Wire Line
+	3750 6100 3550 6100
+$Comp
+L JJH_Library:CC2500RGPR U?
+U 1 1 6230133C
+P 6200 2300
+F 0 "U?" H 6175 3365 50  0000 C CNN
+F 1 "CC2500RGPR" H 6175 3274 50  0000 C CNN
+F 2 "" H 6200 2300 50  0001 C CNN
+F 3 "" H 6200 2300 50  0001 C CNN
+	1    6200 2300
+	1    0    0    -1
+$EndComp
+$Comp
+L power:GND #PWR?
+U 1 1 62302A3B
+P 7100 2650
+F 0 "#PWR?" H 7100 2400 50  0001 C CNN
+F 1 "GND" V 7105 2522 50  0000 R CNN
+F 2 "" H 7100 2650 50  0001 C CNN
+F 3 "" H 7100 2650 50  0001 C CNN
+	1    7100 2650
+	0    -1   -1   0
+$EndComp
+$Comp
+L power:+3V3 #PWR?
+U 1 1 62302D98
+P 7100 2100
+F 0 "#PWR?" H 7100 1950 50  0001 C CNN
+F 1 "+3V3" V 7115 2228 50  0000 L CNN
+F 2 "" H 7100 2100 50  0001 C CNN
+F 3 "" H 7100 2100 50  0001 C CNN
+	1    7100 2100
+	0    1    1    0
+$EndComp
+Wire Wire Line
+	6850 1900 7000 1900
+Wire Wire Line
+	7000 1900 7000 2000
+Wire Wire Line
+	7000 2300 6850 2300
+Wire Wire Line
+	7100 2100 7000 2100
+Connection ~ 7000 2100
+Wire Wire Line
+	7000 2100 7000 2200
+Wire Wire Line
+	6850 2550 7000 2550
+Wire Wire Line
+	7000 2550 7000 2650
+Wire Wire Line
+	7000 2750 6850 2750
+Wire Wire Line
+	6850 2650 7000 2650
+Connection ~ 7000 2650
+Wire Wire Line
+	7000 2650 7000 2750
+Wire Wire Line
+	7000 2650 7100 2650
+Wire Wire Line
+	7000 2100 6850 2100
+Wire Wire Line
+	6850 2200 7000 2200
+Connection ~ 7000 2200
+Wire Wire Line
+	7000 2200 7000 2300
+Wire Wire Line
+	6850 2000 7000 2000
+Connection ~ 7000 2000
+Wire Wire Line
+	7000 2000 7000 2100
+Text GLabel 5300 1550 0    50   Input ~ 0
+SPI_CLK
+Text GLabel 5300 1650 0    50   Input ~ 0
+SPI_CSN
+Text GLabel 5300 1750 0    50   Input ~ 0
+SPI_TX
+Text GLabel 5300 1850 0    50   Input ~ 0
+SPI_RX
+Text GLabel 5300 2100 0    50   Input ~ 0
+GDO2
+Text GLabel 5300 2200 0    50   Input ~ 0
+GDO0
+Wire Wire Line
+	5300 2200 5500 2200
+Wire Wire Line
+	5500 2100 5300 2100
+Wire Wire Line
+	5300 1850 5500 1850
+Wire Wire Line
+	5500 1750 5300 1750
+Wire Wire Line
+	5300 1650 5500 1650
+Wire Wire Line
+	5500 1550 5300 1550
 $EndSCHEMATC

Commit message: Add crystal and decoupling cap
Parts:
- added C?: 100nF, Capacitor_SMD:C_0603_1608Metric, symbol Device:C
- added C? (x2): C, symbol Device:C
- added R?: 56K, Resistor_SMD:R_0603_1608Metric, symbol Device:R
- added XTAL1: 26MHz, symbol Device:Crystal_GND24_Small
Connections:
- net +3V3: now also U?.18 (DGUARD)
- net GND: now also C?.2, C?.2, C?.2, R?.1, XTAL1.2, XTAL1.4
- net at U?.10 (XOSC_Q2): now also C?.1, XTAL1.3
- net at U?.17 (RBIAS): now also R?.2
- net at U?.5 (DCOUPL): now also C?.1
- net at U?.8 (XOSC_Q1): now also C?.1, XTAL1.1
Changed lines of the file:
@@
 Wire Wire Line
 	5500 1550 5300 1550
+$Comp
+L Device:R R?
+U 1 1 6230D792
+P 7100 3050
+F 0 "R?" V 6893 3050 50  0000 C CNN
+F 1 "56K" V 6984 3050 50  0000 C CNN
+F 2 "Resistor_SMD:R_0603_1608Metric" V 7030 3050 50  0001 C CNN
+F 3 "~" H 7100 3050 50  0001 C CNN
+	1    7100 3050
+	0    1    1    0
+$EndComp
+$Comp
+L Device:C C?
+U 1 1 6230DEB2
+P 4800 3200
+F 0 "C?" H 4915 3246 50  0000 L CNN
+F 1 "100nF" H 4915 3155 50  0000 L CNN
+F 2 "Capacitor_SMD:C_0603_1608Metric" H 4838 3050 50  0001 C CNN
+F 3 "~" H 4800 3200 50  0001 C CNN
+	1    4800 3200
+	1    0    0    -1
+$EndComp
+$Comp
+L power:GND #PWR?
+U 1 1 6230EB9D
+P 7450 3050
+F 0 "#PWR?" H 7450 2800 50  0001 C CNN
+F 1 "GND" V 7455 2922 50  0000 R CNN
+F 2 "" H 7450 3050 50  0001 C CNN
+F 3 "" H 7450 3050 50  0001 C CNN
+	1    7450 3050
+	0    -1   -1   0
+$EndComp
+$Comp
+L power:+3V3 #PWR?
+U 1 1 6230EE53
+P 5300 3350
+F 0 "#PWR?" H 5300 3200 50  0001 C CNN
+F 1 "+3V3" H 5315 3523 50  0000 C CNN
+F 2 "" H 5300 3350 50  0001 C CNN
+F 3 "" H 5300 3350 50  0001 C CNN
+	1    5300 3350
+	-1   0    0    1
+$EndComp
+$Comp
+L power:GND #PWR?
+U 1 1 6230F4E2
+P 4800 3350
+F 0 "#PWR?" H 4800 3100 50  0001 C CNN
+F 1 "GND" H 4805 3177 50  0000 C CNN
+F 2 "" H 4800 3350 50  0001 C CNN
+F 3 "" H 4800 3350 50  0001 C CNN
+	1    4800 3350
+	1    0    0    -1
+$EndComp
+Wire Wire Line
+	4800 3050 4800 2950
+Wire Wire Line
+	4800 2950 5500 2950
+Wire Wire Line
+	5500 3050 5300 3050
+Wire Wire Line
+	5300 3050 5300 3350
+Wire Wire Line
+	6850 3050 6950 3050
+Wire Wire Line
+	7250 3050 7450 3050
+$Comp
+L Device:Crystal_GND24_Small XTAL1
+U 1 1 623124BB
+P 4300 2550
+F 0 "XTAL1" V 4200 2600 50  0000 L CNN
+F 1 "26MHz" V 4400 2600 50  0000 L CNN
+F 2 "" H 4300 2550 50  0001 C CNN
+F 3 "~" H 4300 2550 50  0001 C CNN
+	1    4300 2550
+	0    1    1    0
+$EndComp
+$Comp
+L power:GND #PWR?
+U 1 1 62313880
+P 4600 2550
+F 0 "#PWR?" H 4600 2300 50  0001 C CNN
+F 1 "GND" V 4605 2422 50  0000 R CNN
+F 2 "" H 4600 2550 50  0001 C CNN
+F 3 "" H 4600 2550 50  0001 C CNN
+	1    4600 2550
+	0    -1   -1   0
+$EndComp
+$Comp
+L power:GND #PWR?
+U 1 1 62313C1A
+P 4000 2550
+F 0 "#PWR?" H 4000 2300 50  0001 C CNN
+F 1 "GND" V 4005 2422 50  0000 R CNN
+F 2 "" H 4000 2550 50  0001 C CNN
+F 3 "" H 4000 2550 50  0001 C CNN
+	1    4000 2550
+	0    1    1    0
+$EndComp
+Wire Wire Line
+	4000 2550 4200 2550
+Wire Wire Line
+	4400 2550 4600 2550
+$Comp
+L Device:C C?
+U 1 1 6231550C
+P 3950 2350
+F 0 "C?" V 3698 2350 50  0000 C CNN
+F 1 "C" V 3789 2350 50  0000 C CNN
+F 2 "" H 3988 2200 50  0001 C CNN
+F 3 "~" H 3950 2350 50  0001 C CNN
+	1    3950 2350
+	0    1    1    0
+$EndComp
+$Comp
+L Device:C C?
+U 1 1 62315C35
+P 3950 2750
+F 0 "C?" V 4200 2750 50  0000 C CNN
+F 1 "C" V 4100 2750 50  0000 C CNN
+F 2 "" H 3988 2600 50  0001 C CNN
+F 3 "~" H 3950 2750 50  0001 C CNN
+	1    3950 2750
+	0    1    1    0
+$EndComp
+Wire Wire Line
+	4100 2350 4300 2350
+Wire Wire Line
+	4300 2350 4300 2450
+Wire Wire Line
+	4300 2650 4300 2750
+Wire Wire Line
+	4300 2750 4100 2750
+Wire Wire Line
+	5500 2650 4900 2650
+Wire Wire Line
+	4900 2650 4900 2750
+Wire Wire Line
+	4900 2750 4300 2750
+Connection ~ 4300 2750
+Wire Wire Line
+	4300 2350 4900 2350
+Wire Wire Line
+	4900 2350 4900 2450
+Wire Wire Line
+	4900 2450 5500 2450
+Connection ~ 4300 2350
+$Comp
+L power:GND #PWR?
+U 1 1 6231BE16
+P 3550 2350
+F 0 "#PWR?" H 3550 2100 50  0001 C CNN
+F 1 "GND" V 3555 2222 50  0000 R CNN
+F 2 "" H 3550 2350 50  0001 C CNN
+F 3 "" H 3550 2350 50  0001 C CNN
+	1    3550 2350
+	0    1    1    0
+$EndComp
+$Comp
+L power:GND #PWR?
+U 1 1 6231C21F
+P 3550 2750
+F 0 "#PWR?" H 3550 2500 50  0001 C CNN
+F 1 "GND" V 3555 2622 50  0000 R CNN
+F 2 "" H 3550 2750 50  0001 C CNN
+F 3 "" H 3550 2750 50  0001 C CNN
+	1    3550 2750
+	0    1    1    0
+$EndComp
+Wire Wire Line
+	3550 2350 3800 2350
+Wire Wire Line
+	3800 2750 3550 2750
 $EndSCHEMATC

Commit message: Add RF Matching and Filtering
Parts:
- added C?: 1.5pF, Capacitor_SMD:C_0603_1608Metric, symbol Device:C
- added C?: 1.8pF, Capacitor_SMD:C_0603_1608Metric, symbol Device:C
- added C? (x2): 1pF, Capacitor_SMD:C_0603_1608Metric, symbol Device:C
- added C? (x2): 100pF, Capacitor_SMD:C_0603_1608Metric, symbol Device:C
- added J?: Conn_Coaxial, symbol Connector:Conn_Coaxial
- added L? (x3): 1.2nH, Inductor_SMD:L_0603_1608Metric, symbol Device:L
- C? (x2): footprint (none) -> Capacitor_SMD:C_0603_1608Metric
Connections:
- net GND: now also C?.1, C?.2, C?.2, J?.2 (Ext), L?.2
- net at U?.12 (RF_P): now also C?.2
- net at U?.13 (RF_N): now also C?.2
- new net: C?.1, J?.1 (In), L?.1
- new net: C?.1, C?.1, L?.1, L?.2
- new net: C?.1, C?.2, L?.1
- new net: C?.1, C?.2, L?.2
Changed lines of the file:
@@
 F 0 "C?" V 3698 2350 50  0000 C CNN
 F 1 "C" V 3789 2350 50  0000 C CNN
-F 2 "" H 3988 2200 50  0001 C CNN
+F 2 "Capacitor_SMD:C_0603_1608Metric" H 3988 2200 50  0001 C CNN
 F 3 "~" H 3950 2350 50  0001 C CNN
 	1    3950 2350
@@
 F 0 "C?" V 4200 2750 50  0000 C CNN
 F 1 "C" V 4100 2750 50  0000 C CNN
-F 2 "" H 3988 2600 50  0001 C CNN
+F 2 "Capacitor_SMD:C_0603_1608Metric" H 3988 2600 50  0001 C CNN
 F 3 "~" H 3950 2750 50  0001 C CNN
 	1    3950 2750
@@
 Wire Wire Line
 	3800 2750 3550 2750
+$Comp
+L Connector:Conn_Coaxial J?
+U 1 1 6231F9D3
+P 9850 1550
+F 0 "J?" H 9950 1525 50  0000 L CNN
+F 1 "Conn_Coaxial" H 9950 1434 50  0000 L CNN
+F 2 "" H 9850 1550 50  0001 C CNN
+F 3 " ~" H 9850 1550 50  0001 C CNN
+	1    9850 1550
+	1    0    0    -1
+$EndComp
+$Comp
+L Device:C C?
+U 1 1 6231FFA4
+P 9400 2000
+F 0 "C?" H 9515 2046 50  0000 L CNN
+F 1 "1.5pF" H 9515 1955 50  0000 L CNN
+F 2 "Capacitor_SMD:C_0603_1608Metric" H 9438 1850 50  0001 C CNN
+F 3 "~" H 9400 2000 50  0001 C CNN
+	1    9400 2000
+	1    0    0    -1
+$EndComp
+$Comp
+L Device:C C?
+U 1 1 623208C3
+P 8750 2000
+F 0 "C?" H 8865 2046 50  0000 L CNN
+F 1 "1.8pF" H 8865 1955 50  0000 L CNN
+F 2 "Capacitor_SMD:C_0603_1608Metric" H 8788 1850 50  0001 C CNN
+F 3 "~" H 8750 2000 50  0001 C CNN
+	1    8750 2000
+	1    0    0    -1
+$EndComp
+$Comp
+L Device:C C?
+U 1 1 62321099
+P 8200 1750
+F 0 "C?" V 8250 1600 50  0000 C CNN
+F 1 "1pF" V 8250 1900 50  0000 C CNN
+F 2 "Capacitor_SMD:C_0603_1608Metric" H 8238 1600 50  0001 C CNN
+F 3 "~" H 8200 1750 50  0001 C CNN
+	1    8200 1750
+	0    1    1    0
+$EndComp
+$Comp
+L Device:C C?
+U 1 1 623216C5
+P 7900 1200
+F 0 "C?" H 8015 1246 50  0000 L CNN
+F 1 "1pF" H 8015 1155 50  0000 L CNN
+F 2 "Capacitor_SMD:C_0603_1608Metric" H 7938 1050 50  0001 C CNN
+F 3 "~" H 7900 1200 50  0001 C CNN
+	1    7900 1200
+	1    0    0    -1
+$EndComp
+$Comp
+L Device:C C?
+U 1 1 62321D1F
+P 7650 1450
+F 0 "C?" V 7398 1450 50  0000 C CNN
+F 1 "100pF" V 7489 1450 50  0000 C CNN
+F 2 "Capacitor_SMD:C_0603_1608Metric" H 7688 1300 50  0001 C CNN
+F 3 "~" H 7650 1450 50  0001 C CNN
+	1    7650 1450
+	0    1    1    0
+$EndComp
+$Comp
+L Device:C C?
+U 1 1 6232247D
+P 7650 1750
+F 0 "C?" V 7800 1600 50  0000 C CNN
+F 1 "100pF" V 7800 1800 50  0000 C CNN
+F 2 "Capacitor_SMD:C_0603_1608Metric" H 7688 1600 50  0001 C CNN
+F 3 "~" H 7650 1750 50  0001 C CNN
+	1    7650 1750
+	0    1    1    0
+$EndComp
+$Comp
+L Device:L L?
+U 1 1 6232A787
+P 9050 1550
+F 0 "L?" V 8869 1550 50  0000 C CNN
+F 1 "1.2nH" V 8960 1550 50  0000 C CNN
+F 2 "Inductor_SMD:L_0603_1608Metric" H 9050 1550 50  0001 C CNN
+F 3 "~" H 9050 1550 50  0001 C CNN
+	1    9050 1550
+	0    1    1    0
+$EndComp
+$Comp
+L Device:L L?
+U 1 1 6232B3FC
+P 8150 1450
+F 0 "L?" V 8100 1400 50  0000 C CNN
+F 1 "1.2nH" V 8100 1600 50  0000 C CNN
+F 2 "Inductor_SMD:L_0603_1608Metric" H 8150 1450 50  0001 C CNN
+F 3 "~" H 8150 1450 50  0001 C CNN
+	1    8150 1450
+	0    1    1    0
+$EndComp
+$Comp
+L Device:L L?
+U 1 1 6232BEC1
+P 7900 2000
+F 0 "L?" H 7953 2046 50  0000 L CNN
+F 1 "1.2nH" H 7953 1955 50  0000 L CNN
+F 2 "Inductor_SMD:L_0603_1608Metric" H 7900 2000 50  0001 C CNN
+F 3 "~" H 7900 2000 50  0001 C CNN
+	1    7900 2000
+	1    0    0    -1
+$EndComp
+Wire Wire Line
+	6850 1650 7000 1650
+Wire Wire Line
+	7000 1750 7500 1750
+Wire Wire Line
+	7500 1450 7000 1450
+Wire Wire Line
+	7000 1450 7000 1550
+Wire Wire Line
+	7000 1550 6850 1550
+Wire Wire Line
+	7800 1450 7900 1450
+Wire Wire Line
+	7800 1750 7900 1750
+Wire Wire Line
+	7900 1850 7900 1750
+Connection ~ 7900 1750
+Wire Wire Line
+	7900 1750 8050 1750
+Wire Wire Line
+	7900 1350 7900 1450
+Connection ~ 7900 1450
+Wire Wire Line
+	7900 1450 8000 1450
+Wire Wire Line
+	8350 1750 8500 1750
+Wire Wire Line
+	8500 1550 8750 1550
+Wire Wire Line
+	8300 1450 8500 1450
+Wire Wire Line
+	8500 1450 8500 1550
+Connection ~ 8500 1550
+Wire Wire Line
+	7000 1650 7000 1750
+Wire Wire Line
+	8500 1550 8500 1750
+Wire Wire Line
+	8750 1850 8750 1550
+Connection ~ 8750 1550
+Wire Wire Line
+	8750 1550 8900 1550
+Wire Wire Line
+	9200 1550 9400 1550
+Wire Wire Line
+	9400 1850 9400 1550
+Connection ~ 9400 1550
+Wire Wire Line
+	9400 1550 9650 1550
+$Comp
+L power:GND #PWR?
+U 1 1 62356266
+P 9850 2150
+F 0 "#PWR?" H 9850 1900 50  0001 C CNN
+F 1 "GND" H 9855 1977 50  0000 C CNN
+F 2 "" H 9850 2150 50  0001 C CNN
+F 3 "" H 9850 2150 50  0001 C CNN
+	1    9850 2150
+	1    0    0    -1
+$EndComp
+$Comp
+L power:GND #PWR?
+U 1 1 623566EE
+P 9400 2150
+F 0 "#PWR?" H 9400 1900 50  0001 C CNN
+F 1 "GND" H 9405 1977 50  0000 C CNN
+F 2 "" H 9400 2150 50  0001 C CNN
+F 3 "" H 9400 2150 50  0001 C CNN
+	1    9400 2150
+	1    0    0    -1
+$EndComp
+$Comp
+L power:GND #PWR?
+U 1 1 62356B92
+P 8750 2150
+F 0 "#PWR?" H 8750 1900 50  0001 C CNN
+F 1 "GND" H 8755 1977 50  0000 C CNN
+F 2 "" H 8750 2150 50  0001 C CNN
+F 3 "" H 8750 2150 50  0001 C CNN
+	1    8750 2150
+	1    0    0    -1
+$EndComp
+$Comp
+L power:GND #PWR?
+U 1 1 62357052
+P 7900 2150
+F 0 "#PWR?" H 7900 1900 50  0001 C CNN
+F 1 "GND" H 7905 1977 50  0000 C CNN
+F 2 "" H 7900 2150 50  0001 C CNN
+F 3 "" H 7900 2150 50  0001 C CNN
+	1    7900 2150
+	1    0    0    -1
+$EndComp
+$Comp
+L power:GND #PWR?
+U 1 1 62359A30
+P 7900 1050
+F 0 "#PWR?" H 7900 800 50  0001 C CNN
+F 1 "GND" H 7905 877 50  0000 C CNN
+F 2 "" H 7900 1050 50  0001 C CNN
+F 3 "" H 7900 1050 50  0001 C CNN
+	1    7900 1050
+	-1   0    0    1
+$EndComp
+Wire Wire Line
+	9850 2150 9850 1750
 $EndSCHEMATC

Commit message: Add the footprints to key components
Parts:
- J?: footprint (none) -> Connector_Coaxial:SMA_Samtec_SMA-J-P-X-ST-EM1_EdgeMount
- U?: footprint (none) -> jjh:QFN50P400X400X100-21N-D
- XTAL1: footprint (none) -> Crystal:Crystal_SMD_Abracon_ABM8G-4Pin_3.2x2.5mm
Other:
- moved on the sheet: C?, J?, L?, R?, U?, XTAL1
