File: PMod_CC2500/Hardware/pmod_cc2500.sch (KiCad schematic (older format))
At the start: 17 parts

Commit message: initial PCB Layout
Parts:
- J1: renamed from J?; footprint (none) -> Connector_PinHeader_2.54mm:PinHeader_2x06_P2.54mm_Vertical
- gave numbers to parts that had none: 15
Changed lines of the file:
@@
 $EndDescr
 $Comp
-L Connector_Generic:Conn_02x06_Odd_Even J?
+L Connector_Generic:Conn_02x06_Odd_Even J1
 U 1 1 619037E4
 P 3400 5850
-F 0 "J?" H 3450 6267 50  0000 C CNN
+F 0 "J1" H 3450 6267 50  0000 C CNN
 F 1 "Conn_02x06_Counter_Clockwise" H 3450 6176 50  0000 C CNN
-F 2 "" H 3400 5850 50  0001 C CNN
+F 2 "Connector_PinHeader_2.54mm:PinHeader_2x06_P2.54mm_Vertical" H 3400 5850 50  0001 C CNN
 F 3 "~" H 3400 5850 50  0001 C CNN
 	1    3400 5850
@@
 SPI_CSN
 $Comp
-L power:GND #PWR?
+L power:GND #PWR0101
 U 1 1 622EEB9D
 P 3900 6050
-F 0 "#PWR?" H 3900 5800 50  0001 C CNN
+F 0 "#PWR0101" H 3900 5800 50  0001 C CNN
 F 1 "GND" V 3905 5922 50  0000 R CNN
 F 2 "" H 3900 6050 50  0001 C CNN
@@
 $EndComp
 $Comp
-L power:GND #PWR?
+L power:GND #PWR0102
 U 1 1 622EED68
 P 2950 6050
-F 0 "#PWR?" H 2950 5800 50  0001 C CNN
+F 0 "#PWR0102" H 2950 5800 50  0001 C CNN
 F 1 "GND" V 2955 5922 50  0000 R CNN
 F 2 "" H 2950 6050 50  0001 C CNN
@@
 $EndComp
 $Comp
-L power:+3V3 #PWR?
+L power:+3V3 #PWR0103
 U 1 1 622EF08B
 P 2950 6150
-F 0 "#PWR?" H 2950 6000 50  0001 C CNN
+F 0 "#PWR0103" H 2950 6000 50  0001 C CNN
 F 1 "+3V3" V 2965 6278 50  0000 L CNN
 F 2 "" H 2950 6150 50  0001 C CNN
@@
 $EndComp
 $Comp
-L power:+3V3 #PWR?
+L power:+3V3 #PWR0104
 U 1 1 622EF2B3
 P 3900 6150
-F 0 "#PWR?" H 3900 6000 50  0001 C CNN
+F 0 "#PWR0104" H 3900 6000 50  0001 C CNN
 F 1 "+3V3" V 3915 6278 50  0000 L CNN
 F 2 "" H 3900 6150 50  0001 C CNN
@@
 	3900 5750 3700 5750
 $Comp
-L JJH_Library:CC2500RGPR U?
+L JJH_Library:CC2500RGPR U1
 U 1 1 6230133C
 P 5550 2800
-F 0 "U?" H 5525 3865 50  0000 C CNN
+F 0 "U1" H 5525 3865 50  0000 C CNN
 F 1 "CC2500RGPR" H 5525 3774 50  0000 C CNN
 F 2 "jjh:QFN50P400X400X100-21N-D" H 5550 2800 50  0001 C CNN
@@
 $EndComp
 $Comp
-L power:GND #PWR?
+L power:GND #PWR0105
 U 1 1 62302A3B
 P 6450 3150
-F 0 "#PWR?" H 6450 2900 50  0001 C CNN
+F 0 "#PWR0105" H 6450 2900 50  0001 C CNN
 F 1 "GND" V 6455 3022 50  0000 R CNN
 F 2 "" H 6450 3150 50  0001 C CNN
@@
 $EndComp
 $Comp
-L power:+3V3 #PWR?
+L power:+3V3 #PWR0106
 U 1 1 62302D98
 P 6450 2600
-F 0 "#PWR?" H 6450 2450 50  0001 C CNN
+F 0 "#PWR0106" H 6450 2450 50  0001 C CNN
 F 1 "+3V3" V 6465 2728 50  0000 L CNN
 F 2 "" H 6450 2600 50  0001 C CNN
@@
 	4850 2050 4650 2050
 $Comp
-L Device:R R?
+L Device:R R1
 U 1 1 6230D792
 P 6450 3550
-F 0 "R?" V 6243 3550 50  0000 C CNN
+F 0 "R1" V 6243 3550 50  0000 C CNN
 F 1 "56K" V 6334 3550 50  0000 C CNN
 F 2 "Resistor_SMD:R_0603_1608Metric" V 6380 3550 50  0001 C CNN
@@
 $EndComp
 $Comp
-L Device:C C?
+L Device:C C3
 U 1 1 6230DEB2
 P 4150 3700
-F 0 "C?" H 4265 3746 50  0000 L CNN
+F 0 "C3" H 4265 3746 50  0000 L CNN
 F 1 "100nF" H 4265 3655 50  0000 L CNN
 F 2 "Capacitor_SMD:C_0603_1608Metric" H 4188 3550 50  0001 C CNN
@@
 $EndComp
 $Comp
-L power:GND #PWR?
+L power:GND #PWR0107
 U 1 1 6230EB9D
 P 6800 3550
-F 0 "#PWR?" H 6800 3300 50  0001 C CNN
+F 0 "#PWR0107" H 6800 3300 50  0001 C CNN
 F 1 "GND" V 6805 3422 50  0000 R CNN
 F 2 "" H 6800 3550 50  0001 C CNN
@@
 $EndComp
 $Comp
-L power:+3V3 #PWR?
+L power:+3V3 #PWR0108
 U 1 1 6230EE53
 P 4650 3850
-F 0 "#PWR?" H 4650 3700 50  0001 C CNN
+F 0 "#PWR0108" H 4650 3700 50  0001 C CNN
 F 1 "+3V3" H 4665 4023 50  0000 C CNN
 F 2 "" H 4650 3850 50  0001 C CNN
@@
 $EndComp
 $Comp
-L power:GND #PWR?
+L power:GND #PWR0109
 U 1 1 6230F4E2
 P 4150 3850
-F 0 "#PWR?" H 4150 3600 50  0001 C CNN
+F 0 "#PWR0109" H 4150 3600 50  0001 C CNN
 F 1 "GND" H 4155 3677 50  0000 C CNN
 F 2 "" H 4150 3850 50  0001 C CNN
@@
 $EndComp
 $Comp
-L power:GND #PWR?
+L power:GND #PWR0110
 U 1 1 62313880
 P 3950 3050
-F 0 "#PWR?" H 3950 2800 50  0001 C CNN
+F 0 "#PWR0110" H 3950 2800 50  0001 C CNN
 F 1 "GND" V 3955 2922 50  0000 R CNN
 F 2 "" H 3950 3050 50  0001 C CNN
@@
 $EndComp
 $Comp
-L power:GND #PWR?
+L power:GND #PWR0111
 U 1 1 62313C1A
 P 3350 3050
-F 0 "#PWR?" H 3350 2800 50  0001 C CNN
+F 0 "#PWR0111" H 3350 2800 50  0001 C CNN
 F 1 "GND" V 3355 2922 50  0000 R CNN
 F 2 "" H 3350 3050 50  0001 C CNN
@@
 	3750 3050 3950 3050
 $Comp
-L Device:C C?
+L Device:C C1
 U 1 1 6231550C
 P 3300 2850
-F 0 "C?" V 3048 2850 50  0000 C CNN
+F 0 "C1" V 3048 2850 50  0000 C CNN
 F 1 "C" V 3139 2850 50  0000 C CNN
 F 2 "Capacitor_SMD:C_0603_1608Metric" H 3338 2700 50  0001 C CNN
@@
 $EndComp
 $Comp
-L Device:C C?
+L Device:C C2
 U 1 1 62315C35
 P 3300 3250
-F 0 "C?" V 3550 3250 50  0000 C CNN
+F 0 "C2" V 3550 3250 50  0000 C CNN
 F 1 "C" V 3450 3250 50  0000 C CNN
 F 2 "Capacitor_SMD:C_0603_1608Metric" H 3338 3100 50  0001 C CNN
@@
 Connection ~ 3650 2850
 $Comp
-L power:GND #PWR?
+L power:GND #PWR0112
 U 1 1 6231BE16
 P 2900 2850
-F 0 "#PWR?" H 2900 2600 50  0001 C CNN
+F 0 "#PWR0112" H 2900 2600 50  0001 C CNN
 F 1 "GND" V 2905 2722 50  0000 R CNN
 F 2 "" H 2900 2850 50  0001 C CNN
@@
 $EndComp
 $Comp
-L power:GND #PWR?
+L power:GND #PWR0113
 U 1 1 6231C21F
 P 2900 3250
-F 0 "#PWR?" H 2900 3000 50  0001 C CNN
+F 0 "#PWR0113" H 2900 3000 50  0001 C CNN
 F 1 "GND" V 2905 3122 50  0000 R CNN
 F 2 "" H 2900 3250 50  0001 C CNN
@@
 	3150 3250 2900 3250
 $Comp
-L Connector:Conn_Coaxial J?
+L Connector:Conn_Coaxial J2
 U 1 1 6231F9D3
 P 9200 2050
-F 0 "J?" H 9300 2025 50  0000 L CNN
+F 0 "J2" H 9300 2025 50  0000 L CNN
 F 1 "Conn_Coaxial" H 9300 1934 50  0000 L CNN
 F 2 "Connector_Coaxial:SMA_Samtec_SMA-J-P-X-ST-EM1_EdgeMount" H 9200 2050 50  0001 C CNN
@@
 $EndComp
 $Comp
-L Device:C C?
+L Device:C C9
 U 1 1 6231FFA4
 P 8750 2500
-F 0 "C?" H 8865 2546 50  0000 L CNN
+F 0 "C9" H 8865 2546 50  0000 L CNN
 F 1 "1.5pF" H 8865 2455 50  0000 L CNN
 F 2 "Capacitor_SMD:C_0603_1608Metric" H 8788 2350 50  0001 C CNN
@@
 $EndComp
 $Comp
-L Device:C C?
+L Device:C C8
 U 1 1 623208C3
 P 8100 2500
-F 0 "C?" H 8215 2546 50  0000 L CNN
+F 0 "C8" H 8215 2546 50  0000 L CNN
 F 1 "1.8pF" H 8215 2455 50  0000 L CNN
 F 2 "Capacitor_SMD:C_0603_1608Metric" H 8138 2350 50  0001 C CNN
@@
 $EndComp
 $Comp
-L Device:C C?
+L Device:C C7
 U 1 1 62321099
 P 7550 2250
-F 0 "C?" V 7600 2100 50  0000 C CNN
+F 0 "C7" V 7600 2100 50  0000 C CNN
 F 1 "1pF" V 7600 2400 50  0000 C CNN
 F 2 "Capacitor_SMD:C_0603_1608Metric" H 7588 2100 50  0001 C CNN
@@
 $EndComp
 $Comp
-L Device:C C?
+L Device:C C6
 U 1 1 623216C5
 P 7250 1700
-F 0 "C?" H 7365 1746 50  0000 L CNN
+F 0 "C6" H 7365 1746 50  0000 L CNN
 F 1 "1pF" H 7365 1655 50  0000 L CNN
 F 2 "Capacitor_SMD:C_0603_1608Metric" H 7288 1550 50  0001 C CNN
@@
 $EndComp
 $Comp
-L Device:C C?
+L Device:C C4
 U 1 1 62321D1F
 P 7000 1950
-F 0 "C?" V 6748 1950 50  0000 C CNN
+F 0 "C4" V 6748 1950 50  0000 C CNN
 F 1 "100pF" V 6839 1950 50  0000 C CNN
 F 2 "Capacitor_SMD:C_0603_1608Metric" H 7038 1800 50  0001 C CNN
@@
 $EndComp
 $Comp
-L Device:C C?
+L Device:C C5
 U 1 1 6232247D
 P 7000 2250
-F 0 "C?" V 7150 2100 50  0000 C CNN
+F 0 "C5" V 7150 2100 50  0000 C CNN
 F 1 "100pF" V 7150 2300 50  0000 C CNN
 F 2 "Capacitor_SMD:C_0603_1608Metric" H 7038 2100 50  0001 C CNN
@@
 $EndComp
 $Comp
-L Device:L L?
+L Device:L L3
 U 1 1 6232A787
 P 8400 2050
-F 0 "L?" V 8219 2050 50  0000 C CNN
+F 0 "L3" V 8219 2050 50  0000 C CNN
 F 1 "1.2nH" V 8310 2050 50  0000 C CNN
 F 2 "Inductor_SMD:L_0603_1608Metric" H 8400 2050 50  0001 C CNN
@@
 $EndComp
 $Comp
-L Device:L L?
+L Device:L L2
 U 1 1 6232B3FC
 P 7500 1950
-F 0 "L?" V 7450 1850 50  0000 C CNN
+F 0 "L2" V 7450 1850 50  0000 C CNN
 F 1 "1.2nH" V 7450 2100 50  0000 C CNN
 F 2 "Inductor_SMD:L_0603_1608Metric" H 7500 1950 50  0001 C CNN
@@
 $EndComp
 $Comp
-L Device:L L?
+L Device:L L1
 U 1 1 6232BEC1
 P 7250 2500
-F 0 "L?" H 7303 2546 50  0000 L CNN
+F 0 "L1" H 7303 2546 50  0000 L CNN
 F 1 "1.2nH" H 7303 2455 50  0000 L CNN
 F 2 "Inductor_SMD:L_0603_1608Metric" H 7250 2500 50  0001 C CNN
@@
 	8750 2050 9000 2050
 $Comp
-L power:GND #PWR?
+L power:GND #PWR0114
 U 1 1 62356266
 P 9200 2650
-F 0 "#PWR?" H 9200 2400 50  0001 C CNN
+F 0 "#PWR0114" H 9200 2400 50  0001 C CNN
 F 1 "GND" H 9205 2477 50  0000 C CNN
 F 2 "" H 9200 2650 50  0001 C CNN
@@
 $EndComp
 $Comp
-L power:GND #PWR?
+L power:GND #PWR0115
 U 1 1 623566EE
 P 8750 2650
-F 0 "#PWR?" H 8750 2400 50  0001 C CNN
+F 0 "#PWR0115" H 8750 2400 50  0001 C CNN
 F 1 "GND" H 8755 2477 50  0000 C CNN
 F 2 "" H 8750 2650 50  0001 C CNN
@@
 $EndComp
 $Comp
-L power:GND #PWR?
+L power:GND #PWR0116
 U 1 1 62356B92
 P 8100 2650
-F 0 "#PWR?" H 8100 2400 50  0001 C CNN
+F 0 "#PWR0116" H 8100 2400 50  0001 C CNN
 F 1 "GND" H 8105 2477 50  0000 C CNN
 F 2 "" H 8100 2650 50  0001 C CNN
@@
 $EndComp
 $Comp
-L power:GND #PWR?
+L power:GND #PWR0117
 U 1 1 62357052
 P 7250 2650
-F 0 "#PWR?" H 7250 2400 50  0001 C CNN
+F 0 "#PWR0117" H 7250 2400 50  0001 C CNN
 F 1 "GND" H 7255 2477 50  0000 C CNN
 F 2 "" H 7250 2650 50  0001 C CNN
@@
 $EndComp
 $Comp
-L power:GND #PWR?
+L power:GND #PWR0118
 U 1 1 62359A30
 P 7250 1550
-F 0 "#PWR?" H 7250 1300 50  0001 C CNN
+F 0 "#PWR0118" H 7250 1300 50  0001 C CNN
 F 1 "GND" H 7255 1377 50  0000 C CNN
 F 2 "" H 7250 1550 50  0001 C CNN
