File: PMod_Hub75/Hardware/PMod_Hub75.kicad_pcb (KiCad board)
At the start: 2 copper layers, 47.5 x 40 mm, 13 parts, among them IC1 SN74LVC8T245DWR, IC2 SN74LVC8T245DWR, J1 Conn_02x06_Counter_Clockwise, J2 Conn_02x06_Counter_Clockwise, J3 Conn_02x08_Counter_Clockwise

Commit message: Place r and c on pcb
Parts:
- moved R2 37.2 mm to (125.7, 111.1)
- moved R4 35.1 mm to (143.9, 112.1)
- moved C2 31.0 mm to (125.7, 109.5), turned to 180 degrees
- moved C4 29.3 mm to (144.0, 110.0), turned to 180 degrees
- moved R1 20.8 mm to (125.7, 88.0)
- moved C3 16.2 mm to (144.3, 86.7), turned to 180 degrees
- moved R3 15.7 mm to (144.2, 88.6)
- moved C1 8.91 mm to (125.7, 86.3), turned to 180 degrees
Changed lines of the file:
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@@
   )
   (module Capacitor_SMD:C_0603_1608Metric (layer F.Cu)
-    (at 141.51 80.8)
+    (at 144 110 180)
     (descr "Capacitor SMD 0603 (1608 Metric), square (rectangular) end terminal, IPC_7351 nominal, (Body size source: IPC-SM-782 page 76, https://www.pcb-3d.com/wordpress/wp-content/uploads/ipc-sm-782a_amendment_1_and_2.pdf), generated with kicad-footprint-generator")
     (tags capacitor)
     (attr smd)
-    (fp_text reference C4 (at 0 -1.43) (layer F.SilkS)
+    (fp_text reference C4 (at 2.625 0.1) (layer F.SilkS)
       (effects (font (size 1 1) (thickness 0.15)))
     )
@@
     (fp_line (start 1.48 -0.73) (end 1.48 0.73) (layer F.CrtYd) (width 0.05))
     (fp_line (start 1.48 0.73) (end -1.48 0.73) (layer F.CrtYd) (width 0.05))
-    (pad 2 smd roundrect (at 0.775 0) (size 0.9 0.95) (layers F.Cu F.Paste F.Mask) (roundrect_rratio 0.25)
+    (pad 2 smd roundrect (at 0.775 0 180) (size 0.9 0.95) (layers F.Cu F.Paste F.Mask) (roundrect_rratio 0.25)
       (net 3 VCC))
-    (pad 1 smd roundrect (at -0.775 0) (size 0.9 0.95) (layers F.Cu F.Paste F.Mask) (roundrect_rratio 0.25)
+    (pad 1 smd roundrect (at -0.775 0 180) (size 0.9 0.95) (layers F.Cu F.Paste F.Mask) (roundrect_rratio 0.25)
       (net 1 GND))
     (model ${KISYS3DMOD}/Capacitor_SMD.3dshapes/C_0603_1608Metric.wrl
@@
   )
   (module Capacitor_SMD:C_0603_1608Metric (layer F.Cu)
-    (at 137.5 80.8)
+    (at 125.675 109.5 180)
     (descr "Capacitor SMD 0603 (1608 Metric), square (rectangular) end terminal, IPC_7351 nominal, (Body size source: IPC-SM-782 page 76, https://www.pcb-3d.com/wordpress/wp-content/uploads/ipc-sm-782a_amendment_1_and_2.pdf), generated with kicad-footprint-generator")
     (tags capacitor)
     (attr smd)
-    (fp_text reference C2 (at 0 -1.43) (layer F.SilkS)
+    (fp_text reference C2 (at 2.775 0) (layer F.SilkS)
       (effects (font (size 1 1) (thickness 0.15)))
     )
@@
     (fp_line (start 1.48 -0.73) (end 1.48 0.73) (layer F.CrtYd) (width 0.05))
     (fp_line (start 1.48 0.73) (end -1.48 0.73) (layer F.CrtYd) (width 0.05))
-    (pad 2 smd roundrect (at 0.775 0) (size 0.9 0.95) (layers F.Cu F.Paste F.Mask) (roundrect_rratio 0.25)
-      (net 1 GND))
-    (pad 1 smd roundrect (at -0.775 0) (size 0.9 0.95) (layers F.Cu F.Paste F.Mask) (roundrect_rratio 0.25)
+    (pad 2 smd roundrect (at 0.775 0 180) (size 0.9 0.95) (layers F.Cu F.Paste F.Mask) (roundrect_rratio 0.25)
+      (net 1 GND))
+    (pad 1 smd roundrect (at -0.775 0 180) (size 0.9 0.95) (layers F.Cu F.Paste F.Mask) (roundrect_rratio 0.25)
       (net 2 +3V3))
     (model ${KISYS3DMOD}/Capacitor_SMD.3dshapes/C_0603_1608Metric.wrl
@@
   )
   (module Resistor_SMD:R_0603_1608Metric (layer F.Cu)
-    (at 128.7 80.41)
+    (at 143.9 112.1)
     (descr "Resistor SMD 0603 (1608 Metric), square (rectangular) end terminal, IPC_7351 nominal, (Body size source: IPC-SM-782 page 72, https://www.pcb-3d.com/wordpress/wp-content/uploads/ipc-sm-782a_amendment_1_and_2.pdf), generated with kicad-footprint-generator")
     (tags resistor)
     (attr smd)
-    (fp_text reference R4 (at 0 -1.43) (layer F.SilkS)
+    (fp_text reference R4 (at -2.6 0) (layer F.SilkS)
       (effects (font (size 1 1) (thickness 0.15)))
     )
@@
   )
   (module Resistor_SMD:R_0603_1608Metric (layer F.Cu)
-    (at 132.71 77.9)
+    (at 144.225 88.6)
     (descr "Resistor SMD 0603 (1608 Metric), square (rectangular) end terminal, IPC_7351 nominal, (Body size source: IPC-SM-782 page 72, https://www.pcb-3d.com/wordpress/wp-content/uploads/ipc-sm-782a_amendment_1_and_2.pdf), generated with kicad-footprint-generator")
     (tags resistor)
     (attr smd)
-    (fp_text reference R3 (at 0 -1.43) (layer F.SilkS)
+    (fp_text reference R3 (at -2.625 0.1) (layer F.SilkS)
       (effects (font (size 1 1) (thickness 0.15)))
     )
@@
   )
   (module Resistor_SMD:R_0603_1608Metric (layer F.Cu)
-    (at 135.9 75.36)
+    (at 125.675 111.1)
     (descr "Resistor SMD 0603 (1608 Metric), square (rectangular) end terminal, IPC_7351 nominal, (Body size source: IPC-SM-782 page 72, https://www.pcb-3d.com/wordpress/wp-content/uploads/ipc-sm-782a_amendment_1_and_2.pdf), generated with kicad-footprint-generator")
     (tags resistor)
     (attr smd)
-    (fp_text reference R2 (at 0 -1.43) (layer F.SilkS)
+    (fp_text reference R2 (at -2.475 0) (layer F.SilkS)
       (effects (font (size 1 1) (thickness 0.15)))
     )
@@
   )
   (module Resistor_SMD:R_0603_1608Metric (layer F.Cu)
-    (at 139.91 72.85)
+    (at 125.675 88)
     (descr "Resistor SMD 0603 (1608 Metric), square (rectangular) end terminal, IPC_7351 nominal, (Body size source: IPC-SM-782 page 72, https://www.pcb-3d.com/wordpress/wp-content/uploads/ipc-sm-782a_amendment_1_and_2.pdf), generated with kicad-footprint-generator")
     (tags resistor)
     (attr smd)
-    (fp_text reference R1 (at 0 -1.43) (layer F.SilkS)
+    (fp_text reference R1 (at -2.5 0) (layer F.SilkS)
       (effects (font (size 1 1) (thickness 0.15)))
     )
@@
     (descr "Through hole straight pin header, 2x06, 2.54mm pitch, double rows")
     (tags "Through hole pin header THT 2x06 2.54mm double row")
-    (fp_text reference J2 (at 5.2 13.7) (layer F.SilkS)
+    (fp_text reference J2 (at 4.9 13.5) (layer F.SilkS)
       (effects (font (size 1 1) (thickness 0.15)))
     )
@@
     (descr "Through hole straight pin header, 2x06, 2.54mm pitch, double rows")
     (tags "Through hole pin header THT 2x06 2.54mm double row")
-    (fp_text reference J1 (at 5.3 -1.12) (layer F.SilkS)
+    (fp_text reference J1 (at 5.1 13.58) (layer F.SilkS)
       (effects (font (size 1 1) (thickness 0.15)))
     )
@@
   )
   (module Capacitor_SMD:C_0603_1608Metric (layer F.Cu)
-    (at 135.9 72.85)
+    (at 144.275 86.7 180)
     (descr "Capacitor SMD 0603 (1608 Metric), square (rectangular) end terminal, IPC_7351 nominal, (Body size source: IPC-SM-782 page 76, https://www.pcb-3d.com/wordpress/wp-content/uploads/ipc-sm-782a_amendment_1_and_2.pdf), generated with kicad-footprint-generator")
     (tags capacitor)
     (attr smd)
-    (fp_text reference C3 (at 0 -1.43) (layer F.SilkS)
+    (fp_text reference C3 (at 2.575 0) (layer F.SilkS)
       (effects (font (size 1 1) (thickness 0.15)))
     )
@@
     (fp_line (start 1.48 -0.73) (end 1.48 0.73) (layer F.CrtYd) (width 0.05))
     (fp_line (start 1.48 0.73) (end -1.48 0.73) (layer F.CrtYd) (width 0.05))
-    (pad 2 smd roundrect (at 0.775 0) (size 0.9 0.95) (layers F.Cu F.Paste F.Mask) (roundrect_rratio 0.25)
+    (pad 2 smd roundrect (at 0.775 0 180) (size 0.9 0.95) (layers F.Cu F.Paste F.Mask) (roundrect_rratio 0.25)
       (net 3 VCC))
-    (pad 1 smd roundrect (at -0.775 0) (size 0.9 0.95) (layers F.Cu F.Paste F.Mask) (roundrect_rratio 0.25)
+    (pad 1 smd roundrect (at -0.775 0 180) (size 0.9 0.95) (layers F.Cu F.Paste F.Mask) (roundrect_rratio 0.25)
       (net 1 GND))
     (model ${KISYS3DMOD}/Capacitor_SMD.3dshapes/C_0603_1608Metric.wrl
@@
   )
   (module Capacitor_SMD:C_0603_1608Metric (layer F.Cu)
-    (at 128.7 77.9)
+    (at 125.725 86.3 180)
     (descr "Capacitor SMD 0603 (1608 Metric), square (rectangular) end terminal, IPC_7351 nominal, (Body size source: IPC-SM-782 page 76, https://www.pcb-3d.com/wordpress/wp-content/uploads/ipc-sm-782a_amendment_1_and_2.pdf), generated with kicad-footprint-generator")
     (tags capacitor)
     (attr smd)
-    (fp_text reference C1 (at 0 -1.43) (layer F.SilkS)
+    (fp_text reference C1 (at 2.6 0) (layer F.SilkS)
       (effects (font (size 1 1) (thickness 0.15)))
     )
@@
     (fp_line (start 1.48 -0.73) (end 1.48 0.73) (layer F.CrtYd) (width 0.05))
     (fp_line (start 1.48 0.73) (end -1.48 0.73) (layer F.CrtYd) (width 0.05))
-    (pad 2 smd roundrect (at 0.775 0) (size 0.9 0.95) (layers F.Cu F.Paste F.Mask) (roundrect_rratio 0.25)
-      (net 1 GND))
-    (pad 1 smd roundrect (at -0.775 0) (size 0.9 0.95) (layers F.Cu F.Paste F.Mask) (roundrect_rratio 0.25)
+    (pad 2 smd roundrect (at 0.775 0 180) (size 0.9 0.95) (layers F.Cu F.Paste F.Mask) (roundrect_rratio 0.25)
+      (net 1 GND))
+    (pad 1 smd roundrect (at -0.775 0 180) (size 0.9 0.95) (layers F.Cu F.Paste F.Mask) (roundrect_rratio 0.25)
       (net 2 +3V3))
     (model ${KISYS3DMOD}/Capacitor_SMD.3dshapes/C_0603_1608Metric.wrl

Commit message: Add initial routing to PCB
Parts:
- moved C3 1.70 mm to (142.6, 86.7)
- moved R3 1.66 mm to (142.6, 88.7)
- moved R4 1.60 mm to (142.5, 111.3)
- moved C4 1.55 mm to (142.5, 109.7)
Routing:
- net +3V3: track 0.00 -> 71.9 mm, vias 0 -> 1
- net GND: track 0.00 -> 37.0 mm, vias 0 -> 13
- net Out_Latch: track 0.00 -> 26.5 mm
- net Out_B1: track 0.00 -> 22.0 mm
- net Out_A: track 0.00 -> 22.0 mm
- net Out_R1: track 0.00 -> 21.6 mm
- net Out_B0: track 0.00 -> 21.5 mm, vias 0 -> 1
- net Out_E: track 0.00 -> 20.1 mm, vias 0 -> 1
- net Out_R0: track 0.00 -> 19.9 mm
- net Out_B: track 0.00 -> 19.0 mm
- net Out_C: track 0.00 -> 17.9 mm
- net Out_CLK: track 0.00 -> 17.5 mm
- net Out_OE: track 0.00 -> 16.9 mm
- net Out_G1: track 0.00 -> 16.9 mm
- net Out_G0: track 0.00 -> 16.3 mm
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- added copper zone on B.Cu, net GND
Other:
- board size 47.5 x 40 mm -> 45 x 40 mm
- rule trace_min: 0.2 -> 0.1

Commit message: Update the routing of 3v3 and GND
Connections:
- C3 pad 2: VCC -> +3V3
- C4 pad 2: VCC -> +3V3
- IC1 pad 23: VCC -> +3V3
- IC1 pad 24: VCC -> +3V3
- IC2 pad 23: VCC -> +3V3
- IC2 pad 24: VCC -> +3V3
- J3 pad 16: Out_GND -> GND
- J3 pad 4: Out_GND -> GND
Routing:
- net +3V3: track 71.9 -> 133.6 mm, vias 1 -> 3
- net VCC: track 12.8 -> 0.00 mm

Commit message: upgrade to kicad v6
Other:
- net class Default removed

Commit message: Correct DRC error on pcb
Parts:
- added kibuzzard-61DA1109: G***, kibuzzard-61DA1109, F.Cu at (158.1, 108.3)
- added kibuzzard-61DA119E: G***, kibuzzard-61DA119E, F.Cu at (158.1, 95.5)
- added kibuzzard-61DA11BD: G***, kibuzzard-61DA11BD, F.Cu at (157.7, 100.7)
Routing:
- net +3V3: track 133.6 -> 133.1 mm

Commit message: Move connector on the PCB into center of the board
Parts:
- moved J3 1.71 mm to (153.4, 113.4)
- moved kibuzzard-61DA1109 1.71 mm to (156.4, 108.3)
- moved kibuzzard-61DA119E 1.71 mm to (156.4, 95.5)
- moved kibuzzard-61DA11BD 1.71 mm to (156.0, 100.7)
Routing:
- net Out_D: track 14.9 -> 13.2 mm
- net Out_OE: track 16.9 -> 15.2 mm
- net Out_R1: track 21.6 -> 19.9 mm
- net Out_A: track 22.0 -> 20.3 mm
- net Out_G1: track 16.9 -> 15.2 mm
- net Out_R0: track 19.9 -> 18.2 mm
- net Out_C: track 17.9 -> 16.2 mm
- net Out_B0: track 21.5 -> 19.8 mm
- net Out_B1: track 22.0 -> 20.3 mm
- net Out_Latch: track 26.5 -> 24.9 mm
- net Out_CLK: track 17.5 -> 15.9 mm
- net Out_E: track 20.1 -> 18.7 mm
- net Out_G0: track 16.3 -> 15.1 mm
- net Out_B: track 19.0 -> 17.8 mm
