File: PMod_Hub75/Hardware/PMod_Hub75.kicad_sch (KiCad schematic)
At the start: 13 parts, among them IC1 SN74LVC8T245DWR, IC2 SN74LVC8T245DWR, J1 Conn_02x06_Counter_Clockwise, J2 Conn_02x06_Counter_Clockwise, J3 Conn_02x08_Counter_Clockwise

Commit message: Add power flags to resolve erc checks
Changed lines of the file:
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@@
     (comment 4 "Licensed Under CERN Open Hardware Licence Version 2 - Permissive")
   )
+  (junction (at 41.91 48.26) (diameter 0) (color 0 0 0 0)
+  )
   (junction (at 180.34 104.14) (diameter 0) (color 0 0 0 0)
   )
@@
   )
   (junction (at 119.38 52.07) (diameter 0) (color 0 0 0 0)
+  )
+  (junction (at 40.64 132.08) (diameter 0) (color 0 0 0 0)
   )
   (no_connect (at 63.5 60.96))
@@
     (stroke (width 0) (type default) (color 0 0 0 0))
   )
+  (wire (pts (xy 40.64 132.08) (xy 40.64 134.62))
+    (stroke (width 0) (type default) (color 0 0 0 0))
+  )
   (wire (pts (xy 182.88 69.85) (xy 175.26 69.85))
     (stroke (width 0) (type default) (color 0 0 0 0))
@@
     (stroke (width 0) (type default) (color 0 0 0 0))
   )
-  (wire (pts (xy 40.64 124.46) (xy 40.64 134.62))
+  (wire (pts (xy 40.64 124.46) (xy 40.64 132.08))
     (stroke (width 0) (type default) (color 0 0 0 0))
   )
@@
   (symbol (lib_id "power:GND") (at 261.62 104.14 90) (unit 1)
     (in_bom yes) (on_board yes)
-    (property "Reference" "#PWR?" (id 0) (at 267.97 104.14 0)
+    (property "Reference" "#PWR0119" (id 0) (at 267.97 104.14 0)
       (effects (font (size 1.27 1.27)) hide)
     )
@@
   (symbol (lib_id "power:GND") (at 261.62 88.9 90) (unit 1)
     (in_bom yes) (on_board yes)
-    (property "Reference" "#PWR?" (id 0) (at 267.97 88.9 0)
+    (property "Reference" "#PWR0118" (id 0) (at 267.97 88.9 0)
       (effects (font (size 1.27 1.27)) hide)
     )
@@
     (pin "1")
   )
+  (symbol (lib_id "power:PWR_FLAG") (at 40.64 132.08 90) (unit 1)
+    (in_bom yes) (on_board yes) (fields_autoplaced)
+    (property "Reference" "#FLG?" (id 0) (at 38.735 132.08 0)
+      (effects (font (size 1.27 1.27)) hide)
+    )
+    (property "Value" "PWR_FLAG" (id 1) (at 39.37 129.9995 90))
+    (property "Footprint" "" (id 2) (at 40.64 132.08 0)
+      (effects (font (size 1.27 1.27)) hide)
+    )
+    (property "Datasheet" "~" (id 3) (at 40.64 132.08 0)
+      (effects (font (size 1.27 1.27)) hide)
+    )
+    (pin "1")
+  )
+  (symbol (lib_id "power:PWR_FLAG") (at 41.91 48.26 0) (unit 1)
+    (in_bom yes) (on_board yes) (fields_autoplaced)
+    (property "Reference" "#FLG0101" (id 0) (at 41.91 46.355 0)
+      (effects (font (size 1.27 1.27)) hide)
+    )
+    (property "Value" "PWR_FLAG" (id 1) (at 41.91 44.6555 0))
+    (property "Footprint" "" (id 2) (at 41.91 48.26 0)
+      (effects (font (size 1.27 1.27)) hide)
+    )
+    (property "Datasheet" "~" (id 3) (at 41.91 48.26 0)
+      (effects (font (size 1.27 1.27)) hide)
+    )
+    (pin "1")
+  )
   (sheet_instances
     (path "/" (page "1"))
   )
   (symbol_instances
+    (path "/af3a5ad9-3c72-4849-ad9e-dec0a7570455"
+      (reference "#FLG0101") (unit 1) (value "PWR_FLAG") (footprint "")
+    )
+    (path "/9545bfbf-48dd-4146-8d60-6fa543402f0a"
+      (reference "#FLG?") (unit 1) (value "PWR_FLAG") (footprint "")
+    )
     (path "/00000000-0000-0000-0000-000061c461d7"
       (reference "#PWR0101") (unit 1) (value "GND") (footprint "")
@@
       (reference "#PWR0117") (unit 1) (value "GND") (footprint "")
     )
+    (path "/00000000-0000-0000-0000-000061d511b8"
+      (reference "#PWR0118") (unit 1) (value "GND") (footprint "")
+    )
+    (path "/00000000-0000-0000-0000-000061d511b2"
+      (reference "#PWR0119") (unit 1) (value "GND") (footprint "")
+    )
     (path "/00000000-0000-0000-0000-000061d2486a"
       (reference "#PWR0120") (unit 1) (value "VCC") (footprint "")
@@
       (reference "#PWR0121") (unit 1) (value "+3V3") (footprint "")
     )
-    (path "/00000000-0000-0000-0000-000061d511b2"
-      (reference "#PWR?") (unit 1) (value "GND") (footprint "")
-    )
-    (path "/00000000-0000-0000-0000-000061d511b8"
-      (reference "#PWR?") (unit 1) (value "GND") (footprint "")
-    )
     (path "/00000000-0000-0000-0000-000061e30d85"

Commit message: Tidy up the schematic and add titles
Other:
- note added: "Duel PMod Connector"
- note added: "Level Converter Chips"
- note added: "Output to Hub75 Display"
- moved on the sheet: C1, C2, C3, C4, IC1, IC2, J1, J2, J3, R1, R2, R3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

Commit message: Swap A and B pins so they are in order for the RP2040 code
Connections:
- net In_A: now also J2.1 (Pin_1); no longer J2.2 (Pin_2)
- net In_B: now also J2.2 (Pin_2); no longer J2.1 (Pin_1)
Changed lines of the file:
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@@
     )
   )
-  (global_label "In_B" (shape input) (at 35.56 107.95 180) (fields_autoplaced)
-    (effects (font (size 1.27 1.27)) (justify right))
-    (property "Intersheet References" "${INTERSHEET_REFS}" (id 0) (at -2.54 -6.35 0)
+  (global_label "In_B" (shape input) (at 74.93 107.95 0) (fields_autoplaced)
+    (effects (font (size 1.27 1.27)) (justify left))
+    (property "Intersheet References" "${INTERSHEET_REFS}" (id 0) (at 113.03 222.25 0)
       (effects (font (size 1.27 1.27)) hide)
     )
@@
     )
   )
-  (global_label "In_A" (shape input) (at 74.93 107.95 0) (fields_autoplaced)
-    (effects (font (size 1.27 1.27)) (justify left))
-    (property "Intersheet References" "${INTERSHEET_REFS}" (id 0) (at -2.54 -6.35 0)
+  (global_label "In_A" (shape input) (at 35.56 107.95 180) (fields_autoplaced)
+    (effects (font (size 1.27 1.27)) (justify right))
+    (property "Intersheet References" "${INTERSHEET_REFS}" (id 0) (at 113.03 222.25 0)
       (effects (font (size 1.27 1.27)) hide)
     )
@@
   (symbol (lib_id "power:PWR_FLAG") (at 38.1 125.73 90) (unit 1)
     (in_bom yes) (on_board yes) (fields_autoplaced)
-    (property "Reference" "#FLG?" (id 0) (at 36.195 125.73 0)
+    (property "Reference" "#FLG0102" (id 0) (at 36.195 125.73 0)
       (effects (font (size 1.27 1.27)) hide)
     )
@@
     )
     (path "/9545bfbf-48dd-4146-8d60-6fa543402f0a"
-      (reference "#FLG?") (unit 1) (value "PWR_FLAG") (footprint "")
+      (reference "#FLG0102") (unit 1) (value "PWR_FLAG") (footprint "")
     )
     (path "/00000000-0000-0000-0000-000061c461d7"
