File: PMOD_RGB7Segment/Hardware/segment2.kicad_sch (KiCad schematic)
At the start: 22 parts

Commit message: Add the schematics for each of the 7 segment characters
Parts:
- removed D1, D10, D11, D12, D13, D14, D15, D16, D17, D18, D19, D2, D20, D21, D22, D3, D4, D5, D6, D7, D8, D9: LED_ARGB, jjh:SX-0402-RGB, symbol Device:LED_ARGB
- added D23, D24, D25, D26, D27, D28, D29, D30, D31, D32, D33, D34, D35, D36, D37, D38, D39, D40, D41, D42, D43, D44, D45, D46: LED_ARGB, jjh:SX-0402-RGB, symbol Device:LED_ARGB
Connections:
- net CS1: now also D23.2 (RK), D35.2 (RK)
- net CS10: now also D26.2 (RK), D38.2 (RK)
- net CS11: now also D26.3 (GK), D38.3 (GK)
- net CS12: now also D26.4 (BK), D38.4 (BK)
- net CS13: now also D27.2 (RK), D39.2 (RK)
- net CS14: now also D27.3 (GK), D39.3 (GK)
- net CS15: now also D27.4 (BK), D39.4 (BK)
- net CS16: now also D28.2 (RK), D40.2 (RK)
- net CS17: now also D28.3 (GK), D40.3 (GK)
- net CS18: now also D28.4 (BK), D40.4 (BK)
- net CS19: now also D29.2 (RK), D41.2 (RK)
- net CS2: now also D23.3 (GK), D35.3 (GK)
- net CS20: now also D29.3 (GK), D41.3 (GK)
- net CS21: now also D29.4 (BK), D41.4 (BK)
- net CS22: now also D30.2 (RK), D42.2 (RK)
- net CS23: now also D30.3 (GK), D42.3 (GK)
- net CS24: now also D30.4 (BK), D42.4 (BK)
- net CS25: now also D31.2 (RK), D43.2 (RK)
- net CS26: now also D31.3 (GK), D43.3 (GK)
- net CS27: now also D31.4 (BK), D43.4 (BK)
- net CS28: now also D32.2 (RK), D44.2 (RK)
- net CS29: now also D32.3 (GK), D44.3 (GK)
- net CS3: now also D23.4 (BK), D35.4 (BK)
- net CS30: now also D32.4 (BK), D44.4 (BK)
- net CS31: now also D33.2 (RK), D45.2 (RK)
- net CS32: now also D33.3 (GK), D45.3 (GK)
- net CS33: now also D33.4 (BK), D45.4 (BK)
- net CS34: now also D34.2 (RK), D46.2 (RK)
- net CS35: now also D34.3 (GK), D46.3 (GK)
- net CS36: now also D34.4 (BK), D46.4 (BK)
- net CS4: now also D24.2 (RK), D36.2 (RK)
- net CS5: now also D24.3 (GK), D36.3 (GK)
- net CS6: now also D24.4 (BK), D36.4 (BK)
- net CS7: now also D25.2 (RK), D37.2 (RK)
- net CS8: now also D25.3 (GK), D37.3 (GK)
- net CS9: now also D25.4 (BK), D37.4 (BK)
- new net SW3: D23.1 (A), D24.1 (A), D25.1 (A), D26.1 (A), D27.1 (A), D28.1 (A), D29.1 (A), D30.1 (A), D31.1 (A), D32.1 (A), D33.1 (A), D34.1 (A)
- new net SW4: D35.1 (A), D36.1 (A), D37.1 (A), D38.1 (A), D39.1 (A), D40.1 (A), D41.1 (A), D42.1 (A), D43.1 (A), D44.1 (A), D45.1 (A), D46.1 (A)
