File: PMOD_RGB7Segment/Hardware/segment2.kicad_sch (KiCad schematic)
At the start: 24 parts

Commit message: correct the bus naming
Changed lines of the file:
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@@
     (effects (font (size 0.7 0.7) bold) (justify left bottom))
   )
-  (hierarchical_label "SW_Bus" (shape input) (at 31.75 175.26 180)
+  (hierarchical_label "SW[9..1]" (shape input) (at 31.75 175.26 180)
     (effects (font (size 1.27 1.27)) (justify right))
   )
-  (hierarchical_label "CS_Bus" (shape input) (at 34.29 15.24 180)
+  (hierarchical_label "CS[39..1]" (shape input) (at 34.29 15.24 180)
     (effects (font (size 1.27 1.27)) (justify right))
   )

Commit message: start mapping out locations on PCB
Other:
- company: (none) -> James Horton
- title: (none) -> PMod RGB & Segment Display
Changed lines of the file:
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@@
 (kicad_sch (version 20211123) (generator eeschema)
   (paper "A4")
+  (title_block
+    (title "PMod RGB & Segment Display")
+    (rev "v0.1")
+    (company "James Horton")
+    (comment 1 "interface, all LED's are designed to be indivdually addressable ")
+    (comment 2 "This design is a 4 Digit Seven Segment Display made from RGB LED's, controlled using I2C")
+    (comment 4 "Licensed Under CERN Open Hardware Licence Version 2 - Permissive")
+  )
   (junction (at 271.78 130.81) (diameter 0) (color 0 0 0 0)
   )

Commit message: update the pin layout on segment 2
Connections:
- net CS16 is gone; now on net CS10: D28.2 (RK), D40.2 (RK)
- net CS17 is gone; now on net CS11: D28.3 (GK), D40.3 (GK)
- net CS18 is gone; now on net CS12: D28.4 (BK), D40.4 (BK)
- net CS19 is gone; now on net CS13: D29.2 (RK), D41.2 (RK)
- net CS20 is gone; now on net CS14: D29.3 (GK), D41.3 (GK)
- net CS21 is gone; now on net CS15: D29.4 (BK), D41.4 (BK)
- net CS22 is gone; now on net CS13: D30.2 (RK), D42.2 (RK)
- net CS23 is gone; now on net CS14: D30.3 (GK), D42.3 (GK)
- net CS24 is gone; now on net CS15: D30.4 (BK), D42.4 (BK)
- net CS10: now also D23.2 (RK), D24.2 (RK), D25.2 (RK), D27.2 (RK), D39.2 (RK)
- net CS11: now also D23.3 (GK), D24.3 (GK), D25.3 (GK), D27.3 (GK), D39.3 (GK)
- net CS12: now also D23.4 (BK), D24.4 (BK), D25.4 (BK), D27.4 (BK), D39.4 (BK)
- net CS13: now also D31.2 (RK), D35.2 (RK), D36.2 (RK), D37.2 (RK); no longer D27.2 (RK), D39.2 (RK)
- net CS14: now also D31.3 (GK), D35.3 (GK), D36.3 (GK), D37.3 (GK); no longer D27.3 (GK), D39.3 (GK)
- net CS15: now also D31.4 (BK), D35.4 (BK), D36.4 (BK), D37.4 (BK); no longer D27.4 (BK), D39.4 (BK)
- net CS25: no longer D31.2 (RK)
- net CS26: no longer D31.3 (GK)
- net CS27: no longer D31.4 (BK)
- net SW3: no longer D23.1 (A), D24.1 (A), D26.1 (A), D27.1 (A), D28.1 (A), D29.1 (A), D30.1 (A), D31.1 (A), D32.1 (A), D33.1 (A), D34.1 (A)
- net SW4: now also D26.1 (A), D29.1 (A), D30.1 (A), D31.1 (A), D32.1 (A), D33.1 (A), D34.1 (A)
- removed net CS1: D23.2 (RK), D35.2 (RK)
- removed net CS2: D23.3 (GK), D35.3 (GK)
- removed net CS3: D23.4 (BK), D35.4 (BK)
- removed net CS4: D24.2 (RK), D36.2 (RK)
- removed net CS5: D24.3 (GK), D36.3 (GK)
- removed net CS6: D24.4 (BK), D36.4 (BK)
- removed net CS7: D25.2 (RK), D37.2 (RK)
- removed net CS8: D25.3 (GK), D37.3 (GK)
- removed net CS9: D25.4 (BK), D37.4 (BK)
- new net SW1: D23.1 (A)
- new net SW2: D24.1 (A)
- new net SW5: D27.1 (A)
- new net SW6: D28.1 (A)

Commit message: update the pin for segment 2 to improve pcb layout
Connections:
- net CS31 is gone; now on net CS16: D33.2 (RK), D45.2 (RK)
- net CS32 is gone; now on net CS17: D33.3 (GK), D45.3 (GK)
- net CS33 is gone; now on net CS18: D33.4 (BK), D45.4 (BK)
- net CS34 is gone; now on net CS16: D34.2 (RK), D46.2 (RK)
- net CS35 is gone; now on net CS17: D34.3 (GK), D46.3 (GK)
- net CS36 is gone; now on net CS18: D34.4 (BK), D46.4 (BK)
- net CS28 renamed CS16
- net CS29 renamed CS17
- net CS30 renamed CS18
Changed lines of the file:
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@@
     (effects (font (size 1.27 1.27) bold) (justify left bottom))
   )
-  (label "CS34" (at 242.57 146.05 0)
+  (label "CS16" (at 242.57 146.05 0)
     (effects (font (size 0.7 0.7) bold) (justify left bottom))
   )
@@
     (effects (font (size 0.7 0.7) bold) (justify left bottom))
   )
-  (label "CS29" (at 128.27 109.22 0)
+  (label "CS17" (at 128.27 109.22 0)
     (effects (font (size 0.7 0.7) bold) (justify left bottom))
   )
@@
     (effects (font (size 1.27 1.27) bold) (justify left bottom))
   )
-  (label "CS34" (at 128.27 146.05 0)
+  (label "CS16" (at 128.27 146.05 0)
     (effects (font (size 0.7 0.7) bold) (justify left bottom))
   )
-  (label "CS32" (at 128.27 130.81 0)
+  (label "CS17" (at 128.27 130.81 0)
     (effects (font (size 0.7 0.7) bold) (justify left bottom))
   )
@@
     (effects (font (size 0.7 0.7) bold) (justify left bottom))
   )
-  (label "CS36" (at 128.27 156.21 0)
+  (label "CS18" (at 128.27 156.21 0)
     (effects (font (size 0.7 0.7) bold) (justify left bottom))
   )
-  (label "CS28" (at 242.57 104.14 0)
+  (label "CS16" (at 242.57 104.14 0)
     (effects (font (size 0.7 0.7) bold) (justify left bottom))
   )
-  (label "CS32" (at 242.57 130.81 0)
+  (label "CS17" (at 242.57 130.81 0)
     (effects (font (size 0.7 0.7) bold) (justify left bottom))
   )
-  (label "CS28" (at 128.27 104.14 0)
+  (label "CS16" (at 128.27 104.14 0)
     (effects (font (size 0.7 0.7) bold) (justify left bottom))
   )
-  (label "CS36" (at 242.57 156.21 0)
+  (label "CS18" (at 242.57 156.21 0)
     (effects (font (size 0.7 0.7) bold) (justify left bottom))
   )
@@
     (effects (font (size 1.27 1.27) bold) (justify left bottom))
   )
-  (label "CS33" (at 242.57 135.89 0)
+  (label "CS18" (at 242.57 135.89 0)
     (effects (font (size 0.7 0.7) bold) (justify left bottom))
   )
@@
     (effects (font (size 1.27 1.27) bold) (justify left bottom))
   )
-  (label "CS30" (at 242.57 114.3 0)
+  (label "CS18" (at 242.57 114.3 0)
     (effects (font (size 0.7 0.7) bold) (justify left bottom))
   )
@@
     (effects (font (size 1.27 1.27) bold) (justify left bottom))
   )
-  (label "CS35" (at 242.57 151.13 0)
+  (label "CS17" (at 242.57 151.13 0)
     (effects (font (size 0.7 0.7) bold) (justify left bottom))
   )
-  (label "CS30" (at 128.27 114.3 0)
+  (label "CS18" (at 128.27 114.3 0)
     (effects (font (size 0.7 0.7) bold) (justify left bottom))
   )
-  (label "CS35" (at 128.27 151.13 0)
+  (label "CS17" (at 128.27 151.13 0)
     (effects (font (size 0.7 0.7) bold) (justify left bottom))
   )
@@
     (effects (font (size 1.27 1.27) bold) (justify left bottom))
   )
-  (label "CS31" (at 128.27 125.73 0)
+  (label "CS16" (at 128.27 125.73 0)
     (effects (font (size 0.7 0.7) bold) (justify left bottom))
   )
-  (label "CS31" (at 242.57 125.73 0)
+  (label "CS16" (at 242.57 125.73 0)
     (effects (font (size 0.7 0.7) bold) (justify left bottom))
   )
@@
     (effects (font (size 1.27 1.27) bold) (justify left bottom))
   )
-  (label "CS29" (at 242.57 109.22 0)
+  (label "CS17" (at 242.57 109.22 0)
     (effects (font (size 0.7 0.7) bold) (justify left bottom))
   )
@@
     (effects (font (size 0.7 0.7) bold) (justify left bottom))
   )
-  (label "CS33" (at 128.27 135.89 0)
+  (label "CS18" (at 128.27 135.89 0)
     (effects (font (size 0.7 0.7) bold) (justify left bottom))
   )

Commit message: finish remapping the pins to the LEDs
Connections:
- net SW1: now also D32.1 (A), D35.1 (A), D38.1 (A); no longer D23.1 (A)
- net SW2: now also D33.1 (A), D36.1 (A), D39.1 (A); no longer D24.1 (A)
- net SW3: now also D34.1 (A), D37.1 (A), D40.1 (A); no longer D25.1 (A)
- net SW4: now also D23.1 (A); no longer D26.1 (A), D29.1 (A), D30.1 (A), D31.1 (A), D32.1 (A), D33.1 (A), D34.1 (A), D35.1 (A), D36.1 (A), D37.1 (A), D38.1 (A), D39.1 (A), D40.1 (A), D42.1 (A), D43.1 (A), D45.1 (A), D46.1 (A)
- net SW5: now also D24.1 (A), D42.1 (A), D45.1 (A); no longer D27.1 (A)
- net SW6: now also D25.1 (A), D43.1 (A), D46.1 (A); no longer D28.1 (A)
- new net SW7: D26.1 (A), D29.1 (A)
- new net SW8: D27.1 (A), D30.1 (A)
- new net SW9: D28.1 (A), D31.1 (A)
Changed lines of the file:
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@@
     (effects (font (size 0.7 0.7) bold) (justify left bottom))
   )
-  (label "SW4" (at 152.4 151.13 0)
+  (label "SW3" (at 152.4 151.13 0)
     (effects (font (size 1.27 1.27) bold) (justify left bottom))
   )
@@
     (effects (font (size 0.7 0.7) bold) (justify left bottom))
   )
-  (label "SW5" (at 95.25 130.81 0)
+  (label "SW8" (at 95.25 130.81 0)
     (effects (font (size 1.27 1.27) bold) (justify left bottom))
   )
@@
     (effects (font (size 0.7 0.7) bold) (justify left bottom))
   )
-  (label "SW3" (at 95.25 78.74 0)
+  (label "SW6" (at 95.25 78.74 0)
     (effects (font (size 1.27 1.27) bold) (justify left bottom))
   )
@@
     (effects (font (size 0.7 0.7) bold) (justify left bottom))
   )
-  (label "SW4" (at 209.55 78.74 0)
+  (label "SW3" (at 209.55 78.74 0)
     (effects (font (size 1.27 1.27) bold) (justify left bottom))
   )
@@
     (effects (font (size 0.7 0.7) bold) (justify left bottom))
   )
-  (label "SW4" (at 209.55 58.42 0)
+  (label "SW2" (at 209.55 58.42 0)
     (effects (font (size 1.27 1.27) bold) (justify left bottom))
   )
@@
     (effects (font (size 0.7 0.7) bold) (justify left bottom))
   )
-  (label "SW4" (at 266.7 78.74 0)
+  (label "SW6" (at 266.7 78.74 0)
     (effects (font (size 1.27 1.27) bold) (justify left bottom))
   )
@@
     (effects (font (size 0.7 0.7) bold) (justify left bottom))
   )
-  (label "SW4" (at 95.25 109.22 0)
+  (label "SW7" (at 95.25 109.22 0)
     (effects (font (size 1.27 1.27) bold) (justify left bottom))
   )
@@
     (effects (font (size 0.7 0.7) bold) (justify left bottom))
   )
-  (label "SW4" (at 209.55 151.13 0)
+  (label "SW3" (at 209.55 151.13 0)
     (effects (font (size 1.27 1.27) bold) (justify left bottom))
   )
@@
     (effects (font (size 0.7 0.7) bold) (justify left bottom))
   )
-  (label "SW4" (at 152.4 58.42 0)
+  (label "SW8" (at 152.4 58.42 0)
     (effects (font (size 1.27 1.27) bold) (justify left bottom))
   )
@@
     (effects (font (size 0.7 0.7) bold) (justify left bottom))
   )
-  (label "SW6" (at 95.25 151.13 0)
+  (label "SW9" (at 95.25 151.13 0)
     (effects (font (size 1.27 1.27) bold) (justify left bottom))
   )
@@
     (effects (font (size 0.7 0.7) bold) (justify left bottom))
   )
-  (label "SW4" (at 152.4 130.81 0)
+  (label "SW2" (at 152.4 130.81 0)
     (effects (font (size 1.27 1.27) bold) (justify left bottom))
   )
@@
     (effects (font (size 0.7 0.7) bold) (justify left bottom))
   )
-  (label "SW4" (at 209.55 109.22 0)
-    (effects (font (size 1.27 1.27) bold) (justify left bottom))
-  )
-  (label "SW4" (at 209.55 130.81 0)
+  (label "SW1" (at 209.55 109.22 0)
+    (effects (font (size 1.27 1.27) bold) (justify left bottom))
+  )
+  (label "SW2" (at 209.55 130.81 0)
     (effects (font (size 1.27 1.27) bold) (justify left bottom))
   )
@@
     (effects (font (size 0.7 0.7) bold) (justify left bottom))
   )
-  (label "SW4" (at 152.4 78.74 0)
+  (label "SW9" (at 152.4 78.74 0)
     (effects (font (size 1.27 1.27) bold) (justify left bottom))
   )
@@
     (effects (font (size 0.7 0.7) bold) (justify left bottom))
   )
-  (label "SW4" (at 266.7 58.42 0)
+  (label "SW5" (at 266.7 58.42 0)
     (effects (font (size 1.27 1.27) bold) (justify left bottom))
   )
@@
     (effects (font (size 0.7 0.7) bold) (justify left bottom))
   )
-  (label "SW4" (at 209.55 36.83 0)
+  (label "SW1" (at 209.55 36.83 0)
     (effects (font (size 1.27 1.27) bold) (justify left bottom))
   )
@@
     (effects (font (size 0.7 0.7) bold) (justify left bottom))
   )
-  (label "SW4" (at 266.7 130.81 0)
+  (label "SW5" (at 266.7 130.81 0)
     (effects (font (size 1.27 1.27) bold) (justify left bottom))
   )
@@
     (effects (font (size 0.7 0.7) bold) (justify left bottom))
   )
-  (label "SW2" (at 95.25 58.42 0)
+  (label "SW5" (at 95.25 58.42 0)
     (effects (font (size 1.27 1.27) bold) (justify left bottom))
   )
@@
     (effects (font (size 0.7 0.7) bold) (justify left bottom))
   )
-  (label "SW4" (at 266.7 151.13 0)
+  (label "SW6" (at 266.7 151.13 0)
     (effects (font (size 1.27 1.27) bold) (justify left bottom))
   )
@@
     (effects (font (size 0.7 0.7) bold) (justify left bottom))
   )
-  (label "SW1" (at 95.25 36.83 0)
+  (label "SW4" (at 95.25 36.83 0)
     (effects (font (size 1.27 1.27) bold) (justify left bottom))
   )
@@
     (effects (font (size 0.7 0.7) bold) (justify left bottom))
   )
-  (label "SW4" (at 152.4 109.22 0)
-    (effects (font (size 1.27 1.27) bold) (justify left bottom))
-  )
-  (label "SW4" (at 152.4 36.83 0)
-    (effects (font (size 1.27 1.27) bold) (justify left bottom))
-  )
+  (label "SW1" (at 152.4 109.22 0)
+    (effects (font (size 1.27 1.27) bold) (justify left bottom))
+  )
+  (label "SW7" (at 152.4 36.83 0)
+    (effects (font (size 1.27 1.27) bold) (justify left bottom))
+  )

Commit message: correct pins in schematic and continue LED layout on PCB
Connections:
- net CS25 is gone; now on net CS13: D43.2 (RK)
- net CS26 is gone; now on net CS14: D43.3 (GK)
- net CS27 is gone; now on net CS15: D43.4 (BK)
Changed lines of the file:
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@@
     (effects (font (size 0.7 0.7) bold) (justify left bottom))
   )
-  (label "CS26" (at 242.57 78.74 0)
+  (label "CS14" (at 242.57 78.74 0)
     (effects (font (size 0.7 0.7) bold) (justify left bottom))
   )
@@
     (effects (font (size 1.27 1.27) bold) (justify left bottom))
   )
-  (label "CS27" (at 242.57 83.82 0)
+  (label "CS15" (at 242.57 83.82 0)
     (effects (font (size 0.7 0.7) bold) (justify left bottom))
   )
@@
     (effects (font (size 0.7 0.7) bold) (justify left bottom))
   )
-  (label "CS25" (at 242.57 73.66 0)
-    (effects (font (size 0.7 0.7) bold) (justify left bottom))
-  )
+  (label "CS13" (at 242.57 73.66 0)
+    (effects (font (size 0.7 0.7) bold) (justify left bottom))
+  )
