File: PMOD_RGB7Segment/Hardware/PMod_RGB7Segment.kicad_sch (KiCad schematic)
At the start: 1 part

Commit message: Add the schematics for each of the 7 segment characters
Parts:
- gave numbers to parts that had none: 1
Other:
- added sheet Segment2 (segment2.kicad_sch)
- added sheet Segment3 (segment3.kicad_sch)
- added sheet Segment4 (segment4.kicad_sch)

Commit message: Add pmod connector
Parts:
- added J1: Conn_02x06_Counter_Clockwise, Connector_PinHeader_2.54mm:PinHeader_2x06_P2.54mm_Vertical, symbol Connector_Generic:Conn_02x06_Counter_Clockwise
