File: PMOD_RGB7Segment/Hardware/PMod_RGB7Segment.kicad_sch (KiCad schematic)
At the start: 2 parts, among them IC1 IS31FL3741A-QFLS4-TR, J1 Conn_02x06_Counter_Clockwise

Commit message: include changes in moving controller to seperate sheet
Parts:
- removed IC1: IS31FL3741A-QFLS4-TR, QFN40P700X700X80-61N-D, symbol jjh:IS31FL3741A-QFLS4-TR
Connections:
- net GND: now reaches J1.5 (Pin_5)
- net GND: now also J1.8 (Pin_8)
- net +3V3: now reaches J1.6 (Pin_6)
- net +3V3: now also J1.7 (Pin_7)
Other:
- added sheet controller (controller.kicad_sch)
- moved on the sheet: J1

Commit message: correct the bus naming
Other:
- sheet Segment1 ports: added CS[39..1], SW[9..1]; removed CS_Bus, SW_Bus
- sheet Segment2 ports: added CS[39..1], SW[9..1]; removed CS_Bus, SW_Bus
- sheet Segment3 ports: added CS[39..1], SW[9..1]; removed CS_Bus, SW_Bus
- sheet Segment4 ports: added CS[39..1], SW[9..1]; removed CS_Bus, SW_Bus
- sheet controller ports: added CS[39..1], SW[9..1]; removed CS_Bus, SW_Bus
Changed lines of the file:
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@@
       (effects (font (size 1.27 1.27)) (justify left top))
     )
-    (pin "SW_Bus" input (at 233.68 138.43 180)
+    (pin "CS[39..1]" input (at 233.68 128.27 180)
       (effects (font (size 1.27 1.27)) (justify left))
     )
-    (pin "CS_Bus" input (at 233.68 128.27 180)
+    (pin "SW[9..1]" input (at 233.68 138.43 180)
       (effects (font (size 1.27 1.27)) (justify left))
     )
@@
       (effects (font (size 1.27 1.27)) (justify left top))
     )
-    (pin "SW_Bus" input (at 233.68 43.18 180)
+    (pin "CS[39..1]" input (at 233.68 33.02 180)
       (effects (font (size 1.27 1.27)) (justify left))
     )
-    (pin "CS_Bus" input (at 233.68 33.02 180)
+    (pin "SW[9..1]" input (at 233.68 43.18 180)
       (effects (font (size 1.27 1.27)) (justify left))
     )
@@
       (effects (font (size 1.27 1.27)) (justify left top))
     )
-    (pin "SW_Bus" input (at 233.68 106.68 180)
+    (pin "CS[39..1]" input (at 233.68 96.52 180)
       (effects (font (size 1.27 1.27)) (justify left))
     )
-    (pin "CS_Bus" input (at 233.68 96.52 180)
+    (pin "SW[9..1]" input (at 233.68 106.68 180)
       (effects (font (size 1.27 1.27)) (justify left))
     )
@@
       (effects (font (size 1.27 1.27)) (justify left top))
     )
-    (pin "SW_Bus" input (at 233.68 74.93 180)
+    (pin "SW[9..1]" input (at 233.68 74.93 180)
       (effects (font (size 1.27 1.27)) (justify left))
     )
-    (pin "CS_Bus" input (at 233.68 64.77 180)
+    (pin "CS[39..1]" input (at 233.68 64.77 180)
       (effects (font (size 1.27 1.27)) (justify left))
     )
@@
       (effects (font (size 1.27 1.27)) (justify left top))
     )
-    (pin "SW_Bus" input (at 132.08 86.36 0)
+    (pin "SW[9..1]" input (at 132.08 86.36 0)
       (effects (font (size 1.27 1.27)) (justify right))
     )
-    (pin "CS_Bus" input (at 132.08 77.47 0)
+    (pin "CS[39..1]" input (at 132.08 77.47 0)
       (effects (font (size 1.27 1.27)) (justify right))
     )

Commit message: Add power and connections for i2c interface
Connections:
- no-connect marks 0 -> 4
Other:
- sheet controller renamed Controller
- sheet Controller ports: added INTB, SCL, SDA, SDB; removed none
- moved on the sheet: J1

Commit message: start mapping out locations on PCB
Parts:
- removed J1: Conn_02x06_Counter_Clockwise, Connector_PinHeader_2.54mm:PinHeader_2x06_P2.54mm_Vertical, symbol Connector_Generic:Conn_02x06_Counter_Clockwise
- added J1: Conn_02x06_Odd_Even, Connector_PinHeader_2.54mm:PinHeader_2x06_P2.54mm_Vertical, symbol Connector_Generic:Conn_02x06_Odd_Even
Connections:
- net +3V3: now also J1.11 (Pin_11), J1.12 (Pin_12)
- net Controller/INTB: now also J1.6 (Pin_6)
- net Controller/SCL: now also J1.8 (Pin_8)
- net Controller/SDA: now also J1.7 (Pin_7)
- net Controller/SDB: now also J1.5 (Pin_5)
- net GND: now also J1.10 (Pin_10), J1.9 (Pin_9)
Other:
- note added: "PMod Connector"
- company: (none) -> James Horton
- title: (none) -> PMod RGB & Segment Display
