File: PMOD_RGB7Segment/Hardware/segment3.kicad_sch (KiCad schematic)
At the start: 22 parts

Commit message: Add the schematics for each of the 7 segment characters
Parts:
- removed D1, D10, D11, D12, D13, D14, D15, D16, D17, D18, D19, D2, D20, D21, D22, D3, D4, D5, D6, D7, D8, D9: LED_ARGB, jjh:SX-0402-RGB, symbol Device:LED_ARGB
- added D? (x22): LED_ARGB, jjh:SX-0402-RGB, symbol Device:LED_ARGB
Connections:
- net CS1: now also D?.2 (RK), D?.2 (RK)
- net CS10: now also D?.2 (RK), D?.2 (RK)
- net CS11: now also D?.3 (GK), D?.3 (GK)
- net CS12: now also D?.4 (BK), D?.4 (BK)
- net CS13: now also D?.2 (RK), D?.2 (RK)
- net CS14: now also D?.3 (GK), D?.3 (GK)
- net CS15: now also D?.4 (BK), D?.4 (BK)
- net CS16: now also D?.2 (RK), D?.2 (RK)
- net CS17: now also D?.3 (GK), D?.3 (GK)
- net CS18: now also D?.4 (BK), D?.4 (BK)
- net CS19: now also D?.2 (RK), D?.2 (RK)
- net CS2: now also D?.3 (GK), D?.3 (GK)
- net CS20: now also D?.3 (GK), D?.3 (GK)
- net CS21: now also D?.4 (BK), D?.4 (BK)
- net CS22: now also D?.2 (RK), D?.2 (RK)
- net CS23: now also D?.3 (GK), D?.3 (GK)
- net CS24: now also D?.4 (BK), D?.4 (BK)
- net CS25: now also D?.2 (RK), D?.2 (RK)
- net CS26: now also D?.3 (GK), D?.3 (GK)
- net CS27: now also D?.4 (BK), D?.4 (BK)
- net CS28: now also D?.2 (RK), D?.2 (RK)
- net CS29: now also D?.3 (GK), D?.3 (GK)
- net CS3: now also D?.4 (BK), D?.4 (BK)
- net CS30: now also D?.4 (BK), D?.4 (BK)
- net CS31: now also D?.2 (RK)
- net CS32: now also D?.3 (GK)
- net CS33: now also D?.4 (BK)
- net CS34: now also D?.2 (RK)
- net CS35: now also D?.3 (GK)
- net CS36: now also D?.4 (BK)
- net CS4: now also D?.2 (RK), D?.2 (RK)
- net CS5: now also D?.3 (GK), D?.3 (GK)
- net CS6: now also D?.4 (BK), D?.4 (BK)
- net CS7: now also D?.2 (RK), D?.2 (RK)
- net CS8: now also D?.3 (GK), D?.3 (GK)
- net CS9: now also D?.4 (BK), D?.4 (BK)
- new net SW5: D?.1 (A), D?.1 (A), D?.1 (A), D?.1 (A), D?.1 (A), D?.1 (A), D?.1 (A), D?.1 (A), D?.1 (A), D?.1 (A), D?.1 (A), D?.1 (A)
- new net SW6: D?.1 (A), D?.1 (A), D?.1 (A), D?.1 (A), D?.1 (A), D?.1 (A), D?.1 (A), D?.1 (A), D?.1 (A), D?.1 (A)

Commit message: minor changes to segments
Parts:
- gave numbers to parts that had none: 22
Changed lines of the file:
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@@
   (symbol (lib_id "Device:LED_ARGB") (at 195.58 109.22 0)
     (in_bom yes) (on_board yes)
-    (property "Reference" "D?" (id 0) (at 200.66 101.6 0))
+    (property "Reference" "D62" (id 0) (at 200.66 101.6 0))
     (property "Value" "LED_ARGB" (id 1) (at 204.47 115.57 0))
     (property "Footprint" "jjh:SX-0402-RGB" (id 2) (at 195.58 110.49 0)
@@
   (symbol (lib_id "Device:LED_ARGB") (at 195.58 78.74 0)
     (in_bom yes) (on_board yes)
-    (property "Reference" "D?" (id 0) (at 200.66 71.12 0))
+    (property "Reference" "D61" (id 0) (at 200.66 71.12 0))
     (property "Value" "LED_ARGB" (id 1) (at 204.47 85.09 0))
     (property "Footprint" "jjh:SX-0402-RGB" (id 2) (at 195.58 80.01 0)
@@
   (symbol (lib_id "Device:LED_ARGB") (at 252.73 109.22 0)
     (in_bom yes) (on_board yes)
-    (property "Reference" "D?" (id 0) (at 257.81 101.6 0))
+    (property "Reference" "D68" (id 0) (at 257.81 101.6 0))
     (property "Value" "LED_ARGB" (id 1) (at 261.62 115.57 0))
     (property "Footprint" "jjh:SX-0402-RGB" (id 2) (at 252.73 110.49 0)
@@
   (symbol (lib_id "Device:LED_ARGB") (at 81.28 36.83 0)
     (in_bom yes) (on_board yes)
-    (property "Reference" "D?" (id 0) (at 86.36 29.21 0))
+    (property "Reference" "D47" (id 0) (at 86.36 29.21 0))
     (property "Value" "LED_ARGB" (id 1) (at 90.17 43.18 0))
     (property "Footprint" "jjh:SX-0402-RGB" (id 2) (at 81.28 38.1 0)
@@
   (symbol (lib_id "Device:LED_ARGB") (at 138.43 58.42 0)
     (in_bom yes) (on_board yes)
-    (property "Reference" "D?" (id 0) (at 143.51 50.8 0))
+    (property "Reference" "D54" (id 0) (at 143.51 50.8 0))
     (property "Value" "LED_ARGB" (id 1) (at 147.32 64.77 0))
     (property "Footprint" "jjh:SX-0402-RGB" (id 2) (at 138.43 59.69 0)
@@
   (symbol (lib_id "Device:LED_ARGB") (at 195.58 130.81 0)
     (in_bom yes) (on_board yes)
-    (property "Reference" "D?" (id 0) (at 200.66 123.19 0))
+    (property "Reference" "D63" (id 0) (at 200.66 123.19 0))
     (property "Value" "LED_ARGB" (id 1) (at 204.47 137.16 0))
     (property "Footprint" "jjh:SX-0402-RGB" (id 2) (at 195.58 132.08 0)
@@
   (symbol (lib_id "Device:LED_ARGB") (at 81.28 78.74 0)
     (in_bom yes) (on_board yes)
-    (property "Reference" "D?" (id 0) (at 86.36 71.12 0))
+    (property "Reference" "D49" (id 0) (at 86.36 71.12 0))
     (property "Value" "LED_ARGB" (id 1) (at 90.17 85.09 0))
     (property "Footprint" "jjh:SX-0402-RGB" (id 2) (at 81.28 80.01 0)
@@
   (symbol (lib_id "Device:LED_ARGB") (at 138.43 109.22 0)
     (in_bom yes) (on_board yes)
-    (property "Reference" "D?" (id 0) (at 143.51 101.6 0))
+    (property "Reference" "D56" (id 0) (at 143.51 101.6 0))
     (property "Value" "LED_ARGB" (id 1) (at 147.32 115.57 0))
     (property "Footprint" "jjh:SX-0402-RGB" (id 2) (at 138.43 110.49 0)
@@
   (symbol (lib_id "Device:LED_ARGB") (at 252.73 58.42 0)
     (in_bom yes) (on_board yes)
-    (property "Reference" "D?" (id 0) (at 257.81 50.8 0))
+    (property "Reference" "D66" (id 0) (at 257.81 50.8 0))
     (property "Value" "LED_ARGB" (id 1) (at 261.62 64.77 0))
     (property "Footprint" "jjh:SX-0402-RGB" (id 2) (at 252.73 59.69 0)
@@
   (symbol (lib_id "Device:LED_ARGB") (at 138.43 130.81 0)
     (in_bom yes) (on_board yes)
-    (property "Reference" "D?" (id 0) (at 143.51 123.19 0))
+    (property "Reference" "D57" (id 0) (at 143.51 123.19 0))
     (property "Value" "LED_ARGB" (id 1) (at 147.32 137.16 0))
     (property "Footprint" "jjh:SX-0402-RGB" (id 2) (at 138.43 132.08 0)
@@
   (symbol (lib_id "Device:LED_ARGB") (at 138.43 78.74 0)
     (in_bom yes) (on_board yes)
-    (property "Reference" "D?" (id 0) (at 143.51 71.12 0))
+    (property "Reference" "D55" (id 0) (at 143.51 71.12 0))
     (property "Value" "LED_ARGB" (id 1) (at 147.32 85.09 0))
     (property "Footprint" "jjh:SX-0402-RGB" (id 2) (at 138.43 80.01 0)
@@
   (symbol (lib_id "Device:LED_ARGB") (at 252.73 36.83 0)
     (in_bom yes) (on_board yes)
-    (property "Reference" "D?" (id 0) (at 257.81 29.21 0))
+    (property "Reference" "D65" (id 0) (at 257.81 29.21 0))
     (property "Value" "LED_ARGB" (id 1) (at 261.62 43.18 0))
     (property "Footprint" "jjh:SX-0402-RGB" (id 2) (at 252.73 38.1 0)
@@
   (symbol (lib_id "Device:LED_ARGB") (at 195.58 58.42 0)
     (in_bom yes) (on_board yes)
-    (property "Reference" "D?" (id 0) (at 200.66 50.8 0))
+    (property "Reference" "D60" (id 0) (at 200.66 50.8 0))
     (property "Value" "LED_ARGB" (id 1) (at 204.47 64.77 0))
     (property "Footprint" "jjh:SX-0402-RGB" (id 2) (at 195.58 59.69 0)
@@
   (symbol (lib_id "Device:LED_ARGB") (at 195.58 151.13 0)
     (in_bom yes) (on_board yes)
-    (property "Reference" "D?" (id 0) (at 200.66 143.51 0))
+    (property "Reference" "D64" (id 0) (at 200.66 143.51 0))
     (property "Value" "LED_ARGB" (id 1) (at 204.47 157.48 0))
     (property "Footprint" "jjh:SX-0402-RGB" (id 2) (at 195.58 152.4 0)
@@
   (symbol (lib_id "Device:LED_ARGB") (at 138.43 151.13 0)
     (in_bom yes) (on_board yes)
-    (property "Reference" "D?" (id 0) (at 143.51 143.51 0))
+    (property "Reference" "D58" (id 0) (at 143.51 143.51 0))
     (property "Value" "LED_ARGB" (id 1) (at 147.32 157.48 0))
     (property "Footprint" "jjh:SX-0402-RGB" (id 2) (at 138.43 152.4 0)
@@
   (symbol (lib_id "Device:LED_ARGB") (at 138.43 36.83 0)
     (in_bom yes) (on_board yes)
-    (property "Reference" "D?" (id 0) (at 143.51 29.21 0))
+    (property "Reference" "D53" (id 0) (at 143.51 29.21 0))
     (property "Value" "LED_ARGB" (id 1) (at 147.32 43.18 0))
     (property "Footprint" "jjh:SX-0402-RGB" (id 2) (at 138.43 38.1 0)
@@
   (symbol (lib_id "Device:LED_ARGB") (at 195.58 36.83 0)
     (in_bom yes) (on_board yes)
-    (property "Reference" "D?" (id 0) (at 200.66 29.21 0))
+    (property "Reference" "D59" (id 0) (at 200.66 29.21 0))
     (property "Value" "LED_ARGB" (id 1) (at 204.47 43.18 0))
     (property "Footprint" "jjh:SX-0402-RGB" (id 2) (at 195.58 38.1 0)
@@
   (symbol (lib_id "Device:LED_ARGB") (at 81.28 151.13 0)
     (in_bom yes) (on_board yes)
-    (property "Reference" "D?" (id 0) (at 86.36 143.51 0))
+    (property "Reference" "D52" (id 0) (at 86.36 143.51 0))
     (property "Value" "LED_ARGB" (id 1) (at 90.17 157.48 0))
     (property "Footprint" "jjh:SX-0402-RGB" (id 2) (at 81.28 152.4 0)
@@
   (symbol (lib_id "Device:LED_ARGB") (at 252.73 78.74 0)
     (in_bom yes) (on_board yes)
-    (property "Reference" "D?" (id 0) (at 257.81 71.12 0))
+    (property "Reference" "D67" (id 0) (at 257.81 71.12 0))
     (property "Value" "LED_ARGB" (id 1) (at 261.62 85.09 0))
     (property "Footprint" "jjh:SX-0402-RGB" (id 2) (at 252.73 80.01 0)
@@
   (symbol (lib_id "Device:LED_ARGB") (at 81.28 130.81 0)
     (in_bom yes) (on_board yes)
-    (property "Reference" "D?" (id 0) (at 86.36 123.19 0))
+    (property "Reference" "D51" (id 0) (at 86.36 123.19 0))
     (property "Value" "LED_ARGB" (id 1) (at 90.17 137.16 0))
     (property "Footprint" "jjh:SX-0402-RGB" (id 2) (at 81.28 132.08 0)
@@
   (symbol (lib_id "Device:LED_ARGB") (at 81.28 109.22 0)
     (in_bom yes) (on_board yes)
-    (property "Reference" "D?" (id 0) (at 86.36 101.6 0))
+    (property "Reference" "D50" (id 0) (at 86.36 101.6 0))
     (property "Value" "LED_ARGB" (id 1) (at 90.17 115.57 0))
     (property "Footprint" "jjh:SX-0402-RGB" (id 2) (at 81.28 110.49 0)
@@
   (symbol (lib_id "Device:LED_ARGB") (at 81.28 58.42 0)
     (in_bom yes) (on_board yes)
-    (property "Reference" "D?" (id 0) (at 86.36 50.8 0))
+    (property "Reference" "D48" (id 0) (at 86.36 50.8 0))
     (property "Value" "LED_ARGB" (id 1) (at 90.17 64.77 0))
     (property "Footprint" "jjh:SX-0402-RGB" (id 2) (at 81.28 59.69 0)
