File: PMOD_RGB7Segment/Hardware/segment3.kicad_sch (KiCad schematic)
At the start: 22 parts

Commit message: correct the bus naming
Changed lines of the file:
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@@
     (effects (font (size 0.7 0.7) bold) (justify left bottom))
   )
-  (hierarchical_label "SW_Bus" (shape input) (at 31.75 175.26 180)
+  (hierarchical_label "SW[9..1]" (shape input) (at 31.75 175.26 180)
     (effects (font (size 1.27 1.27)) (justify right))
   )
-  (hierarchical_label "CS_Bus" (shape input) (at 34.29 15.24 180)
+  (hierarchical_label "CS[39..1]" (shape input) (at 34.29 15.24 180)
     (effects (font (size 1.27 1.27)) (justify right))
   )

Commit message: start mapping out locations on PCB
Other:
- company: (none) -> James Horton
- title: (none) -> PMod RGB & Segment Display
Changed lines of the file:
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@@
 (kicad_sch (version 20211123) (generator eeschema)
   (paper "A4")
+  (title_block
+    (title "PMod RGB & Segment Display")
+    (rev "v0.1")
+    (company "James Horton")
+    (comment 1 "interface, all LED's are designed to be indivdually addressable ")
+    (comment 2 "This design is a 4 Digit Seven Segment Display made from RGB LED's, controlled using I2C")
+    (comment 4 "Licensed Under CERN Open Hardware Licence Version 2 - Permissive")
+  )
   (junction (at 214.63 78.74) (diameter 0) (color 0 0 0 0)
   )

Commit message: route the bus conections on SW to LEDs
Connections:
- net CS10 is gone; now on net CS19: D50.2 (RK), D62.2 (RK)
- net CS11 is gone; now on net CS20: D50.3 (GK), D62.3 (GK)
- net CS12 is gone; now on net CS21: D50.4 (BK), D62.4 (BK)
- net CS28 is gone; now on net CS25: D56.2 (RK), D68.2 (RK)
- net CS29 is gone; now on net CS26: D56.3 (GK), D68.3 (GK)
- net CS30 is gone; now on net CS27: D56.4 (BK), D68.4 (BK)
- net CS31 is gone; now on net CS25: D57.2 (RK)
- net CS32 is gone; now on net CS26: D57.3 (GK)
- net CS33 is gone; now on net CS27: D57.4 (BK)
- net CS34 is gone; now on net CS25: D58.2 (RK)
- net CS35 is gone; now on net CS26: D58.3 (GK)
- net CS36 is gone; now on net CS27: D58.4 (BK)
- net CS13: no longer D51.2 (RK)
- net CS14: no longer D51.3 (GK)
- net CS15: no longer D51.4 (BK)
- net CS16: no longer D52.2 (RK)
- net CS17: no longer D52.3 (GK)
- net CS18: no longer D52.4 (BK)
- net CS19: now also D47.2 (RK), D48.2 (RK), D49.2 (RK), D51.2 (RK), D52.2 (RK); no longer D53.2 (RK), D65.2 (RK)
- net CS20: now also D47.3 (GK), D48.3 (GK), D49.3 (GK), D51.3 (GK), D52.3 (GK); no longer D53.3 (GK), D65.3 (GK)
- net CS21: now also D47.4 (BK), D48.4 (BK), D49.4 (BK), D51.4 (BK), D52.4 (BK); no longer D53.4 (BK), D65.4 (BK)
- net CS22: now also D53.2 (RK), D55.2 (RK), D59.2 (RK), D60.2 (RK), D61.2 (RK), D65.2 (RK), D67.2 (RK)
- net CS23: now also D53.3 (GK), D55.3 (GK), D59.3 (GK), D60.3 (GK), D61.3 (GK), D65.3 (GK), D67.3 (GK)
- net CS24: now also D53.4 (BK), D55.4 (BK), D59.4 (BK), D60.4 (BK), D61.4 (BK), D65.4 (BK), D67.4 (BK)
- net CS25: no longer D55.2 (RK), D67.2 (RK)
- net CS26: no longer D55.3 (GK), D67.3 (GK)
- net CS27: no longer D55.4 (BK), D67.4 (BK)
- net SW5: now also D66.1 (A); no longer D47.1 (A), D49.1 (A), D50.1 (A), D51.1 (A), D52.1 (A), D53.1 (A), D54.1 (A), D55.1 (A), D56.1 (A), D57.1 (A), D58.1 (A)
- net SW6: now also D49.1 (A); no longer D59.1 (A), D60.1 (A), D61.1 (A), D62.1 (A), D63.1 (A), D64.1 (A), D65.1 (A), D66.1 (A), D68.1 (A)
- removed net CS1: D47.2 (RK), D59.2 (RK)
- removed net CS2: D47.3 (GK), D59.3 (GK)
- removed net CS3: D47.4 (BK), D59.4 (BK)
- removed net CS4: D48.2 (RK), D60.2 (RK)
- removed net CS5: D48.3 (GK), D60.3 (GK)
- removed net CS6: D48.4 (BK), D60.4 (BK)
- removed net CS7: D49.2 (RK), D61.2 (RK)
- removed net CS8: D49.3 (GK), D61.3 (GK)
- removed net CS9: D49.4 (BK), D61.4 (BK)
- new net SW1: D56.1 (A), D59.1 (A), D62.1 (A)
- new net SW2: D57.1 (A), D60.1 (A), D63.1 (A)
- new net SW3: D58.1 (A), D61.1 (A), D64.1 (A)
- new net SW4: D47.1 (A), D65.1 (A), D68.1 (A)
- new net SW7: D50.1 (A), D53.1 (A)
- new net SW8: D51.1 (A), D54.1 (A)
- new net SW9: D52.1 (A), D55.1 (A)

Commit message: correct pins in schematic and continue LED layout on PCB
Connections:
- net CS13 is gone; now on net CS19: D63.2 (RK)
- net CS14 is gone; now on net CS20: D63.3 (GK)
- net CS15 is gone; now on net CS21: D63.4 (BK)
- net CS16 is gone; now on net CS19: D64.2 (RK)
- net CS17 is gone; now on net CS20: D64.3 (GK)
- net CS18 is gone; now on net CS21: D64.4 (BK)
Changed lines of the file:
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@@
     (effects (font (size 1.27 1.27) bold) (justify left bottom))
   )
-  (label "CS14" (at 185.42 130.81 0)
+  (label "CS20" (at 185.42 130.81 0)
     (effects (font (size 0.7 0.7) bold) (justify left bottom))
   )
@@
     (effects (font (size 0.7 0.7) bold) (justify left bottom))
   )
-  (label "CS17" (at 185.42 151.13 0)
+  (label "CS20" (at 185.42 151.13 0)
     (effects (font (size 0.7 0.7) bold) (justify left bottom))
   )
@@
     (effects (font (size 0.7 0.7) bold) (justify left bottom))
   )
-  (label "CS16" (at 185.42 146.05 0)
+  (label "CS19" (at 185.42 146.05 0)
     (effects (font (size 0.7 0.7) bold) (justify left bottom))
   )
@@
     (effects (font (size 1.27 1.27) bold) (justify left bottom))
   )
-  (label "CS15" (at 185.42 135.89 0)
+  (label "CS21" (at 185.42 135.89 0)
     (effects (font (size 0.7 0.7) bold) (justify left bottom))
   )
-  (label "CS18" (at 185.42 156.21 0)
+  (label "CS21" (at 185.42 156.21 0)
     (effects (font (size 0.7 0.7) bold) (justify left bottom))
   )
@@
     (effects (font (size 0.7 0.7) bold) (justify left bottom))
   )
-  (label "CS13" (at 185.42 125.73 0)
+  (label "CS19" (at 185.42 125.73 0)
     (effects (font (size 0.7 0.7) bold) (justify left bottom))
   )

Commit message: continue with placement and layout of digits
Connections:
- net SW1: now also D64.1 (A); no longer D62.1 (A)
- net SW3: now also D62.1 (A); no longer D64.1 (A)
Changed lines of the file:
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@@
     (effects (font (size 1.27 1.27) bold) (justify left bottom))
   )
-  (label "SW3" (at 210.82 151.13 0)
+  (label "SW1" (at 210.82 151.13 0)
     (effects (font (size 1.27 1.27) bold) (justify left bottom))
   )
@@
     (effects (font (size 0.7 0.7) bold) (justify left bottom))
   )
-  (label "SW1" (at 210.82 109.22 0)
+  (label "SW3" (at 210.82 109.22 0)
     (effects (font (size 1.27 1.27) bold) (justify left bottom))
   )
