File: PMOD_RGB7Segment/Hardware/segment1.kicad_sch (KiCad schematic)
At the start: 22 parts

Commit message: correct the bus naming
Changed lines of the file:
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@@
     (effects (font (size 0.7 0.7) bold) (justify left bottom))
+  )
+  (label "CS[39..1]" (at 41.91 15.24 0)
+    (effects (font (size 1.27 1.27) bold) (justify left bottom))
   )
   (label "CS17" (at 71.12 151.13 0)
@@
     (effects (font (size 0.7 0.7) bold) (justify left bottom))
   )
-  (hierarchical_label "SW_Bus" (shape input) (at 31.75 175.26 180)
+  (hierarchical_label "SW[9..1]" (shape input) (at 31.75 175.26 180)
     (effects (font (size 1.27 1.27)) (justify right))
   )
-  (hierarchical_label "CS_Bus" (shape input) (at 34.29 15.24 180)
+  (hierarchical_label "CS[39..1]" (shape input) (at 34.29 15.24 180)
     (effects (font (size 1.27 1.27)) (justify right))
   )

Commit message: start mapping out locations on PCB
Other:
- company: (none) -> James Horton
- title: (none) -> PMod RGB & Segment Display
Changed lines of the file:
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@@
 (kicad_sch (version 20211123) (generator eeschema)
   (paper "A4")
+  (title_block
+    (title "PMod RGB & Segment Display")
+    (rev "v0.1")
+    (company "James Horton")
+    (comment 1 "interface, all LED's are designed to be indivdually addressable ")
+    (comment 2 "This design is a 4 Digit Seven Segment Display made from RGB LED's, controlled using I2C")
+    (comment 4 "Licensed Under CERN Open Hardware Licence Version 2 - Permissive")
+  )
   (junction (at 214.63 78.74) (diameter 0) (color 0 0 0 0)
   )

Commit message: changes to the LED connection ordering
Connections:
- net CS10 is gone; now on net CS1: D16.2 (RK), D4.2 (RK)
- net CS11 is gone; now on net CS2: D16.3 (GK), D4.3 (GK)
- net CS12 is gone; now on net CS3: D16.4 (BK), D4.4 (BK)
- net CS13 is gone; now on net CS1: D17.2 (RK), D5.2 (RK)
- net CS14 is gone; now on net CS2: D17.3 (GK), D5.3 (GK)
- net CS15 is gone; now on net CS3: D17.4 (BK), D5.4 (BK)
- net CS16 is gone; now on net CS1: D18.2 (RK), D6.2 (RK)
- net CS17 is gone; now on net CS2: D18.3 (GK), D6.3 (GK)
- net CS18 is gone; now on net CS3: D18.4 (BK), D6.4 (BK)
- net CS19 is gone; now on net CS4: D19.2 (RK), D7.2 (RK)
- net CS20 is gone; now on net CS5: D19.3 (GK), D7.3 (GK)
- net CS21 is gone; now on net CS6: D19.4 (BK), D7.4 (BK)
- net CS22 is gone; now on net CS4: D20.2 (RK), D8.2 (RK)
- net CS23 is gone; now on net CS5: D20.3 (GK), D8.3 (GK)
- net CS24 is gone; now on net CS6: D20.4 (BK), D8.4 (BK)
- net CS25 is gone; now on net CS4: D21.2 (RK), D9.2 (RK)
- net CS26 is gone; now on net CS5: D21.3 (GK), D9.3 (GK)
- net CS27 is gone; now on net CS6: D21.4 (BK), D9.4 (BK)
- net CS28 is gone; now on net CS7: D10.2 (RK), D22.2 (RK)
- net CS29 is gone; now on net CS8: D10.3 (GK), D22.3 (GK)
- net CS30 is gone; now on net CS9: D10.4 (BK), D22.4 (BK)
- net CS31 is gone; now on net CS7: D11.2 (RK)
- net CS32 is gone; now on net CS8: D11.3 (GK)
- net CS33 is gone; now on net CS9: D11.4 (BK)
- net CS34 is gone; now on net CS7: D12.2 (RK)
- net CS35 is gone; now on net CS8: D12.3 (GK)
- net CS36 is gone; now on net CS9: D12.4 (BK)
- net CS1: now also D2.2 (RK), D3.2 (RK); no longer D13.2 (RK)
- net CS2: now also D2.3 (GK), D3.3 (GK); no longer D13.3 (GK)
- net CS3: now also D2.4 (BK), D3.4 (BK); no longer D13.4 (BK)
- net CS4: now also D13.2 (RK), D15.2 (RK); no longer D2.2 (RK)
- net CS5: now also D13.3 (GK), D15.3 (GK); no longer D2.3 (GK)
- net CS6: now also D13.4 (BK), D15.4 (BK); no longer D2.4 (BK)
- net CS7: no longer D15.2 (RK), D3.2 (RK)
- net CS8: no longer D15.3 (GK), D3.3 (GK)
- net CS9: no longer D15.4 (BK), D3.4 (BK)
- net SW1: now also D13.1 (A), D16.1 (A); no longer D1.1 (A), D11.1 (A), D12.1 (A), D2.1 (A), D3.1 (A), D4.1 (A), D5.1 (A), D6.1 (A), D7.1 (A), D8.1 (A), D9.1 (A)
- net SW2: now also D11.1 (A); no longer D13.1 (A), D15.1 (A), D16.1 (A), D18.1 (A), D19.1 (A), D20.1 (A), D21.1 (A), D22.1 (A)
- new net SW3: D12.1 (A), D15.1 (A), D18.1 (A)
- new net SW4: D1.1 (A), D19.1 (A), D22.1 (A)
- new net SW5: D2.1 (A), D20.1 (A)
- new net SW6: D21.1 (A), D3.1 (A)
- new net SW7: D4.1 (A), D7.1 (A)
- new net SW8: D5.1 (A), D8.1 (A)
- new net SW9: D6.1 (A), D9.1 (A)
