File: PMOD_RGB7Segment/Hardware/PMod_RGB7Segment.kicad_pcb (KiCad board)
At the start: 2 copper layers, 100 x 96 mm, 12 parts

Commit message: Add initial layout for segment 1
Parts:
- added D1: LED_ARGB, jjh:SX-0402-RGB, F.Cu at (115.6, 103.6)
- added D10: LED_ARGB, jjh:SX-0402-RGB, F.Cu at (120.5, 125.5)
- added D11: LED_ARGB, jjh:SX-0402-RGB, F.Cu at (118.0, 125.5)
- added D12: LED_ARGB, jjh:SX-0402-RGB, F.Cu at (115.4, 125.5)
- added D13: LED_ARGB, jjh:SX-0402-RGB, F.Cu at (112.2, 122.2)
- added D14: LED_ARGB, jjh:SX-0402-RGB, F.Cu at (112.2, 119.8)
- added D15: LED_ARGB, jjh:SX-0402-RGB, F.Cu at (112.2, 117.2)
- added D16: LED_ARGB, jjh:SX-0402-RGB, F.Cu at (112.2, 111.5)
- added D17: LED_ARGB, jjh:SX-0402-RGB, F.Cu at (112.2, 109.0)
- added D18: LED_ARGB, jjh:SX-0402-RGB, F.Cu at (112.2, 106.8)
- added D19: LED_ARGB, jjh:SX-0402-RGB, F.Cu at (115.5, 114.5)
- added D2: LED_ARGB, jjh:SX-0402-RGB, F.Cu at (118.0, 103.6)
- added D20: LED_ARGB, jjh:SX-0402-RGB, F.Cu at (118.0, 114.5)
- added D21: LED_ARGB, jjh:SX-0402-RGB, F.Cu at (120.5, 114.5)
- added D22: LED_ARGB, jjh:SX-0402-RGB, F.Cu at (127.5, 125.2)
- added D23: LED_ARGB, jjh:SX-0402-RGB, F.Cu at (64.5, 37.9)
- added D24: LED_ARGB, jjh:SX-0402-RGB, F.Cu at (57.2, 40.4)
- added D25: LED_ARGB, jjh:SX-0402-RGB, F.Cu at (57.2, 42.8)
- added D26: LED_ARGB, jjh:SX-0402-RGB, F.Cu at (59.6, 42.8)
- added D27: LED_ARGB, jjh:SX-0402-RGB, F.Cu at (62.1, 40.4)
- added D28: LED_ARGB, jjh:SX-0402-RGB, F.Cu at (62.1, 45.2)
- added D29: LED_ARGB, jjh:SX-0402-RGB, F.Cu at (59.6, 37.9)
- added D3: LED_ARGB, jjh:SX-0402-RGB, F.Cu at (120.3, 103.6)
- added D30: LED_ARGB, jjh:SX-0402-RGB, F.Cu at (64.5, 42.8)
- added D31: LED_ARGB, jjh:SX-0402-RGB, F.Cu at (57.2, 45.2)
- added D32: LED_ARGB, jjh:SX-0402-RGB, F.Cu at (64.5, 40.4)
- added D33: LED_ARGB, jjh:SX-0402-RGB, F.Cu at (59.6, 40.4)
- added D34: LED_ARGB, jjh:SX-0402-RGB, F.Cu at (52.3, 42.8)
- added D35: LED_ARGB, jjh:SX-0402-RGB, F.Cu at (54.8, 45.2)
- added D36: LED_ARGB, jjh:SX-0402-RGB, F.Cu at (54.8, 40.4)
- added D37: LED_ARGB, jjh:SX-0402-RGB, F.Cu at (62.1, 37.9)
- added D38: LED_ARGB, jjh:SX-0402-RGB, F.Cu at (54.8, 42.8)
- added D39: LED_ARGB, jjh:SX-0402-RGB, F.Cu at (54.8, 37.9)
- added D4: LED_ARGB, jjh:SX-0402-RGB, F.Cu at (123.5, 106.8)
- added D40: LED_ARGB, jjh:SX-0402-RGB, F.Cu at (62.1, 42.8)
- added D41: LED_ARGB, jjh:SX-0402-RGB, F.Cu at (52.3, 37.9)
- added D42: LED_ARGB, jjh:SX-0402-RGB, F.Cu at (67.0, 37.9)
- added D43: LED_ARGB, jjh:SX-0402-RGB, F.Cu at (52.3, 45.2)
- added D44: LED_ARGB, jjh:SX-0402-RGB, F.Cu at (52.3, 40.4)
- added D45: LED_ARGB, jjh:SX-0402-RGB, F.Cu at (57.2, 37.9)
- added D46: LED_ARGB, jjh:SX-0402-RGB, F.Cu at (59.6, 45.2)
- added D47: LED_ARGB, jjh:SX-0402-RGB, F.Cu at (61.0, 64.0)
- added D48: LED_ARGB, jjh:SX-0402-RGB, F.Cu at (51.2, 61.6)
- added D49: LED_ARGB, jjh:SX-0402-RGB, F.Cu at (61.0, 61.6)
- added D5: LED_ARGB, jjh:SX-0402-RGB, F.Cu at (123.5, 108.9)
- added D50: LED_ARGB, jjh:SX-0402-RGB, F.Cu at (53.7, 59.1)
- added D51: LED_ARGB, jjh:SX-0402-RGB, F.Cu at (51.2, 64.0)
- added D52: LED_ARGB, jjh:SX-0402-RGB, F.Cu at (56.1, 59.1)
- added D53: LED_ARGB, jjh:SX-0402-RGB, F.Cu at (53.7, 64.0)
- added D54: LED_ARGB, jjh:SX-0402-RGB, F.Cu at (58.6, 66.4)
- added D55: LED_ARGB, jjh:SX-0402-RGB, F.Cu at (58.6, 61.6)
- added D56: LED_ARGB, jjh:SX-0402-RGB, F.Cu at (58.6, 64.0)
- added D57: LED_ARGB, jjh:SX-0402-RGB, F.Cu at (61.0, 59.1)
- added D58: LED_ARGB, jjh:SX-0402-RGB, F.Cu at (56.1, 61.6)
- added D59: LED_ARGB, jjh:SX-0402-RGB, F.Cu at (51.2, 66.4)
- added D6: LED_ARGB, jjh:SX-0402-RGB, F.Cu at (123.5, 111.2)
- added D60: LED_ARGB, jjh:SX-0402-RGB, F.Cu at (53.7, 66.4)
- added D61: LED_ARGB, jjh:SX-0402-RGB, F.Cu at (65.9, 59.1)
- added D62: LED_ARGB, jjh:SX-0402-RGB, F.Cu at (56.1, 64.0)
- added D63: LED_ARGB, jjh:SX-0402-RGB, F.Cu at (63.4, 59.1)
- added D64: LED_ARGB, jjh:SX-0402-RGB, F.Cu at (58.6, 59.1)
- added D65: LED_ARGB, jjh:SX-0402-RGB, F.Cu at (51.2, 59.1)
- added D66: LED_ARGB, jjh:SX-0402-RGB, F.Cu at (56.1, 66.4)
- added D67: LED_ARGB, jjh:SX-0402-RGB, F.Cu at (53.7, 61.6)
- added D68: LED_ARGB, jjh:SX-0402-RGB, F.Cu at (63.4, 61.6)
- added D69: LED_ARGB, jjh:SX-0402-RGB, F.Cu at (39.7, 59.1)
- added D7: LED_ARGB, jjh:SX-0402-RGB, F.Cu at (123.5, 117.2)
- added D70: LED_ARGB, jjh:SX-0402-RGB, F.Cu at (37.2, 59.1)
- added D71: LED_ARGB, jjh:SX-0402-RGB, F.Cu at (42.1, 59.1)
- added D72: LED_ARGB, jjh:SX-0402-RGB, F.Cu at (34.8, 61.6)
- added D73: LED_ARGB, jjh:SX-0402-RGB, F.Cu at (34.8, 59.1)
- added D74: LED_ARGB, jjh:SX-0402-RGB, F.Cu at (29.9, 64.0)
- added D75: LED_ARGB, jjh:SX-0402-RGB, F.Cu at (39.7, 64.0)
- added D76: LED_ARGB, jjh:SX-0402-RGB, F.Cu at (32.3, 66.4)
- added D77: LED_ARGB, jjh:SX-0402-RGB, F.Cu at (37.2, 61.6)
- added D78: LED_ARGB, jjh:SX-0402-RGB, F.Cu at (32.3, 64.0)
- added D79: LED_ARGB, jjh:SX-0402-RGB, F.Cu at (29.9, 61.6)
- added D8: LED_ARGB, jjh:SX-0402-RGB, F.Cu at (123.5, 119.8)
- added D80: LED_ARGB, jjh:SX-0402-RGB, F.Cu at (44.5, 59.1)
- added D81: LED_ARGB, jjh:SX-0402-RGB, F.Cu at (37.2, 66.4)
- added D82: LED_ARGB, jjh:SX-0402-RGB, F.Cu at (29.9, 66.4)
- added D83: LED_ARGB, jjh:SX-0402-RGB, F.Cu at (32.3, 59.1)
- added D84: LED_ARGB, jjh:SX-0402-RGB, F.Cu at (37.2, 64.0)
- added D85: LED_ARGB, jjh:SX-0402-RGB, F.Cu at (39.7, 61.6)
- added D86: LED_ARGB, jjh:SX-0402-RGB, F.Cu at (42.1, 61.6)
- added D87: LED_ARGB, jjh:SX-0402-RGB, F.Cu at (32.3, 61.6)
- added D88: LED_ARGB, jjh:SX-0402-RGB, F.Cu at (29.9, 59.1)
- added D89: LED_ARGB, jjh:SX-0402-RGB, F.Cu at (34.8, 66.4)
- added D9: LED_ARGB, jjh:SX-0402-RGB, F.Cu at (123.5, 122.2)
- added D90: LED_ARGB, jjh:SX-0402-RGB, F.Cu at (34.8, 64.0)
- added IC1: IS31FL3741A-QFLS4-TR, jjh:QFN40P700X700X80-61N-D, F.Cu at (105.0, 114.5)
- added J1: Conn_02x06_Counter_Clockwise, Connector_PinHeader_2.54mm:PinHeader_2x06_P2.54mm_Vertical, F.Cu at (93.7, 108.7)
- added REF**: NPTH, NPTH, F.Cu at (185.0, 61.8)
- added REF**: NPTH, NPTH, F.Cu at (97.0, 100.2)
- added REF**: NPTH, NPTH, F.Cu at (99.0, 66.2)
- added REF**: NPTH, NPTH, F.Cu at (186.0, 66.2)
- added REF**: NPTH, NPTH, F.Cu at (98.0, 95.8)
- added REF**: NPTH, NPTH, F.Cu at (186.0, 95.8)
- added REF**: NPTH, NPTH, F.Cu at (183.0, 100.2)
- added REF**: NPTH, NPTH, F.Cu at (185.0, 95.8)
- added REF**: NPTH, NPTH, F.Cu at (186.0, 100.2)
- added REF**: NPTH, NPTH, F.Cu at (187.0, 95.8)
- added REF**: NPTH, NPTH, F.Cu at (98.0, 66.2)
- added REF**: NPTH, NPTH, F.Cu at (184.0, 95.8)
- added REF**: NPTH, NPTH, F.Cu at (98.0, 100.2)
- added REF**: NPTH, NPTH, F.Cu at (183.0, 66.2)
- added REF**: NPTH, NPTH, F.Cu at (95.0, 66.2)
- added REF**: NPTH, NPTH, F.Cu at (184.0, 100.2)
- added REF**: NPTH, NPTH, F.Cu at (187.0, 66.2)
- added REF**: NPTH, NPTH, F.Cu at (96.0, 66.2)
- added REF**: NPTH, NPTH, F.Cu at (183.0, 61.8)
- added REF**: NPTH, NPTH, F.Cu at (185.0, 100.2)
- added REF**: NPTH, NPTH, F.Cu at (186.0, 61.8)
- added REF**: NPTH, NPTH, F.Cu at (187.0, 61.8)
- added REF**: NPTH, NPTH, F.Cu at (184.0, 66.2)
- added REF**: NPTH, NPTH, F.Cu at (99.0, 100.2)
- added REF**: NPTH, NPTH, F.Cu at (183.0, 95.8)
- added REF**: NPTH, NPTH, F.Cu at (184.0, 61.8)
- added REF**: NPTH, NPTH, F.Cu at (185.0, 66.2)
- added REF**: NPTH, NPTH, F.Cu at (96.0, 100.2)
- added REF**: NPTH, NPTH, F.Cu at (99.0, 61.8)
- added REF**: NPTH, NPTH, F.Cu at (95.0, 100.2)
- added REF**: NPTH, NPTH, F.Cu at (97.0, 66.2)
- added REF**: NPTH, NPTH, F.Cu at (96.0, 61.8)
- added REF**: NPTH, NPTH, F.Cu at (97.0, 95.8)
- added REF**: NPTH, NPTH, F.Cu at (98.0, 61.8)
- added REF**: NPTH, NPTH, F.Cu at (96.0, 95.8)
- added REF**: NPTH, NPTH, F.Cu at (97.0, 61.8)
- added REF**: NPTH, NPTH, F.Cu at (187.0, 100.2)
- added REF**: NPTH, NPTH, F.Cu at (99.0, 95.8)
- added REF**: NPTH, NPTH, F.Cu at (95.0, 61.8)
- added REF**: NPTH, NPTH, F.Cu at (95.0, 95.8)
- moved G*** 2.00 mm to (140.0, 47.0)
- moved G*** 2.00 mm to (180.0, 47.0)
- moved G*** 2.00 mm to (120.0, 46.8)
- moved G*** 2.00 mm to (160.0, 46.8)
- moved G*** 1.04 mm to (120.0, 80.8)
- moved G*** 1.00 mm to (180.0, 81.0)
- moved G*** 1.00 mm to (160.0, 80.8)
- moved G*** 1.00 mm to (140.0, 81.0)
Other:
- board size 100 x 96 mm -> 100 x 98 mm

Commit message: initial LED placement
Parts:
- moved D90 164.6 mm to (187.5, 125.5)
- moved D79 161.3 mm to (178.0, 125.5)
- moved D74 160.8 mm to (183.5, 111.5)
- moved D78 160.4 mm to (180.5, 125.5)
- moved D76 160.3 mm to (183.5, 119.8)
- moved D77 158.4 mm to (183.5, 122.2)
- moved D88 158.1 mm to (178.0, 114.5)
- moved D73 156.9 mm to (183.5, 109.0)
- moved D72 155.4 mm to (183.5, 106.5)
- moved D89 153.4 mm to (180.5, 114.5)
- moved D75 153.4 mm to (183.5, 117.2)
- moved D87 152.6 mm to (175.5, 114.5)
- moved D82 152.0 mm to (172.2, 119.8)
- moved D83 151.5 mm to (172.2, 117.2)
- moved D70 147.7 mm to (178.0, 103.8)
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
Commit message: include changes in moving controller to seperate sheet
Parts:
- added R1: 20, Resistor_SMD:R_0603_1608Metric, F.Cu at (37.4, 64.9)
- added R10: 20, Resistor_SMD:R_0603_1608Metric, F.Cu at (25.4, 57.4)
- added R11: 20, Resistor_SMD:R_0603_1608Metric, F.Cu at (21.3, 62.4)
- added R12: 20, Resistor_SMD:R_0603_1608Metric, F.Cu at (37.4, 57.4)
- added R13: 20, Resistor_SMD:R_0603_1608Metric, F.Cu at (21.3, 67.4)
- added R14: 20, Resistor_SMD:R_0603_1608Metric, F.Cu at (33.4, 59.9)
- added R15: 20, Resistor_SMD:R_0603_1608Metric, F.Cu at (21.3, 64.9)
- added R16: 20, Resistor_SMD:R_0603_1608Metric, F.Cu at (29.4, 67.4)
- added R17: 20, Resistor_SMD:R_0603_1608Metric, F.Cu at (33.4, 62.4)
- added R18: 20, Resistor_SMD:R_0603_1608Metric, F.Cu at (37.4, 59.9)
- added R19: 20, Resistor_SMD:R_0603_1608Metric, F.Cu at (25.4, 54.9)
- added R2: 20, Resistor_SMD:R_0603_1608Metric, F.Cu at (21.3, 69.9)
- added R20: 20, Resistor_SMD:R_0603_1608Metric, F.Cu at (37.4, 54.9)
- added R21: 20, Resistor_SMD:R_0603_1608Metric, F.Cu at (29.4, 59.9)
- added R22: 20, Resistor_SMD:R_0603_1608Metric, F.Cu at (41.4, 59.9)
- added R23: 20, Resistor_SMD:R_0603_1608Metric, F.Cu at (41.4, 62.4)
- added R24: 20, Resistor_SMD:R_0603_1608Metric, F.Cu at (45.4, 57.4)
- added R25: 20, Resistor_SMD:R_0603_1608Metric, F.Cu at (45.4, 54.9)
- added R26: 20, Resistor_SMD:R_0603_1608Metric, F.Cu at (37.4, 62.4)
- added R27: 20, Resistor_SMD:R_0603_1608Metric, F.Cu at (41.4, 54.9)
- added R28: 20, Resistor_SMD:R_0603_1608Metric, F.Cu at (25.4, 62.4)
- added R29: 20, Resistor_SMD:R_0603_1608Metric, F.Cu at (29.4, 57.4)
- added R3: 20, Resistor_SMD:R_0603_1608Metric, F.Cu at (41.4, 57.4)
- added R30: 20, Resistor_SMD:R_0603_1608Metric, F.Cu at (33.4, 69.9)
- added R31: 20, Resistor_SMD:R_0603_1608Metric, F.Cu at (33.4, 67.4)
- added R32: 20, Resistor_SMD:R_0603_1608Metric, F.Cu at (25.4, 67.4)
- added R33: 20, Resistor_SMD:R_0603_1608Metric, F.Cu at (29.4, 62.4)
- added R34: 20, Resistor_SMD:R_0603_1608Metric, F.Cu at (33.4, 64.9)
- added R35: 20, Resistor_SMD:R_0603_1608Metric, F.Cu at (25.4, 69.9)
- added R36: 20, Resistor_SMD:R_0603_1608Metric, F.Cu at (33.4, 57.4)
- added R37: 20, Resistor_SMD:R_0603_1608Metric, F.Cu at (29.4, 54.9)
- added R38: 20, Resistor_SMD:R_0603_1608Metric, F.Cu at (25.4, 59.9)
- added R39: 20, Resistor_SMD:R_0603_1608Metric, F.Cu at (29.4, 69.9)
- added R4: 20, Resistor_SMD:R_0603_1608Metric, F.Cu at (33.4, 54.9)
- added R5: 20, Resistor_SMD:R_0603_1608Metric, F.Cu at (29.4, 64.9)
- added R6: 20, Resistor_SMD:R_0603_1608Metric, F.Cu at (21.3, 54.9)
- added R7: 20, Resistor_SMD:R_0603_1608Metric, F.Cu at (21.3, 59.9)
- added R8: 20, Resistor_SMD:R_0603_1608Metric, F.Cu at (21.3, 57.4)
- added R9: 20, Resistor_SMD:R_0603_1608Metric, F.Cu at (25.4, 64.9)
Connections:
- J1 pad 5: unconnected-(J1-Pad5) -> GND
- J1 pad 6: unconnected-(J1-Pad6) -> +3V3
- J1 pad 7: unconnected-(J1-Pad7) -> +3V3
- J1 pad 8: unconnected-(J1-Pad8) -> GND

Commit message: start mapping out locations on PCB
Parts:
- added C1: 1u, Capacitor_SMD:C_0603_1608Metric, F.Cu at (76.3, 110.2)
- added C2: 0.1u, Capacitor_SMD:C_0603_1608Metric, F.Cu at (72.3, 112.7)
- added C3: 1u, Capacitor_SMD:C_0603_1608Metric, F.Cu at (67.0, 119.5)
- added C4: 0.1u, Capacitor_SMD:C_0603_1608Metric, F.Cu at (72.3, 107.7)
- added C5: 0.1u, Capacitor_SMD:C_0603_1608Metric, F.Cu at (76.3, 112.7)
- added C6: 1u, Capacitor_SMD:C_0603_1608Metric, F.Cu at (76.3, 107.7)
- added C7: 0.1u, Capacitor_SMD:C_0603_1608Metric, F.Cu at (63.0, 119.5)
- added R40: 100K, Resistor_SMD:R_0603_1608Metric, F.Cu at (71.0, 119.5)
- added R41: 100K, Resistor_SMD:R_0603_1608Metric, F.Cu at (72.3, 110.2)
- added R42: 2K, Resistor_SMD:R_0603_1608Metric, F.Cu at (67.0, 117.0)
- added R43: 2K, Resistor_SMD:R_0603_1608Metric, F.Cu at (71.0, 117.0)
- added R44: 10K, Resistor_SMD:R_0603_1608Metric, F.Cu at (63.0, 117.0)
- J1: value Conn_02x06_Counter_Clockwise -> Conn_02x06_Odd_Even
- moved D45 142.1 mm to (145.8, 148.9)
- moved D46 142.1 mm to (148.2, 156.2)
- moved R1 87.4 mm to (103.5, 122.1), turned to 90 degrees
- moved R10 47.1 mm to (62.7, 86.0)
- moved R14 47.1 mm to (70.7, 88.5)
- moved R17 47.1 mm to (70.7, 91.0)
- moved R24 47.1 mm to (82.8, 86.0)
- moved R25 47.1 mm to (82.8, 83.5)
- moved R29 47.1 mm to (66.7, 86.0)
- moved R3 47.1 mm to (78.8, 86.0)
- moved R30 47.1 mm to (70.7, 98.5)
- moved R31 47.1 mm to (70.7, 96.0)
- moved R34 47.1 mm to (70.7, 93.5)
- moved R36 47.1 mm to (70.7, 86.0)
- moved R4 47.1 mm to (70.7, 83.5)
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Connections:
- net /controller/CS37 renamed /CS37
- net /controller/CS38 renamed /CS38
- net /controller/CS39 renamed /CS39
- D1 pad 1: /Segment1/SW1 -> /SW1
- D1 pad 2: /Segment1/CS1 -> /CS1
- D1 pad 3: /Segment1/CS2 -> /CS2
- D1 pad 4: /Segment1/CS3 -> /CS3
- D10 pad 1: /Segment1/SW1 -> /SW1
- D10 pad 2: /Segment1/CS28 -> /CS28
- D10 pad 3: /Segment1/CS29 -> /CS29
- D10 pad 4: /Segment1/CS30 -> /CS30
- D11 pad 1: /Segment1/SW1 -> /SW1
- D11 pad 2: /Segment1/CS31 -> /CS31
- D11 pad 3: /Segment1/CS32 -> /CS32
- D11 pad 4: /Segment1/CS33 -> /CS33
- D12 pad 1: /Segment1/SW1 -> /SW1
- D12 pad 2: /Segment1/CS34 -> /CS34
- D12 pad 3: /Segment1/CS35 -> /CS35
- D12 pad 4: /Segment1/CS36 -> /CS36
- D13 pad 1: /Segment1/SW2 -> /SW2
- D13 pad 2: /Segment1/CS1 -> /CS1
- D13 pad 3: /Segment1/CS2 -> /CS2
- D13 pad 4: /Segment1/CS3 -> /CS3
- D14 pad 1: /Segment1/SW2 -> /SW2
- D14 pad 2: /Segment1/CS4 -> /CS4
- D14 pad 3: /Segment1/CS5 -> /CS5
- D14 pad 4: /Segment1/CS6 -> /CS6
- D15 pad 1: /Segment1/SW2 -> /SW2
- D15 pad 2: /Segment1/CS7 -> /CS7
- D15 pad 3: /Segment1/CS8 -> /CS8
- D15 pad 4: /Segment1/CS9 -> /CS9
- D16 pad 1: /Segment1/SW2 -> /SW2
- D16 pad 2: /Segment1/CS10 -> /CS10
- D16 pad 3: /Segment1/CS11 -> /CS11
- D16 pad 4: /Segment1/CS12 -> /CS12
- D17 pad 1: /Segment1/SW2 -> /SW2
- D17 pad 2: /Segment1/CS13 -> /CS13
- D17 pad 3: /Segment1/CS14 -> /CS14
- D17 pad 4: /Segment1/CS15 -> /CS15
- D18 pad 1: /Segment1/SW2 -> /SW2
- D18 pad 2: /Segment1/CS16 -> /CS16
- D18 pad 3: /Segment1/CS17 -> /CS17
- D18 pad 4: /Segment1/CS18 -> /CS18
- D19 pad 1: /Segment1/SW2 -> /SW2
- D19 pad 2: /Segment1/CS19 -> /CS19
- D19 pad 3: /Segment1/CS20 -> /CS20
- D19 pad 4: /Segment1/CS21 -> /CS21
- D2 pad 1: /Segment1/SW1 -> /SW1
- D2 pad 2: /Segment1/CS4 -> /CS4
- D2 pad 3: /Segment1/CS5 -> /CS5
- D2 pad 4: /Segment1/CS6 -> /CS6
- D20 pad 1: /Segment1/SW2 -> /SW2
- D20 pad 2: /Segment1/CS22 -> /CS22
- D20 pad 3: /Segment1/CS23 -> /CS23
- D20 pad 4: /Segment1/CS24 -> /CS24
- D21 pad 1: /Segment1/SW2 -> /SW2
- D21 pad 2: /Segment1/CS25 -> /CS25
- D21 pad 3: /Segment1/CS26 -> /CS26
- D21 pad 4: /Segment1/CS27 -> /CS27
- D22 pad 1: /Segment1/SW2 -> /SW2
- D22 pad 2: /Segment1/CS28 -> /CS28
- D22 pad 3: /Segment1/CS29 -> /CS29
- D22 pad 4: /Segment1/CS30 -> /CS30
- D23 pad 1: /Segment2/SW3 -> /SW3
- D23 pad 2: /Segment2/CS1 -> /CS1
- D23 pad 3: /Segment2/CS2 -> /CS2
- D23 pad 4: /Segment2/CS3 -> /CS3
- D24 pad 1: /Segment2/SW3 -> /SW3
- D24 pad 2: /Segment2/CS4 -> /CS4
- D24 pad 3: /Segment2/CS5 -> /CS5
- D24 pad 4: /Segment2/CS6 -> /CS6
- D25 pad 1: /Segment2/SW3 -> /SW3
- D25 pad 2: /Segment2/CS7 -> /CS7
- D25 pad 3: /Segment2/CS8 -> /CS8
- D25 pad 4: /Segment2/CS9 -> /CS9
- D26 pad 1: /Segment2/SW3 -> /SW3
- D26 pad 2: /Segment2/CS10 -> /CS10
- D26 pad 3: /Segment2/CS11 -> /CS11
- D26 pad 4: /Segment2/CS12 -> /CS12
- D27 pad 1: /Segment2/SW3 -> /SW3
- D27 pad 2: /Segment2/CS13 -> /CS13
- D27 pad 3: /Segment2/CS14 -> /CS14
- D27 pad 4: /Segment2/CS15 -> /CS15
- D28 pad 1: /Segment2/SW3 -> /SW3
- D28 pad 2: /Segment2/CS16 -> /CS16
- D28 pad 3: /Segment2/CS17 -> /CS17
- D28 pad 4: /Segment2/CS18 -> /CS18
- D29 pad 1: /Segment2/SW3 -> /SW3
- D29 pad 2: /Segment2/CS19 -> /CS19
- D29 pad 3: /Segment2/CS20 -> /CS20
- D29 pad 4: /Segment2/CS21 -> /CS21
- D3 pad 1: /Segment1/SW1 -> /SW1
- D3 pad 2: /Segment1/CS7 -> /CS7
- D3 pad 3: /Segment1/CS8 -> /CS8
- D3 pad 4: /Segment1/CS9 -> /CS9
- D30 pad 1: /Segment2/SW3 -> /SW3
- D30 pad 2: /Segment2/CS22 -> /CS22
- D30 pad 3: /Segment2/CS23 -> /CS23
- D30 pad 4: /Segment2/CS24 -> /CS24
- D31 pad 1: /Segment2/SW3 -> /SW3
- D31 pad 2: /Segment2/CS25 -> /CS25
- D31 pad 3: /Segment2/CS26 -> /CS26
- D31 pad 4: /Segment2/CS27 -> /CS27
- D32 pad 1: /Segment2/SW3 -> /SW3
- D32 pad 2: /Segment2/CS28 -> /CS28
- D32 pad 3: /Segment2/CS29 -> /CS29
- D32 pad 4: /Segment2/CS30 -> /CS30
- D33 pad 1: /Segment2/SW3 -> /SW3
- D33 pad 2: /Segment2/CS31 -> /CS31
- D33 pad 3: /Segment2/CS32 -> /CS32
- D33 pad 4: /Segment2/CS33 -> /CS33
- D34 pad 1: /Segment2/SW3 -> /SW3
- D34 pad 2: /Segment2/CS34 -> /CS34
- D34 pad 3: /Segment2/CS35 -> /CS35
- D34 pad 4: /Segment2/CS36 -> /CS36
- D35 pad 1: /Segment2/SW4 -> /SW4
- D35 pad 2: /Segment2/CS1 -> /CS1
- D35 pad 3: /Segment2/CS2 -> /CS2
- D35 pad 4: /Segment2/CS3 -> /CS3
- D36 pad 1: /Segment2/SW4 -> /SW4
- D36 pad 2: /Segment2/CS4 -> /CS4
- D36 pad 3: /Segment2/CS5 -> /CS5
- D36 pad 4: /Segment2/CS6 -> /CS6
- D37 pad 1: /Segment2/SW4 -> /SW4
- D37 pad 2: /Segment2/CS7 -> /CS7
- D37 pad 3: /Segment2/CS8 -> /CS8
- D37 pad 4: /Segment2/CS9 -> /CS9
- D38 pad 1: /Segment2/SW4 -> /SW4
- D38 pad 2: /Segment2/CS10 -> /CS10
- D38 pad 3: /Segment2/CS11 -> /CS11
- D38 pad 4: /Segment2/CS12 -> /CS12
- D39 pad 1: /Segment2/SW4 -> /SW4
- D39 pad 2: /Segment2/CS13 -> /CS13
- D39 pad 3: /Segment2/CS14 -> /CS14
- D39 pad 4: /Segment2/CS15 -> /CS15
- D4 pad 1: /Segment1/SW1 -> /SW1
- D4 pad 2: /Segment1/CS10 -> /CS10
- D4 pad 3: /Segment1/CS11 -> /CS11
- D4 pad 4: /Segment1/CS12 -> /CS12
- D40 pad 1: /Segment2/SW4 -> /SW4
- D40 pad 2: /Segment2/CS16 -> /CS16
- D40 pad 3: /Segment2/CS17 -> /CS17
- D40 pad 4: /Segment2/CS18 -> /CS18
- D41 pad 1: /Segment2/SW4 -> /SW4
- D41 pad 2: /Segment2/CS19 -> /CS19
- D41 pad 3: /Segment2/CS20 -> /CS20
- D41 pad 4: /Segment2/CS21 -> /CS21
- D42 pad 1: /Segment2/SW4 -> /SW4
- D42 pad 2: /Segment2/CS22 -> /CS22
- D42 pad 3: /Segment2/CS23 -> /CS23
- D42 pad 4: /Segment2/CS24 -> /CS24
- D43 pad 1: /Segment2/SW4 -> /SW4
- D43 pad 2: /Segment2/CS25 -> /CS25
- D43 pad 3: /Segment2/CS26 -> /CS26
- D43 pad 4: /Segment2/CS27 -> /CS27
- D44 pad 1: /Segment2/SW4 -> /SW4
- D44 pad 2: /Segment2/CS28 -> /CS28
- D44 pad 3: /Segment2/CS29 -> /CS29
- D44 pad 4: /Segment2/CS30 -> /CS30
- D45 pad 1: /Segment2/SW4 -> /SW4
- D45 pad 2: /Segment2/CS31 -> /CS31
- D45 pad 3: /Segment2/CS32 -> /CS32
- D45 pad 4: /Segment2/CS33 -> /CS33
- D46 pad 1: /Segment2/SW4 -> /SW4
- D46 pad 2: /Segment2/CS34 -> /CS34
- D46 pad 3: /Segment2/CS35 -> /CS35
- D46 pad 4: /Segment2/CS36 -> /CS36
- D47 pad 1: /Segment3/SW5 -> /SW5
- D47 pad 2: /Segment3/CS1 -> /CS1
- D47 pad 3: /Segment3/CS2 -> /CS2
- D47 pad 4: /Segment3/CS3 -> /CS3
- D48 pad 1: /Segment3/SW5 -> /SW5
- D48 pad 2: /Segment3/CS4 -> /CS4
- D48 pad 3: /Segment3/CS5 -> /CS5
- D48 pad 4: /Segment3/CS6 -> /CS6
- D49 pad 1: /Segment3/SW5 -> /SW5
- D49 pad 2: /Segment3/CS7 -> /CS7
- D49 pad 3: /Segment3/CS8 -> /CS8
- D49 pad 4: /Segment3/CS9 -> /CS9
- D5 pad 1: /Segment1/SW1 -> /SW1
- D5 pad 2: /Segment1/CS13 -> /CS13
- D5 pad 3: /Segment1/CS14 -> /CS14
- D5 pad 4: /Segment1/CS15 -> /CS15
- D50 pad 1: /Segment3/SW5 -> /SW5
- D50 pad 2: /Segment3/CS10 -> /CS10
- D50 pad 3: /Segment3/CS11 -> /CS11
- D50 pad 4: /Segment3/CS12 -> /CS12
- D51 pad 1: /Segment3/SW5 -> /SW5
- D51 pad 2: /Segment3/CS13 -> /CS13
- D51 pad 3: /Segment3/CS14 -> /CS14
- D51 pad 4: /Segment3/CS15 -> /CS15
- D52 pad 1: /Segment3/SW5 -> /SW5
- D52 pad 2: /Segment3/CS16 -> /CS16
- D52 pad 3: /Segment3/CS17 -> /CS17
- D52 pad 4: /Segment3/CS18 -> /CS18
- D53 pad 1: /Segment3/SW5 -> /SW5
- D53 pad 2: /Segment3/CS19 -> /CS19
- D53 pad 3: /Segment3/CS20 -> /CS20
- D53 pad 4: /Segment3/CS21 -> /CS21
- D54 pad 1: /Segment3/SW5 -> /SW5
- D54 pad 2: /Segment3/CS22 -> /CS22
- D54 pad 3: /Segment3/CS23 -> /CS23
- D54 pad 4: /Segment3/CS24 -> /CS24
- D55 pad 1: /Segment3/SW5 -> /SW5
- D55 pad 2: /Segment3/CS25 -> /CS25
- D55 pad 3: /Segment3/CS26 -> /CS26
- D55 pad 4: /Segment3/CS27 -> /CS27
- D56 pad 1: /Segment3/SW5 -> /SW5
- D56 pad 2: /Segment3/CS28 -> /CS28
- D56 pad 3: /Segment3/CS29 -> /CS29
- D56 pad 4: /Segment3/CS30 -> /CS30
- D57 pad 1: /Segment3/SW5 -> /SW5
- D57 pad 2: /Segment3/CS31 -> /CS31
- D57 pad 3: /Segment3/CS32 -> /CS32
- D57 pad 4: /Segment3/CS33 -> /CS33
- D58 pad 1: /Segment3/SW5 -> /SW5
- D58 pad 2: /Segment3/CS34 -> /CS34
- D58 pad 3: /Segment3/CS35 -> /CS35
- D58 pad 4: /Segment3/CS36 -> /CS36
- D59 pad 1: /Segment3/SW6 -> /SW6
- D59 pad 2: /Segment3/CS1 -> /CS1
- D59 pad 3: /Segment3/CS2 -> /CS2
- D59 pad 4: /Segment3/CS3 -> /CS3
- D6 pad 1: /Segment1/SW1 -> /SW1
- D6 pad 2: /Segment1/CS16 -> /CS16
- D6 pad 3: /Segment1/CS17 -> /CS17
- D6 pad 4: /Segment1/CS18 -> /CS18
- D60 pad 1: /Segment3/SW6 -> /SW6
- D60 pad 2: /Segment3/CS4 -> /CS4
- D60 pad 3: /Segment3/CS5 -> /CS5
- D60 pad 4: /Segment3/CS6 -> /CS6
- D61 pad 1: /Segment3/SW6 -> /SW6
- D61 pad 2: /Segment3/CS7 -> /CS7
- D61 pad 3: /Segment3/CS8 -> /CS8
- D61 pad 4: /Segment3/CS9 -> /CS9
- D62 pad 1: /Segment3/SW6 -> /SW6
- D62 pad 2: /Segment3/CS10 -> /CS10
- D62 pad 3: /Segment3/CS11 -> /CS11
- D62 pad 4: /Segment3/CS12 -> /CS12
- D63 pad 1: /Segment3/SW6 -> /SW6
- D63 pad 2: /Segment3/CS13 -> /CS13
- D63 pad 3: /Segment3/CS14 -> /CS14
- D63 pad 4: /Segment3/CS15 -> /CS15
- D64 pad 1: /Segment3/SW6 -> /SW6
- D64 pad 2: /Segment3/CS16 -> /CS16
- D64 pad 3: /Segment3/CS17 -> /CS17
- D64 pad 4: /Segment3/CS18 -> /CS18
- D65 pad 1: /Segment3/SW6 -> /SW6
- D65 pad 2: /Segment3/CS19 -> /CS19
- D65 pad 3: /Segment3/CS20 -> /CS20
- D65 pad 4: /Segment3/CS21 -> /CS21
- D66 pad 1: /Segment3/SW6 -> /SW6
- D66 pad 2: /Segment3/CS22 -> /CS22
- D66 pad 3: /Segment3/CS23 -> /CS23
- D66 pad 4: /Segment3/CS24 -> /CS24
- D67 pad 1: /Segment3/SW6 -> /SW6
- D67 pad 2: /Segment3/CS25 -> /CS25
- D67 pad 3: /Segment3/CS26 -> /CS26
- D67 pad 4: /Segment3/CS27 -> /CS27
- D68 pad 1: /Segment3/SW6 -> /SW6
- D68 pad 2: /Segment3/CS28 -> /CS28
- D68 pad 3: /Segment3/CS29 -> /CS29
- D68 pad 4: /Segment3/CS30 -> /CS30
- D69 pad 1: /Segment4/SW7 -> /SW7
- D69 pad 2: /Segment4/CS1 -> /CS1
- D69 pad 3: /Segment4/CS2 -> /CS2
- D69 pad 4: /Segment4/CS3 -> /CS3
- D7 pad 1: /Segment1/SW1 -> /SW1
- D7 pad 2: /Segment1/CS19 -> /CS19
- D7 pad 3: /Segment1/CS20 -> /CS20
- D7 pad 4: /Segment1/CS21 -> /CS21
- D70 pad 1: /Segment4/SW7 -> /SW7
- D70 pad 2: /Segment4/CS4 -> /CS4
- D70 pad 3: /Segment4/CS5 -> /CS5
- D70 pad 4: /Segment4/CS6 -> /CS6
- D71 pad 1: /Segment4/SW7 -> /SW7
- D71 pad 2: /Segment4/CS7 -> /CS7
- D71 pad 3: /Segment4/CS8 -> /CS8
- D71 pad 4: /Segment4/CS9 -> /CS9
- D72 pad 1: /Segment4/SW7 -> /SW7
- D72 pad 2: /Segment4/CS10 -> /CS10
- D72 pad 3: /Segment4/CS11 -> /CS11
- D72 pad 4: /Segment4/CS12 -> /CS12
- D73 pad 1: /Segment4/SW7 -> /SW7
- D73 pad 2: /Segment4/CS13 -> /CS13
- D73 pad 3: /Segment4/CS14 -> /CS14
- D73 pad 4: /Segment4/CS15 -> /CS15
- D74 pad 1: /Segment4/SW7 -> /SW7
- D74 pad 2: /Segment4/CS16 -> /CS16
- D74 pad 3: /Segment4/CS17 -> /CS17
- D74 pad 4: /Segment4/CS18 -> /CS18
- D75 pad 1: /Segment4/SW7 -> /SW7
- D75 pad 2: /Segment4/CS19 -> /CS19
- D75 pad 3: /Segment4/CS20 -> /CS20
- D75 pad 4: /Segment4/CS21 -> /CS21
- D76 pad 1: /Segment4/SW7 -> /SW7
- D76 pad 2: /Segment4/CS22 -> /CS22
- D76 pad 3: /Segment4/CS23 -> /CS23
- D76 pad 4: /Segment4/CS24 -> /CS24
- D77 pad 1: /Segment4/SW7 -> /SW7
- D77 pad 2: /Segment4/CS25 -> /CS25
- D77 pad 3: /Segment4/CS26 -> /CS26
- D77 pad 4: /Segment4/CS27 -> /CS27
- D78 pad 1: /Segment4/SW7 -> /SW7
- D78 pad 2: /Segment4/CS28 -> /CS28
- D78 pad 3: /Segment4/CS29 -> /CS29
- D78 pad 4: /Segment4/CS30 -> /CS30
- D79 pad 1: /Segment4/SW7 -> /SW7
- D79 pad 2: /Segment4/CS31 -> /CS31
- D79 pad 3: /Segment4/CS32 -> /CS32
- D79 pad 4: /Segment4/CS33 -> /CS33
- D8 pad 1: /Segment1/SW1 -> /SW1
- D8 pad 2: /Segment1/CS22 -> /CS22
- D8 pad 3: /Segment1/CS23 -> /CS23
- D8 pad 4: /Segment1/CS24 -> /CS24
- D80 pad 1: /Segment4/SW7 -> /SW7
- D80 pad 2: /Segment4/CS34 -> /CS34
- D80 pad 3: /Segment4/CS35 -> /CS35
- D80 pad 4: /Segment4/CS36 -> /CS36
- D81 pad 1: /Segment4/SW8 -> /SW8
- D81 pad 2: /Segment4/CS1 -> /CS1
- D81 pad 3: /Segment4/CS2 -> /CS2
- D81 pad 4: /Segment4/CS3 -> /CS3
- D82 pad 1: /Segment4/SW8 -> /SW8
- D82 pad 2: /Segment4/CS4 -> /CS4
- D82 pad 3: /Segment4/CS5 -> /CS5
- D82 pad 4: /Segment4/CS6 -> /CS6
- D83 pad 1: /Segment4/SW8 -> /SW8
- D83 pad 2: /Segment4/CS7 -> /CS7
- D83 pad 3: /Segment4/CS8 -> /CS8
- D83 pad 4: /Segment4/CS9 -> /CS9
- D84 pad 1: /Segment4/SW8 -> /SW8
- D84 pad 2: /Segment4/CS10 -> /CS10
- D84 pad 3: /Segment4/CS11 -> /CS11
- D84 pad 4: /Segment4/CS12 -> /CS12
- D85 pad 1: /Segment4/SW8 -> /SW8
- D85 pad 2: /Segment4/CS13 -> /CS13
- D85 pad 3: /Segment4/CS14 -> /CS14
- D85 pad 4: /Segment4/CS15 -> /CS15
- D86 pad 1: /Segment4/SW8 -> /SW8
- D86 pad 2: /Segment4/CS16 -> /CS16
- D86 pad 3: /Segment4/CS17 -> /CS17
- D86 pad 4: /Segment4/CS18 -> /CS18
- D87 pad 1: /Segment4/SW8 -> /SW8
- D87 pad 2: /Segment4/CS19 -> /CS19
- D87 pad 3: /Segment4/CS20 -> /CS20
- D87 pad 4: /Segment4/CS21 -> /CS21
- D88 pad 1: /Segment4/SW8 -> /SW8
- D88 pad 2: /Segment4/CS22 -> /CS22
- D88 pad 3: /Segment4/CS23 -> /CS23
- D88 pad 4: /Segment4/CS24 -> /CS24
- D89 pad 1: /Segment4/SW8 -> /SW8
- D89 pad 2: /Segment4/CS25 -> /CS25
- D89 pad 3: /Segment4/CS26 -> /CS26
- D89 pad 4: /Segment4/CS27 -> /CS27
- D9 pad 1: /Segment1/SW1 -> /SW1
- D9 pad 2: /Segment1/CS25 -> /CS25
- D9 pad 3: /Segment1/CS26 -> /CS26
- D9 pad 4: /Segment1/CS27 -> /CS27
- D90 pad 1: /Segment4/SW8 -> /SW8
- D90 pad 2: /Segment4/CS28 -> /CS28
- D90 pad 3: /Segment4/CS29 -> /CS29
- D90 pad 4: /Segment4/CS30 -> /CS30
- IC1 pad 1: unconnected-(IC1-Pad1) -> Net-(IC1-Pad1)
- IC1 pad 10: unconnected-(IC1-Pad10) -> /Controller/SCL
- IC1 pad 11: unconnected-(IC1-Pad11) -> /Controller/SDB
- IC1 pad 12: unconnected-(IC1-Pad12) -> GND
- IC1 pad 13: unconnected-(IC1-Pad13) -> Net-(IC1-Pad13)
- IC1 pad 14: unconnected-(IC1-Pad14) -> +3V3
- IC1 pad 15: unconnected-(IC1-Pad15) -> +3V3
- IC1 pad 16: unconnected-(IC1-Pad16) -> /SW1
- IC1 pad 17: unconnected-(IC1-Pad17) -> /SW2
- IC1 pad 18: unconnected-(IC1-Pad18) -> /SW3
- IC1 pad 19: unconnected-(IC1-Pad19) -> /SW4
- IC1 pad 2: unconnected-(IC1-Pad2) -> Net-(IC1-Pad2)
- IC1 pad 20: unconnected-(IC1-Pad20) -> /SW5
- IC1 pad 21: unconnected-(IC1-Pad21) -> /SW6
- IC1 pad 22: unconnected-(IC1-Pad22) -> /SW7
- IC1 pad 23: unconnected-(IC1-Pad23) -> /SW8
- IC1 pad 24: unconnected-(IC1-Pad24) -> /SW9
- IC1 pad 25: unconnected-(IC1-Pad25) -> +3V3
- IC1 pad 26: unconnected-(IC1-Pad26) -> Net-(IC1-Pad26)
- IC1 pad 27: unconnected-(IC1-Pad27) -> Net-(IC1-Pad27)
- IC1 pad 28: unconnected-(IC1-Pad28) -> Net-(IC1-Pad28)
- IC1 pad 29: unconnected-(IC1-Pad29) -> Net-(IC1-Pad29)
- IC1 pad 3: unconnected-(IC1-Pad3) -> Net-(IC1-Pad3)
- IC1 pad 30: unconnected-(IC1-Pad30) -> Net-(IC1-Pad30)
- IC1 pad 31: unconnected-(IC1-Pad31) -> Net-(IC1-Pad31)
- IC1 pad 32: unconnected-(IC1-Pad32) -> Net-(IC1-Pad32)
- IC1 pad 33: unconnected-(IC1-Pad33) -> Net-(IC1-Pad33)
- IC1 pad 34: unconnected-(IC1-Pad34) -> Net-(IC1-Pad34)
- IC1 pad 35: unconnected-(IC1-Pad35) -> Net-(IC1-Pad35)
- IC1 pad 36: unconnected-(IC1-Pad36) -> GND
- IC1 pad 37: unconnected-(IC1-Pad37) -> Net-(IC1-Pad37)
- IC1 pad 38: unconnected-(IC1-Pad38) -> Net-(IC1-Pad38)
- IC1 pad 39: unconnected-(IC1-Pad39) -> Net-(IC1-Pad39)
- IC1 pad 4: unconnected-(IC1-Pad4) -> Net-(IC1-Pad4)
- IC1 pad 40: unconnected-(IC1-Pad40) -> Net-(IC1-Pad40)
- IC1 pad 41: unconnected-(IC1-Pad41) -> Net-(IC1-Pad41)
- IC1 pad 42: unconnected-(IC1-Pad42) -> Net-(IC1-Pad42)
- IC1 pad 43: unconnected-(IC1-Pad43) -> Net-(IC1-Pad43)
- IC1 pad 44: unconnected-(IC1-Pad44) -> Net-(IC1-Pad44)
- IC1 pad 45: unconnected-(IC1-Pad45) -> Net-(IC1-Pad45)
- IC1 pad 46: unconnected-(IC1-Pad46) -> Net-(IC1-Pad46)
- IC1 pad 47: unconnected-(IC1-Pad47) -> Net-(IC1-Pad47)
- IC1 pad 48: unconnected-(IC1-Pad48) -> Net-(IC1-Pad48)
- IC1 pad 49: unconnected-(IC1-Pad49) -> Net-(IC1-Pad49)
- IC1 pad 5: unconnected-(IC1-Pad5) -> Net-(IC1-Pad5)
- IC1 pad 50: unconnected-(IC1-Pad50) -> Net-(IC1-Pad50)
- IC1 pad 51: unconnected-(IC1-Pad51) -> Net-(IC1-Pad51)
- IC1 pad 52: unconnected-(IC1-Pad52) -> Net-(IC1-Pad52)
- IC1 pad 53: unconnected-(IC1-Pad53) -> Net-(IC1-Pad53)
- IC1 pad 54: unconnected-(IC1-Pad54) -> Net-(IC1-Pad54)
- IC1 pad 55: unconnected-(IC1-Pad55) -> GND
- IC1 pad 56: unconnected-(IC1-Pad56) -> Net-(IC1-Pad56)
- IC1 pad 57: unconnected-(IC1-Pad57) -> Net-(IC1-Pad57)
- IC1 pad 58: unconnected-(IC1-Pad58) -> Net-(IC1-Pad58)
- IC1 pad 59: unconnected-(IC1-Pad59) -> Net-(IC1-Pad59)
- IC1 pad 6: unconnected-(IC1-Pad6) -> Net-(IC1-Pad6)
- IC1 pad 60: unconnected-(IC1-Pad60) -> Net-(IC1-Pad60)
- IC1 pad 61: unconnected-(IC1-Pad61) -> GND
- IC1 pad 7: unconnected-(IC1-Pad7) -> /Controller/INTB
- IC1 pad 8: unconnected-(IC1-Pad8) -> GND
- IC1 pad 9: unconnected-(IC1-Pad9) -> /Controller/SDA
- J1 pad 10: unconnected-(J1-Pad10) -> GND
- J1 pad 11: unconnected-(J1-Pad11) -> +3V3
- J1 pad 12: unconnected-(J1-Pad12) -> +3V3
- J1 pad 5: GND -> /Controller/SDB
- J1 pad 6: +3V3 -> /Controller/INTB
- J1 pad 7: +3V3 -> /Controller/SDA
- J1 pad 8: GND -> /Controller/SCL
- J1 pad 9: unconnected-(J1-Pad9) -> GND
- R1 pad 2: /controller/CS1 -> /CS1
- R10 pad 2: /controller/CS10 -> /CS10
- R11 pad 2: /controller/CS11 -> /CS11
- R12 pad 2: /controller/CS12 -> /CS12
- R13 pad 2: /controller/CS13 -> /CS13
- R14 pad 2: /controller/CS14 -> /CS14
- R15 pad 2: /controller/CS15 -> /CS15
- R16 pad 2: /controller/CS16 -> /CS16
- R17 pad 2: /controller/CS17 -> /CS17
- R18 pad 2: /controller/CS18 -> /CS18
- R19 pad 2: /controller/CS19 -> /CS19
- R2 pad 2: /controller/CS2 -> /CS2
- R20 pad 2: /controller/CS20 -> /CS20
- R21 pad 2: /controller/CS21 -> /CS21
- R22 pad 2: /controller/CS22 -> /CS22
- R23 pad 2: /controller/CS23 -> /CS23
- R24 pad 2: /controller/CS24 -> /CS24
- R25 pad 2: /controller/CS25 -> /CS25
- R26 pad 2: /controller/CS26 -> /CS26
- R27 pad 2: /controller/CS27 -> /CS27
- R28 pad 2: /controller/CS28 -> /CS28
- R29 pad 2: /controller/CS29 -> /CS29
- R3 pad 2: /controller/CS3 -> /CS3
- R30 pad 2: /controller/CS30 -> /CS30
- R31 pad 2: /controller/CS31 -> /CS31
- R32 pad 2: /controller/CS32 -> /CS32
- R33 pad 2: /controller/CS33 -> /CS33
- R34 pad 2: /controller/CS34 -> /CS34
- R35 pad 2: /controller/CS35 -> /CS35
- R36 pad 2: /controller/CS36 -> /CS36
- R4 pad 2: /controller/CS4 -> /CS4
- R5 pad 2: /controller/CS5 -> /CS5
- R6 pad 2: /controller/CS6 -> /CS6
- R7 pad 2: /controller/CS7 -> /CS7
- R8 pad 2: /controller/CS8 -> /CS8
- R9 pad 2: /controller/CS9 -> /CS9
Routing:
- net /SW1: track 0.00 -> 52.6 mm
- net /SW2: track 0.00 -> 34.5 mm
- net /CS5: track 0.00 -> 27.5 mm, vias 0 -> 4
- net /CS6: track 0.00 -> 27.2 mm, vias 0 -> 4
- net /CS9: track 0.00 -> 26.8 mm, vias 0 -> 4
- net /CS3: track 0.00 -> 26.8 mm, vias 0 -> 4
- net /CS4: track 0.00 -> 26.5 mm, vias 0 -> 4
- net /CS1: track 0.00 -> 26.3 mm, vias 0 -> 4
- net /CS2: track 0.00 -> 25.9 mm, vias 0 -> 4
- net /CS8: track 0.00 -> 25.5 mm, vias 0 -> 4
- net /CS7: track 0.00 -> 25.0 mm, vias 0 -> 4

Commit message: changes to the LED connection ordering
Parts:
- moved D35 16.0 mm to (132.5, 106.7)
- moved D13 15.2 mm to (112.2, 107.0)
- moved D18 11.3 mm to (120.5, 114.5)
- moved D21 11.3 mm to (112.2, 122.2)
- moved D36 11.1 mm to (132.5, 108.9)
- moved D43 11.0 mm to (132.4, 122.2)
- moved D40 10.9 mm to (140.3, 114.6)
- moved D14 10.8 mm to (112.2, 109.0)
- moved D17 7.96 mm to (118.0, 114.5)
- moved D20 7.79 mm to (112.2, 119.8)
- moved D42 7.47 mm to (132.5, 119.8)
- moved D39 7.46 mm to (137.7, 114.6)
- moved D37 6.23 mm to (132.5, 111.3)
- moved D15 6.00 mm to (112.2, 111.2)
- moved D16 4.42 mm to (115.5, 114.5)
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Routing:
- net /SW2: track 34.5 -> 3.89 mm
- net /CS12: track 0.00 -> 27.0 mm
- net /CS10: track 0.00 -> 24.3 mm
- net /CS17: track 0.00 -> 13.7 mm
- net /CS11: track 0.00 -> 11.6 mm
- net /CS2: track 25.9 -> 15.9 mm, vias 4 -> 0
- net /CS13: track 0.00 -> 9.94 mm
- net /CS15: track 0.00 -> 8.93 mm
- net /CS3: track 26.8 -> 18.6 mm, vias 4 -> 0
- net /CS1: track 26.3 -> 19.0 mm, vias 4 -> 0
- net /CS5: track 27.5 -> 20.6 mm, vias 4 -> 0
- net /CS14: track 0.00 -> 4.87 mm
- net /CS16: track 0.00 -> 4.50 mm
- net /CS7: track 25.0 -> 29.4 mm, vias 4 -> 0
- net /CS18: track 0.00 -> 3.82 mm
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Other:
- copper layers 2 -> 4

Commit message: update PCB with the schematic for first display
Parts:
- moved D21 11.4 mm to (120.6, 114.5)
- moved D13 10.5 mm to (112.3, 117.5)
- moved D14 10.5 mm to (112.3, 119.5)
- moved D15 10.5 mm to (112.3, 121.7)
- moved D18 8.71 mm to (112.4, 111.3)
- moved D16 8.35 mm to (112.4, 106.8)
- moved D20 7.94 mm to (118.2, 114.5)
- moved D17 7.85 mm to (112.4, 109.0)
- moved D19 4.32 mm to (115.6, 114.5)
Connections:
- D1 pad 1: /SW1 -> /SW4
- D10 pad 2: /CS28 -> /CS7
- D10 pad 3: /CS29 -> /CS8
- D10 pad 4: /CS30 -> /CS9
- D11 pad 1: /SW1 -> /SW2
- D11 pad 2: /CS31 -> /CS7
- D11 pad 3: /CS32 -> /CS8
- D11 pad 4: /CS33 -> /CS9
- D12 pad 1: /SW1 -> /SW3
- D12 pad 2: /CS34 -> /CS7
- D12 pad 3: /CS35 -> /CS8
- D12 pad 4: /CS36 -> /CS9
- D13 pad 1: /SW2 -> /SW1
- D13 pad 2: /CS1 -> /CS4
- D13 pad 3: /CS2 -> /CS5
- D13 pad 4: /CS3 -> /CS6
- D15 pad 1: /SW2 -> /SW3
- D15 pad 2: /CS7 -> /CS4
- D15 pad 3: /CS8 -> /CS5
- D15 pad 4: /CS9 -> /CS6
- D16 pad 1: /SW2 -> /SW1
- D16 pad 2: /CS10 -> /CS1
- D16 pad 3: /CS11 -> /CS2
- D16 pad 4: /CS12 -> /CS3
- D17 pad 2: /CS13 -> /CS1
- D17 pad 3: /CS14 -> /CS2
- D17 pad 4: /CS15 -> /CS3
- D18 pad 1: /SW2 -> /SW3
- D18 pad 2: /CS16 -> /CS1
- D18 pad 3: /CS17 -> /CS2
- D18 pad 4: /CS18 -> /CS3
- D19 pad 1: /SW2 -> /SW4
- D19 pad 2: /CS19 -> /CS4
- D19 pad 3: /CS20 -> /CS5
- D19 pad 4: /CS21 -> /CS6
- D2 pad 1: /SW1 -> /SW5
- D2 pad 2: /CS4 -> /CS1
- D2 pad 3: /CS5 -> /CS2
- D2 pad 4: /CS6 -> /CS3
- D20 pad 1: /SW2 -> /SW5
- D20 pad 2: /CS22 -> /CS4
- D20 pad 3: /CS23 -> /CS5
- D20 pad 4: /CS24 -> /CS6
- D21 pad 1: /SW2 -> /SW6
- D21 pad 2: /CS25 -> /CS4
- D21 pad 3: /CS26 -> /CS5
- D21 pad 4: /CS27 -> /CS6
- D22 pad 1: /SW2 -> /SW4
- D22 pad 2: /CS28 -> /CS7
- D22 pad 3: /CS29 -> /CS8
- D22 pad 4: /CS30 -> /CS9
- D3 pad 1: /SW1 -> /SW6
- D3 pad 2: /CS7 -> /CS1
- D3 pad 3: /CS8 -> /CS2
- D3 pad 4: /CS9 -> /CS3
- D4 pad 1: /SW1 -> /SW7
- D4 pad 2: /CS10 -> /CS1
- D4 pad 3: /CS11 -> /CS2
- D4 pad 4: /CS12 -> /CS3
- D5 pad 1: /SW1 -> /SW8
- D5 pad 2: /CS13 -> /CS1
- D5 pad 3: /CS14 -> /CS2
- D5 pad 4: /CS15 -> /CS3
- D6 pad 1: /SW1 -> /SW9
- D6 pad 2: /CS16 -> /CS1
- D6 pad 3: /CS17 -> /CS2
- D6 pad 4: /CS18 -> /CS3
- D7 pad 1: /SW1 -> /SW7
- D7 pad 2: /CS19 -> /CS4
- D7 pad 3: /CS20 -> /CS5
- D7 pad 4: /CS21 -> /CS6
- D8 pad 1: /SW1 -> /SW8
- D8 pad 2: /CS22 -> /CS4
- D8 pad 3: /CS23 -> /CS5
- D8 pad 4: /CS24 -> /CS6
- D9 pad 1: /SW1 -> /SW9
- D9 pad 2: /CS25 -> /CS4
- D9 pad 3: /CS26 -> /CS5
- D9 pad 4: /CS27 -> /CS6
Routing:
- net /SW1: track 50.0 -> 1.23 mm, vias 0 -> 1
- net /CS7: track 29.4 -> 0.00 mm
- net /CS3: track 18.6 -> 46.8 mm, vias 0 -> 2
- net /CS9: track 28.1 -> 0.05 mm
- net /CS12: track 27.0 -> 0.00 mm
- net /CS8: track 25.7 -> 0.00 mm
- net /CS2: track 15.9 -> 41.2 mm, vias 0 -> 9
- net /CS4: track 24.5 -> 0.01 mm
- net /CS10: track 24.3 -> 0.00 mm
- net /CS6: track 23.7 -> 0.11 mm
- net /CS5: track 20.6 -> 0.00 mm
- net /CS1: track 19.0 -> 39.2 mm
- net /CS17: track 13.7 -> 0.00 mm
- net /CS11: track 11.6 -> 0.00 mm
- net /SW5: track 0.00 -> 11.3 mm, vias 0 -> 1
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