File: PMOD_RGB7Segment/Hardware/PMod_RGB7Segment.kicad_pcb (KiCad board)
At the start: 4 copper layers, 100 x 98 mm, 195 parts, among them IC1 IS31FL3741A-QFLS4-TR, J1 Conn_02x06_Odd_Even

Commit message: update PCB from the segment pin changes
Connections:
- D23 pad 1: /SW3 -> /SW4
- D23 pad 2: /CS1 -> /CS10
- D23 pad 3: /CS2 -> /CS11
- D23 pad 4: /CS3 -> /CS12
- D24 pad 1: /SW3 -> /SW5
- D24 pad 2: /CS4 -> /CS10
- D24 pad 3: /CS5 -> /CS11
- D24 pad 4: /CS6 -> /CS12
- D25 pad 1: /SW3 -> /SW6
- D25 pad 2: /CS7 -> /CS10
- D25 pad 3: /CS8 -> /CS11
- D25 pad 4: /CS9 -> /CS12
- D26 pad 1: /SW3 -> /SW7
- D27 pad 1: /SW3 -> /SW8
- D27 pad 2: /CS13 -> /CS10
- D27 pad 3: /CS14 -> /CS11
- D27 pad 4: /CS15 -> /CS12
- D28 pad 1: /SW3 -> /SW9
- D28 pad 2: /CS16 -> /CS10
- D28 pad 3: /CS17 -> /CS11
- D28 pad 4: /CS18 -> /CS12
- D29 pad 1: /SW3 -> /SW7
- D29 pad 2: /CS19 -> /CS13
- D29 pad 3: /CS20 -> /CS14
- D29 pad 4: /CS21 -> /CS15
- D30 pad 1: /SW3 -> /SW8
- D30 pad 2: /CS22 -> /CS13
- D30 pad 3: /CS23 -> /CS14
- D30 pad 4: /CS24 -> /CS15
- D31 pad 1: /SW3 -> /SW9
- D31 pad 2: /CS25 -> /CS13
- D31 pad 3: /CS26 -> /CS14
- D31 pad 4: /CS27 -> /CS15
- D32 pad 1: /SW3 -> /SW1
- D32 pad 2: /CS28 -> /CS16
- D32 pad 3: /CS29 -> /CS17
- D32 pad 4: /CS30 -> /CS18
- D33 pad 1: /SW3 -> /SW2
- D33 pad 2: /CS31 -> /CS16
- D33 pad 3: /CS32 -> /CS17
- D33 pad 4: /CS33 -> /CS18
- D34 pad 2: /CS34 -> /CS16
- D34 pad 3: /CS35 -> /CS17
- D34 pad 4: /CS36 -> /CS18
- D35 pad 1: /SW4 -> /SW1
- D35 pad 2: /CS1 -> /CS13
- D35 pad 3: /CS2 -> /CS14
- D35 pad 4: /CS3 -> /CS15
- D36 pad 1: /SW4 -> /SW2
- D36 pad 2: /CS4 -> /CS13
- D36 pad 3: /CS5 -> /CS14
- D36 pad 4: /CS6 -> /CS15
- D37 pad 1: /SW4 -> /SW3
- D37 pad 2: /CS7 -> /CS13
- D37 pad 3: /CS8 -> /CS14
- D37 pad 4: /CS9 -> /CS15
- D38 pad 1: /SW4 -> /SW1
- D39 pad 1: /SW4 -> /SW2
- D39 pad 2: /CS13 -> /CS10
- D39 pad 3: /CS14 -> /CS11
- D39 pad 4: /CS15 -> /CS12
- D40 pad 1: /SW4 -> /SW3
- D40 pad 2: /CS16 -> /CS10
- D40 pad 3: /CS17 -> /CS11
- D40 pad 4: /CS18 -> /CS12
- D41 pad 2: /CS19 -> /CS13
- D41 pad 3: /CS20 -> /CS14
- D41 pad 4: /CS21 -> /CS15
- D42 pad 1: /SW4 -> /SW5
- D42 pad 2: /CS22 -> /CS13
- D42 pad 3: /CS23 -> /CS14
- D42 pad 4: /CS24 -> /CS15
- D43 pad 1: /SW4 -> /SW6
- D44 pad 2: /CS28 -> /CS16
- D44 pad 3: /CS29 -> /CS17
- D44 pad 4: /CS30 -> /CS18
- D45 pad 1: /SW4 -> /SW5
- D45 pad 2: /CS31 -> /CS16
- D45 pad 3: /CS32 -> /CS17
- D45 pad 4: /CS33 -> /CS18
- D46 pad 1: /SW4 -> /SW6
- D46 pad 2: /CS34 -> /CS16
- D46 pad 3: /CS35 -> /CS17
- D46 pad 4: /CS36 -> /CS18
- D47 pad 1: /SW5 -> /SW4
- D47 pad 2: /CS1 -> /CS19
- D47 pad 3: /CS2 -> /CS20
- D47 pad 4: /CS3 -> /CS21
- D48 pad 2: /CS4 -> /CS19
- D48 pad 3: /CS5 -> /CS20
- D48 pad 4: /CS6 -> /CS21
- D49 pad 1: /SW5 -> /SW6
- D49 pad 2: /CS7 -> /CS19
- D49 pad 3: /CS8 -> /CS20
- D49 pad 4: /CS9 -> /CS21
- D50 pad 1: /SW5 -> /SW7
- D50 pad 2: /CS10 -> /CS19
- D50 pad 3: /CS11 -> /CS20
- D50 pad 4: /CS12 -> /CS21
- D51 pad 1: /SW5 -> /SW8
- D51 pad 2: /CS13 -> /CS19
- D51 pad 3: /CS14 -> /CS20
- D51 pad 4: /CS15 -> /CS21
- D52 pad 1: /SW5 -> /SW9
- D52 pad 2: /CS16 -> /CS19
- D52 pad 3: /CS17 -> /CS20
- D52 pad 4: /CS18 -> /CS21
- D53 pad 1: /SW5 -> /SW7
- D53 pad 2: /CS19 -> /CS22
- D53 pad 3: /CS20 -> /CS23
- D53 pad 4: /CS21 -> /CS24
- D54 pad 1: /SW5 -> /SW8
- D55 pad 1: /SW5 -> /SW9
- D55 pad 2: /CS25 -> /CS22
- D55 pad 3: /CS26 -> /CS23
- D55 pad 4: /CS27 -> /CS24
- D56 pad 1: /SW5 -> /SW1
- D56 pad 2: /CS28 -> /CS25
- D56 pad 3: /CS29 -> /CS26
- D56 pad 4: /CS30 -> /CS27
- D57 pad 1: /SW5 -> /SW2
- D57 pad 2: /CS31 -> /CS25
- D57 pad 3: /CS32 -> /CS26
- D57 pad 4: /CS33 -> /CS27
- D58 pad 1: /SW5 -> /SW3
- D58 pad 2: /CS34 -> /CS25
- D58 pad 3: /CS35 -> /CS26
- D58 pad 4: /CS36 -> /CS27
- D59 pad 1: /SW6 -> /SW1
- D59 pad 2: /CS1 -> /CS22
- D59 pad 3: /CS2 -> /CS23
- D59 pad 4: /CS3 -> /CS24
- D60 pad 1: /SW6 -> /SW2
- D60 pad 2: /CS4 -> /CS22
- D60 pad 3: /CS5 -> /CS23
- D60 pad 4: /CS6 -> /CS24
- D61 pad 1: /SW6 -> /SW3
- D61 pad 2: /CS7 -> /CS22
- D61 pad 3: /CS8 -> /CS23
- D61 pad 4: /CS9 -> /CS24
- D62 pad 1: /SW6 -> /SW1
- D62 pad 2: /CS10 -> /CS19
- D62 pad 3: /CS11 -> /CS20
- D62 pad 4: /CS12 -> /CS21
- D63 pad 1: /SW6 -> /SW2
- D64 pad 1: /SW6 -> /SW3
- D65 pad 1: /SW6 -> /SW4
- D65 pad 2: /CS19 -> /CS22
- D65 pad 3: /CS20 -> /CS23
- D65 pad 4: /CS21 -> /CS24
- D66 pad 1: /SW6 -> /SW5
- D67 pad 2: /CS25 -> /CS22
- D67 pad 3: /CS26 -> /CS23
- D67 pad 4: /CS27 -> /CS24
- D68 pad 1: /SW6 -> /SW4
- D68 pad 2: /CS28 -> /CS25
- D68 pad 3: /CS29 -> /CS26
- D68 pad 4: /CS30 -> /CS27
- D69 pad 1: /SW7 -> /SW4
- D69 pad 2: /CS1 -> /CS28
- D69 pad 3: /CS2 -> /CS29
- D69 pad 4: /CS3 -> /CS30
- D70 pad 1: /SW7 -> /SW5
- D70 pad 2: /CS4 -> /CS28
- D70 pad 3: /CS5 -> /CS29
- D70 pad 4: /CS6 -> /CS20
- D71 pad 1: /SW7 -> /SW6
- D71 pad 2: /CS7 -> /CS28
- D71 pad 3: /CS8 -> /CS29
- D71 pad 4: /CS9 -> /CS30
- D72 pad 2: /CS10 -> /CS28
- D72 pad 3: /CS11 -> /CS29
- D72 pad 4: /CS12 -> /CS30
- D73 pad 1: /SW7 -> /SW8
- D73 pad 2: /CS13 -> /CS28
- D73 pad 3: /CS14 -> /CS29
- D73 pad 4: /CS15 -> /CS30
- D74 pad 1: /SW7 -> /SW9
- D74 pad 2: /CS16 -> /CS28
- D74 pad 3: /CS17 -> /CS29
- D74 pad 4: /CS18 -> /CS30
- D75 pad 2: /CS19 -> /CS31
- D75 pad 3: /CS20 -> /CS32
- D75 pad 4: /CS21 -> /Segment4/33
- D76 pad 1: /SW7 -> /SW8
- D76 pad 2: /CS22 -> /CS31
- D76 pad 3: /CS23 -> /CS32
- D76 pad 4: /CS24 -> /CS33
- D77 pad 1: /SW7 -> /SW9
- D77 pad 2: /CS25 -> /CS31
- D77 pad 3: /CS26 -> /CS32
- D77 pad 4: /CS27 -> /CS33
- D78 pad 1: /SW7 -> /SW1
- D78 pad 2: /CS28 -> /CS34
- D78 pad 3: /CS29 -> /CS35
- D78 pad 4: /CS30 -> /CS36
- D79 pad 1: /SW7 -> /SW2
- D79 pad 2: /CS31 -> /CS34
- D79 pad 3: /CS32 -> /CS35
- D79 pad 4: /CS33 -> /CS36
- D80 pad 1: /SW7 -> /SW3
- D81 pad 1: /SW8 -> /SW1
- D81 pad 2: /CS1 -> /CS31
- D81 pad 3: /CS2 -> /CS32
- D81 pad 4: /CS3 -> /CS33
- D82 pad 1: /SW8 -> /SW2
- D82 pad 2: /CS4 -> /CS31
- D82 pad 3: /CS5 -> /CS32
- D82 pad 4: /CS6 -> /CS33
- D83 pad 1: /SW8 -> /SW3
- D83 pad 2: /CS7 -> /CS31
- D83 pad 3: /CS8 -> /CS32
- D83 pad 4: /CS9 -> /CS33
- D84 pad 1: /SW8 -> /SW1
- D84 pad 2: /CS10 -> /CS28
- D84 pad 3: /CS11 -> /CS29
- D84 pad 4: /CS12 -> /CS30
- D85 pad 1: /SW8 -> /SW2
- D85 pad 2: /CS13 -> /CS28
- D85 pad 3: /CS14 -> /CS29
- D85 pad 4: /CS15 -> /CS30
- D86 pad 1: /SW8 -> /SW3
- D86 pad 2: /CS16 -> /CS28
- D86 pad 3: /CS17 -> /CS29
- D86 pad 4: /CS18 -> /CS30
- D87 pad 1: /SW8 -> /SW4
- D87 pad 2: /CS19 -> /CS31
- D87 pad 3: /CS20 -> /CS32
- D87 pad 4: /CS21 -> /CS33
- D88 pad 1: /SW8 -> /SW5
- D88 pad 2: /CS22 -> /CS31
- D88 pad 3: /CS23 -> /CS32
- D88 pad 4: /CS24 -> /CS33
- D89 pad 1: /SW8 -> /SW6
- D89 pad 2: /CS25 -> /CS31
- D89 pad 3: /CS26 -> /CS32
- D89 pad 4: /CS27 -> /CS33
- D90 pad 1: /SW8 -> /SW4
- D90 pad 2: /CS28 -> /CS34
- D90 pad 3: /CS29 -> /CS35
- D90 pad 4: /CS30 -> /CS36

Commit message: correct pins in schematic and continue LED layout on PCB
Parts:
- moved D43 11.0 mm to (140.2, 114.5)
- moved D35 11.0 mm to (132.2, 117.7)
- moved D36 11.0 mm to (132.2, 119.9)
- moved D37 11.0 mm to (132.2, 122.2)
- moved D40 8.47 mm to (132.5, 111.3)
- moved D38 8.38 mm to (132.4, 106.7)
- moved D39 7.78 mm to (132.4, 108.9)
- moved D42 7.46 mm to (137.8, 114.5)
- moved D41 3.92 mm to (135.2, 114.5)
Connections:
- D43 pad 2: /CS25 -> /CS13
- D43 pad 3: /CS26 -> /CS14
- D43 pad 4: /CS27 -> /CS15
- D63 pad 2: /CS13 -> /CS19
- D63 pad 3: /CS14 -> /CS20
- D63 pad 4: /CS15 -> /CS21
- D64 pad 2: /CS16 -> /CS19
- D64 pad 3: /CS17 -> /CS20
- D64 pad 4: /CS18 -> /CS21
- D70 pad 4: /CS20 -> /CS30
Routing:
- net /SW1: track 1.23 -> 48.4 mm, vias 1 -> 5
- net /SW3: track 1.25 -> 47.8 mm, vias 1 -> 5
- net /SW2: track 1.35 -> 47.8 mm, vias 1 -> 5
- net /SW9: track 1.13 -> 46.4 mm, vias 1 -> 4
- net /SW7: track 1.13 -> 46.3 mm, vias 1 -> 4
- net /SW8: track 1.08 -> 45.8 mm, vias 1 -> 4
- net /CS13: track 0.00 -> 41.0 mm
- net /CS12: track 0.00 -> 40.9 mm, vias 0 -> 2
- net /CS15: track 0.00 -> 40.5 mm, vias 0 -> 2
- net /CS6: track 0.10 -> 39.6 mm, vias 0 -> 2
- net /CS4: track 0.01 -> 39.4 mm
- net /CS10: track 0.00 -> 38.5 mm
- net /CS11: track 0.00 -> 36.9 mm, vias 0 -> 9
- net /CS14: track 0.00 -> 35.0 mm, vias 0 -> 9
- net /CS5: track 0.00 -> 34.4 mm, vias 0 -> 9
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