File: PMOD_RGB7Segment/Hardware/PMod_RGB7Segment.kicad_pcb (KiCad board)
At the start: 4 copper layers, 100 x 98 mm, 195 parts, among them IC1 IS31FL3741A-QFLS4-TR, J1 Conn_02x06_Odd_Even

Commit message: continue with placement and layout of digits
Parts:
- moved R36 138.6 mm to (171.9, 180.7)
- moved R35 133.8 mm to (171.7, 176.1)
- moved R33 129.9 mm to (172.1, 167.0)
- moved R32 128.0 mm to (172.0, 162.7)
- moved R34 127.7 mm to (171.8, 171.5)
- moved R29 123.0 mm to (172.1, 149.4)
- moved R28 122.2 mm to (172.2, 145.2)
- moved R27 121.6 mm to (153.5, 179.4)
- moved R31 119.0 mm to (172.0, 158.5)
- moved R30 115.4 mm to (171.9, 154.0)
- moved R26 115.0 mm to (153.7, 174.6)
- moved R25 112.3 mm to (153.8, 170.4)
- moved R19 110.3 mm to (154.4, 144.8)
- moved R21 109.1 mm to (154.1, 153.8)
- moved R18 108.2 mm to (138.5, 175.9)
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Connections:
- D62 pad 1: /SW1 -> /SW3
- D64 pad 1: /SW3 -> /SW1
- D75 pad 4: /Segment4/33 -> /CS33
- D84 pad 1: /SW1 -> /SW3
- D86 pad 1: /SW3 -> /SW1
Routing:
- net /SW4: track 26.7 -> 233.5 mm, vias 5 -> 11
- net /SW6: track 35.0 -> 163.6 mm, vias 5 -> 9
- net /SW5: track 31.3 -> 155.0 mm, vias 5 -> 9
- net /SW1: track 48.4 -> 166.9 mm, vias 5 -> 12
- net /SW2: track 47.8 -> 153.0 mm, vias 5 -> 12
- net /SW3: track 47.8 -> 144.0 mm, vias 5 -> 12
- net /SW9: track 46.4 -> 135.7 mm, vias 4 -> 8
- net /SW8: track 45.8 -> 134.3 mm, vias 4 -> 8
- net /SW7: track 46.3 -> 134.6 mm, vias 4 -> 8
- net /CS33: track 0.00 -> 43.5 mm, vias 0 -> 2
- net /CS21: track 0.07 -> 42.3 mm, vias 0 -> 6
- net /CS19: track 0.00 -> 41.6 mm
- net /CS31: track 0.00 -> 41.1 mm
- net /CS22: track 0.00 -> 41.0 mm
- net /CS20: track 0.00 -> 39.2 mm, vias 0 -> 6
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
Commit message: change 20ohms resistors to 4 way resistor arrays
Parts:
- removed R1, R10, R11, R12, R13, R14, R15, R16, R17, R18, R19, R2, R20, R21, R22, R23, R24, R25, R26, R27, R28, R29, R3, R30, R31, R32, R33, R34, R35, R36, R4, R5, R6, R7, R8, R9: 20, Resistor_SMD:R_0603_1608Metric
- added RN1: EXB38V472JV, jjh:EXB38V472JV, B.Cu at (110.2, 102.6)
- added RN2: EXB38V472JV, jjh:EXB38V472JV, B.Cu at (110.0, 126.0)
- added RN3: EXB38V472JV, jjh:EXB38V472JV, F.Cu at (135.0, 156.0)
- added RN4: EXB38V472JV, jjh:EXB38V472JV, F.Cu at (136.0, 164.0)
- added RN5: EXB38V472JV, jjh:EXB38V472JV, F.Cu at (118.0, 165.0)
- added RN6: EXB38V472JV, jjh:EXB38V472JV, F.Cu at (155.0, 156.0)
- added RN7: EXB38V472JV, jjh:EXB38V472JV, F.Cu at (155.6, 168.2)
- added RN8: EXB38V472JV, jjh:EXB38V472JV, F.Cu at (172.0, 167.0)
- added RN9: EXB38V472JV, jjh:EXB38V472JV, F.Cu at (174.0, 156.0)
Connections:
- IC1 pad 4: Net-(IC1-Pad4) -> unconnected-(IC1-Pad4)
- IC1 pad 5: Net-(IC1-Pad5) -> unconnected-(IC1-Pad5)
- IC1 pad 6: Net-(IC1-Pad6) -> unconnected-(IC1-Pad6)
Routing:
- net /SW2: track 153.0 -> 192.4 mm, vias 12 -> 13
- net /SW9: track 135.7 -> 164.4 mm, vias 8 -> 9
- net /SW5: track 155.0 -> 181.4 mm, vias 9 -> 10
- net /SW8: track 134.3 -> 160.4 mm, vias 8 -> 9
- net /SW4: track 233.5 -> 258.8 mm, vias 11 -> 12
- net /SW6: track 163.6 -> 188.3 mm, vias 9 -> 10
- net /SW7: track 134.6 -> 158.8 mm, vias 8 -> 9
- net /CS4: track 39.4 -> 60.6 mm, vias 0 -> 1
- net /CS1: track 39.2 -> 59.9 mm, vias 0 -> 1
- net /SW3: track 144.0 -> 160.3 mm, vias 12 -> 13
- net /SW1: track 166.9 -> 183.2 mm, vias 12 -> 13
- net /CS6: track 39.6 -> 49.6 mm, vias 2 -> 3
- net /CS5: track 34.4 -> 41.4 mm, vias 9 -> 11
- net /CS7: track 16.6 -> 22.4 mm
- net /CS8: track 18.2 -> 23.1 mm, vias 0 -> 1
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
Commit message: PCB layout continued, not completed
Parts:
- removed the G*** at (120.0, 46.8)
- removed the G*** at (180.0, 81.0)
- removed the G*** at (160.0, 80.8)
- removed the G*** at (140.0, 81.0)
- removed the G*** at (120.0, 80.8)
- removed the G*** at (140.0, 47.0)
- removed the G*** at (180.0, 47.0)
- removed the G*** at (160.0, 46.8)
- removed the REF** at (185.0, 61.8)
- removed the REF** at (97.0, 100.2)
- removed the REF** at (99.0, 66.2)
- removed the REF** at (186.0, 66.2)
- removed the REF** at (98.0, 95.8)
- removed the REF** at (186.0, 95.8)
- removed the REF** at (183.0, 100.2)
- removed the REF** at (185.0, 95.8)
- removed the REF** at (186.0, 100.2)
- removed the REF** at (187.0, 95.8)
- removed the REF** at (98.0, 66.2)
- removed the REF** at (184.0, 95.8)
- removed the REF** at (98.0, 100.2)
- removed the REF** at (183.0, 66.2)
- removed the REF** at (95.0, 66.2)
- removed the REF** at (184.0, 100.2)
- removed the REF** at (187.0, 66.2)
- removed the REF** at (96.0, 66.2)
- removed the REF** at (183.0, 61.8)
- removed the REF** at (185.0, 100.2)
- removed the REF** at (186.0, 61.8)
- removed the REF** at (187.0, 61.8)
- removed the REF** at (184.0, 66.2)
- removed the REF** at (99.0, 100.2)
- removed the REF** at (183.0, 95.8)
- removed the REF** at (184.0, 61.8)
- removed the REF** at (185.0, 66.2)
- removed the REF** at (96.0, 100.2)
- removed the REF** at (99.0, 61.8)
- removed the REF** at (95.0, 100.2)
- removed the REF** at (97.0, 66.2)
- removed the REF** at (96.0, 61.8)
- removed the REF** at (97.0, 95.8)
- removed the REF** at (98.0, 61.8)
- removed the REF** at (96.0, 95.8)
- removed the REF** at (97.0, 61.8)
- removed the REF** at (187.0, 100.2)
- removed the REF** at (99.0, 95.8)
- removed the REF** at (95.0, 61.8)
- removed the REF** at (95.0, 95.8)
- added REF**: MountingHole_2.2mm_M2_Pad, MountingHole:MountingHole_2.2mm_M2_Pad, F.Cu at (124.5, 98.5)
- added REF**: MountingHole_2.2mm_M2_Pad, MountingHole:MountingHole_2.2mm_M2_Pad, F.Cu at (184.5, 131.5)
- added REF**: MountingHole_2.2mm_M2_Pad, MountingHole:MountingHole_2.2mm_M2_Pad, F.Cu at (184.5, 98.5)
- added REF**: MountingHole_2.2mm_M2_Pad, MountingHole:MountingHole_2.2mm_M2_Pad, F.Cu at (124.5, 131.5)
- RN1, RN2: moved to F.Cu
- moved RN8 99.0 mm to (100.5, 98.5), turned to 180 degrees
- moved RN7 85.5 mm to (106.0, 98.5), turned to 180 degrees
- moved RN6 72.1 mm to (111.5, 98.5), turned to 180 degrees
- moved RN5 71.8 mm to (145.7, 98.8)
- moved RN4 67.0 mm to (151.4, 98.8)
- moved C7 39.3 mm to (102.0, 124.4), turned to -90 degrees
- moved RN3 39.0 mm to (105.8, 130.1)
- moved RN9 33.7 mm to (152.0, 130.5), turned to 180 degrees
- moved C3 33.5 mm to (100.4, 121.3), turned to -90 degrees
- moved R44 33.4 mm to (96.0, 122.0)
- moved C4 31.3 mm to (98.8, 124.4), turned to -90 degrees
- moved RN1 31.2 mm to (95.4, 130.1), turned to 0 degrees
- moved C6 29.3 mm to (100.4, 124.4), turned to -90 degrees
- moved R42 29.0 mm to (96.0, 118.0), turned to 180 degrees
- moved C2 26.9 mm to (96.0, 125.5), turned to 180 degrees
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Connections:
- RN1 pad 1: /CS4 -> /CS1
- RN1 pad 2: /CS3 -> /CS2
- RN1 pad 3: /CS2 -> /CS3
- RN1 pad 4: /CS1 -> /CS4
- RN1 pad 5: Net-(IC1-Pad26) -> Net-(IC1-Pad29)
- RN1 pad 6: Net-(IC1-Pad27) -> Net-(IC1-Pad28)
- RN1 pad 7: Net-(IC1-Pad28) -> Net-(IC1-Pad27)
- RN1 pad 8: Net-(IC1-Pad29) -> Net-(IC1-Pad26)
- RN2 pad 1: /CS8 -> /CS5
- RN2 pad 2: /CS7 -> /CS6
- RN2 pad 3: /CS6 -> /CS7
- RN2 pad 4: /CS5 -> /CS8
- RN2 pad 5: Net-(IC1-Pad30) -> Net-(IC1-Pad33)
- RN2 pad 6: Net-(IC1-Pad31) -> Net-(IC1-Pad32)
- RN2 pad 7: Net-(IC1-Pad32) -> Net-(IC1-Pad31)
- RN2 pad 8: Net-(IC1-Pad33) -> Net-(IC1-Pad30)
- RN3 pad 1: /CS12 -> /CS9
- RN3 pad 2: /CS11 -> /CS10
- RN3 pad 3: /CS10 -> /CS11
- RN3 pad 4: /CS9 -> /CS12
- RN3 pad 5: Net-(IC1-Pad34) -> Net-(IC1-Pad38)
- RN3 pad 6: Net-(IC1-Pad35) -> Net-(IC1-Pad37)
- RN3 pad 7: Net-(IC1-Pad37) -> Net-(IC1-Pad35)
- RN3 pad 8: Net-(IC1-Pad38) -> Net-(IC1-Pad34)
- RN6 pad 1: /CS24 -> /CS21
- RN6 pad 2: /CS23 -> /CS22
- RN6 pad 3: /CS22 -> /CS23
- RN6 pad 4: /CS21 -> /CS24
- RN6 pad 5: Net-(IC1-Pad47) -> Net-(IC1-Pad50)
- RN6 pad 6: Net-(IC1-Pad48) -> Net-(IC1-Pad49)
- RN6 pad 7: Net-(IC1-Pad49) -> Net-(IC1-Pad48)
- RN6 pad 8: Net-(IC1-Pad50) -> Net-(IC1-Pad47)
- RN7 pad 1: /CS28 -> /CS25
- RN7 pad 2: /CS27 -> /CS26
- RN7 pad 3: /CS26 -> /CS27
- RN7 pad 4: /CS25 -> /CS28
- RN7 pad 5: Net-(IC1-Pad51) -> Net-(IC1-Pad54)
- RN7 pad 6: Net-(IC1-Pad52) -> Net-(IC1-Pad53)
- RN7 pad 7: Net-(IC1-Pad53) -> Net-(IC1-Pad52)
- RN7 pad 8: Net-(IC1-Pad54) -> Net-(IC1-Pad51)
- RN8 pad 1: /CS32 -> /CS29
- RN8 pad 2: /CS31 -> /CS30
- RN8 pad 3: /CS30 -> /CS31
- RN8 pad 4: /CS29 -> /CS32
- RN8 pad 5: Net-(IC1-Pad56) -> Net-(IC1-Pad59)
- RN8 pad 6: Net-(IC1-Pad57) -> Net-(IC1-Pad58)
- RN8 pad 7: Net-(IC1-Pad58) -> Net-(IC1-Pad57)
- RN8 pad 8: Net-(IC1-Pad59) -> Net-(IC1-Pad56)
Routing:
- net Net-(IC1-Pad3): track 0.00 -> 83.1 mm, vias 0 -> 1
- net /CS32: track 36.1 -> 118.9 mm, vias 9 -> 10
- net /CS31: track 41.1 -> 122.2 mm, vias 0 -> 1
- net Net-(IC1-Pad2): track 0.00 -> 79.9 mm, vias 0 -> 1
- net /CS26: track 18.1 -> 96.9 mm, vias 0 -> 3
- net Net-(IC1-Pad60): track 0.00 -> 78.5 mm, vias 0 -> 1
- net /CS25: track 16.8 -> 94.4 mm, vias 4 -> 6
- net Net-(IC1-Pad1): track 0.00 -> 77.3 mm, vias 0 -> 1
- net /CS27: track 22.2 -> 95.5 mm, vias 0 -> 3
- net GND: track 0.00 -> 71.9 mm, vias 0 -> 7
- net /CS24: track 39.2 -> 107.4 mm, vias 2 -> 4
- net /CS22: track 41.0 -> 107.9 mm, vias 0 -> 3
- net /CS23: track 35.1 -> 99.6 mm, vias 9 -> 11
- net +3V3: track 0.00 -> 56.3 mm
- net Net-(IC1-Pad39): track 0.00 -> 55.8 mm, vias 0 -> 2
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Other:
- board size 100 x 98 mm -> 100 x 38 mm

Commit message: Complete initial PCB layout
Parts:
- removed R37, R38, R39: 20, Resistor_SMD:R_0603_1608Metric
- moved RN5 0.10 mm to (145.6, 98.8)
Connections:
- RN5 pad 1: /CS20 -> /CS17
- RN5 pad 2: /CS19 -> /CS18
- RN5 pad 3: /CS18 -> /CS19
- RN5 pad 4: /CS17 -> /CS20
- RN5 pad 5: Net-(IC1-Pad43) -> Net-(IC1-Pad46)
- RN5 pad 6: Net-(IC1-Pad44) -> Net-(IC1-Pad45)
- RN5 pad 7: Net-(IC1-Pad45) -> Net-(IC1-Pad44)
- RN5 pad 8: Net-(IC1-Pad46) -> Net-(IC1-Pad43)
- RN9 pad 1: /CS36 -> /CS33
- RN9 pad 2: /CS35 -> /CS34
- RN9 pad 3: /CS34 -> /CS35
- RN9 pad 4: /CS33 -> /CS36
- RN9 pad 5: Net-(IC1-Pad60) -> Net-(IC1-Pad3)
- RN9 pad 6: Net-(IC1-Pad1) -> Net-(IC1-Pad2)
- RN9 pad 7: Net-(IC1-Pad2) -> Net-(IC1-Pad1)
- RN9 pad 8: Net-(IC1-Pad3) -> Net-(IC1-Pad60)
Routing:
- net /CS28: track 69.0 -> 193.5 mm, vias 1 -> 6
- net /CS29: track 71.5 -> 121.1 mm, vias 7 -> 9
- net /CS32: track 118.9 -> 166.1 mm
- net /CS30: track 75.6 -> 121.8 mm, vias 7 -> 9
- net /CS31: track 122.2 -> 164.2 mm, vias 1 -> 2
- net /CS33: track 43.5 -> 77.9 mm, vias 2 -> 4
- net GND: track 71.9 -> 101.7 mm
- net /CS36: track 18.9 -> 47.5 mm
- net /CS35: track 18.1 -> 45.0 mm
- net /CS34: track 18.2 -> 44.6 mm, vias 4 -> 5
- net /CS14: track 35.0 -> 60.9 mm, vias 9 -> 11
- net /CS16: track 31.9 -> 54.2 mm
- net /CS13: track 41.4 -> 63.3 mm, vias 0 -> 2
- net /SW1: track 201.9 -> 222.8 mm
- net /CS15: track 42.4 -> 61.7 mm, vias 2 -> 4
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