File: PMOD_RGB7Segment/Hardware/PMod_RGB7Segment.kicad_pcb (KiCad board)
At the start: 4 copper layers, 100 x 38 mm, 121 parts, among them IC1 IS31FL3741A-QFLS4-TR, J1 Conn_02x06_Odd_Even

Commit message: Chane required clearance to 0.19mm from 0.2mm
Other:
- rule pad_to_mask_clearance: 0 -> 0.19
Changed lines of the file:
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@@
       (dielectric_constraints no)
     )
-    (pad_to_mask_clearance 0)
+    (pad_to_mask_clearance 0.19)
     (pcbplotparams
       (layerselection 0x00010fc_ffffffff)
