File: PMOD_RGB7Segment/Hardware/segment4.kicad_sch (KiCad schematic)
At the start: 22 parts

Commit message: Add the schematics for each of the 7 segment characters
Parts:
- removed D1, D10, D11, D12, D13, D14, D15, D16, D17, D18, D19, D2, D20, D21, D22, D3, D4, D5, D6, D7, D8, D9: LED_ARGB, jjh:SX-0402-RGB, symbol Device:LED_ARGB
- added D? (x22): LED_ARGB, jjh:SX-0402-RGB, symbol Device:LED_ARGB
Connections:
- net CS1: now also D?.2 (RK), D?.2 (RK)
- net CS10: now also D?.2 (RK), D?.2 (RK)
- net CS11: now also D?.3 (GK), D?.3 (GK)
- net CS12: now also D?.4 (BK), D?.4 (BK)
- net CS13: now also D?.2 (RK), D?.2 (RK)
- net CS14: now also D?.3 (GK), D?.3 (GK)
- net CS15: now also D?.4 (BK), D?.4 (BK)
- net CS16: now also D?.2 (RK), D?.2 (RK)
- net CS17: now also D?.3 (GK), D?.3 (GK)
- net CS18: now also D?.4 (BK), D?.4 (BK)
- net CS19: now also D?.2 (RK), D?.2 (RK)
- net CS2: now also D?.3 (GK), D?.3 (GK)
- net CS20: now also D?.3 (GK), D?.3 (GK)
- net CS21: now also D?.4 (BK), D?.4 (BK)
- net CS22: now also D?.2 (RK), D?.2 (RK)
- net CS23: now also D?.3 (GK), D?.3 (GK)
- net CS24: now also D?.4 (BK), D?.4 (BK)
- net CS25: now also D?.2 (RK), D?.2 (RK)
- net CS26: now also D?.3 (GK), D?.3 (GK)
- net CS27: now also D?.4 (BK), D?.4 (BK)
- net CS28: now also D?.2 (RK), D?.2 (RK)
- net CS29: now also D?.3 (GK), D?.3 (GK)
- net CS3: now also D?.4 (BK), D?.4 (BK)
- net CS30: now also D?.4 (BK), D?.4 (BK)
- net CS31: now also D?.2 (RK)
- net CS32: now also D?.3 (GK)
- net CS33: now also D?.4 (BK)
- net CS34: now also D?.2 (RK)
- net CS35: now also D?.3 (GK)
- net CS36: now also D?.4 (BK)
- net CS4: now also D?.2 (RK), D?.2 (RK)
- net CS5: now also D?.3 (GK), D?.3 (GK)
- net CS6: now also D?.4 (BK), D?.4 (BK)
- net CS7: now also D?.2 (RK), D?.2 (RK)
- net CS8: now also D?.3 (GK), D?.3 (GK)
- net CS9: now also D?.4 (BK), D?.4 (BK)
- new net SW7: D?.1 (A), D?.1 (A), D?.1 (A), D?.1 (A), D?.1 (A), D?.1 (A), D?.1 (A), D?.1 (A), D?.1 (A), D?.1 (A), D?.1 (A), D?.1 (A)
- new net SW8: D?.1 (A), D?.1 (A), D?.1 (A), D?.1 (A), D?.1 (A), D?.1 (A), D?.1 (A), D?.1 (A), D?.1 (A), D?.1 (A)

Commit message: minor changes to segments
Parts:
- removed D? (x22): LED_ARGB, jjh:SX-0402-RGB, symbol Device:LED_ARGB
- added D69, D70, D71, D72, D73, D74, D75, D76, D77, D78, D79, D80, D81, D82, D83, D84, D85, D86, D87, D88, D89, D90: LED_ARGB, jjh:SX-0402-RGB, symbol Device:LED_ARGB
Connections:
- net CS1: now also D69.2 (RK), D81.2 (RK)
- net CS10: now also D72.2 (RK), D84.2 (RK)
- net CS11: now also D72.3 (GK), D84.3 (GK)
- net CS12: now also D72.4 (BK), D84.4 (BK)
- net CS13: now also D73.2 (RK), D85.2 (RK)
- net CS14: now also D73.3 (GK), D85.3 (GK)
- net CS15: now also D73.4 (BK), D85.4 (BK)
- net CS16: now also D74.2 (RK), D86.2 (RK)
- net CS17: now also D74.3 (GK), D86.3 (GK)
- net CS18: now also D74.4 (BK), D86.4 (BK)
- net CS19: now also D75.2 (RK), D87.2 (RK)
- net CS2: now also D69.3 (GK), D81.3 (GK)
- net CS20: now also D75.3 (GK), D87.3 (GK)
- net CS21: now also D75.4 (BK), D87.4 (BK)
- net CS22: now also D76.2 (RK), D88.2 (RK)
- net CS23: now also D76.3 (GK), D88.3 (GK)
- net CS24: now also D76.4 (BK), D88.4 (BK)
- net CS25: now also D77.2 (RK), D89.2 (RK)
- net CS26: now also D77.3 (GK), D89.3 (GK)
- net CS27: now also D77.4 (BK), D89.4 (BK)
- net CS28: now also D78.2 (RK), D90.2 (RK)
- net CS29: now also D78.3 (GK), D90.3 (GK)
- net CS3: now also D69.4 (BK), D81.4 (BK)
- net CS30: now also D78.4 (BK), D90.4 (BK)
- net CS31: now also D79.2 (RK)
- net CS32: now also D79.3 (GK)
- net CS33: now also D79.4 (BK)
- net CS34: now also D80.2 (RK)
- net CS35: now also D80.3 (GK)
- net CS36: now also D80.4 (BK)
- net CS4: now also D70.2 (RK), D82.2 (RK)
- net CS5: now also D70.3 (GK), D82.3 (GK)
- net CS6: now also D70.4 (BK), D82.4 (BK)
- net CS7: now also D71.2 (RK), D83.2 (RK)
- net CS8: now also D71.3 (GK), D83.3 (GK)
- net CS9: now also D71.4 (BK), D83.4 (BK)
- net SW7: now also D69.1 (A), D70.1 (A), D71.1 (A), D72.1 (A), D73.1 (A), D74.1 (A), D75.1 (A), D76.1 (A), D77.1 (A), D78.1 (A), D79.1 (A), D80.1 (A)
- net SW8: now also D81.1 (A), D82.1 (A), D83.1 (A), D84.1 (A), D85.1 (A), D86.1 (A), D87.1 (A), D88.1 (A), D89.1 (A), D90.1 (A)

Commit message: correct the bus naming
Changed lines of the file:
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@@
     (effects (font (size 0.7 0.7) bold) (justify left bottom))
   )
-  (hierarchical_label "SW_Bus" (shape input) (at 31.75 175.26 180)
+  (hierarchical_label "SW[9..1]" (shape input) (at 31.75 175.26 180)
     (effects (font (size 1.27 1.27)) (justify right))
   )
-  (hierarchical_label "CS_Bus" (shape input) (at 34.29 15.24 180)
+  (hierarchical_label "CS[39..1]" (shape input) (at 34.29 15.24 180)
     (effects (font (size 1.27 1.27)) (justify right))
   )

Commit message: start mapping out locations on PCB
Other:
- company: (none) -> James Horton
- title: (none) -> PMod RGB & Segment Display
Changed lines of the file:
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@@
 (kicad_sch (version 20211123) (generator eeschema)
   (paper "A4")
+  (title_block
+    (title "PMod RGB & Segment Display")
+    (rev "v0.1")
+    (company "James Horton")
+    (comment 1 "interface, all LED's are designed to be indivdually addressable ")
+    (comment 2 "This design is a 4 Digit Seven Segment Display made from RGB LED's, controlled using I2C")
+    (comment 4 "Licensed Under CERN Open Hardware Licence Version 2 - Permissive")
+  )
   (junction (at 214.63 78.74) (diameter 0) (color 0 0 0 0)
   )

Commit message: update the pin for segment 4 to improve pcb layout
Connections:
- net CS10 is gone; now on net CS28: D72.2 (RK), D84.2 (RK)
- net CS11 is gone; now on net CS29: D72.3 (GK), D84.3 (GK)
- net CS12 is gone; now on net CS30: D72.4 (BK), D84.4 (BK)
- net CS13 is gone; now on net CS28: D73.2 (RK), D85.2 (RK)
- net CS14 is gone; now on net CS29: D73.3 (GK), D85.3 (GK)
- net CS15 is gone; now on net CS30: D73.4 (BK), D85.4 (BK)
- net CS16 is gone; now on net CS28: D74.2 (RK), D86.2 (RK)
- net CS17 is gone; now on net CS29: D74.3 (GK), D86.3 (GK)
- net CS18 is gone; now on net CS30: D74.4 (BK), D86.4 (BK)
- net CS19 is gone; now on net CS31: D75.2 (RK), D87.2 (RK)
- net CS22 is gone; now on net CS31: D76.2 (RK), D88.2 (RK)
- net CS23 is gone; now on net CS32: D76.3 (GK), D88.3 (GK)
- net CS24 is gone; now on net CS33: D76.4 (BK), D88.4 (BK)
- net CS25 is gone; now on net CS31: D77.2 (RK), D89.2 (RK)
- net CS26 is gone; now on net CS32: D77.3 (GK), D89.3 (GK)
- net CS27 is gone; now on net CS33: D77.4 (BK), D89.4 (BK)
- net CS20: now also D70.4 (BK); no longer D75.3 (GK), D87.3 (GK)
- net CS28: now also D69.2 (RK), D70.2 (RK), D71.2 (RK); no longer D78.2 (RK), D90.2 (RK)
- net CS29: now also D69.3 (GK), D70.3 (GK), D71.3 (GK); no longer D78.3 (GK), D90.3 (GK)
- net CS30: now also D69.4 (BK), D71.4 (BK); no longer D78.4 (BK), D90.4 (BK)
- net CS31: now also D81.2 (RK), D82.2 (RK), D83.2 (RK); no longer D79.2 (RK)
- net CS32: now also D75.3 (GK), D81.3 (GK), D82.3 (GK), D83.3 (GK), D87.3 (GK); no longer D79.3 (GK)
- net CS33: now also D81.4 (BK), D82.4 (BK), D83.4 (BK), D87.4 (BK); no longer D79.4 (BK)
- net CS34: now also D78.2 (RK), D79.2 (RK), D90.2 (RK)
- net CS35: now also D78.3 (GK), D79.3 (GK), D90.3 (GK)
- net CS36: now also D78.4 (BK), D79.4 (BK), D90.4 (BK)
- net SW7: no longer D69.1 (A), D70.1 (A), D71.1 (A), D73.1 (A), D74.1 (A), D76.1 (A), D77.1 (A), D78.1 (A), D79.1 (A), D80.1 (A)
- net SW8: now also D73.1 (A), D76.1 (A); no longer D81.1 (A), D82.1 (A), D83.1 (A), D84.1 (A), D85.1 (A), D86.1 (A), D87.1 (A), D88.1 (A), D89.1 (A), D90.1 (A)
- removed net CS1: D69.2 (RK), D81.2 (RK)
- removed net CS2: D69.3 (GK), D81.3 (GK)
- net CS21 renamed 33
- net 33: no longer D87.4 (BK)
- removed net CS3: D69.4 (BK), D81.4 (BK)
- removed net CS4: D70.2 (RK), D82.2 (RK)
- removed net CS5: D70.3 (GK), D82.3 (GK)
- removed net CS6: D70.4 (BK), D82.4 (BK)
- removed net CS7: D71.2 (RK), D83.2 (RK)
- removed net CS8: D71.3 (GK), D83.3 (GK)
- removed net CS9: D71.4 (BK), D83.4 (BK)
- new net SW1: D78.1 (A), D81.1 (A), D84.1 (A)
- new net SW2: D79.1 (A), D82.1 (A), D85.1 (A)
- new net SW3: D80.1 (A), D83.1 (A), D86.1 (A)
- new net SW4: D69.1 (A), D87.1 (A), D90.1 (A)
- new net SW5: D70.1 (A), D88.1 (A)
- new net SW6: D71.1 (A), D89.1 (A)
- new net SW9: D74.1 (A), D77.1 (A)

Commit message: correct pins in schematic and continue LED layout on PCB
Connections:
- net CS20 is gone; now on net CS30: D70.4 (BK)
Changed lines of the file:
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@@
     (effects (font (size 1.27 1.27) bold) (justify left bottom))
   )
-  (label "CS20" (at 71.12 63.5 0)
+  (label "CS30" (at 71.12 63.5 0)
     (effects (font (size 0.7 0.7) bold) (justify left bottom))
   )

Commit message: continue with placement and layout of digits
Connections:
- net 33 is gone; now on net CS33: D75.4 (BK)
- net SW1: now also D86.1 (A); no longer D84.1 (A)
- net SW3: now also D84.1 (A); no longer D86.1 (A)
Changed lines of the file:
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@@
     (effects (font (size 0.7 0.7) bold) (justify left bottom))
   )
-  (label "33" (at 128.27 41.91 0)
+  (label "CS33" (at 128.27 41.91 0)
     (effects (font (size 0.7 0.7) bold) (justify left bottom))
   )
@@
     (effects (font (size 1.27 1.27) bold) (justify left bottom))
   )
-  (label "SW3" (at 210.82 151.13 0)
+  (label "SW1" (at 210.82 151.13 0)
     (effects (font (size 1.27 1.27) bold) (justify left bottom))
   )
@@
     (effects (font (size 0.7 0.7) bold) (justify left bottom))
   )
-  (label "SW1" (at 210.82 109.22 0)
+  (label "SW3" (at 210.82 109.22 0)
     (effects (font (size 1.27 1.27) bold) (justify left bottom))
   )
