File: PMOD_RGB7Segment/Hardware/controller.kicad_sch (KiCad schematic)
At the start: 40 parts, among them IC1 IS31FL3741A-QFLS4-TR

Commit message: correct the bus naming
Changed lines of the file:
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@@
     (effects (font (size 1.27 1.27)) (justify left bottom))
   )
-  (hierarchical_label "CS_Bus" (shape input) (at 217.17 24.13 0)
+  (hierarchical_label "CS[39..1]" (shape input) (at 217.17 24.13 0)
     (effects (font (size 1.27 1.27)) (justify left))
   )
-  (hierarchical_label "SW_Bus" (shape input) (at 219.71 125.73 0)
+  (hierarchical_label "SW[9..1]" (shape input) (at 219.71 125.73 0)
     (effects (font (size 1.27 1.27)) (justify left))
   )

Commit message: Add power and connections for i2c interface
Parts:
- added C1, C3, C6: 1u, Capacitor_SMD:C_0603_1608Metric, symbol Device:C
- added C2, C4, C5, C7: 0.1u, Capacitor_SMD:C_0603_1608Metric, symbol Device:C
- added R40, R41: 100K, Resistor_SMD:R_0603_1608Metric, symbol Device:R
- added R42, R43: 2K, Resistor_SMD:R_0603_1608Metric, symbol Device:R
- added R44: 10K, Resistor_SMD:R_0603_1608Metric, symbol Device:R
Connections:
- net GND: now also IC1.12 (GND_1), IC1.36 (GND_2), IC1.55 (GND_3), IC1.8 (ADDR), C1.2, C2.2, C3.2, C4.2, C5.2, C6.2, C7.2, R41.1, R44.1
- net SCL: now reaches IC1.10 (SCL)
- net SCL: now also R42.1
- net SDB: now reaches IC1.11 (SDB)
- net SDB: now also C5.1, R41.2
- net at IC1.13 (ISET): now also R44.2
- net +3V3: now reaches IC1.14 (AVCC)
- net +3V3: now also IC1.15 (PVCC_1), IC1.25 (PVCC_2), C1.1, C2.1, C3.1, C4.1, C6.1, C7.1, R40.2, R42.2, R43.2
- net INTB: now reaches IC1.7 (INTB)
- net INTB: now also R40.1
- net SDA: now reaches IC1.9 (SDA)
- net SDA: now also R43.1

Commit message: start mapping out locations on PCB
Other:
- company: (none) -> James Horton
- title: (none) -> PMod RGB & Segment Display
Changed lines of the file:
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@@
 (kicad_sch (version 20211123) (generator eeschema)
   (paper "A4")
+  (title_block
+    (title "PMod RGB & Segment Display")
+    (rev "v0.1")
+    (company "James Horton")
+    (comment 1 "interface, all LED's are designed to be indivdually addressable ")
+    (comment 2 "This design is a 4 Digit Seven Segment Display made from RGB LED's, controlled using I2C")
+    (comment 4 "Licensed Under CERN Open Hardware Licence Version 2 - Permissive")
+  )
   (junction (at 48.26 30.48) (diameter 0) (color 0 0 0 0)
   )

Commit message: update PCB from the segment pin changes
Parts:
- IC1: footprint QFN40P700X700X80-61N-D -> jjh:QFN40P700X700X80-61N-D
Changed lines of the file:
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@@
     (property "Reference" "IC1" (id 0) (at 146.05 20.32 0))
     (property "Value" "IS31FL3741A-QFLS4-TR" (id 1) (at 146.05 22.86 0))
-    (property "Footprint" "QFN40P700X700X80-61N-D" (id 2) (at 193.04 69.85 0)
+    (property "Footprint" "jjh:QFN40P700X700X80-61N-D" (id 2) (at 193.04 69.85 0)
       (effects (font (size 1.27 1.27)) (justify left) hide)
     )

Commit message: change 20ohms resistors to 4 way resistor arrays
Parts:
- removed R1, R10, R11, R12, R13, R14, R15, R16, R17, R18, R19, R2, R20, R21, R22, R23, R24, R25, R26, R27, R28, R29, R3, R30, R31, R32, R33, R34, R35, R36, R37, R38, R39, R4, R5, R6, R7, R8, R9: 20, Resistor_SMD:R_0603_1608Metric, symbol Device:R
- added RN1, RN2, RN3, RN4, RN5, RN6, RN7, RN8, RN9: EXB38V472JV, jjh:EXB38V472JV, symbol Device:R_Pack04
Connections:
- net CS1: now also RN1.4 (R4.1)
- net CS10: now also RN3.3 (R3.1)
- net CS11: now also RN3.2 (R2.1)
- net CS12: now also RN3.1 (R1.1)
- net CS13: now also RN4.4 (R4.1)
- net CS14: now also RN4.3 (R3.1)
- net CS15: now also RN4.2 (R2.1)
- net CS16: now also RN4.1 (R1.1)
- net CS17: now also RN5.4 (R4.1)
- net CS18: now also RN5.3 (R3.1)
- net CS19: now also RN5.2 (R2.1)
- net CS2: now also RN1.3 (R3.1)
- net CS20: now also RN5.1 (R1.1)
- net CS21: now also RN6.4 (R4.1)
- net CS22: now also RN6.3 (R3.1)
- net CS23: now also RN6.2 (R2.1)
- net CS24: now also RN6.1 (R1.1)
- net CS25: now also RN7.4 (R4.1)
- net CS26: now also RN7.3 (R3.1)
- net CS27: now also RN7.2 (R2.1)
- net CS28: now also RN7.1 (R1.1)
- net CS29: now also RN8.4 (R4.1)
- net CS3: now also RN1.2 (R2.1)
- net CS30: now also RN8.3 (R3.1)
- net CS31: now also RN8.2 (R2.1)
- net CS32: now also RN8.1 (R1.1)
- net CS33: now also RN9.4 (R4.1)
- net CS34: now also RN9.3 (R3.1)
- net CS35: now also RN9.2 (R2.1)
- net CS36: now also RN9.1 (R1.1)
- net CS4: now also RN1.1 (R1.1)
- net CS5: now also RN2.4 (R4.1)
- net CS6: now also RN2.3 (R3.1)
- net CS7: now also RN2.2 (R2.1)
- net CS8: now also RN2.1 (R1.1)
- net CS9: now also RN3.4 (R4.1)
- net at IC1.31 (CS6): now also RN2.6 (R3.2)
- net at IC1.33 (CS8): now also RN2.8 (R1.2)
- net at IC1.45 (CS19): now also RN5.7 (R2.2)
- net at IC1.32 (CS7): now also RN2.7 (R2.2)
- net at IC1.35 (CS10): now also RN3.6 (R3.2)
- net at IC1.37 (CS11): now also RN3.7 (R2.2)
- net at IC1.56 (CS29): now also RN8.5 (R4.2)
- net at IC1.41 (CS15): now also RN4.7 (R2.2)
- net at IC1.29 (CS4): now also RN1.8 (R1.2)
- net at IC1.1 (CS34): now also RN9.6 (R3.2)
- net at IC1.2 (CS35): now also RN9.7 (R2.2)
- net at IC1.26 (CS1): now also RN1.5 (R4.2)
- net at IC1.27 (CS2): now also RN1.6 (R3.2)
- net at IC1.28 (CS3): now also RN1.7 (R2.2)
- net at IC1.3 (CS36): now also RN9.8 (R1.2)
- net at IC1.30 (CS5): now also RN2.5 (R4.2)
- net at IC1.34 (CS9): now also RN3.5 (R4.2)
- net at IC1.38 (CS12): now also RN3.8 (R1.2)
- net at IC1.39 (CS13): now also RN4.5 (R4.2)
- net at IC1.40 (CS14): now also RN4.6 (R3.2)
- net at IC1.42 (CS16): now also RN4.8 (R1.2)
- net at IC1.43 (CS17): now also RN5.5 (R4.2)
- net at IC1.44 (CS18): now also RN5.6 (R3.2)
- net at IC1.46 (CS20): now also RN5.8 (R1.2)
- net at IC1.47 (CS21): now also RN6.5 (R4.2)
- net at IC1.48 (CS22): now also RN6.6 (R3.2)
- net at IC1.49 (CS23): now also RN6.7 (R2.2)
- net at IC1.50 (CS24): now also RN6.8 (R1.2)
- net at IC1.51 (CS25): now also RN7.5 (R4.2)
- net at IC1.52 (CS26): now also RN7.6 (R3.2)
- net at IC1.53 (CS27): now also RN7.7 (R2.2)
- net at IC1.54 (CS28): now also RN7.8 (R1.2)
- net at IC1.57 (CS30): now also RN8.6 (R3.2)
- net at IC1.58 (CS31): now also RN8.7 (R2.2)
- net at IC1.59 (CS32): now also RN8.8 (R1.2)
- net at IC1.60 (CS33): now also RN9.5 (R4.2)

Commit message: PCB layout continued, not completed
Connections:
- net CS1: now also RN1.1 (R1.1); no longer RN1.4 (R4.1)
- net CS10: now also RN3.2 (R2.1); no longer RN3.3 (R3.1)
- net CS11: now also RN3.3 (R3.1); no longer RN3.2 (R2.1)
- net CS12: now also RN3.4 (R4.1); no longer RN3.1 (R1.1)
- net CS2: now also RN1.2 (R2.1); no longer RN1.3 (R3.1)
- net CS21: now also RN6.1 (R1.1); no longer RN6.4 (R4.1)
- net CS22: now also RN6.2 (R2.1); no longer RN6.3 (R3.1)
- net CS23: now also RN6.3 (R3.1); no longer RN6.2 (R2.1)
- net CS24: now also RN6.4 (R4.1); no longer RN6.1 (R1.1)
- net CS25: now also RN7.1 (R1.1); no longer RN7.4 (R4.1)
- net CS26: now also RN7.2 (R2.1); no longer RN7.3 (R3.1)
- net CS27: now also RN7.3 (R3.1); no longer RN7.2 (R2.1)
- net CS28: now also RN7.4 (R4.1); no longer RN7.1 (R1.1)
- net CS29: now also RN8.1 (R1.1); no longer RN8.4 (R4.1)
- net CS3: now also RN1.3 (R3.1); no longer RN1.2 (R2.1)
- net CS30: now also RN8.2 (R2.1); no longer RN8.3 (R3.1)
- net CS31: now also RN8.3 (R3.1); no longer RN8.2 (R2.1)
- net CS32: now also RN8.4 (R4.1); no longer RN8.1 (R1.1)
- net CS4: now also RN1.4 (R4.1); no longer RN1.1 (R1.1)
- net CS5: now also RN2.1 (R1.1); no longer RN2.4 (R4.1)
- net CS6: now also RN2.2 (R2.1); no longer RN2.3 (R3.1)
- net CS7: now also RN2.3 (R3.1); no longer RN2.2 (R2.1)
- net CS8: now also RN2.4 (R4.1); no longer RN2.1 (R1.1)
- net CS9: now also RN3.1 (R1.1); no longer RN3.4 (R4.1)
- net at RN2.5 (R4.2): now also IC1.33 (CS8); no longer IC1.30 (CS5)
- net at RN2.6 (R3.2): now also IC1.32 (CS7); no longer IC1.31 (CS6)
- net at RN2.7 (R2.2): now also IC1.31 (CS6); no longer IC1.32 (CS7)
- net at RN2.8 (R1.2): now also IC1.30 (CS5); no longer IC1.33 (CS8)
- net at RN3.5 (R4.2): now also IC1.38 (CS12); no longer IC1.34 (CS9)
- net at RN3.6 (R3.2): now also IC1.37 (CS11); no longer IC1.35 (CS10)
- net at RN3.7 (R2.2): now also IC1.35 (CS10); no longer IC1.37 (CS11)
- net at RN3.8 (R1.2): now also IC1.34 (CS9); no longer IC1.38 (CS12)
- net at RN8.5 (R4.2): now also IC1.59 (CS32); no longer IC1.56 (CS29)
- net at RN8.6 (R3.2): now also IC1.58 (CS31); no longer IC1.57 (CS30)
- net at RN8.7 (R2.2): now also IC1.57 (CS30); no longer IC1.58 (CS31)
- net at RN8.8 (R1.2): now also IC1.56 (CS29); no longer IC1.59 (CS32)
- net at IC1.26 (CS1): now also RN1.8 (R1.2); no longer RN1.5 (R4.2)
- net at IC1.27 (CS2): now also RN1.7 (R2.2); no longer RN1.6 (R3.2)
- net at IC1.28 (CS3): now also RN1.6 (R3.2); no longer RN1.7 (R2.2)
- net at IC1.29 (CS4): now also RN1.5 (R4.2); no longer RN1.8 (R1.2)
- net at IC1.47 (CS21): now also RN6.8 (R1.2); no longer RN6.5 (R4.2)
- net at IC1.48 (CS22): now also RN6.7 (R2.2); no longer RN6.6 (R3.2)
- net at IC1.49 (CS23): now also RN6.6 (R3.2); no longer RN6.7 (R2.2)
- net at IC1.50 (CS24): now also RN6.5 (R4.2); no longer RN6.8 (R1.2)
- net at IC1.51 (CS25): now also RN7.8 (R1.2); no longer RN7.5 (R4.2)
- net at IC1.52 (CS26): now also RN7.7 (R2.2); no longer RN7.6 (R3.2)
- net at IC1.53 (CS27): now also RN7.6 (R3.2); no longer RN7.7 (R2.2)
- net at IC1.54 (CS28): now also RN7.5 (R4.2); no longer RN7.8 (R1.2)
Changed lines of the file:
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@@
     (pin "1")
   )
-  (symbol (lib_id "Device:R_Pack04") (at 181.61 39.37 90) (unit 1)
-    (in_bom yes) (on_board yes)
-    (property "Reference" "RN2" (id 0) (at 175.26 38.1 90))
-    (property "Value" "EXB38V472JV" (id 1) (at 193.04 35.56 90)
-      (effects (font (size 1.27 1.27)) hide)
-    )
-    (property "Footprint" "jjh:EXB38V472JV" (id 2) (at 181.61 32.385 90)
-      (effects (font (size 1.27 1.27)) hide)
-    )
-    (property "Datasheet" "~" (id 3) (at 181.61 39.37 0)
+  (symbol (lib_id "Device:R_Pack04") (at 181.61 41.91 90) (mirror x) (unit 1)
+    (in_bom yes) (on_board yes)
+    (property "Reference" "RN2" (id 0) (at 175.26 43.18 90))
+    (property "Value" "EXB38V472JV" (id 1) (at 193.04 45.72 90)
+      (effects (font (size 1.27 1.27)) hide)
+    )
+    (property "Footprint" "jjh:EXB38V472JV" (id 2) (at 181.61 48.895 90)
+      (effects (font (size 1.27 1.27)) hide)
+    )
+    (property "Datasheet" "~" (id 3) (at 181.61 41.91 0)
       (effects (font (size 1.27 1.27)) hide)
     )
@@
     (pin "1")
   )
-  (symbol (lib_id "Device:R_Pack04") (at 181.61 49.53 90) (unit 1)
-    (in_bom yes) (on_board yes)
-    (property "Reference" "RN3" (id 0) (at 175.26 48.26 90))
-    (property "Value" "EXB38V472JV" (id 1) (at 193.04 45.72 90)
-      (effects (font (size 1.27 1.27)) hide)
-    )
-    (property "Footprint" "jjh:EXB38V472JV" (id 2) (at 181.61 42.545 90)
-      (effects (font (size 1.27 1.27)) hide)
-    )
-    (property "Datasheet" "~" (id 3) (at 181.61 49.53 0)
-      (effects (font (size 1.27 1.27)) hide)
-    )
-    (pin "1")
-    (pin "2")
-    (pin "3")
-    (pin "4")
-    (pin "5")
-    (pin "6")
-    (pin "7")
-    (pin "8")
-  )
-  (symbol (lib_id "Device:R_Pack04") (at 181.61 100.33 90) (unit 1)
-    (in_bom yes) (on_board yes)
-    (property "Reference" "RN8" (id 0) (at 175.26 99.06 90))
-    (property "Value" "EXB38V472JV" (id 1) (at 193.04 96.52 90)
-      (effects (font (size 1.27 1.27)) hide)
-    )
-    (property "Footprint" "jjh:EXB38V472JV" (id 2) (at 181.61 93.345 90)
-      (effects (font (size 1.27 1.27)) hide)
-    )
-    (property "Datasheet" "~" (id 3) (at 181.61 100.33 0)
+  (symbol (lib_id "Device:R_Pack04") (at 181.61 52.07 90) (mirror x) (unit 1)
+    (in_bom yes) (on_board yes)
+    (property "Reference" "RN3" (id 0) (at 175.26 53.34 90))
+    (property "Value" "EXB38V472JV" (id 1) (at 193.04 55.88 90)
+      (effects (font (size 1.27 1.27)) hide)
+    )
+    (property "Footprint" "jjh:EXB38V472JV" (id 2) (at 181.61 59.055 90)
+      (effects (font (size 1.27 1.27)) hide)
+    )
+    (property "Datasheet" "~" (id 3) (at 181.61 52.07 0)
+      (effects (font (size 1.27 1.27)) hide)
+    )
+    (pin "1")
+    (pin "2")
+    (pin "3")
+    (pin "4")
+    (pin "5")
+    (pin "6")
+    (pin "7")
+    (pin "8")
+  )
+  (symbol (lib_id "Device:R_Pack04") (at 181.61 102.87 90) (mirror x) (unit 1)
+    (in_bom yes) (on_board yes)
+    (property "Reference" "RN8" (id 0) (at 175.26 104.14 90))
+    (property "Value" "EXB38V472JV" (id 1) (at 193.04 106.68 90)
+      (effects (font (size 1.27 1.27)) hide)
+    )
+    (property "Footprint" "jjh:EXB38V472JV" (id 2) (at 181.61 109.855 90)
+      (effects (font (size 1.27 1.27)) hide)
+    )
+    (property "Datasheet" "~" (id 3) (at 181.61 102.87 0)
       (effects (font (size 1.27 1.27)) hide)
     )
@@
     (pin "1")
   )
-  (symbol (lib_id "Device:R_Pack04") (at 181.61 29.21 90) (unit 1)
-    (in_bom yes) (on_board yes)
-    (property "Reference" "RN1" (id 0) (at 175.26 27.94 90))
-    (property "Value" "EXB38V472JV" (id 1) (at 181.61 22.86 90))
-    (property "Footprint" "jjh:EXB38V472JV" (id 2) (at 181.61 22.225 90)
-      (effects (font (size 1.27 1.27)) hide)
-    )
-    (property "Datasheet" "~" (id 3) (at 181.61 29.21 0)
+  (symbol (lib_id "Device:R_Pack04") (at 181.61 31.75 90) (mirror x) (unit 1)
+    (in_bom yes) (on_board yes)
+    (property "Reference" "RN1" (id 0) (at 175.26 33.02 90))
+    (property "Value" "EXB38V472JV" (id 1) (at 181.61 38.1 90)
+      (effects (font (size 1.27 1.27)) hide)
+    )
+    (property "Footprint" "jjh:EXB38V472JV" (id 2) (at 181.61 38.735 90)
+      (effects (font (size 1.27 1.27)) hide)
+    )
+    (property "Datasheet" "~" (id 3) (at 181.61 31.75 0)
       (effects (font (size 1.27 1.27)) hide)
     )
@@
     (pin "1")
   )
-  (symbol (lib_id "Device:R_Pack04") (at 181.61 90.17 90) (unit 1)
-    (in_bom yes) (on_board yes)
-    (property "Reference" "RN7" (id 0) (at 175.26 88.9 90))
-    (property "Value" "EXB38V472JV" (id 1) (at 193.04 86.36 90)
-      (effects (font (size 1.27 1.27)) hide)
-    )
-    (property "Footprint" "jjh:EXB38V472JV" (id 2) (at 181.61 83.185 90)
-      (effects (font (size 1.27 1.27)) hide)
-    )
-    (property "Datasheet" "~" (id 3) (at 181.61 90.17 0)
+  (symbol (lib_id "Device:R_Pack04") (at 181.61 92.71 90) (mirror x) (unit 1)
+    (in_bom yes) (on_board yes)
+    (property "Reference" "RN7" (id 0) (at 175.26 93.98 90))
+    (property "Value" "EXB38V472JV" (id 1) (at 193.04 96.52 90)
+      (effects (font (size 1.27 1.27)) hide)
+    )
+    (property "Footprint" "jjh:EXB38V472JV" (id 2) (at 181.61 99.695 90)
+      (effects (font (size 1.27 1.27)) hide)
+    )
+    (property "Datasheet" "~" (id 3) (at 181.61 92.71 0)
       (effects (font (size 1.27 1.27)) hide)
     )
@@
     (pin "2")
   )
-  (symbol (lib_id "Device:R_Pack04") (at 181.61 80.01 90) (unit 1)
-    (in_bom yes) (on_board yes)
-    (property "Reference" "RN6" (id 0) (at 175.26 78.74 90))
-    (property "Value" "EXB38V472JV" (id 1) (at 193.04 76.2 90)
-      (effects (font (size 1.27 1.27)) hide)
-    )
-    (property "Footprint" "jjh:EXB38V472JV" (id 2) (at 181.61 73.025 90)
-      (effects (font (size 1.27 1.27)) hide)
-    )
-    (property "Datasheet" "~" (id 3) (at 181.61 80.01 0)
-      (effects (font (size 1.27 1.27)) hide)
-    )
+  (symbol (lib_id "Device:R_Pack04") (at 181.61 82.55 90) (mirror x) (unit 1)
+    (in_bom yes) (on_board yes)
+    (property "Reference" "RN6" (id 0) (at 175.26 83.82 90))
+    (property "Value" "EXB38V472JV" (id 1) (at 193.04 86.36 90)
+      (effects (font (size 1.27 1.27)) hide)
+    )
+    (property "Footprint" "jjh:EXB38V472JV" (id 2) (at 181.61 89.535 90)
+      (effects (font (size 1.27 1.27)) hide)
+    )
+    (property "Datasheet" "~" (id 3) (at 181.61 82.55 0)
+      (effects (font (size 1.27 1.27)) hide)
+    )

Commit message: Complete initial PCB layout
Connections:
- net CS17: now also RN5.1 (R1.1); no longer RN5.4 (R4.1)
- net CS18: now also RN5.2 (R2.1); no longer RN5.3 (R3.1)
- net CS19: now also RN5.3 (R3.1); no longer RN5.2 (R2.1)
- net CS20: now also RN5.4 (R4.1); no longer RN5.1 (R1.1)
- net CS33: now also RN9.1 (R1.1); no longer RN9.4 (R4.1)
- net CS34: now also RN9.2 (R2.1); no longer RN9.3 (R3.1)
- net CS35: now also RN9.3 (R3.1); no longer RN9.2 (R2.1)
- net CS36: now also RN9.4 (R4.1); no longer RN9.1 (R1.1)
- net at IC1.1 (CS34): now also RN9.7 (R2.2); no longer RN9.6 (R3.2)
- net at IC1.2 (CS35): now also RN9.6 (R3.2); no longer RN9.7 (R2.2)
- net at IC1.3 (CS36): now also RN9.5 (R4.2); no longer RN9.8 (R1.2)
- net at IC1.43 (CS17): now also RN5.8 (R1.2); no longer RN5.5 (R4.2)
- net at IC1.44 (CS18): now also RN5.7 (R2.2); no longer RN5.6 (R3.2)
- net at IC1.45 (CS19): now also RN5.6 (R3.2); no longer RN5.7 (R2.2)
- net at IC1.46 (CS20): now also RN5.5 (R4.2); no longer RN5.8 (R1.2)
- net at IC1.60 (CS33): now also RN9.8 (R1.2); no longer RN9.5 (R4.2)
- no-connect marks 0 -> 3
Changed lines of the file:
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@@
   (junction (at 93.98 73.66) (diameter 0) (color 0 0 0 0)
   )
-  (bus_entry (at 201.93 123.19) (size 2.54 -2.54)
-    (stroke (width 0) (type default) (color 0 0 0 0))
-  )
+  (no_connect (at 176.53 123.19))
+  (no_connect (at 176.53 118.11))
+  (no_connect (at 176.53 120.65))
   (bus_entry (at 201.93 100.33) (size 2.54 -2.54)
     (stroke (width 0) (type default) (color 0 0 0 0))
@@
     (stroke (width 0) (type default) (color 0 0 0 0))
   )
-  (bus_entry (at 201.93 118.11) (size 2.54 -2.54)
-    (stroke (width 0) (type default) (color 0 0 0 0))
-  )
   (bus_entry (at 201.93 90.17) (size 2.54 -2.54)
     (stroke (width 0) (type default) (color 0 0 0 0))
@@
     (stroke (width 0) (type default) (color 0 0 0 0))
   )
-  (bus_entry (at 201.93 120.65) (size 2.54 -2.54)
-    (stroke (width 0) (type default) (color 0 0 0 0))
-  )
   (bus_entry (at 201.93 41.91) (size 2.54 -2.54)
     (stroke (width 0) (type default) (color 0 0 0 0))
@@
     (stroke (width 0) (type default) (color 0 0 0 0))
   )
-  (wire (pts (xy 184.15 120.65) (xy 201.93 120.65))
-    (stroke (width 0) (type default) (color 0 0 0 0))
-  )
-  (wire (pts (xy 184.15 118.11) (xy 201.93 118.11))
-    (stroke (width 0) (type default) (color 0 0 0 0))
-  )
   (bus (pts (xy 204.47 107.95) (xy 204.47 105.41))
     (stroke (width 0) (type default) (color 0 0 0 0))
@@
     (stroke (width 0) (type default) (color 0 0 0 0))
   )
-  (bus (pts (xy 204.47 120.65) (xy 204.47 118.11))
-    (stroke (width 0) (type default) (color 0 0 0 0))
-  )
   (wire (pts (xy 186.69 74.93) (xy 201.93 74.93))
     (stroke (width 0) (type default) (color 0 0 0 0))
@@
     (stroke (width 0) (type default) (color 0 0 0 0))
   )
-  (bus (pts (xy 204.47 118.11) (xy 204.47 115.57))
-    (stroke (width 0) (type default) (color 0 0 0 0))
-  )
   (bus (pts (xy 204.47 80.01) (xy 204.47 77.47))
     (stroke (width 0) (type default) (color 0 0 0 0))
@@
     (stroke (width 0) (type default) (color 0 0 0 0))
   )
-  (bus (pts (xy 204.47 115.57) (xy 204.47 113.03))
+  (bus (pts (xy 204.47 113.03) (xy 204.47 118.11))
     (stroke (width 0) (type default) (color 0 0 0 0))
   )
@@
     (stroke (width 0) (type default) (color 0 0 0 0))
   )
-  (wire (pts (xy 184.15 123.19) (xy 201.93 123.19))
-    (stroke (width 0) (type default) (color 0 0 0 0))
-  )
   (wire (pts (xy 172.72 62.23) (xy 176.53 62.23))
     (stroke (width 0) (type default) (color 0 0 0 0))
@@
     (effects (font (size 1.27 1.27)) (justify left bottom))
   )
-  (label "CS38" (at 195.58 120.65 0)
-    (effects (font (size 1.27 1.27)) (justify left bottom))
-  )
-  (label "CS37" (at 195.58 118.11 0)
-    (effects (font (size 1.27 1.27)) (justify left bottom))
-  )
   (label "SW3" (at 177.8 133.35 0)
     (effects (font (size 1.27 1.27)) (justify left bottom))
@@
   )
   (label "CS1" (at 195.58 26.67 0)
-    (effects (font (size 1.27 1.27)) (justify left bottom))
-  )
-  (label "CS39" (at 195.58 123.19 0)
     (effects (font (size 1.27 1.27)) (justify left bottom))
   )
@@
     (pin "1")
   )
-  (symbol (lib_id "Device:R_Pack04") (at 181.61 110.49 90) (unit 1)
+  (symbol (lib_id "Device:R_Pack04") (at 181.61 113.03 90) (mirror x) (unit 1)
     (in_bom yes) (on_board yes)
-    (property "Reference" "RN9" (id 0) (at 175.26 109.22 90))
-    (property "Value" "EXB38V472JV" (id 1) (at 193.04 106.68 90)
-      (effects (font (size 1.27 1.27)) hide)
-    )
-    (property "Footprint" "jjh:EXB38V472JV" (id 2) (at 181.61 103.505 90)
-      (effects (font (size 1.27 1.27)) hide)
-    )
-    (property "Datasheet" "~" (id 3) (at 181.61 110.49 0)
+    (property "Reference" "RN9" (id 0) (at 175.26 114.3 90))
+    (property "Value" "EXB38V472JV" (id 1) (at 193.04 116.84 90)
+      (effects (font (size 1.27 1.27)) hide)
+    )
+    (property "Footprint" "jjh:EXB38V472JV" (id 2) (at 181.61 120.015 90)
+      (effects (font (size 1.27 1.27)) hide)
+    )
+    (property "Datasheet" "~" (id 3) (at 181.61 113.03 0)
       (effects (font (size 1.27 1.27)) hide)
     )
@@
     (pin "8")
   )
-  (symbol (lib_id "Device:R_Pack04") (at 181.61 69.85 90) (unit 1)
+  (symbol (lib_id "Device:R_Pack04") (at 181.61 72.39 90) (mirror x) (unit 1)
     (in_bom yes) (on_board yes)
-    (property "Reference" "RN5" (id 0) (at 175.26 68.58 90))
-    (property "Value" "EXB38V472JV" (id 1) (at 193.04 66.04 90)
-      (effects (font (size 1.27 1.27)) hide)
-    )
-    (property "Footprint" "jjh:EXB38V472JV" (id 2) (at 181.61 62.865 90)
-      (effects (font (size 1.27 1.27)) hide)
-    )
-    (property "Datasheet" "~" (id 3) (at 181.61 69.85 0)
-      (effects (font (size 1.27 1.27)) hide)
-    )
+    (property "Reference" "RN5" (id 0) (at 175.26 73.66 90))
+    (property "Value" "EXB38V472JV" (id 1) (at 193.04 76.2 90)
+      (effects (font (size 1.27 1.27)) hide)
+    )
+    (property "Footprint" "jjh:EXB38V472JV" (id 2) (at 181.61 79.375 90)
+      (effects (font (size 1.27 1.27)) hide)
+    )
+    (property "Datasheet" "~" (id 3) (at 181.61 72.39 0)
+      (effects (font (size 1.27 1.27)) hide)
+    )
