File: PMod_LED/Hardware/PMod_LED.kicad_pcb (KiCad board)
At the start: 2 copper layers, 25.5 x 17 mm, 17 parts, among them J1 Conn_02x06_Odd_Even

Commit message: Start work in kicad v6 to add duel pmod version
Parts:
- added D10: LED, LED_SMD:LED_0603_1608Metric, F.Cu at (146.5, 112.2)
- added D11: LED, LED_SMD:LED_0603_1608Metric, F.Cu at (146.5, 110.2)
- added D12: LED, LED_SMD:LED_0603_1608Metric, F.Cu at (146.5, 108.2)
- added D13: LED, LED_SMD:LED_0603_1608Metric, F.Cu at (146.5, 106.2)
- added D14: LED, LED_SMD:LED_0603_1608Metric, F.Cu at (146.5, 104.2)
- added D15: LED, LED_SMD:LED_0603_1608Metric, F.Cu at (146.5, 102.2)
- added D16: LED, LED_SMD:LED_0603_1608Metric, F.Cu at (146.5, 100.2)
- added D17: LED, LED_SMD:LED_0603_1608Metric, F.Cu at (146.4, 137.3)
- added D18: LED, LED_SMD:LED_0603_1608Metric, F.Cu at (146.4, 135.3)
- added D19: LED, LED_SMD:LED_0603_1608Metric, F.Cu at (146.4, 133.3)
- added D20: LED, LED_SMD:LED_0603_1608Metric, F.Cu at (146.4, 131.3)
- added D21: LED, LED_SMD:LED_0603_1608Metric, F.Cu at (146.4, 129.3)
- added D22: LED, LED_SMD:LED_0603_1608Metric, F.Cu at (146.4, 127.3)
- added D23: LED, LED_SMD:LED_0603_1608Metric, F.Cu at (146.4, 125.3)
- added D24: LED, LED_SMD:LED_0603_1608Metric, F.Cu at (146.4, 123.3)
- added D9: LED, LED_SMD:LED_0603_1608Metric, F.Cu at (146.5, 114.2)
- added G***: LOGO, jjh:j2h_small, F.Cu at (142.4, 118.7)
- added G***: LOGO, jjh:Untitled, B.Cu at (143.0, 87.5)
- added G***: LOGO, jjh:Untitled, B.Cu at (146.0, 118.5)
- added J2: Conn_02x06_Odd_Even, Connector_PinSocket_2.54mm:PinSocket_2x06_P2.54mm_Vertical, F.Cu at (134.8, 100.8)
- added J3: Conn_02x06_Odd_Even, Connector_PinSocket_2.54mm:PinSocket_2x06_P2.54mm_Vertical, F.Cu at (134.8, 123.8)
- added R10: 330, Resistor_SMD:R_0603_1608Metric, F.Cu at (141.5, 112.2)
- added R11: 330, Resistor_SMD:R_0603_1608Metric, F.Cu at (141.5, 110.2)
- added R12: 330, Resistor_SMD:R_0603_1608Metric, F.Cu at (141.5, 108.2)
- added R13: 330, Resistor_SMD:R_0603_1608Metric, F.Cu at (141.5, 106.2)
- added R14: 330, Resistor_SMD:R_0603_1608Metric, F.Cu at (141.5, 104.2)
- added R15: 330, Resistor_SMD:R_0603_1608Metric, F.Cu at (141.5, 102.2)
- added R16: 330, Resistor_SMD:R_0603_1608Metric, F.Cu at (141.5, 100.2)
- added R17: 330, Resistor_SMD:R_0603_1608Metric, F.Cu at (141.4, 137.3)
- added R18: 330, Resistor_SMD:R_0603_1608Metric, F.Cu at (141.4, 135.3)
- added R19: 330, Resistor_SMD:R_0603_1608Metric, F.Cu at (141.4, 133.3)
- added R20: 330, Resistor_SMD:R_0603_1608Metric, F.Cu at (141.4, 131.3)
- added R21: 330, Resistor_SMD:R_0603_1608Metric, F.Cu at (141.4, 129.3)
- added R22: 330, Resistor_SMD:R_0603_1608Metric, F.Cu at (141.4, 127.3)
- added R23: 330, Resistor_SMD:R_0603_1608Metric, F.Cu at (141.4, 125.3)
- added R24: 330, Resistor_SMD:R_0603_1608Metric, F.Cu at (141.4, 123.3)
- added R9: 330, Resistor_SMD:R_0603_1608Metric, F.Cu at (141.5, 114.2)
- added REF**: OSHW-Logo2_7.3x6mm_SilkScreen, Symbol:OSHW-Logo2_7.3x6mm_SilkScreen, F.Cu at (151.4, 118.8)
- added kibuzzard-62214D6E: G***, kibuzzard-62214D6E, F.Cu at (151.5, 90.0)
- added kibuzzard-62214D6E: G***, kibuzzard-62214D6E, F.Cu at (151.4, 133.6)
- added kibuzzard-62214D83: G***, kibuzzard-62214D83, F.Cu at (151.4, 135.6)
- added kibuzzard-62214D83: G***, kibuzzard-62214D83, F.Cu at (151.5, 92.0)
- added kibuzzard-62214D8E: G***, kibuzzard-62214D8E, F.Cu at (151.4, 137.6)
- added kibuzzard-62214D8E: G***, kibuzzard-62214D8E, F.Cu at (151.5, 94.0)
- added kibuzzard-62214D9F: G***, kibuzzard-62214D9F, F.Cu at (151.5, 88.0)
- added kibuzzard-62214D9F: G***, kibuzzard-62214D9F, F.Cu at (151.4, 131.6)
- added kibuzzard-62214DA9: G***, kibuzzard-62214DA9, F.Cu at (151.5, 86.0)
- added kibuzzard-62214DA9: G***, kibuzzard-62214DA9, F.Cu at (151.4, 129.6)
- added kibuzzard-62214DB4: G***, kibuzzard-62214DB4, F.Cu at (151.5, 84.0)
- added kibuzzard-62214DB4: G***, kibuzzard-62214DB4, F.Cu at (151.4, 127.6)
- added kibuzzard-62214DC1: G***, kibuzzard-62214DC1, F.Cu at (151.4, 125.6)
- added kibuzzard-62214DC1: G***, kibuzzard-62214DC1, F.Cu at (151.5, 82.0)
- added kibuzzard-62214DCC: G***, kibuzzard-62214DCC, F.Cu at (151.5, 80.0)
- added kibuzzard-62214DCC: G***, kibuzzard-62214DCC, F.Cu at (151.4, 123.6)
- added kibuzzard-62214EC6: G***, kibuzzard-62214EC6, F.Cu at (151.5, 100.2)
- added kibuzzard-62214ED8: G***, kibuzzard-62214ED8, F.Cu at (151.5, 102.2)
- added kibuzzard-62214EE5: G***, kibuzzard-62214EE5, F.Cu at (151.5, 104.2)
- added kibuzzard-62214EF3: G***, kibuzzard-62214EF3, F.Cu at (151.5, 106.2)
- added kibuzzard-62214F07: G***, kibuzzard-62214F07, F.Cu at (151.5, 108.2)
- added kibuzzard-62214F11: G***, kibuzzard-62214F11, F.Cu at (151.5, 110.2)
- added kibuzzard-62214F38: G***, kibuzzard-62214F38, F.Cu at (151.5, 112.2)
- added kibuzzard-62214F50: G***, kibuzzard-62214F50, F.Cu at (151.5, 114.2)
- added kibuzzard-62215596: G***, kibuzzard-62215596, F.Cu at (138.0, 130.0)
- added kibuzzard-622155A9: G***, kibuzzard-622155A9, F.Cu at (138.0, 107.5)
- added kibuzzard-62215645: G***, kibuzzard-62215645, F.Cu at (138.0, 87.0)
- moved D1 5.09 mm to (147.0, 94.0)
- moved D8 5.06 mm to (147.0, 80.0)
- moved D2 5.05 mm to (147.0, 92.0)
- moved D7 5.04 mm to (147.0, 82.0)
- moved D3 5.03 mm to (147.0, 90.0)
- moved D6 5.02 mm to (147.0, 84.0)
- moved D4 5.00 mm to (147.0, 88.0)
- moved D5 5.00 mm to (147.0, 86.1)
- moved R1 2.60 mm to (141.5, 94.0)
- moved R2 2.50 mm to (141.5, 92.0)
- moved R3 2.46 mm to (141.5, 90.0)
- moved R8 2.44 mm to (141.5, 80.0)
- moved R5 2.41 mm to (141.5, 86.0)
- moved R4 2.40 mm to (141.5, 88.0)
- moved R7 2.38 mm to (141.5, 82.0)
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Connections:
- net LED0 renamed P1_LED0
- net LED1 renamed P1_LED1
- net LED2 renamed P1_LED2
- net LED3 renamed P1_LED3
- net LED4 renamed P1_LED4
- net LED5 renamed P1_LED5
- net LED6 renamed P1_LED6
- net LED7 renamed P1_LED7
- J1 pad 11: Net-(J1-Pad11) -> unconnected-(J1-Pad11)
- J1 pad 12: Net-(J1-Pad12) -> unconnected-(J1-Pad12)
Routing:
- net GND: track 52.3 -> 5.16 mm, vias 3 -> 0
- net P2A_LED0: track 0.00 -> 10.8 mm
- net P2B_LED0: track 0.00 -> 10.7 mm
- net P2A_LED2: track 0.00 -> 10.2 mm
- net P2B_LED2: track 0.00 -> 10.1 mm
- net P2A_LED4: track 0.00 -> 9.58 mm
- net P2B_LED4: track 0.00 -> 9.51 mm
- net P2A_LED6: track 0.00 -> 8.97 mm
- net P2B_LED6: track 0.00 -> 8.91 mm
- net P1_LED7: track 8.23 -> 0.00 mm
- net P1_LED3: track 9.17 -> 1.68 mm
- net P2A_LED1: track 0.00 -> 7.42 mm
- net P2B_LED1: track 0.00 -> 7.35 mm
- net P1_LED1: track 9.53 -> 2.58 mm
- net P1_LED2: track 12.4 -> 5.51 mm
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- removed copper zone on B.Cu, net GND
Other:
- board size 25.5 x 17 mm -> 25.5 x 60.2 mm
- net class Default removed
- board text removed: "1 2"
- board text removed: "3 4"
- board text removed: "3V3"
- board text removed: "5 6"
- board text removed: "7 8"
- board text removed: "GND"

Commit message: update the pcb, complete connections and add logos
Parts:
- removed the G*** at (143.0, 87.5)
- added G***: LOGO, jjh:j2h_small, B.Cu at (139.0, 86.7)
- added REF**: OSHW-Logo2_7.3x6mm_SilkScreen, Symbol:OSHW-Logo2_7.3x6mm_SilkScreen, B.Cu at (152.2, 87.2)
Routing:
- net P1_LED7: track 0.00 -> 6.21 mm
- net P1_LED3: track 1.68 -> 6.81 mm
- net P1_LED1: track 2.58 -> 7.42 mm
- net P1_LED0: track 6.05 -> 10.8 mm
- net P1_LED2: track 5.51 -> 10.2 mm
- net Net-(D5-Pad2): track 0.00 -> 3.93 mm
- net Net-(D8-Pad2): track 0.00 -> 3.89 mm
- net Net-(D7-Pad2): track 0.00 -> 3.89 mm
- net Net-(D6-Pad2): track 0.00 -> 3.89 mm
- net Net-(D4-Pad2): track 0.00 -> 3.89 mm
- net Net-(D3-Pad2): track 0.00 -> 3.89 mm
- net Net-(D2-Pad2): track 0.00 -> 3.89 mm
- net Net-(D1-Pad2): track 0.00 -> 3.89 mm
- net P1_LED5: track 3.10 -> 6.21 mm
- net P1_LED6: track 6.14 -> 8.97 mm
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- added copper zone on B.Cu, net GND
- added copper zone on F.Cu, net GND
Other:
- outline, holes or cut-outs redrawn

Commit message: Add join between the two PCB's
Parts:
- added REF**: NPTH, NPTH, F.Cu at (141.4, 95.2)
- added REF**: NPTH, NPTH, F.Cu at (140.4, 90.8)
- added REF**: NPTH, NPTH, F.Cu at (142.4, 90.8)
- added REF**: NPTH, NPTH, F.Cu at (141.4, 90.8)
- added REF**: NPTH, NPTH, F.Cu at (143.4, 90.8)
- added REF**: NPTH, NPTH, F.Cu at (142.4, 95.2)
- added REF**: NPTH, NPTH, F.Cu at (140.4, 95.2)
- added REF**: NPTH, NPTH, F.Cu at (144.4, 90.8)
- added REF**: NPTH, NPTH, F.Cu at (143.4, 95.2)
- added REF**: NPTH, NPTH, F.Cu at (144.4, 95.2)
- moved D1 4.53 mm to (146.5, 89.5)
- moved D2 4.53 mm to (146.5, 87.5)
- moved D3 4.53 mm to (146.5, 85.5)
- moved D4 4.53 mm to (146.5, 83.5)
- moved D5 4.53 mm to (146.5, 81.6)
- moved D6 4.53 mm to (146.5, 79.5)
- moved D7 4.53 mm to (146.5, 77.5)
- moved D8 4.53 mm to (146.5, 75.5)
- moved G*** 4.53 mm to (138.5, 82.2)
- moved J1 4.53 mm to (134.3, 76.2)
- moved R1 4.53 mm to (141.0, 89.5)
- moved R2 4.53 mm to (141.0, 87.5)
- moved R3 4.53 mm to (141.0, 85.5)
- moved R4 4.53 mm to (141.0, 83.5)
- moved R5 4.53 mm to (141.0, 81.5)
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Other:
- board size 25.5 x 60.2 mm -> 25.5 x 61 mm

Commit message: Fix the DRC errors on duel LED board
Connections:
- D1 pad 1: GND -> GND2
- D2 pad 1: GND -> GND2
- D3 pad 1: GND -> GND2
- D4 pad 1: GND -> GND2
- D5 pad 1: GND -> GND2
- D6 pad 1: GND -> GND2
- D7 pad 1: GND -> GND2
- D8 pad 1: GND -> GND2
- J1 pad 10: GND -> GND2
- J1 pad 9: GND -> GND2
Routing:
- net GND2: track 0.00 -> 2.54 mm, vias 0 -> 4
- net GND: track 2.54 -> 0.00 mm, vias 12 -> 8
- added copper zone on B.Cu, net GND2
- added copper zone on F.Cu, net GND2
