File: PMod_LED/Hardware/PMod_LED.kicad_pcb (KiCad board)
At the start: 2 copper layers, 25.5 x 61 mm, 93 parts, among them J1 Conn_02x06_Odd_Even, J2 Conn_02x06_Odd_Even, J3 Conn_02x06_Odd_Even

Commit message: Change the logo references
Parts:
- renumbered G*** to Logo1, REF** to Logo2, G*** to Logo3, G*** to Logo4, REF** to Logo5

Commit message: Change the pmod logo references
Parts:
- kibuzzard-62215596: value G*** -> Logo6
- kibuzzard-622155A9: value G*** -> Logo7
- kibuzzard-62215645: value G*** -> Logo8
Changed lines of the file:
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@@
     (attr board_only exclude_from_pos_files exclude_from_bom)
     (fp_text reference "kibuzzard-622155A9" (at 0 -0.923348 90) (layer "F.SilkS") hide
-        (effects (font (size 0.000254 0.000254) (thickness 0.000003)))
-    )
-    (fp_text value "G***" (at 0 0.923348 90) (layer "F.SilkS") hide
-        (effects (font (size 0.000254 0.000254) (thickness 0.000003)))
+        (effects (font (size 0.0254 0.0254) (thickness 0.000003)))
+    )
+    (fp_text value "Logo7" (at 0 0.923348 90) (layer "F.SilkS") hide
+        (effects (font (size 0.0254 0.0254) (thickness 0.000003)))
     )
     (fp_poly
@@
     (attr board_only exclude_from_pos_files exclude_from_bom)
     (fp_text reference "kibuzzard-62215596" (at 0 -0.923348 90) (layer "F.SilkS") hide
-        (effects (font (size 0.000254 0.000254) (thickness 0.000003)))
-    )
-    (fp_text value "G***" (at 0 0.923348 90) (layer "F.SilkS") hide
-        (effects (font (size 0.000254 0.000254) (thickness 0.000003)))
+        (effects (font (size 0.0254 0.0254) (thickness 0.000003)))
+    )
+    (fp_text value "Logo6" (at 0 0.923348 90) (layer "F.SilkS") hide
+        (effects (font (size 0.0254 0.0254) (thickness 0.000003)))
     )
     (fp_poly
@@
     (attr board_only exclude_from_pos_files exclude_from_bom)
     (fp_text reference "kibuzzard-62215645" (at 0 -0.923348 90) (layer "F.SilkS") hide
-        (effects (font (size 0.000254 0.000254) (thickness 0.000003)))
-    )
-    (fp_text value "G***" (at 0 0.923348 90) (layer "F.SilkS") hide
-        (effects (font (size 0.000254 0.000254) (thickness 0.000003)))
-    )
-    (fp_poly
+        (effects (font (size 0.0254 0.0254) (thickness 0.000003)))
+    )
+    (fp_text value "Logo8" (at 0 0.923348 90) (layer "F.SilkS") hide
+        (effects (font (size 0.0254 0.0254) (thickness 0.000003)))
+    )
+    (fp_poly
