File: PMod_LED/Hardware/PMod_LED.kicad_pcb (KiCad board)
At the start: 2 copper layers, 25.5 x 61 mm, 93 parts, among them J1 Conn_02x06_Odd_Even, J2 Conn_02x06_Odd_Even, J3 Conn_02x06_Odd_Even

Commit message: Change LED desigantors
Parts:
- kibuzzard-62214D6E, kibuzzard-62214D83, kibuzzard-62214D8E, kibuzzard-62214D9F, kibuzzard-62214DA9, kibuzzard-62214DB4, kibuzzard-62214DC1, kibuzzard-62214DCC: value G*** -> LED
Changed lines of the file:
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@@
     (attr board_only exclude_from_pos_files exclude_from_bom)
     (fp_text reference "kibuzzard-62214DA9" (at 0 -0.915728) (layer "F.SilkS") hide
-        (effects (font (size 0.000254 0.000254) (thickness 0.000003)))
+        (effects (font (size 0.0254 0.0254) (thickness 0.000003)))
     )
-    (fp_text value "G***" (at 0 0.915728) (layer "F.SilkS") hide
-        (effects (font (size 0.000254 0.000254) (thickness 0.000003)))
+    (fp_text value "LED" (at 0 0.915728) (layer "F.SilkS") hide
+        (effects (font (size 0.0254 0.0254) (thickness 0.000003)))
     )
     (fp_poly
@@
     (attr board_only exclude_from_pos_files exclude_from_bom)
     (fp_text reference "kibuzzard-62214DCC" (at 0 -0.915728) (layer "F.SilkS") hide
-        (effects (font (size 0.000254 0.000254) (thickness 0.000003)))
+        (effects (font (size 0.0254 0.0254) (thickness 0.000003)))
     )
-    (fp_text value "G***" (at 0 0.915728) (layer "F.SilkS") hide
-        (effects (font (size 0.000254 0.000254) (thickness 0.000003)))
+    (fp_text value "LED" (at 0 0.915728) (layer "F.SilkS") hide
+        (effects (font (size 0.0254 0.0254) (thickness 0.000003)))
     )
     (fp_poly
@@
     (attr board_only exclude_from_pos_files exclude_from_bom)
     (fp_text reference "kibuzzard-62214DB4" (at 0 -0.918903) (layer "F.SilkS") hide
-        (effects (font (size 0.000254 0.000254) (thickness 0.000003)))
+        (effects (font (size 0.0254 0.0254) (thickness 0.000003)))
     )
-    (fp_text value "G***" (at 0 0.918903) (layer "F.SilkS") hide
-        (effects (font (size 0.000254 0.000254) (thickness 0.000003)))
+    (fp_text value "LED" (at 0 0.918903) (layer "F.SilkS") hide
+        (effects (font (size 0.0254 0.0254) (thickness 0.000003)))
     )
     (fp_poly
@@
     (attr board_only exclude_from_pos_files exclude_from_bom)
     (fp_text reference "kibuzzard-62214D6E" (at 0 -0.920173) (layer "F.SilkS") hide
-        (effects (font (size 0.000254 0.000254) (thickness 0.000003)))
+        (effects (font (size 0.0254 0.0254) (thickness 0.000003)))
     )
-    (fp_text value "G***" (at 0 0.920173) (layer "F.SilkS") hide
-        (effects (font (size 0.000254 0.000254) (thickness 0.000003)))
+    (fp_text value "LED" (at 0 0.920173) (layer "F.SilkS") hide
+        (effects (font (size 0.0254 0.0254) (thickness 0.000003)))
     )
     (fp_poly
@@
     (attr board_only exclude_from_pos_files exclude_from_bom)
     (fp_text reference "kibuzzard-62214D8E" (at 0 -0.923348) (layer "F.SilkS") hide
-        (effects (font (size 0.000254 0.000254) (thickness 0.000003)))
+        (effects (font (size 0.0254 0.0254) (thickness 0.000003)))
     )
-    (fp_text value "G***" (at 0 0.923348) (layer "F.SilkS") hide
-        (effects (font (size 0.000254 0.000254) (thickness 0.000003)))
+    (fp_text value "LED" (at 0 0.923348) (layer "F.SilkS") hide
+        (effects (font (size 0.0254 0.0254) (thickness 0.000003)))
     )
     (fp_poly
@@
     (attr board_only exclude_from_pos_files exclude_from_bom)
     (fp_text reference "kibuzzard-62214D83" (at 0 -0.915728) (layer "F.SilkS") hide
-        (effects (font (size 0.000254 0.000254) (thickness 0.000003)))
+        (effects (font (size 0.0254 0.0254) (thickness 0.000003)))
     )
-    (fp_text value "G***" (at 0 0.915728) (layer "F.SilkS") hide
-        (effects (font (size 0.000254 0.000254) (thickness 0.000003)))
+    (fp_text value "LED" (at 0 0.915728) (layer "F.SilkS") hide
+        (effects (font (size 0.0254 0.0254) (thickness 0.000003)))
     )
     (fp_poly
@@
     (attr board_only exclude_from_pos_files exclude_from_bom)
     (fp_text reference "kibuzzard-62214DC1" (at 0 -0.918903) (layer "F.SilkS") hide
-        (effects (font (size 0.000254 0.000254) (thickness 0.000003)))
+        (effects (font (size 0.0254 0.0254) (thickness 0.000003)))
     )
-    (fp_text value "G***" (at 0 0.918903) (layer "F.SilkS") hide
-        (effects (font (size 0.000254 0.000254) (thickness 0.000003)))
+    (fp_text value "LED" (at 0 0.918903) (layer "F.SilkS") hide
+        (effects (font (size 0.0254 0.0254) (thickness 0.000003)))
     )
     (fp_poly
@@
     (attr board_only exclude_from_pos_files exclude_from_bom)
     (fp_text reference "kibuzzard-62214D9F" (at 0 -0.923348) (layer "F.SilkS") hide
-        (effects (font (size 0.000254 0.000254) (thickness 0.000003)))
+        (effects (font (size 0.0254 0.0254) (thickness 0.000003)))
     )
-    (fp_text value "G***" (at 0 0.923348) (layer "F.SilkS") hide
-        (effects (font (size 0.000254 0.000254) (thickness 0.000003)))
+    (fp_text value "LED" (at 0 0.923348) (layer "F.SilkS") hide
+        (effects (font (size 0.0254 0.0254) (thickness 0.000003)))
     )
     (fp_poly

Commit message: remove ref** designators
Parts:
- renumbered REF** to HOLE
Changed lines of the file:
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@@
     (at 141.4 95.2)
     (attr through_hole)
-    (fp_text reference "REF**" (at 0 0.5) (layer "F.SilkS") hide
+    (fp_text reference "HOLE" (at 0 0.5) (layer "F.SilkS") hide
         (effects (font (size 1 1) (thickness 0.15)))
     )
@@
     (at 142.4 90.798)
     (attr through_hole)
-    (fp_text reference "REF**" (at 0 0.5) (layer "F.SilkS") hide
+    (fp_text reference "HOLE" (at 0 0.5) (layer "F.SilkS") hide
         (effects (font (size 1 1) (thickness 0.15)))
     )
@@
     (at 141.4 90.798)
     (attr through_hole)
-    (fp_text reference "REF**" (at 0 0.5) (layer "F.SilkS") hide
+    (fp_text reference "HOLE" (at 0 0.5) (layer "F.SilkS") hide
         (effects (font (size 1 1) (thickness 0.15)))
     )
@@
     (at 143.4 90.798)
     (attr through_hole)
-    (fp_text reference "REF**" (at 0 0.5) (layer "F.SilkS") hide
+    (fp_text reference "HOLE" (at 0 0.5) (layer "F.SilkS") hide
         (effects (font (size 1 1) (thickness 0.15)))
     )
@@
     (at 142.4 95.2)
     (attr through_hole)
-    (fp_text reference "REF**" (at 0 0.5) (layer "F.SilkS") hide
+    (fp_text reference "HOLE" (at 0 0.5) (layer "F.SilkS") hide
         (effects (font (size 1 1) (thickness 0.15)))
     )
@@
     (at 140.4 95.2)
     (attr through_hole)
-    (fp_text reference "REF**" (at 0 0.5) (layer "F.SilkS") hide
+    (fp_text reference "HOLE" (at 0 0.5) (layer "F.SilkS") hide
         (effects (font (size 1 1) (thickness 0.15)))
     )
@@
     (at 144.4 90.798)
     (attr through_hole)
-    (fp_text reference "REF**" (at 0 0.5) (layer "F.SilkS") hide
+    (fp_text reference "HOLE" (at 0 0.5) (layer "F.SilkS") hide
         (effects (font (size 1 1) (thickness 0.15)))
     )
@@
     (at 143.4 95.2)
     (attr through_hole)
-    (fp_text reference "REF**" (at 0 0.5) (layer "F.SilkS") hide
+    (fp_text reference "HOLE" (at 0 0.5) (layer "F.SilkS") hide
         (effects (font (size 1 1) (thickness 0.15)))
     )
@@
     (at 144.4 95.2)
     (attr through_hole)
-    (fp_text reference "REF**" (at 0 0.5) (layer "F.SilkS") hide
+    (fp_text reference "HOLE" (at 0 0.5) (layer "F.SilkS") hide
         (effects (font (size 1 1) (thickness 0.15)))
     )
@@
     (at 140.4 90.798)
     (attr through_hole)
-    (fp_text reference "REF**" (at 0 0.5) (layer "F.SilkS") hide
+    (fp_text reference "HOLE" (at 0 0.5) (layer "F.SilkS") hide
         (effects (font (size 1 1) (thickness 0.15)))
     )

Commit message: remove hole designators
Parts:
- renumbered HOLE to HOLE1, HOLE to HOLE2, HOLE to HOLE3, HOLE to HOLE4, HOLE to HOLE5, HOLE to HOLE6, HOLE to HOLE7, HOLE to HOLE8, HOLE to HOLE9
Changed lines of the file:
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@@
     (at 141.4 95.2)
     (attr through_hole)
-    (fp_text reference "HOLE" (at 0 0.5) (layer "F.SilkS") hide
+    (fp_text reference "HOLE6" (at 0 0.5) (layer "F.SilkS") hide
         (effects (font (size 1 1) (thickness 0.15)))
     )
@@
     (at 142.4 90.798)
     (attr through_hole)
-    (fp_text reference "HOLE" (at 0 0.5) (layer "F.SilkS") hide
+    (fp_text reference "HOLE2" (at 0 0.5) (layer "F.SilkS") hide
         (effects (font (size 1 1) (thickness 0.15)))
     )
@@
     (at 141.4 90.798)
     (attr through_hole)
-    (fp_text reference "HOLE" (at 0 0.5) (layer "F.SilkS") hide
+    (fp_text reference "HOLE1" (at 0 0.5) (layer "F.SilkS") hide
         (effects (font (size 1 1) (thickness 0.15)))
     )
@@
     (at 143.4 90.798)
     (attr through_hole)
-    (fp_text reference "HOLE" (at 0 0.5) (layer "F.SilkS") hide
+    (fp_text reference "HOLE3" (at 0 0.5) (layer "F.SilkS") hide
         (effects (font (size 1 1) (thickness 0.15)))
     )
@@
     (at 142.4 95.2)
     (attr through_hole)
-    (fp_text reference "HOLE" (at 0 0.5) (layer "F.SilkS") hide
+    (fp_text reference "HOLE7" (at 0 0.5) (layer "F.SilkS") hide
         (effects (font (size 1 1) (thickness 0.15)))
     )
@@
     (at 140.4 95.2)
     (attr through_hole)
-    (fp_text reference "HOLE" (at 0 0.5) (layer "F.SilkS") hide
+    (fp_text reference "HOLE5" (at 0 0.5) (layer "F.SilkS") hide
         (effects (font (size 1 1) (thickness 0.15)))
     )
@@
     (at 144.4 90.798)
     (attr through_hole)
-    (fp_text reference "HOLE" (at 0 0.5) (layer "F.SilkS") hide
+    (fp_text reference "HOLE4" (at 0 0.5) (layer "F.SilkS") hide
         (effects (font (size 1 1) (thickness 0.15)))
     )
@@
     (at 143.4 95.2)
     (attr through_hole)
-    (fp_text reference "HOLE" (at 0 0.5) (layer "F.SilkS") hide
+    (fp_text reference "HOLE8" (at 0 0.5) (layer "F.SilkS") hide
         (effects (font (size 1 1) (thickness 0.15)))
     )
@@
     (at 144.4 95.2)
     (attr through_hole)
-    (fp_text reference "HOLE" (at 0 0.5) (layer "F.SilkS") hide
+    (fp_text reference "HOLE9" (at 0 0.5) (layer "F.SilkS") hide
         (effects (font (size 1 1) (thickness 0.15)))
     )

Commit message: update pcb from schematic
Parts:
- renumbered HOLE to HOLE10
