File: PMod_LED/Hardware/PMod_LED.kicad_sch (KiCad schematic)
At the start: 51 parts, among them J1 Conn_02x06_Odd_Even

Commit message: update the pcb, complete connections and add logos
Parts:
- gave numbers to parts that had none: 34

Commit message: Fix the DRC errors on duel LED board
Connections:
- net GND: no longer D1.1 (K), D2.1 (K), D3.1 (K), D4.1 (K), D5.1 (K), D6.1 (K), D7.1 (K), D8.1 (K), J1.10 (Pin_10), J1.9 (Pin_9)
- new net GND2: D1.1 (K), D2.1 (K), D3.1 (K), D4.1 (K), D5.1 (K), D6.1 (K), D7.1 (K), D8.1 (K), J1.10 (Pin_10), J1.9 (Pin_9)

Commit message: Add power ports
Changed lines of the file:
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@@
     (pin "2")
+  )
+  (symbol (lib_id "power:PWR_FLAG") (at 111.76 45.72 0) (unit 1)
+    (in_bom yes) (on_board yes) (fields_autoplaced)
+    (property "Reference" "#FLG?" (id 0) (at 111.76 43.815 0)
+      (effects (font (size 1.27 1.27)) hide)
+    )
+    (property "Value" "PWR_FLAG" (id 1) (at 111.76 42.1442 0))
+    (property "Footprint" "" (id 2) (at 111.76 45.72 0)
+      (effects (font (size 1.27 1.27)) hide)
+    )
+    (property "Datasheet" "~" (id 3) (at 111.76 45.72 0)
+      (effects (font (size 1.27 1.27)) hide)
+    )
+    (pin "1")
   )
   (symbol (lib_id "power:GND") (at 193.04 105.41 0) (unit 1)
@@
     )
     (property "Datasheet" "" (id 3) (at 59.69 146.05 0)
+      (effects (font (size 1.27 1.27)) hide)
+    )
+    (pin "1")
+  )
+  (symbol (lib_id "power:GND") (at 111.76 93.98 0) (unit 1)
+    (in_bom yes) (on_board yes)
+    (property "Reference" "#PWR?" (id 0) (at 111.76 100.33 0)
+      (effects (font (size 1.27 1.27)) hide)
+    )
+    (property "Value" "GND" (id 1) (at 111.887 97.2312 90)
+      (effects (font (size 1.27 1.27)) (justify right))
+    )
+    (property "Footprint" "" (id 2) (at 111.76 93.98 0)
+      (effects (font (size 1.27 1.27)) hide)
+    )
+    (property "Datasheet" "" (id 3) (at 111.76 93.98 0)
       (effects (font (size 1.27 1.27)) hide)
     )
@@
     (pin "2")
   )
+  (symbol (lib_id "power:PWR_FLAG") (at 111.76 93.98 0) (unit 1)
+    (in_bom yes) (on_board yes) (fields_autoplaced)
+    (property "Reference" "#FLG?" (id 0) (at 111.76 92.075 0)
+      (effects (font (size 1.27 1.27)) hide)
+    )
+    (property "Value" "PWR_FLAG" (id 1) (at 111.76 90.4042 0))
+    (property "Footprint" "" (id 2) (at 111.76 93.98 0)
+      (effects (font (size 1.27 1.27)) hide)
+    )
+    (property "Datasheet" "~" (id 3) (at 111.76 93.98 0)
+      (effects (font (size 1.27 1.27)) hide)
+    )
+    (pin "1")
+  )
   (symbol (lib_id "Device:LED") (at 193.04 97.79 90) (unit 1)
     (in_bom yes) (on_board yes)
@@
     (pin "1")
     (pin "2")
+  )
+  (symbol (lib_id "power:GND2") (at 111.76 45.72 0) (unit 1)
+    (in_bom yes) (on_board yes) (fields_autoplaced)
+    (property "Reference" "#PWR?" (id 0) (at 111.76 52.07 0)
+      (effects (font (size 1.27 1.27)) hide)
+    )
+    (property "Value" "GND2" (id 1) (at 113.665 47.4238 0)
+      (effects (font (size 1.27 1.27)) (justify left))
+    )
+    (property "Footprint" "" (id 2) (at 111.76 45.72 0)
+      (effects (font (size 1.27 1.27)) hide)
+    )
+    (property "Datasheet" "" (id 3) (at 111.76 45.72 0)
+      (effects (font (size 1.27 1.27)) hide)
+    )
+    (pin "1")
   )
   (symbol (lib_id "power:GND") (at 80.01 146.05 90) (unit 1)
@@
   )
   (symbol_instances
+    (path "/38f1f681-d503-49fe-ab87-4225bebb7b32"
+      (reference "#FLG?") (unit 1) (value "PWR_FLAG") (footprint "")
+    )
+    (path "/a65a0ec5-b875-4912-98d6-d80bfa23e356"
+      (reference "#FLG?") (unit 1) (value "PWR_FLAG") (footprint "")
+    )
     (path "/054e6357-b3a2-41dd-bdee-db9c4bb94842"
       (reference "#PWR0101") (unit 1) (value "GND2") (footprint "")
@@
       (reference "#PWR0130") (unit 1) (value "GND") (footprint "")
     )
+    (path "/5f7b9d88-eb12-47e8-8ae8-265c4903ec29"
+      (reference "#PWR?") (unit 1) (value "GND") (footprint "")
+    )
+    (path "/b437d0ad-354b-4121-8f7d-c3f7ed4b8537"
+      (reference "#PWR?") (unit 1) (value "GND2") (footprint "")
+    )
     (path "/00000000-0000-0000-0000-000060871e3a"
