File: PMod_Test/Hardware/PMod_Tester.kicad_pcb (KiCad board)
At the start: 2 copper layers, 40 x 17.5 mm, 4 parts, among them J1 Conn_02x06, J2 Conn_02x06, J3 Conn_02x06

Commit message: minor pcb edits
Routing:
- added copper zone on B.Cu, net GND

Commit message: update the PCB to kicad v6
Parts:
- added kibuzzard-622FB67C: G***, kibuzzard-622FB67C, F.Cu at (107.9, 53.8)
- added kibuzzard-622FB6A0: G***, kibuzzard-622FB6A0, F.Cu at (131.8, 53.9)
- added kibuzzard-622FB70B: G***, kibuzzard-622FB70B, F.Cu at (115.6, 57.8)
- added kibuzzard-622FB71B: G***, kibuzzard-622FB71B, F.Cu at (115.6, 60.3)
- added kibuzzard-622FB72D: G***, kibuzzard-622FB72D, F.Cu at (115.6, 47.6)
- added kibuzzard-622FB73D: G***, kibuzzard-622FB73D, F.Cu at (115.6, 50.2)
- added kibuzzard-622FB74A: G***, kibuzzard-622FB74A, F.Cu at (115.6, 52.7)
- added kibuzzard-622FB757: G***, kibuzzard-622FB757, F.Cu at (115.6, 55.2)
- added kibuzzard-622FB76E: G***, kibuzzard-622FB76E, F.Cu at (126.0, 47.6)
- added kibuzzard-622FB788: G***, kibuzzard-622FB788, F.Cu at (126.0, 50.0)
- added kibuzzard-622FB795: G***, kibuzzard-622FB795, F.Cu at (126.0, 52.6)
- added kibuzzard-622FB7A1: G***, kibuzzard-622FB7A1, F.Cu at (126.0, 55.1)
- added kibuzzard-622FB7B1: G***, kibuzzard-622FB7B1, F.Cu at (126.0, 57.7)
- added kibuzzard-622FB7C8: G***, kibuzzard-622FB7C8, F.Cu at (126.0, 60.2)
Other:
- net class Default removed
- board text removed: "Client"
- board text removed: "Host"

Commit message: sort out some pcb drc errors
Other:
- board text removed: "1"
- board text removed: "2"
- board text removed: "3"
- board text removed: "3v3"
- board text removed: "4"
- board text removed: "5"
- board text removed: "6"
- board text removed: "7"
- board text removed: "8"
- board text removed: "GND"
Changed lines of the file:
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@@
   )
   (setup
+    (stackup
+      (layer "F.SilkS" (type "Top Silk Screen"))
+      (layer "F.Paste" (type "Top Solder Paste"))
+      (layer "F.Mask" (type "Top Solder Mask") (thickness 0.01))
+      (layer "F.Cu" (type "copper") (thickness 0.035))
+      (layer "dielectric 1" (type "core") (thickness 1.51) (material "FR4") (epsilon_r 4.5) (loss_tangent 0.02))
+      (layer "B.Cu" (type "copper") (thickness 0.035))
+      (layer "B.Mask" (type "Bottom Solder Mask") (thickness 0.01))
+      (layer "B.Paste" (type "Bottom Solder Paste"))
+      (layer "B.SilkS" (type "Bottom Silk Screen"))
+      (copper_finish "None")
+      (dielectric_constraints no)
+    )
     (pad_to_mask_clearance 0)
     (pcbplotparams
@@
       ) (layer "B.SilkS") (width 0.01) (fill solid))
   )
-  (gr_line (start 114.62 79.67) (end 114.62 82.17) (layer "F.SilkS") (width 0.12))
-  (gr_line (start 119 82.2) (end 114.62 82.17) (layer "F.SilkS") (width 0.12))
-  (gr_line (start 124.2 82.4) (end 129.2 82.4) (layer "F.SilkS") (width 0.12))
-  (gr_line (start 114.87 79.67) (end 114.62 79.67) (layer "F.SilkS") (width 0.12))
-  (gr_line (start 114.62 82.17) (end 114.62 66.82) (layer "F.SilkS") (width 0.12))
-  (gr_line (start 129.2 82.4) (end 129.2 67.05) (layer "F.SilkS") (width 0.12))
   (gr_line (start 139 45) (end 101 45) (layer "Edge.Cuts") (width 0.05))
   (gr_arc (start 101 62.5) (mid 100.292893 62.207107) (end 100 61.5) (layer "Edge.Cuts") (width 0.05))
@@
     (effects (font (size 1 1) (thickness 0.15)) (justify mirror))
   )
-  (gr_text "3v3\n" (at 126.5 81.2) (layer "F.SilkS")
-    (effects (font (size 1 1) (thickness 0.15)))
-  )
-  (gr_text "GND\n" (at 116.87 78.37) (layer "F.SilkS")
-    (effects (font (size 1 1) (thickness 0.15)))
-  )
-  (gr_text "GND\n" (at 126.5 78.6) (layer "F.SilkS")
-    (effects (font (size 1 1) (thickness 0.15)))
-  )
-  (gr_text "3" (at 117.37 73.17) (layer "F.SilkS")
-    (effects (font (size 1 1) (thickness 0.15)))
-  )
-  (gr_text "5" (at 125.7 68.3) (layer "F.SilkS")
-    (effects (font (size 1 1) (thickness 0.15)))
-  )
-  (gr_text "7" (at 125.7 73.5) (layer "F.SilkS")
-    (effects (font (size 1 1) (thickness 0.15)))
-  )
-  (gr_text "6" (at 125.7 71) (layer "F.SilkS")
-    (effects (font (size 1 1) (thickness 0.15)))
-  )
-  (gr_text "2\n" (at 117.37 70.77) (layer "F.SilkS")
-    (effects (font (size 1 1) (thickness 0.15)))
-  )
-  (gr_text "3v3" (at 116.97 80.97) (layer "F.SilkS")
-    (effects (font (size 1 1) (thickness 0.15)))
-  )
-  (gr_text "1\n" (at 117.37 68.17) (layer "F.SilkS")
-    (effects (font (size 1 1) (thickness 0.15)))
-  )
-  (gr_text "4" (at 117.27 75.87) (layer "F.SilkS")
-    (effects (font (size 1 1) (thickness 0.15)))
-  )
-  (gr_text "8" (at 125.7 76.1) (layer "F.SilkS")
-    (effects (font (size 1 1) (thickness 0.15)))
-  )
-  (segment (start 137.42 60.2) (end 137.5 60.12) (width 1) (layer "B.Cu") (net 1))
   (segment (start 102.46 60.2) (end 137.42 60.2) (width 1) (layer "B.Cu") (net 1))
   (segment (start 133.864999 53.944999) (end 118.055001 53.944999) (width 0.25) (layer "B.Cu") (net 3))
@@
   (zone (net 2) (net_name "GND") (layer "F.Cu") (hatch edge 0.508)
     (connect_pads (clearance 0.508))
-    (min_thickness 0.254)
+    (min_thickness 0.254) (filled_areas_thickness no)
     (fill yes (thermal_gap 0.508) (thermal_bridge_width 0.508))
     (polygon
@@
   (zone (net 2) (net_name "GND") (layer "B.Cu") (hatch edge 0.508)
     (connect_pads (clearance 0.508))
-    (min_thickness 0.254)
+    (min_thickness 0.254) (filled_areas_thickness no)
     (fill yes (thermal_gap 0.508) (thermal_bridge_width 0.508))
     (polygon
