File: PMod_RGB7Segment/Hardware/PMod_RGB7Segment.kicad_pcb (KiCad board)
At the start: 4 copper layers, 100 x 38 mm, 121 parts, among them IC1 IS31FL3741A-QFLS4-TR, J1 Conn_02x06_Odd_Even

Commit message: update with vias that are 0.45mm/0.2mm
Parts:
- added G***: LOGO, jjh:Untitled, B.Cu at (140.6, 116.2)
Routing:
- net Net-(IC1-Pad44): track 47.9 -> 55.1 mm
- net Net-(IC1-Pad2): track 84.6 -> 81.8 mm
- net /SW4: track 271.1 -> 273.7 mm
- net /CS2: track 76.3 -> 78.8 mm
- net /CS5: track 55.5 -> 57.0 mm
- net /CS28: track 193.5 -> 195.0 mm
- net /SW6: track 200.5 -> 202.0 mm
- net /CS11: track 81.8 -> 83.1 mm
- net /CS30: track 121.8 -> 123.1 mm
- net /SW5: track 188.7 -> 190.0 mm
- net /CS29: track 121.1 -> 122.3 mm
- net /SW9: track 182.2 -> 183.4 mm
- net Net-(IC1-Pad37): track 19.3 -> 20.5 mm
- net /CS12: track 84.0 -> 85.2 mm
- net /CS24: track 105.6 -> 106.7 mm
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
Commit message: fix drc errors in ci
Routing:
- net Net-(IC1-Pad44): track 55.1 -> 48.0 mm
- net /SW1: track 223.8 -> 225.0 mm
- net Net-(IC1-Pad39): track 56.4 -> 55.6 mm
- net /CS28: track 195.0 -> 195.7 mm
- net /CS9: track 33.4 -> 34.0 mm
- net /CS8: track 34.8 -> 35.4 mm
- net /CS7: track 35.9 -> 36.6 mm
- net /SW7: track 175.2 -> 175.7 mm
- net Net-(IC1-Pad41): track 53.6 -> 53.1 mm
- net Net-(IC1-Pad40): track 54.8 -> 54.3 mm
- net Net-(IC1-Pad42): track 52.9 -> 52.4 mm
- net /CS21: track 88.8 -> 89.3 mm
