File: PMod_GPS/Hardware/PMod_GPS.kicad_sch (KiCad schematic)
At the start: 3 parts, among them J1 Conn_02x06_Odd_Even, U1 NEO-M8M

Commit message: add driven flag to the antenna
Changed lines of the file:
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@@
   (junction (at 63.5 93.98) (diameter 0) (color 0 0 0 0)
+  )
+  (junction (at 181.61 80.01) (diameter 0) (color 0 0 0 0)
   )
   (junction (at 55.88 93.98) (diameter 0) (color 0 0 0 0)
@@
     (stroke (width 0) (type default) (color 0 0 0 0))
   )
-  (wire (pts (xy 173.99 80.01) (xy 218.44 80.01))
+  (wire (pts (xy 173.99 80.01) (xy 181.61 80.01))
+    (stroke (width 0) (type default) (color 0 0 0 0))
+  )
+  (wire (pts (xy 181.61 77.47) (xy 181.61 80.01))
     (stroke (width 0) (type default) (color 0 0 0 0))
   )
@@
   )
   (wire (pts (xy 125.73 82.55) (xy 138.43 82.55))
+    (stroke (width 0) (type default) (color 0 0 0 0))
+  )
+  (wire (pts (xy 181.61 80.01) (xy 218.44 80.01))
     (stroke (width 0) (type default) (color 0 0 0 0))
   )
@@
     )
     (property "Mouser No." "673-W3213" (id 4) (at 218.44 74.93 0)
+      (effects (font (size 1.27 1.27)) hide)
+    )
+    (pin "1")
+  )
+  (symbol (lib_id "power:PWR_FLAG") (at 181.61 77.47 0) (unit 1)
+    (in_bom yes) (on_board yes) (fields_autoplaced)
+    (property "Reference" "#FLG0103" (id 0) (at 181.61 75.565 0)
+      (effects (font (size 1.27 1.27)) hide)
+    )
+    (property "Value" "PWR_FLAG" (id 1) (at 181.61 73.8655 0)
+      (effects (font (size 1.27 1.27)) hide)
+    )
+    (property "Footprint" "" (id 2) (at 181.61 77.47 0)
+      (effects (font (size 1.27 1.27)) hide)
+    )
+    (property "Datasheet" "~" (id 3) (at 181.61 77.47 0)
       (effects (font (size 1.27 1.27)) hide)
     )
@@
       (reference "#FLG0102") (unit 1) (value "PWR_FLAG") (footprint "")
     )
+    (path "/4081599c-4187-4b0c-8b58-f14d38f5e3d3"
+      (reference "#FLG0103") (unit 1) (value "PWR_FLAG") (footprint "")
+    )
     (path "/1d7caddf-09e0-4491-b8d7-93c1daf281d7"

Commit message: correct the error for the RX and TX being the wrong way round #73 on schematic
Connections:
- net RXD: now also J1.7 (Pin_7); no longer J1.8 (Pin_8)
- net TXD: now also J1.8 (Pin_8); no longer J1.7 (Pin_7)
Changed lines of the file:
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@@
     )
   )
-  (global_label "RXD" (shape input) (at 66.04 74.93 0) (fields_autoplaced)
-    (effects (font (size 1.27 1.27)) (justify left))
-    (property "Intersheet References" "${INTERSHEET_REFS}" (id 0) (at 72.2026 75.0094 0)
-      (effects (font (size 1.27 1.27)) (justify left) hide)
+  (global_label "RXD" (shape input) (at 53.34 74.93 180) (fields_autoplaced)
+    (effects (font (size 1.27 1.27)) (justify right))
+    (property "Intersheet References" "${INTERSHEET_REFS}" (id 0) (at 47.1774 74.8506 0)
+      (effects (font (size 1.27 1.27)) (justify right) hide)
     )
   )
@@
     )
   )
-  (global_label "TXD" (shape input) (at 53.34 74.93 180) (fields_autoplaced)
-    (effects (font (size 1.27 1.27)) (justify right))
-    (property "Intersheet References" "${INTERSHEET_REFS}" (id 0) (at 47.4798 74.8506 0)
-      (effects (font (size 1.27 1.27)) (justify right) hide)
+  (global_label "TXD" (shape input) (at 66.04 74.93 0) (fields_autoplaced)
+    (effects (font (size 1.27 1.27)) (justify left))
+    (property "Intersheet References" "${INTERSHEET_REFS}" (id 0) (at 71.9002 75.0094 0)
+      (effects (font (size 1.27 1.27)) (justify left) hide)
     )
   )
