File: PMod_GPS/Hardware/PMod_GPS.kicad_pcb (KiCad board)
At the start: 2 copper layers, 47 x 17 mm, 5 parts, among them J1 Conn_02x06_Odd_Even, U1 NEO-M8M

Commit message: change board clearance settings
Parts:
- renumbered G*** to G1
Changed lines of the file:
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@@
       (effects (font (size 1.27 1.27) (thickness 0.254)))
     )
-    (fp_text user "${REFERENCE}" (at 0 -0.7) (layer "F.Fab")
+    (fp_text user "${REFERENCE}" (at 0 -3.85) (layer "F.Fab")
       (effects (font (size 1.27 1.27) (thickness 0.254)))
     )
@@
     (at 143 91 180)
     (attr through_hole)
-    (fp_text reference "G***" (at 0 0) (layer "B.SilkS") hide
+    (fp_text reference "G1" (at 0 0) (layer "B.SilkS") hide
       (effects (font (size 1.524 1.524) (thickness 0.3)) (justify mirror))
     )

Commit message: correct the error for the RX and TX being the wrong way round #73 on PCB
Connections:
- J1 pad 7: TXD -> RXD
- J1 pad 8: RXD -> TXD
Routing:
- net TXD: track 18.5 -> 14.9 mm
- net RXD: track 14.1 -> 17.1 mm
Changed lines of the file:
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@@
     (descr "ublox NEO 6/7/8, (https://www.u-blox.com/sites/default/files/NEO-8Q-NEO-M8-FW3_HardwareIntegrationManual_%28UBX-15029985%29_0.pdf)")
     (tags "GPS ublox NEO 6/7/8")
-    (property "Sheetfile" "PMod_GPS.kicad_sch")
+    (property "Sheetfile" "File: PMod_GPS.kicad_sch")
     (property "Sheetname" "")
     (attr smd)
@@
     (descr "Through hole straight pin header, 2x06, 2.54mm pitch, double rows")
     (tags "Through hole pin header THT 2x06 2.54mm double row")
-    (property "Sheetfile" "PMod_GPS.kicad_sch")
+    (property "Sheetfile" "File: PMod_GPS.kicad_sch")
     (property "Sheetname" "")
     (attr through_hole)
@@
       (net 16 "SCL") (pinfunction "Pin_6") (pintype "passive"))
     (pad "7" thru_hole oval (at 0 7.62) (size 1.7 1.7) (drill 1) (layers *.Cu *.Mask)
-      (net 17 "TXD") (pinfunction "Pin_7") (pintype "passive"))
+      (net 18 "RXD") (pinfunction "Pin_7") (pintype "passive"))
     (pad "8" thru_hole oval (at 2.54 7.62) (size 1.7 1.7) (drill 1) (layers *.Cu *.Mask)
-      (net 18 "RXD") (pinfunction "Pin_8") (pintype "passive"))
+      (net 17 "TXD") (pinfunction "Pin_8") (pintype "passive"))
     (pad "9" thru_hole oval (at 0 10.16) (size 1.7 1.7) (drill 1) (layers *.Cu *.Mask)
       (net 8 "GND") (pinfunction "Pin_9") (pintype "passive"))
@@
     (tags "Antenna")
     (property "Mouser No." "673-W3213")
-    (property "Sheetfile" "PMod_GPS.kicad_sch")
+    (property "Sheetfile" "File: PMod_GPS.kicad_sch")
     (property "Sheetname" "")
     (attr through_hole)
@@
   (via (at 146 83) (size 0.8) (drill 0.4) (layers "F.Cu" "B.Cu") (free) (net 8))
   (via (at 133 92) (size 0.8) (drill 0.4) (layers "F.Cu" "B.Cu") (free) (net 8))
-  (via (at 125.5 90.5) (size 0.8) (drill 0.4) (layers "F.Cu" "B.Cu") (free) (net 8))
+  (via (at 125.8 88.7) (size 0.8) (drill 0.4) (layers "F.Cu" "B.Cu") (free) (net 8))
   (via (at 130 92) (size 0.8) (drill 0.4) (layers "F.Cu" "B.Cu") (free) (net 8))
   (via (at 163 98) (size 0.8) (drill 0.4) (layers "F.Cu" "B.Cu") (free) (net 8))
@@
   (segment (start 134.6 84.7) (end 134.6 84.158217) (width 0.25) (layer "F.Cu") (net 16))
   (segment (start 133.5 85.241783) (end 133.5 84.7) (width 0.25) (layer "F.Cu") (net 17))
-  (segment (start 120.499511 92.944511) (end 120.499511 92.949511) (width 0.25) (layer "F.Cu") (net 17))
-  (segment (start 125.691783 93.05) (end 133.5 85.241783) (width 0.25) (layer "F.Cu") (net 17))
-  (segment (start 120.499511 92.949511) (end 120.6 93.05) (width 0.25) (layer "F.Cu") (net 17))
-  (segment (start 120.6 93.05) (end 125.691783 93.05) (width 0.25) (layer "F.Cu") (net 17))
-  (segment (start 119.325 91.77) (end 120.499511 92.944511) (width 0.25) (layer "F.Cu") (net 17))
-  (segment (start 126.336065 91.77) (end 132.4 85.706065) (width 0.25) (layer "F.Cu") (net 18))
-  (segment (start 132.4 85.706065) (end 132.4 84.7) (width 0.25) (layer "F.Cu") (net 18))
-  (segment (start 121.865 91.77) (end 126.336065 91.77) (width 0.25) (layer "F.Cu") (net 18))
+  (segment (start 127.220892 91.520892) (end 133.5 85.241783) (width 0.25) (layer "F.Cu") (net 17))
+  (segment (start 121.865 91.77) (end 126.971784 91.77) (width 0.25) (layer "F.Cu") (net 17))
+  (segment (start 126.971784 91.77) (end 127.220892 91.520892) (width 0.25) (layer "F.Cu") (net 17))
+  (segment (start 119.325 91.77) (end 120.695 90.4) (width 0.25) (layer "F.Cu") (net 18))
+  (segment (start 122.7 90.4) (end 123.5 91.2) (width 0.25) (layer "F.Cu") (net 18))
+  (segment (start 120.695 90.4) (end 122.7 90.4) (width 0.25) (layer "F.Cu") (net 18))
+  (segment (start 126.611163 91.2) (end 132.4 85.411163) (width 0.25) (layer "F.Cu") (net 18))
+  (segment (start 123.5 91.2) (end 126.611163 91.2) (width 0.25) (layer "F.Cu") (net 18))
+  (segment (start 132.4 85.411163) (end 132.4 84.7) (width 0.25) (layer "F.Cu") (net 18))
   (zone (net 8) (net_name "GND") (layers F&B.Cu) (hatch edge 0.508)
     (connect_pads (clearance 0.508))

Commit message: Add Gitrev to PCB using github action
Other:
- board text added: "%%GITHASH%%"
Changed lines of the file:
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@@
     )
   )
+  (property "VER" "GITVER")
   (net 0 "")
   (net 1 "Net-(AE1-Pad1)")
@@
     (effects (font (size 1 1) (thickness 0.15)) (justify mirror))
   )
+  (gr_text "%%GITHASH%%" (at 126 91 90) (layer "B.SilkS")
+    (effects (font (size 1 1) (thickness 0.15)) (justify mirror))
+  )

Commit message: rotate the text to match others
Other:
- board text added: "Ver: %%GITHASH%%"
- board text removed: "%%GITHASH%%"
Changed lines of the file:
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@@
     (effects (font (size 1 1) (thickness 0.15)) (justify mirror))
   )
-  (gr_text "%%GITHASH%%" (at 126 91 90) (layer "B.SilkS")
+  (gr_text "Ver: %%GITHASH%%" (at 126 91 270) (layer "B.SilkS")
     (effects (font (size 1 1) (thickness 0.15)) (justify mirror))
   )
