File: Pmod_StepAttenuator/Hardware/StepAttenuator.kicad_sch (KiCad schematic)
At the start: 0 parts

Commit message: starting work on the schematic
Parts:
- added C1: 0.1uf, Capacitor_SMD:C_0402_1005Metric, symbol Device:C
- added C2: 100pF, Capacitor_SMD:C_0402_1005Metric, symbol Device:C
- added J1: Conn_02x06_Odd_Even, Connector_PinHeader_2.54mm:PinHeader_2x06_P2.54mm_Vertical, symbol Connector_Generic:Conn_02x06_Odd_Even
- added J2, J3: Conn_Coaxial, symbol Connector:Conn_Coaxial
- added U1: PE4312C-Z, easyeda2kicad:QFN-20_L4.0-W4.0-P0.50-BL-EP2.2, symbol easyead:PE4312C-Z
Connections:
- new net: J2.1 (In), U1.14 (RFOUT)
- new net +3V3: C1.1, C2.1, J1.11 (Pin_11), J1.12 (Pin_12), U1.6 (VDD), U1.9 (VDD)
- new net Data_C1: J1.3 (Pin_3), U1.19 (C1)
- new net Data_C16: J1.6 (Pin_6), U1.1 (C16)
- new net Data_C2: J1.5 (Pin_5), U1.17 (C2)
- new net Data_C4: J1.2 (Pin_2), U1.16 (C4)
- new net Data_C5: J1.1 (Pin_1), U1.20 (C5)
- new net Data_C8: J1.4 (Pin_4), U1.15 (C8)
- new net GND: C1.2, C2.2, J1.10 (Pin_10), J1.9 (Pin_9), J2.2 (Ext), J3.2 (Ext), U1.10 (GND), U1.11 (GND), U1.12 (VSS/GND), U1.13 (PS), U1.18 (GND), U1.21 (GND), U1.7 (PUP1), U1.8 (PUP2)
- new net LE: J1.7 (Pin_7), U1.5 (LE)
Other:
- note added: "Both Power up state control pulled to ground, as not used"
- note added: "PS is pulled Low to enable the parellel interface."
- note added: "Pin 12 pulled to ground to enable internal neg Voltage generator"

Commit message: schematic capture and board layout
Parts:
- J1: now left out of the parts list
- J2: footprint (none) -> Connector_Coaxial:SMA_Amphenol_132289_EdgeMount; now not fitted
- J3: footprint (none) -> Connector_Coaxial:SMA_Amphenol_132289_EdgeMount; now left out of the parts list
- U1: footprint easyeda2kicad:QFN-20_L4.0-W4.0-P0.50-BL-EP2.2 -> easyeda:QFN-20_L4.0-W4.0-P0.50-BL-EP2.2
Connections:
- net Data_C1: now also J1.6 (Pin_6); no longer J1.3 (Pin_3)
- net Data_C16: now also J1.2 (Pin_2); no longer J1.6 (Pin_6)
- net Data_C2: now also J1.3 (Pin_3); no longer J1.5 (Pin_5)
- net Data_C4: now also J1.4 (Pin_4); no longer J1.2 (Pin_2)
- net Data_C5: now also J1.5 (Pin_5); no longer J1.1 (Pin_1)
- net Data_C8: now also J1.1 (Pin_1); no longer J1.4 (Pin_4)
- net at J3.1 (In): now also U1.2 (RFIN)
- no-connect marks 0 -> 2
Changed lines of the file:
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@@
 		(color 0 0 0 0)
 	)
+	(no_connect
+		(at 176.53 93.98)
+	)
+	(no_connect
+		(at 176.53 91.44)
+	)
 	(wire
 		(pts
@@
 	(wire
 		(pts
-			(xy 133.35 88.9) (xy 175.26 88.9)
+			(xy 133.35 88.9) (xy 176.53 88.9)
 		)
 		(stroke
@@
 	(global_label "Data_C16"
 		(shape input)
-		(at 85.09 90.17 0)
+		(at 85.09 85.09 0)
 		(fields_autoplaced yes)
 		(effects
@@
 		)
 		(property "Intersheetrefs" "${INTERSHEET_REFS}"
-			(at 97.0255 90.17 0)
+			(at 97.0255 85.09 0)
 			(effects
 				(font
@@
 	(global_label "Data_C1"
 		(shape input)
-		(at 50.8 87.63 180)
+		(at 85.09 90.17 0)
 		(fields_autoplaced yes)
 		(effects
@@
 				(size 1.27 1.27)
 			)
-			(justify right)
+			(justify left)
 		)
 		(property "Intersheetrefs" "${INTERSHEET_REFS}"
-			(at 40.074 87.63 0)
-			(effects
-				(font
-					(size 1.27 1.27)
-				)
-				(justify right)
+			(at 95.816 90.17 0)
+			(effects
+				(font
+					(size 1.27 1.27)
+				)
+				(justify left)
 				(hide yes)
 			)
@@
 	(global_label "Data_C4"
 		(shape input)
-		(at 85.09 85.09 0)
+		(at 85.09 87.63 0)
 		(fields_autoplaced yes)
 		(effects
@@
 		)
 		(property "Intersheetrefs" "${INTERSHEET_REFS}"
-			(at 95.816 85.09 0)
+			(at 95.816 87.63 0)
 			(effects
 				(font
@@
 	(global_label "Data_C5"
 		(shape input)
-		(at 50.8 85.09 180)
+		(at 50.8 90.17 180)
 		(fields_autoplaced yes)
 		(effects
@@
 		)
 		(property "Intersheetrefs" "${INTERSHEET_REFS}"
-			(at 40.074 85.09 0)
+			(at 40.074 90.17 0)
 			(effects
 				(font
@@
 	(global_label "Data_C2"
 		(shape input)
-		(at 50.8 90.17 180)
+		(at 50.8 87.63 180)
 		(fields_autoplaced yes)
 		(effects
@@
 		)
 		(property "Intersheetrefs" "${INTERSHEET_REFS}"
-			(at 40.074 90.17 0)
+			(at 40.074 87.63 0)
 			(effects
 				(font
@@
 	(global_label "Data_C8"
 		(shape input)
-		(at 85.09 87.63 0)
+		(at 50.8 85.09 180)
 		(fields_autoplaced yes)
 		(effects
@@
 				(size 1.27 1.27)
 			)
-			(justify left)
+			(justify right)
 		)
 		(property "Intersheetrefs" "${INTERSHEET_REFS}"
-			(at 95.816 87.63 0)
-			(effects
-				(font
-					(size 1.27 1.27)
-				)
-				(justify left)
+			(at 40.074 85.09 0)
+			(effects
+				(font
+					(size 1.27 1.27)
+				)
+				(justify right)
 				(hide yes)
 			)
@@
 		(unit 1)
 		(exclude_from_sim no)
-		(in_bom yes)
-		(on_board yes)
+		(in_bom no)
+		(on_board no)
 		(dnp no)
 		(fields_autoplaced yes)
@@
 		(unit 1)
 		(exclude_from_sim no)
-		(in_bom yes)
-		(on_board yes)
+		(in_bom no)
+		(on_board no)
 		(dnp no)
 		(property "Reference" "J3"
@@
 			)
 		)
-		(property "Footprint" ""
+		(property "Footprint" "Connector_Coaxial:SMA_Amphenol_132289_EdgeMount"
 			(at 128.27 88.9 0)
 			(effects
@@
 			)
 		)
-		(property "Footprint" "easyeda2kicad:QFN-20_L4.0-W4.0-P0.50-BL-EP2.2"
+		(property "Footprint" "easyeda:QFN-20_L4.0-W4.0-P0.50-BL-EP2.2"
 			(at 190.5 115.57 0)
 			(effects
@@
 		(in_bom yes)
 		(on_board yes)
-		(dnp no)
+		(dnp yes)
 		(fields_autoplaced yes)
 		(property "Reference" "J2"
@@
 			)
 		)
-		(property "Footprint" ""
+		(property "Footprint" "Connector_Coaxial:SMA_Amphenol_132289_EdgeMount"
 			(at 265.43 88.9 0)
 			(effects
