File: Pmod_StepAttenuator/Hardware/StepAttenuator.kicad_sch (KiCad schematic)
At the start: 6 parts, among them J1 Conn_02x06_Odd_Even, J2 Conn_Coaxial, J3 Conn_Coaxial, U1 PE4312C-Z

Commit message: update with cap part numbers for the bom
Parts:
- C1: LCSC Part (none) -> C1525
- C2: LCSC Part (none) -> C1546
Changed lines of the file:
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@@
+			)
+		)
+		(property "LCSC Part" "C1546"
+			(at 176.53 125.73 0)
+			(effects
+				(font
+					(size 1.27 1.27)
+				)
+				(hide yes)
 			)
 		)
@@
 			(at 163.83 125.73 0)
 			(effects
+				(font
+					(size 1.27 1.27)
+				)
+				(hide yes)
+			)
+		)
+		(property "LCSC Part" "C1525"
+			(at 163.83 125.73 0)
+			(effects
